File: LedBarController/4xFet.sch (KiCad schematic (older format))
At the start: 6 parts, among them Q701 Si2302DS, Q702 Si2302DS, Q703 Si2302DS, Q704 Si2302DS

Commit message: Restarted PCB
Parts:
- removed C701: 0.1uF, Capacitor_SMD:C_0805_2012Metric_Pad1.18x1.45mm_HandSolder, symbol Device:C
- removed C702: 470uF/35V, Capacitor_THT:CP_Radial_D10.0mm_P5.00mm, symbol Device:CP
- renumbered Q701 to Q301, Q702 to Q302, Q703 to Q303, Q704 to Q304

Commit message: Updated labels in schematic and moved RTC to sub-schematic
Changed lines of the file:
@@
 $Descr A4 11693 8268
 encoding utf-8
-Sheet 5 13
+Sheet 5 14
 Title ""
 Date ""
@@
 AR Path="/5F8F2E1B/5F902D83/5F88FE81" Ref="Q504"  Part="1"
 AR Path="/5F8F2E1B/5F902E61/5F88FE81" Ref="Q604"  Part="1"
-F 0 "Q504" H 7854 3846 50  0000 L CNN
+F 0 "Q604" H 7854 3846 50  0000 L CNN
 F 1 "Si2302DS" H 7854 3755 50  0000 L CNN
 F 2 "Package_TO_SOT_SMD:SOT-23_Handsoldering" H 7850 3900 50  0001 C CNN
@@
 AR Path="/5F8F2E1B/5F902D83/5F88FE73" Ref="Q503"  Part="1"
 AR Path="/5F8F2E1B/5F902E61/5F88FE73" Ref="Q603"  Part="1"
-F 0 "Q503" H 6104 3846 50  0000 L CNN
+F 0 "Q603" H 6104 3846 50  0000 L CNN
 F 1 "Si2302DS" H 6104 3755 50  0000 L CNN
 F 2 "Package_TO_SOT_SMD:SOT-23_Handsoldering" H 6100 3900 50  0001 C CNN
@@
 AR Path="/5F8F2E1B/5F902D83/5F88FE65" Ref="Q502"  Part="1"
 AR Path="/5F8F2E1B/5F902E61/5F88FE65" Ref="Q602"  Part="1"
-F 0 "Q502" H 4354 3846 50  0000 L CNN
+F 0 "Q602" H 4354 3846 50  0000 L CNN
 F 1 "Si2302DS" H 4354 3755 50  0000 L CNN
 F 2 "Package_TO_SOT_SMD:SOT-23_Handsoldering" H 4350 3900 50  0001 C CNN
@@
 AR Path="/5F8F2E1B/5F902D83/5F88FE58" Ref="Q501"  Part="1"
 AR Path="/5F8F2E1B/5F902E61/5F88FE58" Ref="Q601"  Part="1"
-F 0 "Q501" H 2604 3846 50  0000 L CNN
+F 0 "Q601" H 2604 3846 50  0000 L CNN
 F 1 "Si2302DS" H 2604 3755 50  0000 L CNN
 F 2 "Package_TO_SOT_SMD:SOT-23_Handsoldering" H 2600 3900 50  0001 C CNN

Commit message: Work in progress
Parts:
- Q301, Q302: Feature (none) -> PWM_SUPPORTED_2STRIPS; Price (none) -> 0.0146; is stock (none) -> yes
- Q303, Q304: Feature (none) -> PWM_SUPPORTED_4STRIPS; Price (none) -> 0.0146; is stock (none) -> yes
Changed lines of the file:
@@
 $Descr A4 11693 8268
 encoding utf-8
-Sheet 5 14
+Sheet 3 14
 Title ""
 Date ""
@@
 F 2 "Package_TO_SOT_SMD:SOT-23_Handsoldering" H 7850 3900 50  0001 C CNN
 F 3 "~" H 7650 3800 50  0001 C CNN
+F 4 "PWM_SUPPORTED_4STRIPS" H 7650 3800 50  0001 C CNN "Feature"
+F 5 "0.0146" H 7650 3800 50  0001 C CNN "Price"
+F 6 "yes" H 7650 3800 50  0001 C CNN "is stock"
 	1    7650 3800
 	1    0    0    -1
@@
 F 2 "Package_TO_SOT_SMD:SOT-23_Handsoldering" H 6100 3900 50  0001 C CNN
 F 3 "~" H 5900 3800 50  0001 C CNN
+F 4 "PWM_SUPPORTED_4STRIPS" H 5900 3800 50  0001 C CNN "Feature"
+F 5 "0.0146" H 5900 3800 50  0001 C CNN "Price"
+F 6 "yes" H 5900 3800 50  0001 C CNN "is stock"
 	1    5900 3800
 	1    0    0    -1
@@
 F 2 "Package_TO_SOT_SMD:SOT-23_Handsoldering" H 4350 3900 50  0001 C CNN
 F 3 "~" H 4150 3800 50  0001 C CNN
+F 4 "PWM_SUPPORTED_2STRIPS" H 4150 3800 50  0001 C CNN "Feature"
+F 5 "0.0146" H 4150 3800 50  0001 C CNN "Price"
+F 6 "yes" H 4150 3800 50  0001 C CNN "is stock"
 	1    4150 3800
 	1    0    0    -1
@@
 F 2 "Package_TO_SOT_SMD:SOT-23_Handsoldering" H 2600 3900 50  0001 C CNN
 F 3 "~" H 2400 3800 50  0001 C CNN
+F 4 "PWM_SUPPORTED_2STRIPS" H 2400 3800 50  0001 C CNN "Feature"
+F 5 "0.0146" H 2400 3800 50  0001 C CNN "Price"
+F 6 "yes" H 2400 3800 50  0001 C CNN "is stock"
 	1    2400 3800
 	1    0    0    -1
