File: LedBarController/LedBarController.kicad_pcb (KiCad board)
At the start: 2 copper layers, 99.8 x 23.6 mm, 115 parts, among them J1001 Conn_01x03, J1002 Conn_01x03, J1003 Conn_01x03, J1004 Conn_01x03, J1005 Conn_01x06, J1006 Conn_01x06, J1101 Conn_01x02, J1102 Conn_01x02, J1201 Barrel_Jack_Switch, J1301 Screw_Terminal_01x03, J1302 Screw_Terminal_01x03, J201 Conn_01x05, J202 Conn_02x07_Odd_Even, J203 Conn_01x05, J701 Conn_01x05, J702 Conn_01x05, J703 Conn_01x05, J801 Conn_01x05, J802 Conn_02x07_Odd_Even, J803 Conn_01x05, J804 Conn_01x05, J805 Conn_01x05, J901 Conn_01x05, J902 Conn_01x05, J903 Conn_01x05, Q1201 FQP47P06, Q301 Si2302DS, Q302 Si2302DS, Q303 Si2302DS, Q304 Si2302DS, Q401 Si2302DS, Q402 Si2302DS, Q403 Si2302DS, Q404 Si2302DS, Q501 Si2302DS, Q502 Si2302DS, Q503 Si2302DS, Q504 Si2302DS, Q601 Si2302DS, Q602 Si2302DS, Q603 Si2302DS, Q604 Si2302DS, SW1001 SW_Push, SW801 SW_Push, U1001 ATmega328P-AU, U1101 LM358, U1201 AMS1117-5.0, U1301 MAX485E, U201 PCA9685PW, Y1001 Crystal

Commit message: Changed components and moved center connector upwards
Parts:
- C1001, C1002, C1003, C1004, C1005, R1002, R1005, U1001: moved to B.Cu
- J1005: value Conn_01x06 -> AVR-ISP-6; footprint Connector_PinSocket_2.54mm:PinSocket_1x06_P2.54mm_Vertical -> Connector_PinSocket_1.27mm:PinSocket_1x06_P1.27mm_Vertical
- SW1001, SW801: footprint Button_Switch_SMD:SW_Push_1P1T_NO_CK_KSC7xxJ -> Button_Switch_SMD:SW_SPST_SKQG_WithStem
- moved J802 197.2 mm to (150.1, 28.1)
- moved J803 190.2 mm to (157.4, 26.0)
- moved J801 187.3 mm to (157.4, 37.0)
- moved J805 186.1 mm to (144.0, 37.0)
- moved J804 180.9 mm to (144.0, 26.0)
- moved SW801 174.9 mm to (151.1, 44.5)
- moved J1005 114.1 mm to (69.7, 100.3), turned to 90 degrees
- moved C1002 111.3 mm to (77.1, 96.1), turned to 315 degrees
- moved J1006 110.4 mm to (54.6, 37.3), turned to 90 degrees
- moved Y1001 108.3 mm to (62.7, 100.6), turned to 270 degrees
- moved U1001 108.2 mm to (72.4, 100.5), turned to 45 degrees
- moved R1002 100.1 mm to (76.7, 123.2), turned to 90 degrees
- moved SW1001 99.4 mm to (72.9, 105.5)
- moved C1003 99.1 mm to (64.8, 104.9), turned to 315 degrees
- moved C1001 98.9 mm to (69.1, 106.2), turned to 315 degrees
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Connections:
- U201 pad 1: +5V -> GND
- U201 pad 3: +5V -> GND
- U201 pad 5: +5V -> GND
Routing:
- net /Microcontroller/Reset: track 0.00 -> 31.7 mm, vias 0 -> 1
- net +5V: track 26.7 -> 45.6 mm
- net /Microcontroller/MOSI: track 0.00 -> 17.2 mm, vias 0 -> 1
- net GND: track 186.7 -> 199.8 mm, vias 7 -> 10
- net /Microcontroller/Rx_: track 0.00 -> 12.4 mm
- net /Microcontroller/Tx: track 0.00 -> 11.4 mm
- net /Microcontroller/TxEn: track 0.00 -> 9.51 mm
- net /Microcontroller/I2C_SCL: track 0.00 -> 8.18 mm
- net /Microcontroller/I2C_SDA: track 0.00 -> 7.42 mm
- net /Microcontroller/button: track 39.5 -> 46.4 mm
- net Net-(C1003-Pad1): track 0.00 -> 6.65 mm
- net /PWM/CenterStrips/red_left_: track 0.00 -> 6.47 mm
- net /PWM/CenterStrips/green_left_: track 0.00 -> 6.47 mm
- net /PWM/CenterStrips/blue_left_: track 0.00 -> 6.47 mm
- net Net-(C1004-Pad1): track 0.00 -> 6.00 mm
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Other:
- board size 99.8 x 23.6 mm -> 146.8 x 25 mm

Commit message: Routed center board
Parts:
- J802: moved to B.Cu
- moved J804 12.9 mm to (156.9, 26.0)
- moved J803 12.1 mm to (145.3, 26.0)
- moved J802 2.00 mm to (152.1, 28.1), turned to 180 degrees
- moved J805 1.30 mm to (145.3, 37.0)
- moved J801 0.50 mm to (156.9, 37.0)
Routing:
- net /PWM/CenterStrips/red_right_: track 0.00 -> 16.8 mm
- net /PWM/CenterStrips/white_right_: track 0.00 -> 16.5 mm
- net /PWM/CenterStrips/blue_right_: track 0.00 -> 16.3 mm
- net /PWM/CenterStrips/white_left_: track 0.00 -> 16.1 mm
- net /PWM/CenterStrips/GND_: track 0.00 -> 16.1 mm
- net /PWM/CenterStrips/green_right_: track 0.00 -> 16.0 mm
- net /PWM/CenterStrips/red_left_: track 6.47 -> 16.7 mm
- net /PWM/CenterStrips/button_: track 0.00 -> 10.0 mm
- net /PWM/CenterStrips/blue_left_: track 6.47 -> 16.2 mm
- net /PWM/CenterStrips/green_left_: track 6.47 -> 15.9 mm
- net /PWM/CenterStrips/VDD_: track 0.00 -> 7.85 mm, vias 0 -> 2
- added copper zone on B.Cu, net /PWM/CenterStrips/VDD_
- added copper zone on F.Cu, net /PWM/CenterStrips/VDD_
Other:
- board size 146.8 x 25 mm -> 132.1 x 25 mm

Commit message: Added side boards
Parts:
- J701, J901: moved to B.Cu
- moved J902 203.5 mm to (169.9, 26.0)
- moved J901 201.4 mm to (163.8, 28.6), turned to 180 degrees
- moved J903 199.4 mm to (169.9, 37.0)
- moved J703 179.7 mm to (132.3, 37.0)
- moved J701 176.0 mm to (138.4, 28.6), turned to 180 degrees
- moved J702 173.5 mm to (132.3, 26.0)
Routing:
- net /PWM/SideStrip_right/green_: track 0.00 -> 19.0 mm
- net /PWM/SideStrip_left/red_: track 0.00 -> 18.8 mm
- net /PWM/SideStrip_left/green_: track 0.00 -> 18.8 mm
- net /PWM/SideStrip_left/blue_: track 0.00 -> 18.8 mm
- net /PWM/SideStrip_right/red_: track 0.00 -> 18.7 mm
- net /PWM/SideStrip_right/blue_: track 0.00 -> 18.7 mm
- net /PWM/SideStrip_left/white_: track 0.00 -> 18.7 mm
- net /PWM/SideStrip_right/white_: track 0.00 -> 18.6 mm
- net /PWM/CenterStrips/GND_: track 16.1 -> 16.9 mm
- added copper zone on B.Cu, net /PWM/SideStrip_left/VDD_
- added copper zone on F.Cu, net /PWM/SideStrip_left/VDD_
- added copper zone on B.Cu, net /PWM/SideStrip_right/VDD_
- added copper zone on F.Cu, net /PWM/SideStrip_right/VDD_
Other:
- board size 132.1 x 25 mm -> 145.1 x 25 mm
- board text added: "TODO: dead-end"

Commit message: Updated schematic, added ds1307, replaced gpio-headers for LEDs and solder-jumpers and remove ISP-connector
Parts:
- removed C1005: C, Capacitor_SMD:C_0805_2012Metric_Pad1.18x1.45mm_HandSolder
- removed J1001, J1002, J1003, J1004: Conn_01x03, Connector_PinSocket_2.54mm:PinSocket_1x03_P2.54mm_Vertical
- removed J1006: Conn_01x06, Connector_PinHeader_2.54mm:PinHeader_1x06_P2.54mm_Vertical
- removed TP1001: ~PWM_OE, TestPoint:TestPoint_Pad_D1.0mm
- removed TP1002: SCA, TestPoint:TestPoint_Pad_D1.0mm
- removed TP1003: SCL, TestPoint:TestPoint_Pad_D1.0mm
- added C1007: 100nF, Capacitor_SMD:C_0805_2012Metric_Pad1.18x1.45mm_HandSolder, F.Cu at (121.1, 83.3)
- added D1003: LED, LED_SMD:LED_0805_2012Metric_Pad1.15x1.40mm_HandSolder, F.Cu at (130.7, 83.3)
- added D1004: LED, LED_SMD:LED_0805_2012Metric_Pad1.15x1.40mm_HandSolder, F.Cu at (121.1, 86.4)
- added D1005: LED, LED_SMD:LED_0805_2012Metric_Pad1.15x1.40mm_HandSolder, F.Cu at (125.9, 86.4)
- added D1006: 1N5819, Diode_SMD:D_SOD-123, F.Cu at (115.8, 83.5)
- added JP1001: SolderJumper_2_Open, Jumper:SolderJumper-2_P1.3mm_Open_TrianglePad1.0x1.5mm, F.Cu at (135.3, 84.3)
- added JP1002: SolderJumper_2_Open, Jumper:SolderJumper-2_P1.3mm_Open_TrianglePad1.0x1.5mm, F.Cu at (134.9, 87.8)
- added JP1003: SolderJumper_2_Open, Jumper:SolderJumper-2_P1.3mm_Open_TrianglePad1.0x1.5mm, F.Cu at (139.6, 84.3)
- added JP1004: SolderJumper_2_Open, Jumper:SolderJumper-2_P1.3mm_Open_TrianglePad1.0x1.5mm, F.Cu at (139.2, 87.8)
- added RN1001: 1k, Resistor_SMD:R_Array_Concave_4x0603, F.Cu at (115.2, 75.3)
- added RN1002: 10k, Resistor_SMD:R_Array_Concave_4x0603, F.Cu at (115.2, 79.6)
- added U1002: DS1307ZN+, Package_SO:SOIC-8_3.9x4.9mm_P1.27mm, F.Cu at (139.4, 76.3)
- added Y1002: 32.768kHz, Crystal:Crystal_DS26_D2.0mm_L6.0mm_Vertical, F.Cu at (129.6, 87.1)
- D1001: value Blue -> LED
- R1001: value 330 -> 100R
- SW1001: value SW_Push -> reset
- moved D1001 176.2 mm to (125.9, 83.3), turned to 0 degrees
- moved R1001 165.8 mm to (115.3, 86.6), turned to 0 degrees
- moved R1004 155.0 mm to (137.6, 81.0)
Connections:
- net /Microcontroller/MISO renamed /Microcontroller/isp_miso
- net /Microcontroller/MOSI renamed /Microcontroller/isp_mosi
- net /Microcontroller/Reset renamed /Microcontroller/reset
- net /Microcontroller/Tx renamed /RS485/Tx
- net Net-(C1002-Pad1) renamed /Microcontroller/aref
- C1006 pad 1: /Microcontroller/ADC_PWR -> /Microcontroller/adc_vdd
- D1002 pad 2: /Microcontroller/ADC_PWR -> /Microcontroller/adc_vdd
- J1005 pad 3: /Microcontroller/SCK -> /Microcontroller/isp_sck
- R1001 pad 1: /Microcontroller/SCK -> Net-(C1005-Pad1)
- R1001 pad 2: Net-(D1001-Pad2) -> Net-(R1001-Pad2)
- R1002 pad 2: /Microcontroller/I2C_SCL -> /Microcontroller/I2C_SDA
- R1003 pad 2: /Microcontroller/I2C_SDA -> /Microcontroller/I2C_SCL
- R1004 pad 1: /Microcontroller/Rx -> +5V
- R1004 pad 2: /Microcontroller/Rx_ -> /Microcontroller/rtc_sqw
- R1007 pad 2: /Microcontroller/ADC_PWR -> /Microcontroller/adc_vdd
- R1008 pad 1: /Microcontroller/ADC_PWR -> /Microcontroller/adc_vdd
- TP1004 pad 1: /Microcontroller/ADC_PWR -> /Microcontroller/adc_vdd
- TP1302 pad 1: /Microcontroller/Rx -> /RS485/Rx
- TP1305 pad 1: /Microcontroller/TxEn -> /RS485/TxEn
- U1001 pad 1: /Microcontroller/button -> /RS485/TxEn
- U1001 pad 10: /Microcontroller/GPIO3 -> /Microcontroller/addr2
- U1001 pad 11: /Microcontroller/GPIO4 -> /Microcontroller/addr3
- U1001 pad 12: (no net) -> /Microcontroller/addr4
- U1001 pad 13: (no net) -> /Microcontroller/button
- U1001 pad 14: /PWM/~OE -> /Microcontroller/led1
- U1001 pad 17: /Microcontroller/SCK -> /Microcontroller/isp_sck
- U1001 pad 19: /Microcontroller/ADC_PWR -> (no net)
- U1001 pad 2: /Microcontroller/GPIO1 -> /PWM/~OE
- U1001 pad 22: (no net) -> /Microcontroller/adc_vdd
- U1001 pad 30: /Microcontroller/Rx_ -> /RS485/Rx
- U1001 pad 32: /Microcontroller/TxEn -> /Microcontroller/rtc_sqw
- U1001 pad 9: /Microcontroller/GPIO2 -> /Microcontroller/addr1
- U1301 pad 1: /Microcontroller/Rx -> /RS485/Rx
- U1301 pad 2: /Microcontroller/TxEn -> /RS485/TxEn
- U1301 pad 3: /Microcontroller/TxEn -> /RS485/TxEn
Routing:
- net /Microcontroller/Reset: track 0.00 -> 19.0 mm
- net /Microcontroller/reset: track 31.7 -> 12.7 mm
- net /Microcontroller/MOSI: track 0.00 -> 11.5 mm
- net /Microcontroller/isp_mosi: track 17.2 -> 5.65 mm
- net /RS485/Tx: track 11.4 -> 0.00 mm
- net /Microcontroller/Tx: track 0.00 -> 11.4 mm

Commit message: Added missing capacitor for MAX485
Parts:
- removed C1007: 100nF, Capacitor_SMD:C_0805_2012Metric_Pad1.18x1.45mm_HandSolder
- removed D1006: 1N5819, Diode_SMD:D_SOD-123
- removed R1001: 100R, Resistor_SMD:R_0805_2012Metric_Pad1.20x1.40mm_HandSolder
- removed R1004: R, Resistor_SMD:R_0805_2012Metric_Pad1.20x1.40mm_HandSolder
- removed U1002: DS1307ZN+, Package_SO:SOIC-8_3.9x4.9mm_P1.27mm
- removed Y1002: 32.768kHz, Crystal:Crystal_DS26_D2.0mm_L6.0mm_Vertical
- added C1301: 0.1uF, Capacitor_SMD:C_0805_2012Metric_Pad1.18x1.45mm_HandSolder, F.Cu at (-55.1, 32.8)
- added C1402: 100nF, Capacitor_SMD:C_0805_2012Metric_Pad1.18x1.45mm_HandSolder, F.Cu at (70.8, -46.7)
- added C1403: 0.1uF, Capacitor_SMD:C_0805_2012Metric_Pad1.18x1.45mm_HandSolder, F.Cu at (68.1, -40.2)
- added D1401: 1N5819, Diode_SMD:D_SOD-123, F.Cu at (62.8, -40.1)
- added R1401: 100R, Resistor_SMD:R_0805_2012Metric_Pad1.20x1.40mm_HandSolder, F.Cu at (70.7, -43.7)
- added R1402: 10k, Resistor_SMD:R_0805_2012Metric_Pad1.20x1.40mm_HandSolder, F.Cu at (72.8, -40.8)
- added U1401: DS1307ZN+, Package_SO:SOIC-8_3.9x4.9mm_P1.27mm, F.Cu at (64.1, -45.0)
- added Y1401: 32.768kHz, Crystal:Crystal_DS26_D2.0mm_L6.0mm_Vertical, F.Cu at (74.4, -46.0)
- U1301: footprint Package_TO_SOT_SMD:SOT-23-8_Handsoldering -> Package_SO:SOP-8_3.76x4.96mm_P1.27mm
- moved TP1305 67.2 mm to (-67.3, 36.8)
- moved TP1302 57.9 mm to (-63.2, 34.5)
- moved TP1303 53.5 mm to (-63.5, 38.9)
- moved JP1301 52.4 mm to (-48.0, 31.5)
- moved TP1301 48.9 mm to (-39.9, 27.4)
- moved R1303 48.2 mm to (-45.0, 27.4), turned to 90 degrees
- moved U1301 40.7 mm to (-56.6, 36.8)
- moved R1302 40.4 mm to (-48.0, 39.1), turned to 270 degrees
- moved R1301 34.0 mm to (-46.0, 40.1), turned to 90 degrees
- moved TP1304 32.1 mm to (-42.4, 40.1)
- moved R1005 21.4 mm to (48.3, 97.8)
Connections:
- net /0-10V/0-10Va1 renamed /Microcontroller/0_10v_ain_1
- net /0-10V/0-10Va2 renamed /Microcontroller/0_10v_ain_2
- net /0-10V/0-10Vd1 renamed /Microcontroller/0_10v_dout_1
- net /0-10V/0-10Vd2 renamed /Microcontroller/0_10v_dout_2
- net /Microcontroller/I2C_SCL renamed /Microcontroller/scl
- net /Microcontroller/I2C_SDA renamed /Microcontroller/sda
- net /PWM/~OE renamed /PWM/~oe
- net /RS485/Rx renamed /Microcontroller/rxd
- net /RS485/Tx renamed /Microcontroller/txd
- net /RS485/TxEn renamed /Microcontroller/tx_en
Routing:
- net /RS485/B: track 105.8 -> 134.7 mm
- net /RS485/A: track 100.7 -> 125.2 mm
- net GND: track 199.8 -> 178.2 mm, vias 10 -> 7
- net /Microcontroller/Reset: track 19.0 -> 0.00 mm
- net /Microcontroller/Rx_: track 12.4 -> 0.00 mm
- net /Microcontroller/MOSI: track 11.5 -> 0.00 mm
- net /Microcontroller/Tx: track 11.4 -> 0.00 mm
- net /Microcontroller/tx_en: track 0.00 -> 9.66 mm
- net /Microcontroller/TxEn: track 9.51 -> 0.00 mm
- net /Microcontroller/scl: track 8.18 -> 0.00 mm
- net /Microcontroller/sda: track 7.42 -> 0.00 mm
- net /Microcontroller/adc_vdd: track 0.00 -> 7.36 mm
- net /Microcontroller/button: track 46.4 -> 39.5 mm
- net /Microcontroller/SCK: track 5.52 -> 0.00 mm, vias 1 -> 0
- net /Microcontroller/txd: track 0.00 -> 4.37 mm
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
Commit message: routed RS485 circuit
Parts:
- R1301, R1302, TP1301, TP1304: moved to B.Cu
- moved TP1305 119.6 mm to (49.8, 61.2), turned to 180 degrees
- moved TP1302 112.7 mm to (45.7, 63.5), turned to 180 degrees
- moved TP1303 111.3 mm to (46.0, 59.2), turned to 180 degrees
- moved U1301 98.9 mm to (42.2, 39.9), turned to 180 degrees
- moved C1301 96.2 mm to (40.4, 44.5), turned to 0 degrees
- moved JP1301 85.2 mm to (36.6, 41.4), turned to 180 degrees
- moved R1303 83.3 mm to (36.6, 44.5), turned to 0 degrees
- moved R1302 81.8 mm to (33.8, 38.9), turned to 180 degrees
- moved R1301 79.8 mm to (33.8, 42.7), turned to 180 degrees
- moved TP1304 75.5 mm to (33.0, 36.8), turned to 180 degrees
- moved TP1301 74.7 mm to (32.8, 44.7), turned to 180 degrees
- moved J1302 5.08 mm to (30.7, 37.6), turned to 270 degrees
Routing:
- net /RS485/B: track 134.7 -> 112.0 mm
- net GND: track 178.2 -> 161.7 mm
- net /RS485/A: track 125.2 -> 109.5 mm
- net +5V: track 44.4 -> 33.5 mm
- net Net-(JP1301-Pad2): track 4.08 -> 1.78 mm

Commit message: Routed LEDs and solder jumpers, renumbered diodes (and LEDs) on microcontroller schematic
Parts:
- C1301, JP1001, JP1002, JP1003, JP1004, R1303: moved to B.Cu
- moved JP1004 108.8 mm to (39.6, 44.1), turned to 90 degrees
- moved JP1002 107.0 mm to (37.1, 44.5), turned to 90 degrees
- moved JP1003 103.4 mm to (44.7, 43.3), turned to 90 degrees
- moved JP1001 101.6 mm to (42.2, 43.7), turned to 90 degrees
- moved D1002 100.4 mm to (37.8, 45.2), turned to 90 degrees
- moved D1001 97.8 mm to (35.8, 45.2), turned to 90 degrees
- moved D1004 93.5 mm to (41.9, 45.2), turned to 90 degrees
- moved D1003 91.1 mm to (39.9, 45.2), turned to 90 degrees
- moved RN1001 76.9 mm to (44.6, 44.7), turned to 180 degrees
- moved C1301 4.68 mm to (39.4, 39.9), turned to 90 degrees
- moved R1303 4.52 mm to (33.8, 40.9)
- moved TP1301 0.68 mm to (33.4, 45.0)
- moved R1301 0.25 mm to (33.8, 42.9)
- renumbered D1003 to D1002, D1004 to D1003, D1005 to D1004, D1002 to D1005
Routing:
- net +5V: track 33.5 -> 53.5 mm, vias 0 -> 1
- net /RS485/A: track 109.5 -> 120.3 mm
- net Net-(D1001-Pad2): track 0.00 -> 8.15 mm
- net Net-(D1002-Pad2): track 0.00 -> 5.77 mm
- net /Microcontroller/addr2: track 0.00 -> 5.58 mm
- net /Microcontroller/addr4: track 0.00 -> 5.49 mm
- net /Microcontroller/tx_en: track 9.66 -> 5.21 mm
- net /Microcontroller/rxd: track 4.22 -> 0.00 mm
- net Net-(D1003-Pad2): track 0.00 -> 4.22 mm
- net /Microcontroller/addr1: track 0.00 -> 3.88 mm
- net /RS485/B: track 112.0 -> 114.2 mm, vias 0 -> 1
- net GND: track 161.7 -> 163.8 mm, vias 7 -> 10
Other:
- board text added: "-"
- board text added: "A"
- board text added: "B"
- board text added: "GND"
- board text added: "TODO: move LEDs upwards, increase coardyard of jumer?"

Commit message: Routed resistor-pack
Parts:
- RN1002: moved to B.Cu
- moved RN1002 75.7 mm to (48.5, 43.7), turned to 180 degrees
- moved JP1002 5.14 mm to (42.2, 43.7)
- moved JP1003 5.13 mm to (39.6, 44.0)
- moved JP1004 2.58 mm to (37.1, 44.5)
- moved JP1001 2.57 mm to (44.7, 43.3)
Connections:
- RN1001 pad 2: Net-(D1001-Pad2) -> /Microcontroller/isp_sck
- RN1001 pad 3: /Microcontroller/isp_mosi -> /Microcontroller/isp_miso
- RN1001 pad 4: Net-(D1002-Pad2) -> /Microcontroller/isp_mosi
- RN1001 pad 5: /Microcontroller/isp_miso -> Net-(D1002-Pad2)
- RN1001 pad 7: /Microcontroller/isp_sck -> Net-(D1004-Pad2)
- RN1001 pad 8: Net-(D1004-Pad2) -> Net-(D1001-Pad2)
- RN1002 pad 2: /Microcontroller/addr1 -> GND
- RN1002 pad 4: /Microcontroller/addr2 -> GND
- RN1002 pad 5: GND -> /Microcontroller/addr4
- RN1002 pad 7: GND -> /Microcontroller/addr2
- RN1002 pad 8: /Microcontroller/addr4 -> /Microcontroller/addr1
Routing:
- net /Microcontroller/addr3: track 0.00 -> 11.8 mm
- net /Microcontroller/addr4: track 5.49 -> 13.5 mm
- net GND: track 163.8 -> 171.6 mm, vias 10 -> 12
- net /Microcontroller/addr2: track 5.58 -> 9.94 mm
- net Net-(D1004-Pad2): track 0.00 -> 2.20 mm
- net /Microcontroller/addr1: track 3.88 -> 2.14 mm
- net Net-(D1001-Pad2): track 8.15 -> 9.08 mm
- net Net-(D1002-Pad2): track 5.77 -> 6.65 mm
- net Net-(D1003-Pad2): track 4.22 -> 4.92 mm
Other:
- board text added: "TODO: Place here some text about how to use this and where to find additional information. line 5 line 4"
