File: LedBarController/LedBarController.kicad_pcb (KiCad board)
At the start: 2 copper layers, 145.1 x 25 mm, 121 parts, among them J1005 AVR-ISP-6, J1101 Conn_01x02, J1102 Conn_01x02, J1201 Barrel_Jack_Switch, J1301 Screw_Terminal_01x03, J1302 Screw_Terminal_01x03, J201 Conn_01x05, J202 Conn_02x07_Odd_Even, J203 Conn_01x05, J701 Conn_01x05, J702 Conn_01x05, J703 Conn_01x05, J801 Conn_01x05, J802 Conn_02x07_Odd_Even, J803 Conn_01x05, J804 Conn_01x05, J805 Conn_01x05, J901 Conn_01x05, J902 Conn_01x05, J903 Conn_01x05, Q1201 FQP47P06, Q301 Si2302DS, Q302 Si2302DS, Q303 Si2302DS, Q304 Si2302DS, Q401 Si2302DS, Q402 Si2302DS, Q403 Si2302DS, Q404 Si2302DS, Q501 Si2302DS, Q502 Si2302DS, Q503 Si2302DS, Q504 Si2302DS, Q601 Si2302DS, Q602 Si2302DS, Q603 Si2302DS, Q604 Si2302DS, SW1001 reset, SW801 SW_Push, U1001 ATmega328P-AU, U1101 LM358, U1201 AMS1117-5.0, U1301 MAX485E, U1401 DS1307ZN+, U201 PCA9685PW, Y1001 Crystal, Y1401 32.768kHz

Commit message: Added INA219 current/voltage sensor
Parts:
- added C1206: 1uF/ceramic, Capacitor_SMD:C_0805_2012Metric_Pad1.18x1.45mm_HandSolder, F.Cu at (80.0, 28.6)
- added C1207: 0.1uF, Capacitor_SMD:C_0805_2012Metric_Pad1.18x1.45mm_HandSolder, F.Cu at (77.1, 31.5)
- added R1204: 10R, Resistor_SMD:R_0805_2012Metric_Pad1.20x1.40mm_HandSolder, F.Cu at (81.0, 31.5)
- added R1205: 10R, Resistor_SMD:R_0805_2012Metric_Pad1.20x1.40mm_HandSolder, F.Cu at (79.1, 31.5)
- added R1206: R001/2W, Resistor_SMD:R_2512_6332Metric_Pad1.40x3.35mm_HandSolder, B.Cu at (80.0, 29.6)
- added U1202: INA219AxD, Package_SO:SOIC-8_3.9x4.9mm_P1.27mm, B.Cu at (79.2, 38.5)
- C1204: footprint Capacitor_THT:CP_Radial_D6.3mm_P2.50mm -> Capacitor_SMD:C_1206_3216Metric_Pad1.33x1.80mm_HandSolder; moved to B.Cu
- C1402, C1403, C201, C204, D1401, R1401, R1402, U1401: moved to B.Cu
- moved C201 111.9 mm to (109.2, 32.3), turned to 270 degrees
- moved C204 94.1 mm to (91.7, 32.1), turned to 270 degrees
- moved Y1401 78.0 mm to (38.6, 23.3), turned to 90 degrees
- moved C1402 69.5 mm to (53.2, 20.5)
- moved U1401 69.3 mm to (43.0, 21.0)
- moved R1401 63.7 mm to (53.2, 17.6)
- moved R1402 58.1 mm to (55.3, 14.6)
- moved C1403 57.1 mm to (50.5, 14.1)
- moved D1401 56.8 mm to (45.2, 13.9)
- moved D1202 25.4 mm to (12.4, 4.78)
- moved C1204 16.3 mm to (63.8, 31.4), turned to 90 degrees
- moved R1201 9.63 mm to (70.5, 31.3)
- moved C1102 8.11 mm to (75.6, 56.5)
- moved C1103 8.11 mm to (79.7, 56.5)
- moved R1101 8.11 mm to (69.7, 58.5)
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Connections:
- C1201 pad 1: VDD -> Net-(C1201-Pad1)
- D1201 pad 1: VDD -> Net-(C1201-Pad1)
- Q1201 pad 3: VDD -> Net-(C1201-Pad1)
Routing:
- net Net-(C1201-Pad1): track 0.00 -> 33.0 mm, vias 0 -> 1
- net +5V: track 53.5 -> 80.0 mm, vias 1 -> 2
- net GND: track 171.6 -> 197.8 mm, vias 12 -> 14
- net VDD: track 35.9 -> 52.0 mm, vias 0 -> 1
- net Net-(C1202-Pad1): track 24.4 -> 12.4 mm
- net /Microcontroller/sda: track 0.00 -> 11.1 mm, vias 0 -> 1
- net /Microcontroller/scl: track 0.00 -> 8.57 mm, vias 0 -> 1
- net Net-(R1205-Pad2): track 0.00 -> 3.81 mm, vias 0 -> 1
- net Net-(R1204-Pad2): track 0.00 -> 3.55 mm, vias 0 -> 1
- net Net-(D1201-Pad2): track 7.23 -> 6.51 mm

Commit message: Work in progress
Parts:
- added C1005: 0.1uF, Capacitor_SMD:C_0805_2012Metric_Pad1.18x1.45mm_HandSolder, F.Cu at (76.5, 13.6)
- added C1208: 0.1uF, Capacitor_SMD:C_0805_2012Metric_Pad1.18x1.45mm_HandSolder, B.Cu at (75.5, 37.0)
- added C1401: 0.47F/5.5V, LedBarController:CP_Disc_D11.5mm_H12.3mm_P4.7mm_Vertical, F.Cu at (66.0, 17.0)
- added U1002: CAT24C256, Package_SO:SOIC-8_3.9x4.9mm_P1.27mm, F.Cu at (76.2, 17.3)
- C1003, C1004: value C -> 22pF
- C1006: value C -> 1uF
- C1101, C1103: value 0.1uF -> 1uF
- C1102, C1104, C1105, C1202, C1203, C203: value C -> 0.1uF
- C1204: value 100uF/35V -> 10uF/35V; footprint Capacitor_SMD:C_1206_3216Metric_Pad1.33x1.80mm_HandSolder -> Capacitor_Tantalum_SMD:CP_EIA-6032-28_Kemet-C_Pad2.25x2.35mm_HandSolder
- C1205: value 47uF/50V -> 10uF/10V; footprint Capacitor_SMD:C_1206_3216Metric_Pad1.33x1.80mm_HandSolder -> Capacitor_Tantalum_SMD:CP_EIA-3216-18_Kemet-A_Pad1.58x1.35mm_HandSolder
- C1206: value 1uF/ceramic -> 1uF
- C1402: value 100nF -> 0.1uF
- D1001: value LED -> Green
- D1002: value LED -> Yellow
- D1003: value LED -> Orange
- D1004: value LED -> Red
- D1005: value D -> 1N4148
- D1202: value LED -> Blue
- F1201: value Fuse -> 5A
- JP1001, JP1002, JP1003, JP1004: footprint Jumper:SolderJumper-2_P1.3mm_Open_TrianglePad1.0x1.5mm -> LedBarController:SolderJumper-2_P1.3mm_Open_TrianglePad1.0x1.5mm
- R1002, R1003: value R -> 4k7
- R1005, R1007: value R -> 10k
- R1006: value 10K -> 10k
- R1008: value R -> 1k8
- R1101, R1105: value 1k -> 10k
- R1203: value 330 -> 470R
- R1301, R1303: value 20K -> 1K
- RN1001: value 1k -> 470R
- TP1004: value ADC1 -> ADC_VDD
- TP1101: value 0-10Va1 -> a1
- TP1102: value 0-10Vd1 -> d1
- TP1103: value 0-10Va2 -> a2
- TP1104: value 0-10Vd2 -> d2
- U1101: value LM358 -> LM358DR
- Y1001: value Crystal -> 14.7456Mhz
- moved R1002 135.3 mm to (9.08, 5.95)
- moved R1005 134.7 mm to (-15.6, -20.8)
- moved C1001 113.8 mm to (-3.68, 18.7), turned to 135 degrees
- moved C1002 111.4 mm to (-11.7, 28.8), turned to 135 degrees
- moved U1001 109.9 mm to (-6.99, 24.4), turned to 225 degrees
- moved C1003 106.4 mm to (0.64, 20.0), turned to 135 degrees
- moved C1004 105.9 mm to (-0.89, 21.5), turned to 135 degrees
- moved J1005 98.9 mm to (-15.6, 50.3)
- moved SW1001 98.9 mm to (-12.4, 55.5)
- moved Y1001 98.9 mm to (-22.6, 50.5)
- moved R1006 97.2 mm to (3.05, 55.6)
- moved C1101 59.8 mm to (98.3, 2.87)
- moved C1102 59.8 mm to (102.1, 2.87)
- moved C1103 59.8 mm to (106.2, 2.87)
- moved R1101 59.8 mm to (96.2, 4.90)
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Routing:
- net GND: track 197.8 -> 226.1 mm, vias 14 -> 15
- net +5V: track 80.0 -> 64.1 mm, vias 2 -> 1
- net /Microcontroller/reset: track 12.7 -> 1.46 mm
- net Net-(C1202-Pad1): track 12.4 -> 19.1 mm
- net /Microcontroller/addr1: track 2.14 -> 6.26 mm
- net /Microcontroller/isp_mosi: track 5.65 -> 2.23 mm
- net /Microcontroller/addr4: track 13.1 -> 10.7 mm
- net Net-(U1401-Pad2): track 0.00 -> 2.04 mm
- net Net-(U1401-Pad1): track 0.00 -> 2.04 mm

Commit message: Changed Something dont known anymore
Parts:
- removed TP1004: ADC_VDD, TestPoint:TestPoint_Pad_D1.0mm
- removed TP1101: a1, TestPoint:TestPoint_Pad_D1.0mm
- removed TP1102: d1, TestPoint:TestPoint_Pad_D1.0mm
- removed TP1103: a2, TestPoint:TestPoint_Pad_D1.0mm
- removed TP1104: d2, TestPoint:TestPoint_Pad_D1.0mm
- removed TP1201: VDD, TestPoint:TestPoint_Pad_D1.0mm
- removed TP1202: 5V+, TestPoint:TestPoint_Pad_D1.0mm
- removed TP1203: GND, TestPoint:TestPoint_Pad_D1.0mm
- removed TP1302: Rx, TestPoint:TestPoint_Pad_D1.0mm
- removed TP1303: Tx, TestPoint:TestPoint_Pad_D1.0mm
- removed TP1305: TxEn, TestPoint:TestPoint_Pad_D1.0mm
- moved Y1001 82.8 mm to (59.6, 60.5), turned to 90 degrees
- moved C1004 71.3 mm to (60.5, 57.9), turned to 0 degrees
- moved C1001 68.6 mm to (56.8, 51.2)
- moved C1003 68.4 mm to (60.5, 53.2), turned to 0 degrees
- moved U1001 67.1 mm to (52.3, 55.8)
- moved C1002 66.8 mm to (47.4, 59.8)
- moved J1005 65.0 mm to (49.1, 55.8)
- moved SW1001 64.9 mm to (52.2, 61.0)
- moved R1006 49.3 mm to (52.3, 53.0)
- moved RN1002 3.96 mm to (43.2, 40.9)
- moved C1205 3.89 mm to (43.3, 27.3), turned to 180 degrees
- moved C1204 2.75 mm to (63.1, 29.6), turned to 90 degrees
- moved U1201 2.35 mm to (50.3, 29.2)
- moved C1202 2.16 mm to (58.5, 27.5)
- moved C1203 2.16 mm to (56.2, 27.5)
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Routing:
- net /Microcontroller/reset: track 1.46 -> 19.0 mm, vias 1 -> 0
- net GND: track 226.1 -> 215.8 mm, vias 15 -> 14
- net +5V: track 64.1 -> 57.3 mm
- net /Microcontroller/addr3: track 11.4 -> 4.77 mm
- net /Microcontroller/isp_miso: track 5.95 -> 0.00 mm
- net /Microcontroller/isp_sck: track 0.00 -> 5.51 mm
- net Net-(C1202-Pad1): track 19.1 -> 14.0 mm
- net /Microcontroller/addr4: track 10.7 -> 5.55 mm
- net /Microcontroller/txd: track 3.94 -> 0.00 mm
- net /Microcontroller/tx_en: track 5.21 -> 1.27 mm
- net /Microcontroller/addr2: track 9.66 -> 6.79 mm
- net /Microcontroller/addr1: track 6.26 -> 8.90 mm
- net /Microcontroller/isp_mosi: track 2.23 -> 4.87 mm, vias 1 -> 0
- net Net-(C1003-Pad1): track 6.65 -> 4.13 mm

Commit message: Reduced circuit by remove extra features. Routed whole board. Needs refinement
Parts:
- removed C1005, C1105, C1402, C1403: 0.1uF, Capacitor_SMD:C_0805_2012Metric_Pad1.18x1.45mm_HandSolder
- removed C1006, C1103: 1uF, Capacitor_SMD:C_0805_2012Metric_Pad1.18x1.45mm_HandSolder
- removed C1401: 0.47F/5.5V, LedBarController:CP_Disc_D11.5mm_H12.3mm_P4.7mm_Vertical
- removed D1005: 1N4148, Diode_SMD:D_1206_3216Metric_Pad1.42x1.75mm_HandSolder
- removed D1401: 1N5819, Diode_SMD:D_SOD-123
- removed J1102: Conn_01x02, Connector_JST:JST_PH_B2B-PH-K_1x02_P2.00mm_Vertical
- removed J1302: Screw_Terminal_01x03, TerminalBlock_TE-Connectivity:TerminalBlock_TE_282834-3_1x03_P2.54mm_Horizontal
- removed R1007, R1105, R1107, R1108, R1402: 10k, Resistor_SMD:R_0805_2012Metric_Pad1.20x1.40mm_HandSolder
- removed R1008: 1k8, Resistor_SMD:R_0805_2012Metric_Pad1.20x1.40mm_HandSolder
- removed R1106: 1k, Resistor_SMD:R_0805_2012Metric_Pad1.20x1.40mm_HandSolder
- removed R1401: 100R, Resistor_SMD:R_0805_2012Metric_Pad1.20x1.40mm_HandSolder
- removed U1002: CAT24C256, Package_SO:SOIC-8_3.9x4.9mm_P1.27mm
- removed U1401: DS1307ZN+, Package_SO:SOIC-8_3.9x4.9mm_P1.27mm
- removed Y1401: 32.768kHz, Crystal:Crystal_DS26_D2.0mm_L6.0mm_Vertical
- added TP1101: a1, TestPoint:TestPoint_Pad_D1.0mm, B.Cu at (66.4, 36.8)
- added TP1102: d1, TestPoint:TestPoint_Pad_D1.0mm, B.Cu at (62.8, 36.3)
- added TP1201: VDD, TestPoint:TestPoint_Pad_D1.0mm, B.Cu at (86.0, 26.5)
- added TP1202: 5V+, TestPoint:TestPoint_Pad_D1.0mm, B.Cu at (64.8, 34.7)
- added TP1203: GND, TestPoint:TestPoint_Pad_D1.0mm, B.Cu at (69.6, 36.8)
- D1202: footprint LED_THT:LED_D3.0mm -> LED_SMD:LED_0805_2012Metric_Pad1.15x1.40mm_HandSolder
- J201, J203: value Conn_01x05 -> Female pitch strip 1x7 pins 2.0mm pitch
- J202: value Conn_02x07_Odd_Even -> Female 2x7 pins 2.0mm pitch
- J701, J901: value Conn_01x05 -> Male pitch strip 1x7 pins 2.0mm pitch
- J802: value Conn_02x07_Odd_Even -> Male pitch strip 2x7pins 2.0mm pitch
- R1003: moved to B.Cu
- R1203: moved to F.Cu
- SW1001: value reset -> 4x42.3mm PCB Tactile Push Button Switch
- SW801: value SW_Push -> 4x42.3mm PCB Tactile Push Button Switch
- moved R1003 115.4 mm to (76.6, 44.1), turned to 90 degrees
- moved J1301 91.3 mm to (30.5, 42.7), turned to 90 degrees
- moved R1005 85.3 mm to (49.4, 34.4)
- moved R1002 79.2 mm to (78.5, 44.1)
- moved D1202 66.5 mm to (67.2, 42.5), turned to 90 degrees
- moved R1102 49.6 mm to (63.8, 44.3)
- moved U1101 48.4 mm to (69.5, 42.5)
- moved C1102 47.3 mm to (71.4, 38.8)
- moved C1101 47.3 mm to (67.5, 38.8)
- moved R1101 46.6 mm to (63.7, 38.3)
- moved R1104 46.5 mm to (63.8, 40.3)
- moved R1103 46.4 mm to (63.8, 42.3)
- moved R1203 36.7 mm to (65.8, 37.5)
- moved C1002 27.9 mm to (59.9, 34.9), turned to 315 degrees
- moved Y1001 24.4 mm to (48.5, 38.7), turned to 270 degrees
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Connections:
- RN1002 pad 5: /Microcontroller/addr4 -> /Microcontroller/addr1
- RN1002 pad 6: /Microcontroller/addr3 -> /Microcontroller/addr2
- RN1002 pad 7: /Microcontroller/addr2 -> /Microcontroller/addr3
- RN1002 pad 8: /Microcontroller/addr1 -> /Microcontroller/addr4
- U1001 pad 1: /Microcontroller/tx_en -> (no net)
- U1001 pad 22: /Microcontroller/adc_vdd -> (no net)
- U1001 pad 25: /Microcontroller/0_10v_dout_2 -> (no net)
- U1001 pad 26: /Microcontroller/0_10v_ain_2 -> (no net)
- U1001 pad 32: /Microcontroller/rtc_sqw -> /Microcontroller/tx_en
- U1101 pad 5: /Microcontroller/0_10v_ain_2 -> Net-(R1103-Pad1)
- U1101 pad 6: Net-(R1107-Pad1) -> Net-(U1101-Pad6)
- U1101 pad 7: Net-(R1106-Pad2) -> Net-(U1101-Pad6)
Routing:
- net /RS485/A: track 120.3 -> 17.0 mm
- net /RS485/B: track 114.2 -> 17.9 mm, vias 1 -> 0
- net GND: track 215.8 -> 310.9 mm, vias 14 -> 39
- net +5V: track 57.3 -> 138.2 mm, vias 1 -> 2
- net /Microcontroller/tx_en: track 1.27 -> 39.8 mm, vias 0 -> 1
- net /Microcontroller/txd: track 0.00 -> 35.9 mm, vias 0 -> 1
- net /Microcontroller/rxd: track 0.00 -> 34.7 mm, vias 0 -> 1
- net /PWM/~oe: track 0.00 -> 33.2 mm, vias 0 -> 1
- net /Microcontroller/button: track 39.5 -> 72.5 mm, vias 1 -> 2
- net /Microcontroller/scl: track 8.70 -> 35.9 mm
- net /Microcontroller/isp_sck: track 5.51 -> 32.3 mm
- net /Microcontroller/sda: track 10.8 -> 36.1 mm
- net /Microcontroller/isp_miso: track 0.00 -> 24.5 mm, vias 0 -> 2
- net VDD: track 52.0 -> 70.5 mm, vias 1 -> 2
- net /Microcontroller/led1: track 0.00 -> 18.3 mm, vias 0 -> 1
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
Commit message: Added surge protection
Parts:
- added D1203: SMBJ30CA CK, Diode_SMD:D_SMB_Handsoldering, B.Cu at (30.6, 30.7)
- moved R1201 0.06 mm to (70.5, 29.1)
- moved R1202 0.06 mm to (71.0, 33.3)
Connections:
- net Net-(F1201-Pad1) renamed /Power/surge_bypass
Routing:
- net /Power/surge_bypass: track 17.3 -> 67.8 mm, vias 0 -> 3
- net GND: track 310.9 -> 324.2 mm, vias 39 -> 40
Other:
- net class surge_bypass added: clearance 0.25, trace_width 2, via_dia 0.8, via_drill 0.4
- board text removed: "TODO: dead-end"

Commit message: Update silk layer
Parts:
- D1203: value SMBJ30CA CK -> SMBJ30CA CK /SMBJ15CA BM
- F1201: value 5A -> max. 5A F
- J1005: value AVR-ISP-6 -> ISP
- SW1001: value 4x42.3mm PCB Tactile Push Button Switch -> reset
- moved TP1203 26.9 mm to (42.7, 34.8)
- moved TP1202 22.1 mm to (42.7, 36.8)
- moved TP1201 5.55 mm to (91.4, 27.6)
- moved R1203 0.38 mm to (65.4, 37.5)
- moved D1202 0.13 mm to (67.1, 42.5)
- moved C203 0.10 mm to (68.3, 37.5)
Routing:
- net GND: track 324.2 -> 326.3 mm, vias 40 -> 45
Other:
- board text removed: "TODO: move LEDs upwards, increase coardyard of jumer?"

Commit message: Improved ISP connector silk layer
Parts:
- J1005: footprint Connector_PinSocket_1.27mm:PinSocket_1x06_P1.27mm_Vertical -> LedBarController:ISP_P1.27mm_single_row
- moved J1005 6.35 mm to (52.3, 39.4), turned to 90 degrees
Changed lines of the file:
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@@
     (add_net /Power/surge_bypass)
   )
+  (module LedBarController:ISP_P1.27mm_single_row (layer F.Cu)
+    (at 52.324 39.37 90)
+    (descr "Through hole straight socket strip, 1x06, 1.27mm pitch, single row (from Kicad 4.0.7), script generated")
+    (tags "Through hole socket strip THT 1x06 1.27mm single row")
+    (fp_text reference J1005 (at 2.286 7.493 90) (layer F.SilkS)
+      (effects (font (size 0.7 0.7) (thickness 0.15)))
+    )
+    (fp_text value ISP (at 0 8.485 90) (layer F.Fab)
+      (effects (font (size 1 1) (thickness 0.15)))
+    )
+    (fp_text user ISP (at -1.143 3.175 180) (layer F.SilkS)
+      (effects (font (size 0.7 0.7) (thickness 0.15)))
+    )
+    (fp_text user SCK (at 2.032 3.81 90) (layer F.SilkS)
+      (effects (font (size 0.7 0.7) (thickness 0.15)))
+    )
+    (fp_text user %R (at 0 3.175) (layer F.Fab)
+      (effects (font (size 1 1) (thickness 0.15)))
+    )
+    (fp_line (start 3.81 -0.635) (end 3.81 6.985) (layer F.CrtYd) (width 0.05))
+    (fp_line (start -1.75 -1.15) (end 1.778 -1.15) (layer F.CrtYd) (width 0.05))
+    (fp_line (start -1.75 7.5) (end -1.75 -1.15) (layer F.CrtYd) (width 0.05))
+    (fp_line (start 1.778 7.5) (end -1.75 7.5) (layer F.CrtYd) (width 0.05))
+    (fp_line (start 1.27 -0.635) (end 1.27 6.985) (layer F.Fab) (width 0.1))
+    (fp_line (start -1.27 -0.635) (end 1.27 -0.635) (layer F.Fab) (width 0.1))
+    (fp_line (start -1.27 6.35) (end -1.27 -0.635) (layer F.Fab) (width 0.1))
+    (fp_line (start -0.635 6.985) (end -1.27 6.35) (layer F.Fab) (width 0.1))
+    (fp_line (start 1.27 6.985) (end -0.635 6.985) (layer F.Fab) (width 0.1))
+    (fp_line (start -1.143 2.159) (end -1.143 -0.635) (layer F.SilkS) (width 0.12))
+    (fp_line (start -1.143 -0.635) (end 3.81 -0.635) (layer F.SilkS) (width 0.12))
+    (fp_line (start 3.81 -0.635) (end 3.81 6.985) (layer F.SilkS) (width 0.12))
+    (fp_line (start 3.81 6.985) (end -1.143 6.985) (layer F.SilkS) (width 0.12))
+    (fp_line (start -1.143 6.985) (end -1.143 4.191) (layer F.SilkS) (width 0.12))
+    (fp_line (start 1.778 -1.143) (end 1.778 -0.635) (layer F.CrtYd) (width 0.05))
+    (fp_line (start 1.778 -0.635) (end 3.81 -0.635) (layer F.CrtYd) (width 0.05))
+    (fp_line (start 1.778 7.493) (end 1.778 6.985) (layer F.CrtYd) (width 0.05))
+    (fp_line (start 1.778 6.985) (end 3.81 6.985) (layer F.CrtYd) (width 0.05))
+    (fp_text user GND (at 2.032 0 90) (layer F.SilkS)
+      (effects (font (size 0.7 0.7) (thickness 0.15)))
+    )
+    (fp_text user ~Reset (at 2.032 1.397 90) (layer F.SilkS)
+      (effects (font (size 0.7 0.7) (thickness 0.15)))
+    )
+    (fp_text user MOSI (at 1.905 2.54 90) (layer F.SilkS)
+      (effects (font (size 0.7 0.7) (thickness 0.15)))
+    )
+    (fp_text user +5V (at 2.032 5.08 90) (layer F.SilkS)
+      (effects (font (size 0.7 0.7) (thickness 0.15)))
+    )
+    (fp_text user MISO (at 2.032 6.35 90) (layer F.SilkS)
+      (effects (font (size 0.7 0.7) (thickness 0.15)))
+    )
+    (pad 6 thru_hole oval (at 0 0 270) (size 1 1) (drill 0.7) (layers *.Cu *.Mask)
+      (net 1 GND))
+    (pad 5 thru_hole oval (at 0 1.27 270) (size 1 1) (drill 0.7) (layers *.Cu *.Mask)
+      (net 74 /Microcontroller/reset))
+    (pad 4 thru_hole oval (at 0 2.54 270) (size 1 1) (drill 0.7) (layers *.Cu *.Mask)
+      (net 75 /Microcontroller/isp_mosi))
+    (pad 3 thru_hole oval (at 0 3.81 270) (size 1 1) (drill 0.7) (layers *.Cu *.Mask)
+      (net 76 /Microcontroller/isp_sck))
+    (pad 2 thru_hole oval (at 0 5.08 270) (size 1 1) (drill 0.7) (layers *.Cu *.Mask)
+      (net 3 +5V))
+    (pad 1 thru_hole rect (at 0 6.35 270) (size 1 1) (drill 0.7) (layers *.Cu *.Mask)
+      (net 77 /Microcontroller/isp_miso))
+    (model ${KISYS3DMOD}/Connector_PinSocket_1.27mm.3dshapes/PinSocket_1x06_P1.27mm_Vertical.wrl
+      (at (xyz 0 0 0))
+      (scale (xyz 1 1 1))
+      (rotate (xyz 0 0 0))
+    )
+  )
   (module Diode_SMD:D_SMB_Handsoldering (layer B.Cu)
     (at 30.607 30.734 270)
@@
       (effects (font (size 0.8 0.8) (thickness 0.15)))
     )
-    (fp_text value "max. 5A F" (at 7.874 -5.842) (layer F.SilkS)
+    (fp_text value "max. 5A F" (at -7.366 -15.875) (layer F.SilkS)
       (effects (font (size 1 1) (thickness 0.15)))
     )
@@
     )
   )
-  (module Connector_PinSocket_1.27mm:PinSocket_1x06_P1.27mm_Vertical (layer F.Cu)
-    (at 58.674 39.37 270)
-    (descr "Through hole straight socket strip, 1x06, 1.27mm pitch, single row (from Kicad 4.0.7), script generated")
-    (tags "Through hole socket strip THT 1x06 1.27mm single row")
-    (fp_text reference J1005 (at -1.778 3.429 180) (layer F.Fab)
-      (effects (font (size 1 1) (thickness 0.15)))
-    )
-    (fp_text value ISP (at -2.032 5.715 180) (layer F.SilkS)
-      (effects (font (size 1.3 1.3) (thickness 0.15)))
-    )
-    (fp_line (start -1.8 7.5) (end -1.8 -1.15) (layer F.CrtYd) (width 0.05))
-    (fp_line (start 1.75 7.5) (end -1.8 7.5) (layer F.CrtYd) (width 0.05))
-    (fp_line (start 1.75 -1.15) (end 1.75 7.5) (layer F.CrtYd) (width 0.05))
-    (fp_line (start -1.8 -1.15) (end 1.75 -1.15) (layer F.CrtYd) (width 0.05))
-    (fp_line (start 0 -0.76) (end 1.33 -0.76) (layer F.SilkS) (width 0.12))
-    (fp_line (start 1.33 -0.76) (end 1.33 0) (layer F.SilkS) (width 0.12))
-    (fp_line (start 1.33 0.635) (end 1.33 7.045) (layer F.SilkS) (width 0.12))
-    (fp_line (start 0.30753 7.045) (end 1.33 7.045) (layer F.SilkS) (width 0.12))
-    (fp_line (start -1.33 7.045) (end -0.30753 7.045) (layer F.SilkS) (width 0.12))
-    (fp_line (start -1.33 0.635) (end -1.33 7.045) (layer F.SilkS) (width 0.12))
-    (fp_line (start 0.76 0.635) (end 1.33 0.635) (layer F.SilkS) (width 0.12))
-    (fp_line (start -1.33 0.635) (end -0.76 0.635) (layer F.SilkS) (width 0.12))
-    (fp_line (start -1.27 6.985) (end -1.27 -0.635) (layer F.Fab) (width 0.1))
-    (fp_line (start 1.27 6.985) (end -1.27 6.985) (layer F.Fab) (width 0.1))
-    (fp_line (start 1.27 0) (end 1.27 6.985) (layer F.Fab) (width 0.1))
-    (fp_line (start 0.635 -0.635) (end 1.27 0) (layer F.Fab) (width 0.1))
-    (fp_line (start -1.27 -0.635) (end 0.635 -0.635) (layer F.Fab) (width 0.1))
-    (fp_text user %R (at 0 3.175) (layer F.Fab)
-      (effects (font (size 1 1) (thickness 0.15)))
-    )
-    (pad 6 thru_hole oval (at 0 6.35 270) (size 1 1) (drill 0.7) (layers *.Cu *.Mask)
-      (net 1 GND))
-    (pad 5 thru_hole oval (at 0 5.08 270) (size 1 1) (drill 0.7) (layers *.Cu *.Mask)
-      (net 74 /Microcontroller/reset))
-    (pad 4 thru_hole oval (at 0 3.81 270) (size 1 1) (drill 0.7) (layers *.Cu *.Mask)
-      (net 75 /Microcontroller/isp_mosi))
-    (pad 3 thru_hole oval (at 0 2.54 270) (size 1 1) (drill 0.7) (layers *.Cu *.Mask)
-      (net 76 /Microcontroller/isp_sck))
-    (pad 2 thru_hole oval (at 0 1.27 270) (size 1 1) (drill 0.7) (layers *.Cu *.Mask)
-      (net 3 +5V))
-    (pad 1 thru_hole rect (at 0 0 270) (size 1 1) (drill 0.7) (layers *.Cu *.Mask)
-      (net 77 /Microcontroller/isp_miso))
-    (model ${KISYS3DMOD}/Connector_PinSocket_1.27mm.3dshapes/PinSocket_1x06_P1.27mm_Vertical.wrl
-      (at (xyz 0 0 0))
-      (scale (xyz 1 1 1))
-      (rotate (xyz 0 0 0))
-    )
-  )
   (module Capacitor_THT:CP_Radial_D13.0mm_P5.00mm (layer F.Cu)
     (at 91.44 29.718 270)
@@
     (attr smd)
     (fp_text reference R1006 (at 0 -1.65 90) (layer F.SilkS)
-      (effects (font (size 1 1) (thickness 0.15)))
+      (effects (font (size 0.7 0.7) (thickness 0.15)))
     )
     (fp_text value 10k (at 0 1.65 90) (layer F.Fab)
@@
     )
   )
-  (gr_line (start 62.611 35.56) (end 55.118 35.56) (layer F.SilkS) (width 0.12))
-  (gr_line (start 55.118 36.83) (end 62.611 36.83) (layer F.SilkS) (width 0.12))
-  (gr_arc (start 55.118 36.195) (end 55.118 35.56) (angle -180) (layer F.SilkS) (width 0.12))
-  (gr_arc (start 62.611 36.195) (end 62.611 36.83) (angle -180) (layer F.SilkS) (width 0.12))
+  (gr_line (start 77.851 45.593) (end 70.358 45.593) (layer F.SilkS) (width 0.12))
+  (gr_line (start 70.358 46.863) (end 77.851 46.863) (layer F.SilkS) (width 0.12))
+  (gr_arc (start 70.358 46.228) (end 70.358 45.593) (angle -180) (layer F.SilkS) (width 0.12))
+  (gr_arc (start 77.851 46.228) (end 77.851 46.863) (angle -180) (layer F.SilkS) (width 0.12))
   (gr_line (start 42.545 42.926) (end 42.291 42.926) (layer F.SilkS) (width 0.12))
   (gr_line (start 42.545 42.926) (end 42.799 43.18) (layer F.SilkS) (width 0.12))
@@
   (segment (start 55.7007 37.2618) (end 55.18 37.7825) (width 0.2) (layer F.Cu) (net 77))
   (segment (start 57.3024 37.2618) (end 55.7007 37.2618) (width 0.2) (layer F.Cu) (net 77))
-  (segment (start 57.3024 37.9984) (end 58.674 39.37) (width 0.2) (layer B.Cu) (net 77))
-  (segment (start 57.3024 37.2618) (end 57.3024 37.9984) (width 0.2) (layer B.Cu) (net 77))
   (segment (start 45.739 44.304) (end 45.173 44.304) (width 0.2) (layer F.Cu) (net 77))
   (segment (start 45.923001 44.119999) (end 45.739 44.304) (width 0.2) (layer F.Cu) (net 77))
@@
   (segment (start 49.441688 40.863711) (end 50.658289 40.863711) (width 0.2) (layer F.Cu) (net 77))
   (segment (start 50.7775 40.7445) (end 50.65829 40.863711) (width 0.2) (layer F.Cu) (net 77))
+  (segment (start 57.3024 37.9984) (end 58.674 39.37) (width 0.2) (layer B.Cu) (net 77))
+  (segment (start 57.3024 37.2618) (end 57.3024 37.9984) (width 0.2) (layer B.Cu) (net 77))
   (segment (start 42.10799 42.64119) (end 42.1016 42.6348) (width 0.2) (layer B.Cu) (net 78))
   (segment (start 42.605789 42.64119) (end 42.10799 42.64119) (width 0.2) (layer B.Cu) (net 78))
