File: LedBarController/LedBarController.kicad_pcb (KiCad board)
At the start: 2 copper layers, 145.1 x 25 mm, 104 parts, among them J1005 ISP, J1101 Conn_01x02, J1201 Barrel_Jack_Switch, J1301 Screw_Terminal_01x03, J201 Female pitch strip 1x7 pins 2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, J202 Female 2x7 pins 2.0mm pitch, J203 Female pitch strip 1x7 pins 2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, J701 Male pitch strip 1x7 pins 2.0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, J702 Conn_01x05, J703 Conn_01x05, J801 Conn_01x05, J802 Male pitch strip 2x7pins 2.0m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, J803 Conn_01x05, J804 Conn_01x05, J805 Conn_01x05, J901 Male pitch strip 1x7 pins 2.0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, J902 Conn_01x05, J903 Conn_01x05, Q1201 FQP47P06, Q301 Si2302DS, Q302 Si2302DS, Q303 Si2302DS, Q304 Si2302DS, Q401 Si2302DS, Q402 Si2302DS, Q403 Si2302DS, Q404 Si2302DS, Q501 Si2302DS, Q502 Si2302DS, Q503 Si2302DS, Q504 Si2302DS, Q601 Si2302DS, Q602 Si2302DS, Q603 Si2302DS, Q604 Si2302DS, SW1001 reset, SW801 4x42.3mm PCB Tactile Push But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, U1001 ATmega328P-AU, U1101 LM358DR, U1201 AMS1117-5.0, U1202 INA219AxD, U1301 MAX485E, U201 PCA9685PW, Y1001 14.7456Mhz

Commit message: Added AT24C256
Parts:
- added C1005: 0.1uF, Capacitor_SMD:C_0805_2012Metric_Pad1.18x1.45mm_HandSolder, B.Cu at (67.9, 40.1)
- added U1002: AT24C256, Package_SO:SOP-8_3.76x4.96mm_P1.27mm, B.Cu at (71.8, 40.1)
- C1101, C1102, R1101, R1102, R1103, R1104, U1101: moved to F.Cu
- moved TP1102 54.6 mm to (116.6, 45.7)
- moved TP1101 54.2 mm to (119.9, 46.0)
- moved R1101 52.4 mm to (115.6, 45.4)
- moved C1101 52.3 mm to (119.5, 44.9)
- moved C1102 52.3 mm to (123.3, 44.9)
- moved R1102 52.2 mm to (115.7, 39.4)
- moved R1104 52.0 mm to (115.7, 43.4)
- moved U1101 52.0 mm to (121.4, 41.1)
- moved R1103 52.0 mm to (115.7, 41.4)
Routing:
- net /Microcontroller/0_10v_ain_1: track 14.7 -> 76.6 mm, vias 0 -> 3
- net /Microcontroller/0_10v_dout_1: track 5.13 -> 65.2 mm, vias 0 -> 2
- net Net-(C1104-Pad2): track 71.7 -> 17.3 mm, vias 1 -> 0
- net GND: track 326.3 -> 374.8 mm, vias 45 -> 48
- net +5V: track 138.6 -> 148.0 mm
- net Net-(R1103-Pad1): track 15.4 -> 13.2 mm, vias 2 -> 0
- net /Microcontroller/sda: track 36.1 -> 34.8 mm
- net VDD: track 70.4 -> 71.5 mm, vias 2 -> 1
- net Net-(R1102-Pad2): track 2.87 -> 2.30 mm
Other:
- board text added: "TODO: Move 0-10V circuit to the most right on the board. So we might add the AT24C256 anyway"
- board text added: "TODO: No copper on the Back where it could touch the aluminum profile! TODO: Make customized footprint to connect GRB(W) strips. (e.g. compatible with GRB)"
- board text added: "TODO: Place here some text about how to use this and where to find additional information. line 4"
- board text removed: "TODO: No copper on the Back where it could touch the aluminum profile! TODO: Make customized footprint to connect GRB(W) strips. (e.g. compatible with GRB) TODO: Make single row ISP connector, with silklayer explaining the pinout"
- board text removed: "TODO: Place here some text about how to use this and where to find additional information. line 5 line 4"
