File: LedBarController/LedBarController.kicad_pcb (KiCad board)
At the start: 2 copper layers, 145.1 x 25 mm, 106 parts, among them J1005 ISP, J1101 Conn_01x02, J1201 Barrel_Jack_Switch, J1301 Screw_Terminal_01x03, J201 Female pitch strip 1x7 pins 2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, J202 Female 2x7 pins 2.0mm pitch, J203 Female pitch strip 1x7 pins 2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, J701 Male pitch strip 1x7 pins 2.0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, J702 Conn_01x05, J703 Conn_01x05, J801 Conn_01x05, J802 Male pitch strip 2x7pins 2.0m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, J803 Conn_01x05, J804 Conn_01x05, J805 Conn_01x05, J901 Male pitch strip 1x7 pins 2.0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, J902 Conn_01x05, J903 Conn_01x05, Q1201 FQP47P06, Q301 Si2302DS, Q302 Si2302DS, Q303 Si2302DS, Q304 Si2302DS, Q401 Si2302DS, Q402 Si2302DS, Q403 Si2302DS, Q404 Si2302DS, Q501 Si2302DS, Q502 Si2302DS, Q503 Si2302DS, Q504 Si2302DS, Q601 Si2302DS, Q602 Si2302DS, Q603 Si2302DS, Q604 Si2302DS, SW1001 reset, SW801 4x42.3mm PCB Tactile Push But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, U1001 ATmega328P-AU, U1002 AT24C256, U1101 LM358DR, U1201 AMS1117-5.0, U1202 INA219AxD, U1301 MAX485E, U201 PCA9685PW, Y1001 14.7456Mhz

Commit message: Updated slik layer
Parts:
- moved C1005 1.50 mm to (67.9, 41.6)
Routing:
- net +5V: track 148.0 -> 148.8 mm
- net GND: vias 48 -> 49

Commit message: Refined routing
Parts:
- moved TP1102 0.25 mm to (116.6, 46.0)
Routing:
- net GND: track 374.8 -> 345.4 mm, vias 49 -> 53
- net +5V: track 148.8 -> 151.7 mm
- net /PWM/strip1_r: track 49.6 -> 48.1 mm
- net /PWM/strip2_w: track 44.5 -> 43.2 mm
- net /PWM/strip2_b: track 35.4 -> 34.2 mm
- net /Power/surge_bypass: track 67.8 -> 66.6 mm
- net /PWM/strip3_b: track 20.6 -> 19.6 mm
- net /PWM/strip1_g: track 52.1 -> 51.3 mm
Other:
- net class surge_bypass: clearance 0.25 -> 0.2

Commit message: Route complete
Parts:
- removed R1005: 10k, Resistor_SMD:R_0805_2012Metric_Pad1.20x1.40mm_HandSolder
- removed RN1002: 10k, Resistor_SMD:R_Array_Concave_4x0603
- removed TP1101: a1, TestPoint:TestPoint_Pad_D1.0mm
- removed TP1102: d1, TestPoint:TestPoint_Pad_D1.0mm
- added C1006: 0.1uF, Capacitor_SMD:C_0805_2012Metric_Pad1.18x1.45mm_HandSolder, B.Cu at (60.6, 35.2)
- added C1103: 1uF, Capacitor_SMD:C_0805_2012Metric_Pad1.18x1.45mm_HandSolder, B.Cu at (45.7, 37.5)
- added C1105: 0.1uF, Capacitor_SMD:C_0805_2012Metric_Pad1.18x1.45mm_HandSolder, B.Cu at (120.0, 35.4)
- added J1102: Conn_01x02, TerminalBlock_TE-Connectivity:TerminalBlock_TE_282834-2_1x02_P2.54mm_Horizontal, F.Cu at (122.2, 34.2)
- added JP1005: SolderJumper_2_Open, LedBarController:SolderJumper-2_P1.3mm_Open_TrianglePad1.0x1.5mm, B.Cu at (32.6, 45.6)
- added R1105: 10k, Resistor_SMD:R_0805_2012Metric_Pad1.20x1.40mm_HandSolder, B.Cu at (48.6, 34.5)
- added R1106: 1k, Resistor_SMD:R_0805_2012Metric_Pad1.20x1.40mm_HandSolder, F.Cu at (123.8, 41.4)
- added R1107: 10k, Resistor_SMD:R_0805_2012Metric_Pad1.20x1.40mm_HandSolder, F.Cu at (123.7, 43.5)
- added R1108: 10k, Resistor_SMD:R_0805_2012Metric_Pad1.20x1.40mm_HandSolder, F.Cu at (123.8, 45.5)
- C1101, R1101: moved to B.Cu
- J1101: footprint Connector_JST:JST_PH_S2B-PH-K_1x02_P2.00mm_Horizontal -> TerminalBlock_TE-Connectivity:TerminalBlock_TE_282834-2_1x02_P2.54mm_Horizontal
- SW1001: footprint Button_Switch_SMD:SW_SPST_SKQG_WithStem -> Button_Switch_SMD:SW_SPST_CK_RS282G05A3
- U1101: value LM358DR -> LM393
- moved C1101 76.2 mm to (43.7, 37.5), turned to 270 degrees
- moved R1101 67.6 mm to (48.6, 36.6), turned to 0 degrees
- moved TP1203 8.42 mm to (34.4, 33.3)
- moved C1102 6.03 mm to (120.0, 39.9), turned to 0 degrees
- moved R1203 4.76 mm to (68.3, 41.3)
- moved U1101 4.40 mm to (117.9, 43.8)
- moved J1101 4.37 mm to (122.2, 27.6), turned to 270 degrees
- moved C1002 3.96 mm to (63.7, 36.2), turned to 270 degrees
- moved TP1202 3.62 mm to (41.5, 33.4)
- moved D1202 3.42 mm to (69.3, 45.1), turned to 180 degrees
- moved C1005 3.01 mm to (68.0, 38.6)
- moved R1104 2.98 mm to (112.9, 44.4), turned to 90 degrees
- moved R1103 2.92 mm to (112.9, 40.5), turned to 90 degrees
- moved C1104 2.73 mm to (120.0, 28.9), turned to 90 degrees
- moved TP1301 2.67 mm to (30.5, 45.0)
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Connections:
- net /PWM/CenterStrips/button_ renamed /PWM/CenterStrips/~button~_
- C1101 pad 1: /Microcontroller/0_10v_ain_1 -> Net-(C1101-Pad1)
- J202 pad 14: /Microcontroller/button -> /Microcontroller/~button~
- JP1001 pad 2: +5V -> GND
- JP1002 pad 2: +5V -> GND
- JP1003 pad 2: +5V -> GND
- JP1004 pad 2: +5V -> GND
- R1101 pad 1: /Microcontroller/0_10v_ain_1 -> Net-(C1101-Pad1)
- R1101 pad 2: /Microcontroller/0_10v_dout_1 -> /0-10V/pwm1
- U1001 pad 1: (no net) -> /Microcontroller/addr1
- U1001 pad 10: /Microcontroller/addr2 -> /0-10V/pwm2
- U1001 pad 13: /Microcontroller/button -> /Microcontroller/addr5
- U1001 pad 2: /PWM/~oe -> /Microcontroller/addr2
- U1001 pad 23: /Microcontroller/0_10v_dout_1 -> /Microcontroller/~button~
- U1001 pad 24: /Microcontroller/0_10v_ain_1 -> (no net)
- U1001 pad 26: (no net) -> /Microcontroller/tx_en
- U1001 pad 32: /Microcontroller/tx_en -> /PWM/~oe
- U1001 pad 9: /Microcontroller/addr1 -> /0-10V/pwm1
- U1101 pad 3: /Microcontroller/0_10v_ain_1 -> Net-(C1101-Pad1)
- U1101 pad 5: Net-(R1103-Pad1) -> Net-(C1103-Pad1)
- U1101 pad 6: Net-(U1101-Pad6) -> Net-(R1107-Pad1)
- U1101 pad 7: Net-(U1101-Pad6) -> Net-(R1106-Pad2)
Routing:
- net GND: track 345.4 -> 610.5 mm, vias 53 -> 49
- net Net-(C1101-Pad1): track 0.00 -> 96.7 mm, vias 0 -> 3
- net Net-(C1103-Pad1): track 0.00 -> 93.6 mm, vias 0 -> 1
- net /Microcontroller/0_10v_ain_1: track 76.6 -> 0.00 mm, vias 3 -> 0
- net /Microcontroller/button: track 72.6 -> 0.00 mm, vias 2 -> 0
- net /Microcontroller/0_10v_dout_1: track 65.1 -> 0.00 mm, vias 2 -> 0
- net /Microcontroller/~button~: track 0.00 -> 61.5 mm, vias 0 -> 2
- net /Microcontroller/addr5: track 0.00 -> 31.3 mm
- net /Microcontroller/led1: track 18.3 -> 34.9 mm
- net Net-(C1105-Pad2): track 0.00 -> 13.4 mm
- net +5V: track 151.7 -> 139.6 mm
- net /Microcontroller/reset: track 17.4 -> 29.2 mm
- net VDD: track 71.5 -> 62.0 mm
- net Net-(R1103-Pad1): track 13.2 -> 4.46 mm
- net /Microcontroller/addr4: track 20.5 -> 28.7 mm
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
Commit message: Added custom footprint for LED strip connection
Parts:
- added TP1101: a1, TestPoint:TestPoint_Pad_D1.0mm, F.Cu at (135.3, 55.7)
- added TP1102: d1, TestPoint:TestPoint_Pad_D1.0mm, F.Cu at (135.3, 58.8)
- added TP1103: d2, TestPoint:TestPoint_Pad_D1.0mm, F.Cu at (138.3, 55.7)
- added TP1104: a2, TestPoint:TestPoint_Pad_D1.0mm, F.Cu at (138.3, 58.8)
- J702, J703, J902, J903: footprint Connector_PinHeader_2.00mm:PinHeader_1x05_P2.00mm_Vertical -> LedBarController:LED_Strip_10mm_5pins_Left
- moved J702 4.00 mm to (132.3, 30.0)
- moved J703 4.00 mm to (132.3, 41.0)
Routing:
- net /PWM/SideStrip_left/VDD_: track 0.00 -> 8.21 mm
- net GND: track 610.5 -> 615.7 mm, vias 49 -> 50
- net (no net): track 1.90 -> 0.00 mm
- net /Microcontroller/addr3: track 25.9 -> 26.5 mm

Commit message: moved board on schema to same sheet
Parts:
- added J704: Male pitch strip 1x7 pins 2.0mm pitch, Connector_PinHeader_2.00mm:PinHeader_1x05_P2.00mm_Vertical, F.Cu at (183.9, 24.9)
- added J705: Male pitch strip 1x7 pins 2.0mm pitch, LedBarController:LED_Strip_10mm_5pins_Right, F.Cu at (187.0, 28.9)
- added J904: Male pitch strip 1x7 pins 2.0mm pitch, LedBarController:LED_Strip_10mm_5pins_Left, F.Cu at (183.9, 42.1)
- added J905: Male pitch strip 1x7 pins 2.0mm pitch, Connector_PinHeader_2.00mm:PinHeader_1x05_P2.00mm_Vertical, F.Cu at (187.0, 38.1)
- J801, J804: footprint Connector_PinHeader_2.00mm:PinHeader_1x05_P2.00mm_Vertical -> LedBarController:LED_Strip_10mm_5pins_Left
- J803, J805: footprint Connector_PinHeader_2.00mm:PinHeader_1x05_P2.00mm_Vertical -> LedBarController:LED_Strip_10mm_5pins_Right
- J902, J903: footprint LedBarController:LED_Strip_10mm_5pins_Left -> LedBarController:LED_Strip_10mm_5pins_Right
- moved J804 19.0 mm to (145.3, 41.0)
- moved J801 13.5 mm to (145.3, 30.0)
- moved J803 12.3 mm to (156.9, 30.0)
- moved J805 12.3 mm to (156.9, 41.0)
- moved J902 4.00 mm to (169.9, 30.0)
- moved J903 4.00 mm to (169.9, 41.0)
Connections:
- net /PWM/CenterStrips/GND_ renamed /PWM/CenterStrips/~button~
- net /PWM/CenterStrips/VDD_ renamed /PWM/CenterStrips/center_front_vdd
- net /PWM/CenterStrips/~button~_ renamed /PWM/CenterStrips/gnd
- net /PWM/SideStrip_left/VDD_ renamed /PWM/CenterStrips/left_front_vdd
- net /PWM/SideStrip_left/blue_ renamed /PWM/CenterStrips/blue_left_front
- net /PWM/SideStrip_left/green_ renamed /PWM/CenterStrips/left_front_green
- net /PWM/SideStrip_left/red_ renamed /PWM/CenterStrips/red_left_front
- net /PWM/SideStrip_left/white_ renamed /PWM/CenterStrips/white_left_front
- net /PWM/SideStrip_right/VDD_ renamed /PWM/CenterStrips/right_front_vdd
- net /PWM/SideStrip_right/blue_ renamed /PWM/CenterStrips/right_front_blue
- net /PWM/SideStrip_right/green_ renamed /PWM/CenterStrips/right_front_green
- net /PWM/SideStrip_right/red_ renamed /PWM/CenterStrips/right_front_red
- net /PWM/SideStrip_right/white_ renamed /PWM/CenterStrips/right_front_white
- J801 pad 2: /PWM/CenterStrips/green_left_ -> /PWM/CenterStrips/center_front_l_green
- J801 pad 3: /PWM/CenterStrips/red_left_ -> /PWM/CenterStrips/center_front_l_red
- J801 pad 4: /PWM/CenterStrips/blue_left_ -> /PWM/CenterStrips/center_front_l_blue
- J801 pad 5: /PWM/CenterStrips/white_left_ -> /PWM/CenterStrips/center_front_l_white
- J802 pad 10: /PWM/CenterStrips/blue_right_ -> /PWM/CenterStrips/center_front_l_blue
- J802 pad 11: /PWM/CenterStrips/white_left_ -> /PWM/CenterStrips/center_front_r_white
- J802 pad 12: /PWM/CenterStrips/white_right_ -> /PWM/CenterStrips/center_front_l_white
- J802 pad 5: /PWM/CenterStrips/green_left_ -> /PWM/CenterStrips/center_front_r_green
- J802 pad 6: /PWM/CenterStrips/green_right_ -> /PWM/CenterStrips/center_front_l_green
- J802 pad 7: /PWM/CenterStrips/red_left_ -> /PWM/CenterStrips/center_front_r_red
- J802 pad 8: /PWM/CenterStrips/red_right_ -> /PWM/CenterStrips/center_front_l_red
- J802 pad 9: /PWM/CenterStrips/blue_left_ -> /PWM/CenterStrips/center_front_r_blue
- J803 pad 2: /PWM/CenterStrips/green_right_ -> /PWM/CenterStrips/center_front_r_green
- J803 pad 3: /PWM/CenterStrips/red_right_ -> /PWM/CenterStrips/center_front_r_red
- J803 pad 4: /PWM/CenterStrips/blue_right_ -> /PWM/CenterStrips/center_front_r_blue
- J803 pad 5: /PWM/CenterStrips/white_right_ -> /PWM/CenterStrips/center_front_r_white
- J804 pad 2: /PWM/CenterStrips/green_left_ -> /PWM/CenterStrips/center_front_l_green
- J804 pad 3: /PWM/CenterStrips/red_left_ -> /PWM/CenterStrips/center_front_l_red
- J804 pad 4: /PWM/CenterStrips/blue_left_ -> /PWM/CenterStrips/center_front_l_blue
- J804 pad 5: /PWM/CenterStrips/white_left_ -> /PWM/CenterStrips/center_front_l_white
- J805 pad 2: /PWM/CenterStrips/green_right_ -> /PWM/CenterStrips/center_front_r_green
- J805 pad 3: /PWM/CenterStrips/red_right_ -> /PWM/CenterStrips/center_front_r_red
- J805 pad 4: /PWM/CenterStrips/blue_right_ -> /PWM/CenterStrips/center_front_r_blue
- J805 pad 5: /PWM/CenterStrips/white_right_ -> /PWM/CenterStrips/center_front_r_white
Routing:
- net /PWM/CenterStrips/red_right_: track 16.8 -> 0.00 mm
- net /PWM/CenterStrips/red_left_: track 16.7 -> 0.00 mm
- net /PWM/CenterStrips/white_right_: track 16.5 -> 0.00 mm
- net /PWM/CenterStrips/center_front_r_red: track 0.00 -> 16.4 mm
- net /PWM/CenterStrips/center_front_r_blue: track 0.00 -> 16.3 mm
- net /PWM/CenterStrips/blue_right_: track 16.3 -> 0.00 mm
- net /PWM/CenterStrips/blue_left_: track 16.2 -> 0.00 mm
- net /PWM/CenterStrips/center_front_l_red: track 0.00 -> 16.2 mm
- net /PWM/CenterStrips/center_front_l_blue: track 0.00 -> 16.1 mm
- net /PWM/CenterStrips/white_left_: track 16.1 -> 0.00 mm
- net /PWM/CenterStrips/center_front_l_white: track 0.00 -> 16.1 mm
- net /PWM/CenterStrips/center_front_r_white: track 0.00 -> 16.0 mm
- net /PWM/CenterStrips/green_right_: track 16.0 -> 0.00 mm
- net /PWM/CenterStrips/center_front_l_green: track 0.00 -> 16.0 mm
- net /PWM/CenterStrips/green_left_: track 15.9 -> 0.00 mm
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Other:
- board size 145.1 x 25 mm -> 162.2 x 25 mm
- board text added: "+"
- board text added: "Front Center"
- board text added: "Front Left"
- board text added: "Front Right"

Commit message: Moved FETs to PWM sheet
Parts:
- removed TP1101: a1, TestPoint:TestPoint_Pad_D1.0mm
- removed TP1102: d1, TestPoint:TestPoint_Pad_D1.0mm
- removed TP1103: d2, TestPoint:TestPoint_Pad_D1.0mm
- removed TP1104: a2, TestPoint:TestPoint_Pad_D1.0mm

Commit message: Rearanged sheets
Connections:
- net /0-10V/pwm1 renamed /CenterBack/0-10V/pwm1
- net /0-10V/pwm2 renamed /CenterBack/0-10V/pwm2
- net /Microcontroller/addr1 renamed /CenterBack/Microcontroller/addr1
- net /Microcontroller/addr2 renamed /CenterBack/Microcontroller/addr2
- net /Microcontroller/addr3 renamed /CenterBack/Microcontroller/addr3
- net /Microcontroller/addr4 renamed /CenterBack/Microcontroller/addr4
- net /Microcontroller/addr5 renamed /CenterBack/Microcontroller/addr5
- net /Microcontroller/aref renamed /CenterBack/Microcontroller/aref
- net /Microcontroller/isp_miso renamed /CenterBack/Microcontroller/isp_miso
- net /Microcontroller/isp_mosi renamed /CenterBack/Microcontroller/isp_mosi
- net /Microcontroller/isp_sck renamed /CenterBack/Microcontroller/isp_sck
- net /Microcontroller/led1 renamed /CenterBack/Microcontroller/led1
- net /Microcontroller/reset renamed /CenterBack/Microcontroller/reset
- net /Microcontroller/rxd renamed /CenterBack/Microcontroller/rxd
- net /Microcontroller/scl renamed /CenterBack/Microcontroller/scl
- net /Microcontroller/sda renamed /CenterBack/Microcontroller/sda
- net /Microcontroller/tx_en renamed /CenterBack/Microcontroller/tx_en
- net /Microcontroller/txd renamed /CenterBack/Microcontroller/txd
- net /Microcontroller/~button~ renamed /CenterBack/Microcontroller/~button~
- net /PWM/CenterStrips/blue_left_front renamed /blue_left_front
- net /PWM/CenterStrips/center_front_l_blue renamed /center_front_l_blue
- net /PWM/CenterStrips/center_front_l_green renamed /center_front_l_green
- net /PWM/CenterStrips/center_front_l_red renamed /center_front_l_red
- net /PWM/CenterStrips/center_front_l_white renamed /center_front_l_white
- net /PWM/CenterStrips/center_front_r_blue renamed /center_front_r_blue
- net /PWM/CenterStrips/center_front_r_green renamed /center_front_r_green
- net /PWM/CenterStrips/center_front_r_red renamed /center_front_r_red
- net /PWM/CenterStrips/center_front_r_white renamed /center_front_r_white
- net /PWM/CenterStrips/center_front_vdd renamed /center_front_vdd
- net /PWM/CenterStrips/gnd renamed /gnd
- net /PWM/CenterStrips/left_back_blue renamed /left_back_blue
- net /PWM/CenterStrips/left_back_green renamed /left_back_green
- net /PWM/CenterStrips/left_back_red renamed /left_back_red
- net /PWM/CenterStrips/left_back_vdd renamed /left_back_vdd
- net /PWM/CenterStrips/left_back_white renamed /left_back_white
- net /PWM/CenterStrips/left_front_green renamed /left_front_green
- net /PWM/CenterStrips/left_front_vdd renamed /left_front_vdd
- net /PWM/CenterStrips/red_left_front renamed /red_left_front
- net /PWM/CenterStrips/right_back_blue renamed /right_back_blue
- net /PWM/CenterStrips/right_back_green renamed /right_back_green
- net /PWM/CenterStrips/right_back_red renamed /right_back_red
- net /PWM/CenterStrips/right_back_vdd renamed /right_back_vdd
- net /PWM/CenterStrips/right_back_white renamed /right_back_white
- net /PWM/CenterStrips/right_front_blue renamed /right_front_blue
- net /PWM/CenterStrips/right_front_green renamed /right_front_green
- net /PWM/CenterStrips/right_front_red renamed /right_front_red
- net /PWM/CenterStrips/right_front_vdd renamed /right_front_vdd
- net /PWM/CenterStrips/right_front_white renamed /right_front_white
- net /PWM/CenterStrips/white_left_front renamed /white_left_front
- net /PWM/CenterStrips/~button~ renamed /~button~
- net /PWM/strip1_b renamed /CenterBack/PWM/strip1_b
- net /PWM/strip1_b_out renamed /CenterBack/PWM/strip1_b_out
- net /PWM/strip1_g renamed /CenterBack/PWM/strip1_g
- net /PWM/strip1_g_out renamed /CenterBack/PWM/strip1_g_out
- net /PWM/strip1_r renamed /CenterBack/PWM/strip1_r
- net /PWM/strip1_r_out renamed /CenterBack/PWM/strip1_r_out
- net /PWM/strip1_w renamed /CenterBack/PWM/strip1_w
- net /PWM/strip1_w_out renamed /CenterBack/PWM/strip1_w_out
- net /PWM/strip2_b renamed /CenterBack/PWM/strip2_b
- net /PWM/strip2_b_out renamed /CenterBack/PWM/strip2_b_out
- net /PWM/strip2_g renamed /CenterBack/PWM/strip2_g
- net /PWM/strip2_g_out renamed /CenterBack/PWM/strip2_g_out
- net /PWM/strip2_r renamed /CenterBack/PWM/strip2_r
- net /PWM/strip2_r_out renamed /CenterBack/PWM/strip2_r_out
- net /PWM/strip2_w renamed /CenterBack/PWM/strip2_w
- net /PWM/strip2_w_out renamed /CenterBack/PWM/strip2_w_out
- net /PWM/strip3_b renamed /CenterBack/PWM/strip3_b
- net /PWM/strip3_b_out renamed /CenterBack/PWM/strip3_b_out
- net /PWM/strip3_g renamed /CenterBack/PWM/strip3_g
- net /PWM/strip3_g_out renamed /CenterBack/PWM/strip3_g_out
- net /PWM/strip3_r renamed /CenterBack/PWM/strip3_r
- net /PWM/strip3_r_out renamed /CenterBack/PWM/strip3_r_out
- net /PWM/strip3_w renamed /CenterBack/PWM/strip3_w
- net /PWM/strip3_w_out renamed /CenterBack/PWM/strip3_w_out
- net /PWM/strip4_b renamed /CenterBack/PWM/strip4_b
- net /PWM/strip4_b_out renamed /CenterBack/PWM/strip4_b_out
- net /PWM/strip4_g renamed /CenterBack/PWM/strip4_g
- net /PWM/strip4_g_out renamed /CenterBack/PWM/strip4_g_out
- net /PWM/strip4_r renamed /CenterBack/PWM/strip4_r
- net /PWM/strip4_r_out renamed /CenterBack/PWM/strip4_r_out
- net /PWM/strip4_w renamed /CenterBack/PWM/strip4_w
- net /PWM/strip4_w_out renamed /CenterBack/PWM/strip4_w_out
- net /PWM/~oe renamed /CenterBack/PWM/~oe
- net /Power/surge_bypass renamed /CenterBack/Power/surge_bypass
- net /RS485/A renamed /CenterBack/RS485/A
- net /RS485/B renamed /CenterBack/RS485/B

Commit message: Reanotate
Parts:
- removed C1103: 1uF, Capacitor_SMD:C_0805_2012Metric_Pad1.18x1.45mm_HandSolder
- removed C1105, C1301, C203: 0.1uF, Capacitor_SMD:C_0805_2012Metric_Pad1.18x1.45mm_HandSolder
- removed F1201: max. 5A F, Fuse:Fuseholder_Cylinder-5x20mm_Stelvio-Kontek_PTF78_Horizontal_Open
- removed SW1001: reset, Button_Switch_SMD:SW_SPST_CK_RS282G05A3
- removed TP1203: GND, TestPoint:TestPoint_Pad_D1.0mm
- added C501: 0.1uF, Capacitor_SMD:C_0805_2012Metric_Pad1.18x1.45mm_HandSolder, B.Cu at (39.1, 39.9)
- added C601: 0.1uF, Capacitor_SMD:C_0805_2012Metric_Pad1.18x1.45mm_HandSolder, F.Cu at (68.3, 37.5)
- added C704: 1uF, Capacitor_SMD:C_0805_2012Metric_Pad1.18x1.45mm_HandSolder, B.Cu at (45.7, 37.5)
- added C705: 0.1uF, Capacitor_SMD:C_0805_2012Metric_Pad1.18x1.45mm_HandSolder, B.Cu at (120.0, 35.4)
- added F301: max. 5A F, Fuse:Fuseholder_Cylinder-5x20mm_Stelvio-Kontek_PTF78_Horizontal_Open, F.Cu at (66.7, 30.5)
- added SW401: reset, Button_Switch_SMD:SW_SPST_CK_RS282G05A3, F.Cu at (56.1, 43.4)
- added TP303: GND, TestPoint:TestPoint_Pad_D1.0mm, B.Cu at (37.4, 30.5)
- renumbered C1208 to C301, C1206 to C302, C1201 to C303, C1207 to C304, C1202 to C305, C1203 to C306, C1204 to C307, C1205 to C308, C1001 to C401, C1006 to C402, C1002 to C403, C1003 to C404, C1004 to C405, C1005 to C406, C201 to C602, C202 to C603, C204 to C604, C205 to C605, C1101 to C701, C1104 to C702, C1102 to C703, D1201 to D301, D1203 to D302, D1202 to D303, D1001 to D401, D1002 to D402, D1003 to D403, D1004 to D404, J704 to J101, J705 to J102, J904 to J103, J905 to J104, J702 to J105, J701 to J106, J801 to J107, J802 to J108, J803 to J109, J901 to J110, J902 to J111, J703 to J112, J804 to J113, J805 to J114, J903 to J115, J1201 to J301, J1005 to J401, J1301 to J501, J201 to J601, J202 to J602, J203 to J603, J1101 to J701, J1102 to J702, JP1001 to JP401, JP1002 to JP402, JP1003 to JP403, JP1004 to JP404, JP1005 to JP405, JP1301 to JP501, Q1201 to Q301, Q301 to Q601, Q302 to Q602, Q303 to Q603, Q304 to Q604, Q401 to Q605, Q402 to Q606, Q403 to Q607, Q404 to Q608, Q501 to Q609, Q502 to Q610, Q503 to Q611, Q504 to Q612, Q601 to Q613, Q602 to Q614, Q603 to Q615, Q604 to Q616, R1204 to R301, R1205 to R302, R1206 to R303, R1201 to R304, R1202 to R305, R1203 to R306, R1006 to R401, R1003 to R402, R1002 to R403, R1301 to R501, R1302 to R502, R1303 to R503, R1101 to R701, R1102 to R702, R1103 to R703, R1104 to R704, R1105 to R705, R1106 to R706, R1107 to R707, R1108 to R708, RN1001 to RN401, SW801 to SW101, TP1201 to TP301, TP1202 to TP302, TP1301 to TP501, TP1304 to TP502, U1202 to U301, U1201 to U302, U1001 to U401, U1002 to U402, U1301 to U501, U201 to U601, U1101 to U701, Y1001 to Y401
Routing:
- net /CenterBack/Power/surge_bypass: track 66.6 -> 65.4 mm, vias 3 -> 2
