File: LedBarController/Microcontroller.sch (KiCad schematic (older format))
At the start: 25 parts, among them J501 Conn_01x03, J502 Conn_01x03, J503 Conn_01x03, J504 Conn_01x03, J505 AVR-ISP-6, J506 Conn_01x06, SW501 SW_Push, U501 ATmega328P-AU, Y501 Crystal

Commit message: Restarted PCB
Parts:
- removed J505: AVR-ISP-6, Connector_IDC:IDC-Header_2x03_P2.54mm_Vertical, symbol Connector:AVR-ISP-6
- added C1006: C, Capacitor_SMD:C_0805_2012Metric_Pad1.18x1.45mm_HandSolder, symbol Device:C
- added D1002: D, Diode_SMD:D_1206_3216Metric_Pad1.42x1.75mm_HandSolder, symbol Device:D
- added J1005: Conn_01x06, Connector_PinSocket_2.54mm:PinSocket_1x06_P2.54mm_Vertical, symbol Connector_Generic:Conn_01x06
- added R1007, R1008: R, Resistor_SMD:R_0805_2012Metric_Pad1.20x1.40mm_HandSolder, symbol Device:R
- renumbered C501 to C1001, C502 to C1002, C503 to C1003, C504 to C1004, C505 to C1005, D501 to D1001, J501 to J1001, J502 to J1002, J503 to J1003, J504 to J1004, J506 to J1006, R501 to R1001, R502 to R1002, R503 to R1003, R504 to R1004, R505 to R1005, R506 to R1006, SW501 to SW1001, TP502 to TP1001, TP503 to TP1002, TP504 to TP1003, TP501 to TP1004, U501 to U1001, Y501 to Y1001
Connections:
- net labels added: ADC_PWR, VDD
- net labels removed: ADC1
- wire segments 95 -> 109
Other:
- moved on the sheet: TP1004

Commit message: Changed components and moved center connector upwards
Parts:
- removed J1005: Conn_01x06, Connector_PinSocket_2.54mm:PinSocket_1x06_P2.54mm_Vertical, symbol Connector_Generic:Conn_01x06
- added J1005: AVR-ISP-6, Connector_PinSocket_1.27mm:PinSocket_1x06_P1.27mm_Vertical, symbol Connector:AVR-ISP-6
- SW1001: footprint Button_Switch_SMD:SW_Push_1P1T_NO_CK_KSC7xxJ -> Button_Switch_SMD:SW_SPST_SKQG_WithStem
Connections:
- wire segments 109 -> 107
Changed lines of the file:
@@
 F 0 "SW1001" V 7654 5852 50  0000 R CNN
 F 1 "SW_Push" V 7745 5852 50  0000 R CNN
-F 2 "Button_Switch_SMD:SW_Push_1P1T_NO_CK_KSC7xxJ" H 7700 6100 50  0001 C CNN
+F 2 "Button_Switch_SMD:SW_SPST_SKQG_WithStem" H 7700 6100 50  0001 C CNN
 F 3 "~" H 7700 6100 50  0001 C CNN
 	1    7700 5900
@@
 L power:GND #PWR01016
 U 1 1 5F8B3A11
-P 8450 5900
-F 0 "#PWR01016" H 8450 5650 50  0001 C CNN
-F 1 "GND" H 8455 5727 50  0000 C CNN
-F 2 "" H 8450 5900 50  0001 C CNN
-F 3 "" H 8450 5900 50  0001 C CNN
-	1    8450 5900
-	1    0    0    -1
-$EndComp
-Wire Wire Line
-	8450 5700 8450 5900
+P 9000 6000
+F 0 "#PWR01016" H 9000 5750 50  0001 C CNN
+F 1 "GND" H 9005 5827 50  0000 C CNN
+F 2 "" H 9000 6000 50  0001 C CNN
+F 3 "" H 9000 6000 50  0001 C CNN
+	1    9000 6000
+	1    0    0    -1
+$EndComp
 Wire Wire Line
 	6100 2700 6400 2700
@@
 	8500 5400 8200 5400
 Wire Wire Line
-	8500 5200 8200 5200
-Wire Wire Line
 	8200 5500 8500 5500
+Text Label 8250 5400 0    50   ~ 0
+MOSI
 Text Label 8250 5500 0    50   ~ 0
-MOSI
-Text Label 8250 5400 0    50   ~ 0
 SCK
 $Comp
@@
 Text Label 4750 2500 2    50   ~ 0
 ADC_PWR
-$Comp
-L Connector_Generic:Conn_01x06 J1005
-U 1 1 5FA7583B
-P 8700 5400
-F 0 "J1005" H 8780 5392 50  0000 L CNN
-F 1 "Conn_01x06" H 8780 5301 50  0000 L CNN
-F 2 "Connector_PinSocket_2.54mm:PinSocket_1x06_P2.54mm_Vertical" H 8700 5400 50  0001 C CNN
-F 3 "~" H 8700 5400 50  0001 C CNN
-	1    8700 5400
-	1    0    0    -1
-$EndComp
-Text Label 8250 5200 0    50   ~ 0
+Text Label 8250 5300 0    50   ~ 0
 MISO
-Wire Wire Line
-	8450 5300 8500 5300
-Wire Wire Line
-	8450 5700 8500 5700
 $Comp
 L power:+5V #PWR01012
 U 1 1 5F8B3F3B
-P 8450 5000
-F 0 "#PWR01012" H 8450 4850 50  0001 C CNN
-F 1 "+5V" H 8465 5173 50  0000 C CNN
-F 2 "" H 8450 5000 50  0001 C CNN
-F 3 "" H 8450 5000 50  0001 C CNN
-	1    8450 5000
-	1    0    0    -1
-$EndComp
-Wire Wire Line
-	8450 5000 8450 5300
+P 9000 4900
+F 0 "#PWR01012" H 9000 4750 50  0001 C CNN
+F 1 "+5V" H 9015 5073 50  0000 C CNN
+F 2 "" H 9000 4900 50  0001 C CNN
+F 3 "" H 9000 4900 50  0001 C CNN
+	1    9000 4900
+	1    0    0    -1
+$EndComp
 Wire Wire Line
 	7700 5000 7700 5200
+$Comp
+L Connector:AVR-ISP-6 J1005
+U 1 1 5FACD200
+P 8900 5500
+F 0 "J1005" H 8570 5596 50  0000 R CNN
+F 1 "AVR-ISP-6" H 8570 5505 50  0000 R CNN
+F 2 "Connector_PinSocket_1.27mm:PinSocket_1x06_P1.27mm_Vertical" V 8650 5550 50  0001 C CNN
+F 3 " ~" H 7625 4950 50  0001 C CNN
+	1    8900 5500
+	-1   0    0    -1
+$EndComp
+Wire Wire Line
+	8500 5300 8200 5300
+Wire Wire Line
+	9000 4900 9000 5000
+Wire Wire Line
+	9000 5900 9000 6000
 $EndSCHEMATC

Commit message: Updated schematic, added ds1307, replaced gpio-headers for LEDs and solder-jumpers and remove ISP-connector
Parts:
- removed C1005: C, Capacitor_SMD:C_0805_2012Metric_Pad1.18x1.45mm_HandSolder, symbol Device:C
- removed J1001, J1002, J1003, J1004: Conn_01x03, Connector_PinSocket_2.54mm:PinSocket_1x03_P2.54mm_Vertical, symbol Connector_Generic:Conn_01x03
- removed J1006: Conn_01x06, Connector_PinHeader_2.54mm:PinHeader_1x06_P2.54mm_Vertical, symbol Connector_Generic:Conn_01x06
- removed TP1001: ~PWM_OE, TestPoint:TestPoint_Pad_D1.0mm, symbol Connector:TestPoint
- removed TP1002: SCA, TestPoint:TestPoint_Pad_D1.0mm, symbol Connector:TestPoint
- removed TP1003: SCL, TestPoint:TestPoint_Pad_D1.0mm, symbol Connector:TestPoint
- added C1005: 0.47uF/5.5V, symbol Device:CP
- added C1007: 100nF, Capacitor_SMD:C_0805_2012Metric_Pad1.18x1.45mm_HandSolder, symbol Device:C
- added D1003, D1004, D1005: LED, LED_SMD:LED_0805_2012Metric_Pad1.15x1.40mm_HandSolder, symbol Device:LED
- added D1006: 1N5819, Diode_SMD:D_SOD-123, symbol Device:D
- added JP1001, JP1002, JP1003, JP1004: SolderJumper_2_Open, Jumper:SolderJumper-2_P1.3mm_Open_TrianglePad1.0x1.5mm, symbol Jumper:SolderJumper_2_Open
- added RN1001: 1k, Resistor_SMD:R_Array_Concave_4x0603, symbol Device:R_Pack04_SIP_Split
- added RN1002: 10k, Resistor_SMD:R_Array_Concave_4x0603, symbol Device:R_Pack04_SIP_Split
- added U1002: DS1307ZN+, Package_SO:SOIC-8_3.9x4.9mm_P1.27mm, symbol Timer_RTC:DS1307ZN+
- added Y1002: 32.768kHz, Crystal:Crystal_DS26_D2.0mm_L6.0mm_Vertical, symbol Device:Crystal_Small
- D1001: value Blue -> LED
- R1001: value 330 -> 100R
- SW1001: value SW_Push -> reset
Connections:
- net labels added: 0_10v_ain_1, 0_10v_ain_2, 0_10v_dout_1, 0_10v_dout_2, adc_vdd, addr1, addr2, addr3, addr4, aref, isp_miso, isp_mosi, isp_sck, led1, led2, led3, led4, reset, rtc_sqw, rxd, scl, sda, tx_en, txd, ~pwm_OE
- net labels removed: 0_10V_ain_1, 0_10V_ain_2, 0_10V_dout_1, 0_10V_dout_2, ADC_PWR, DTR, GPIO1, GPIO2, GPIO3, GPIO4, MISO, MOSI, Reset, Rx, Rx_, SCK, Tx, TxEn, ~PWM_OE
- wire segments 107 -> 157
- no-connect marks 3 -> 1
Other:
- moved on the sheet: C1001, C1002, C1003, C1004, C1006, D1002, J1005, R1002, R1003, R1005, R1006, R1007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

Commit message: Added capacitor for DS1307 and changed package of MAX485
Parts:
- added C1008: 0.1uF, Capacitor_SMD:C_0805_2012Metric_Pad1.18x1.45mm_HandSolder, symbol Device:C
Connections:
- wire segments 157 -> 159
Other:
- note added: "TODO: Wrong RN package"
Changed lines of the file:
@@
 $EndComp
 Connection ~ 8700 4450
+$Comp
+L power:GND #PWR01009
+U 1 1 5FD8F2F4
+P 10300 6200
+F 0 "#PWR01009" H 10300 5950 50  0001 C CNN
+F 1 "GND" H 10305 6027 50  0000 C CNN
+F 2 "" H 10300 6200 50  0001 C CNN
+F 3 "" H 10300 6200 50  0001 C CNN
+	1    10300 6200
+	1    0    0    -1
+$EndComp
+$Comp
+L power:+5V #PWR01008
+U 1 1 5FD8F2FA
+P 10300 5700
+F 0 "#PWR01008" H 10300 5550 50  0001 C CNN
+F 1 "+5V" H 10315 5873 50  0000 C CNN
+F 2 "" H 10300 5700 50  0001 C CNN
+F 3 "" H 10300 5700 50  0001 C CNN
+	1    10300 5700
+	1    0    0    -1
+$EndComp
+Wire Wire Line
+	10300 5700 10300 5800
+Wire Wire Line
+	10300 6100 10300 6200
+$Comp
+L Device:C C1008
+U 1 1 5FD8F302
+P 10300 5950
+F 0 "C1008" H 10415 5996 50  0000 L CNN
+F 1 "0.1uF" H 10415 5905 50  0000 L CNN
+F 2 "Capacitor_SMD:C_0805_2012Metric_Pad1.18x1.45mm_HandSolder" H 10338 5800 50  0001 C CNN
+F 3 "~" H 10300 5950 50  0001 C CNN
+	1    10300 5950
+	1    0    0    -1
+$EndComp
+Text Notes 7650 900  0    50   ~ 0
+TODO: Wrong RN package
 $EndSCHEMATC

Commit message: Updated labels in schematic and moved RTC to sub-schematic
Parts:
- removed C1005: 0.47uF/5.5V, symbol Device:CP
- removed C1007: 100nF, Capacitor_SMD:C_0805_2012Metric_Pad1.18x1.45mm_HandSolder, symbol Device:C
- removed C1008: 0.1uF, Capacitor_SMD:C_0805_2012Metric_Pad1.18x1.45mm_HandSolder, symbol Device:C
- removed D1006: 1N5819, Diode_SMD:D_SOD-123, symbol Device:D
- removed R1001: 100R, Resistor_SMD:R_0805_2012Metric_Pad1.20x1.40mm_HandSolder, symbol Device:R
- removed R1004: R, Resistor_SMD:R_0805_2012Metric_Pad1.20x1.40mm_HandSolder, symbol Device:R
- removed U1002: DS1307ZN+, Package_SO:SOIC-8_3.9x4.9mm_P1.27mm, symbol Timer_RTC:DS1307ZN+
- removed Y1002: 32.768kHz, Crystal:Crystal_DS26_D2.0mm_L6.0mm_Vertical, symbol Device:Crystal_Small
Connections:
- net labels added: ~pwm_oe
- net labels removed: I2C_SCL, I2C_SDA, ~pwm_OE
- wire segments 159 -> 135
Other:
- moved on the sheet: J1005, R1002, R1003, R1005, R1006, SW1001

Commit message: Routed LEDs and solder jumpers, renumbered diodes (and LEDs) on microcontroller schematic
Parts:
- renumbered D1003 to D1002, D1004 to D1003, D1005 to D1004, D1002 to D1005
Changed lines of the file:
@@
 $EndComp
 $Comp
-L Device:D D1002
+L Device:D D1005
 U 1 1 5FA48C9E
 P 2950 6350
-AR Path="/5F829319/5FA48C9E" Ref="D1002"  Part="1"
+AR Path="/5F829319/5FA48C9E" Ref="D1005"  Part="1"
 AR Path="/5F7C8D58/5FA48C9E" Ref="D?"  Part="1"
-F 0 "D1002" V 2904 6430 50  0000 L CNN
+F 0 "D1005" V 2904 6430 50  0000 L CNN
 F 1 "D" V 2995 6430 50  0000 L CNN
 F 2 "Diode_SMD:D_1206_3216Metric_Pad1.42x1.75mm_HandSolder" H 2950 6350 50  0001 C CNN
@@
 	7200 1400 7200 1800
 $Comp
-L Device:LED D1003
+L Device:LED D1002
 U 1 1 5F8E2DAF
 P 6950 1400
-F 0 "D1003" H 7000 1200 50  0000 R CNN
+F 0 "D1002" H 7000 1200 50  0000 R CNN
 F 1 "LED" H 7050 1300 50  0000 R CNN
 F 2 "LED_SMD:LED_0805_2012Metric_Pad1.15x1.40mm_HandSolder" H 6950 1400 50  0001 C CNN
@@
 $EndComp
 $Comp
-L Device:LED D1004
+L Device:LED D1003
 U 1 1 5F8E3481
 P 6950 1800
-F 0 "D1004" H 7000 1600 50  0000 R CNN
+F 0 "D1003" H 7000 1600 50  0000 R CNN
 F 1 "LED" H 7050 1700 50  0000 R CNN
 F 2 "LED_SMD:LED_0805_2012Metric_Pad1.15x1.40mm_HandSolder" H 6950 1800 50  0001 C CNN
@@
 $EndComp
 $Comp
-L Device:LED D1005
+L Device:LED D1004
 U 1 1 5F8E37DA
 P 6950 2200
-F 0 "D1005" H 7000 2000 50  0000 R CNN
+F 0 "D1004" H 7000 2000 50  0000 R CNN
 F 1 "LED" H 7050 2100 50  0000 R CNN
 F 2 "LED_SMD:LED_0805_2012Metric_Pad1.15x1.40mm_HandSolder" H 6950 2200 50  0001 C CNN

Commit message: Routed resistor-pack
Parts:
- RN1001, RN1002: symbol Device:R_Pack04_SIP_Split -> Device:R_Pack04_Split
Other:
- moved on the sheet: RN1001B, RN1001D
Changed lines of the file:
@@
 $EndComp
 $Comp
-L Device:R_Pack04_SIP_Split RN1001
+L Device:R_Pack04_Split RN1001
 U 1 1 5F8B2985
 P 6450 1000
@@
 F 3 "http://www.vishay.com/docs/31509/csc.pdf" H 6450 1000 50  0001 C CNN
 	1    6450 1000
-	0    1    1    0
-$EndComp
-$Comp
-L Device:R_Pack04_SIP_Split RN1001
-U 2 1 5F8B9A58
-P 6450 1400
-F 0 "RN1001" V 6243 1400 50  0000 C CNN
-F 1 "1k" V 6334 1400 50  0000 C CNN
-F 2 "Resistor_SMD:R_Array_Concave_4x0603" V 6370 1400 50  0001 C CNN
-F 3 "http://www.vishay.com/docs/31509/csc.pdf" H 6450 1400 50  0001 C CNN
-	2    6450 1400
-	0    1    1    0
-$EndComp
-$Comp
-L Device:R_Pack04_SIP_Split RN1001
-U 3 1 5F8B9E96
-P 6450 1800
-F 0 "RN1001" V 6243 1800 50  0000 C CNN
-F 1 "1k" V 6334 1800 50  0000 C CNN
-F 2 "Resistor_SMD:R_Array_Concave_4x0603" V 6370 1800 50  0001 C CNN
-F 3 "http://www.vishay.com/docs/31509/csc.pdf" H 6450 1800 50  0001 C CNN
-	3    6450 1800
-	0    1    1    0
-$EndComp
-$Comp
-L Device:R_Pack04_SIP_Split RN1001
-U 4 1 5F8BA948
-P 6450 2200
-F 0 "RN1001" V 6243 2200 50  0000 C CNN
-F 1 "1k" V 6334 2200 50  0000 C CNN
-F 2 "Resistor_SMD:R_Array_Concave_4x0603" V 6370 2200 50  0001 C CNN
-F 3 "http://www.vishay.com/docs/31509/csc.pdf" H 6450 2200 50  0001 C CNN
-	4    6450 2200
 	0    1    1    0
 $EndComp
@@
 $EndComp
 $Comp
-L Device:R_Pack04_SIP_Split RN1002
+L Device:R_Pack04_Split RN1002
 U 1 1 5F8A23F3
 P 9850 1250
@@
 $EndComp
 $Comp
-L Device:R_Pack04_SIP_Split RN1002
+L Device:R_Pack04_Split RN1002
 U 2 1 5F8A28A0
 P 9850 1650
@@
 $EndComp
 $Comp
-L Device:R_Pack04_SIP_Split RN1002
+L Device:R_Pack04_Split RN1002
 U 3 1 5F8A2D89
 P 9850 2050
@@
 $EndComp
 $Comp
-L Device:R_Pack04_SIP_Split RN1002
+L Device:R_Pack04_Split RN1002
 U 4 1 5F8A31E6
 P 9850 2450
@@
 Text HLabel 4000 3450 2    50   Output ~ 0
 rtc_sqw
+$Comp
+L Device:R_Pack04_Split RN1001
+U 4 1 5F8BA948
+P 6450 1400
+F 0 "RN1001" V 6243 1400 50  0000 C CNN
+F 1 "1k" V 6334 1400 50  0000 C CNN
+F 2 "Resistor_SMD:R_Array_Concave_4x0603" V 6370 1400 50  0001 C CNN
+F 3 "http://www.vishay.com/docs/31509/csc.pdf" H 6450 1400 50  0001 C CNN
+	4    6450 1400
+	0    1    1    0
+$EndComp
+$Comp
+L Device:R_Pack04_Split RN1001
+U 3 1 5F8B9E96
+P 6450 1800
+F 0 "RN1001" V 6243 1800 50  0000 C CNN
+F 1 "1k" V 6334 1800 50  0000 C CNN
+F 2 "Resistor_SMD:R_Array_Concave_4x0603" V 6370 1800 50  0001 C CNN
+F 3 "http://www.vishay.com/docs/31509/csc.pdf" H 6450 1800 50  0001 C CNN
+	3    6450 1800
+	0    1    1    0
+$EndComp
+$Comp
+L Device:R_Pack04_Split RN1001
+U 2 1 5F8B9A58
+P 6450 2200
+F 0 "RN1001" V 6243 2200 50  0000 C CNN
+F 1 "1k" V 6334 2200 50  0000 C CNN
+F 2 "Resistor_SMD:R_Array_Concave_4x0603" V 6370 2200 50  0001 C CNN
+F 3 "http://www.vishay.com/docs/31509/csc.pdf" H 6450 2200 50  0001 C CNN
+	2    6450 2200
+	0    1    1    0
+$EndComp
 $EndSCHEMATC

Commit message: Work in progress
Parts:
- added C1005: 0.1uF, Capacitor_SMD:C_0805_2012Metric_Pad1.18x1.45mm_HandSolder, symbol Device:C
- added U1002: CAT24C256, Package_SO:SOIC-8_3.9x4.9mm_P1.27mm, symbol Memory_EEPROM:CAT24C256
- C1001: Feature (none) -> UC; Price (none) -> 0.0057; is stock (none) -> yes
- C1002: Feature (none) -> 10V_SUPPORTED VDDADC_SUPPORTED; Price (none) -> 0.0057; is stock (none) -> yes
- C1003, C1004: value C -> 22pF; Feature (none) -> UC; Price (none) -> 0.0057; is stock (none) -> yes
- C1006: value C -> 1uF; Feature (none) -> VDDADC_SUPPORTED; Price (none) -> 0.015; is stock (none) -> no
- D1001: value LED -> Green; Feature (none) -> GPLED; Price (none) -> 0.00675; is stock (none) -> yes
- D1002: value LED -> Yellow; Feature (none) -> GPLED; Price (none) -> 0.00675; is stock (none) -> yes
- D1003: value LED -> Orange; Feature (none) -> GPLED; Price (none) -> 0.00675; is stock (none) -> yes
- D1004: value LED -> Red; Feature (none) -> GPLED; Price (none) -> 0.00675; is stock (none) -> yes
- D1005: value D -> 1N4148; Feature (none) -> VDDADC_SUPPORTED; Price (none) -> 0.0048; is stock (none) -> yes
- J1005: Feature (none) -> UC; Price (none) -> 0; is stock (none) -> yes
- JP1001, JP1002, JP1003, JP1004: Feature (none) -> GPJUMPER; Price (none) -> 0; is stock (none) -> n.a.
- R1002, R1003: value R -> 4k7; Feature (none) -> INA219_SUPPORTED PWM_SUPPORTED RTC_SUPPORTED EEPROM_SUPPORT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; Price (none) -> 0.0036; is stock (none) -> yes
- R1005: value R -> 10k; Feature (none) -> PWM_SUPPORTED_2STRIPS; Price (none) -> 0.0036; is stock (none) -> yes
- R1006: value 10K -> 10k; Feature (none) -> UC; Price (none) -> 0.0036; is stock (none) -> yes
- R1007: value R -> 10k; Feature (none) -> VDDADC_SUPPORTED; Price (none) -> 0.0036; is stock (none) -> yes
- R1008: value R -> 1k8; Feature (none) -> VDDADC_SUPPORTED; Price (none) -> 0.0036; is stock (none) -> yes
- RN1001: value 1k -> 470R; Feature (none) -> GPLED; Price (none) -> 0.0134; is stock (none) -> no
- RN1002: Feature (none) -> GPJUMPER; Price (none) -> 0.0134; is stock (none) -> no
- SW1001: value reset -> 4x42.3mm PCB Tactile Push Button Switch; Feature (none) -> UC; Price (none) -> 0.0356; is stock (none) -> no
- TP1004: value ADC1 -> ADC_VDD; Feature (none) -> VDDADC_SUPPORTED; Price (none) -> 0; is stock (none) -> n.a.
- U1001: Feature (none) -> UC; Price (none) -> 1.106; is stock (none) -> yes
- Y1001: value Crystal -> 14.7456Mhz; Feature (none) -> RTC_SUPPORTED; Price (none) -> 0.178; is stock (none) -> yes
Connections:
- wire segments 135 -> 149
