File: LedBarController/Microcontroller.sch (KiCad schematic (older format))
At the start: 29 parts, among them J1005 AVR-ISP-6, SW1001 4x42.3mm PCB Tactile Push But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, U1001 ATmega328P-AU, U1002 CAT24C256, Y1001 14.7456Mhz

Commit message: Reduced circuit by remove extra features. Routed whole board. Needs refinement
Parts:
- removed C1005: 0.1uF, Capacitor_SMD:C_0805_2012Metric_Pad1.18x1.45mm_HandSolder, symbol Device:C
- removed C1006: 1uF, Capacitor_SMD:C_0805_2012Metric_Pad1.18x1.45mm_HandSolder, symbol Device:C
- removed D1005: 1N4148, Diode_SMD:D_1206_3216Metric_Pad1.42x1.75mm_HandSolder, symbol Device:D
- removed R1007: 10k, Resistor_SMD:R_0805_2012Metric_Pad1.20x1.40mm_HandSolder, symbol Device:R
- removed R1008: 1k8, Resistor_SMD:R_0805_2012Metric_Pad1.20x1.40mm_HandSolder, symbol Device:R
- removed TP1004: ADC_VDD, TestPoint:TestPoint_Pad_D1.0mm, symbol Connector:TestPoint
- removed U1002: CAT24C256, Package_SO:SOIC-8_3.9x4.9mm_P1.27mm, symbol Memory_EEPROM:CAT24C256
- JP1001, JP1002, JP1003, JP1004: footprint Jumper:SolderJumper-2_P1.3mm_Open_TrianglePad1.0x1.5mm -> LedBarController:SolderJumper-2_P1.3mm_Open_TrianglePad1.0x1.5mm
Connections:
- net labels removed: 0_10v_ain_2, 0_10v_dout_2, VDD, adc_vdd, rtc_sqw
- wire segments 149 -> 117
- no-connect marks 1 -> 5
Other:
- moved on the sheet: RN1002A, RN1002B, RN1002C, RN1002D

Commit message: Update silk layer
Parts:
- J1005: value AVR-ISP-6 -> ISP
- SW1001: value 4x42.3mm PCB Tactile Push Button Switch -> reset
Changed lines of the file:
@@
 P 8350 4650
 F 0 "SW1001" V 8304 4602 50  0000 R CNN
-F 1 "4x42.3mm PCB Tactile Push Button Switch" V 8395 4602 50  0000 R CNN
+F 1 "reset" V 8395 4602 50  0000 R CNN
 F 2 "Button_Switch_SMD:SW_SPST_SKQG_WithStem" H 8350 4850 50  0001 C CNN
 F 3 "~" H 8350 4850 50  0001 C CNN
@@
 P 6100 4450
 F 0 "J1005" H 5770 4546 50  0000 R CNN
-F 1 "AVR-ISP-6" H 5770 4455 50  0000 R CNN
+F 1 "ISP" H 5770 4455 50  0000 R CNN
 F 2 "Connector_PinSocket_1.27mm:PinSocket_1x06_P1.27mm_Vertical" V 5850 4500 50  0001 C CNN
 F 3 " ~" H 4825 3900 50  0001 C CNN

Commit message: Improved ISP connector silk layer
Parts:
- J1005: footprint Connector_PinSocket_1.27mm:PinSocket_1x06_P1.27mm_Vertical -> LedBarController:ISP_P1.27mm_single_row
Changed lines of the file:
@@
 F 0 "J1005" H 5770 4546 50  0000 R CNN
 F 1 "ISP" H 5770 4455 50  0000 R CNN
-F 2 "Connector_PinSocket_1.27mm:PinSocket_1x06_P1.27mm_Vertical" V 5850 4500 50  0001 C CNN
+F 2 "LedBarController:ISP_P1.27mm_single_row" V 5850 4500 50  0001 C CNN
 F 3 " ~" H 4825 3900 50  0001 C CNN
 F 4 "UC" H 6100 4450 50  0001 C CNN "Feature"

Commit message: Added AT24C256
Parts:
- added C1005: 0.1uF, Capacitor_SMD:C_0805_2012Metric_Pad1.18x1.45mm_HandSolder, symbol Device:C
- added U1002: AT24C256, Package_SO:SOP-8_3.76x4.96mm_P1.27mm, symbol Memory_EEPROM:CAT24C256
Connections:
- wire segments 117 -> 131
Changed lines of the file:
@@
 NoConn ~ 3100 2750
 NoConn ~ 1900 1850
+$Comp
+L Memory_EEPROM:CAT24C256 U1002
+U 1 1 5FD8CA5F
+P 3000 6250
+F 0 "U1002" H 2750 6500 50  0000 C CNN
+F 1 "AT24C256" H 3250 6500 50  0000 C CNN
+F 2 "Package_SO:SOP-8_3.76x4.96mm_P1.27mm" H 3000 6250 50  0001 C CNN
+F 3 "https://www.onsemi.cn/PowerSolutions/document/CAT24C256-D.PDF" H 3000 6250 50  0001 C CNN
+	1    3000 6250
+	1    0    0    -1
+$EndComp
+$Comp
+L power:GND #PWR01009
+U 1 1 5FD8DA85
+P 3000 6650
+F 0 "#PWR01009" H 3000 6400 50  0001 C CNN
+F 1 "GND" H 3005 6477 50  0000 C CNN
+F 2 "" H 3000 6650 50  0001 C CNN
+F 3 "" H 3000 6650 50  0001 C CNN
+	1    3000 6650
+	1    0    0    -1
+$EndComp
+Wire Wire Line
+	3000 6650 3000 6550
+$Comp
+L power:+5V #PWR01008
+U 1 1 5FD9311B
+P 3000 5850
+F 0 "#PWR01008" H 3000 5700 50  0001 C CNN
+F 1 "+5V" H 3015 6023 50  0000 C CNN
+F 2 "" H 3000 5850 50  0001 C CNN
+F 3 "" H 3000 5850 50  0001 C CNN
+	1    3000 5850
+	1    0    0    -1
+$EndComp
+Wire Wire Line
+	3000 5850 3000 5950
+Wire Wire Line
+	2600 6150 2600 6250
+Wire Wire Line
+	2600 6550 3000 6550
+Connection ~ 2600 6250
+Wire Wire Line
+	2600 6250 2600 6350
+Connection ~ 2600 6350
+Wire Wire Line
+	2600 6350 2600 6550
+Connection ~ 3000 6550
+Wire Wire Line
+	3400 6150 3750 6150
+Wire Wire Line
+	3400 6250 3750 6250
+Text Label 3700 6250 2    50   ~ 0
+scl
+Text Label 3700 6150 2    50   ~ 0
+sda
+Wire Wire Line
+	3400 6350 3400 6550
+Wire Wire Line
+	3400 6550 3000 6550
+$Comp
+L Device:C C1005
+U 1 1 5FDBE069
+P 2200 6250
+F 0 "C1005" H 2315 6296 50  0000 L CNN
+F 1 "0.1uF" H 2315 6205 50  0000 L CNN
+F 2 "Capacitor_SMD:C_0805_2012Metric_Pad1.18x1.45mm_HandSolder" H 2238 6100 50  0001 C CNN
+F 3 "~" H 2200 6250 50  0001 C CNN
+F 4 "UC" H 2200 6250 50  0001 C CNN "Feature"
+F 5 "0.0057" H 2200 6250 50  0001 C CNN "Price"
+F 6 "yes" H 2200 6250 50  0001 C CNN "is stock"
+	1    2200 6250
+	1    0    0    -1
+$EndComp
+Wire Wire Line
+	2600 6550 2200 6550
+Wire Wire Line
+	2200 6550 2200 6400
+Connection ~ 2600 6550
+Wire Wire Line
+	2200 6100 2200 5950
+Wire Wire Line
+	2200 5950 3000 5950
+Connection ~ 3000 5950
 $EndSCHEMATC

Commit message: Route complete
Parts:
- removed R1005: 10k, Resistor_SMD:R_0805_2012Metric_Pad1.20x1.40mm_HandSolder, symbol Device:R
- removed RN1002: 10k, Resistor_SMD:R_Array_Concave_4x0603, symbol Device:R_Pack04_Split
- added C1006: 0.1uF, Capacitor_SMD:C_0805_2012Metric_Pad1.18x1.45mm_HandSolder, symbol Device:C
- added JP1005: SolderJumper_2_Open, LedBarController:SolderJumper-2_P1.3mm_Open_TrianglePad1.0x1.5mm, symbol Jumper:SolderJumper_2_Open
- SW1001: footprint Button_Switch_SMD:SW_SPST_SKQG_WithStem -> Button_Switch_SMD:SW_SPST_CK_RS282G05A3; Price 0.0356 -> 0.023
- U1002: Feature (none) -> Memory; Price (none) -> 0.05; is stock (none) -> yes
Connections:
- net labels added: addr5, pwm1, pwm2, ~button~
- net labels removed: 0_10v_ain_1, 0_10v_dout_1, button
- wire segments 131 -> 113
- no-connect marks 5 -> 4
Other:
- note added: "Add extra capacitor for AVCC"
- note added: "Make use of the internal pull-ups of the microcontoller"
- note added: "We could use the internal pull-up of the uC,\nso no need to place these external pull-up resistors.\nBut in case of problems we can place them any-way."
- note removed: "TODO: Wrong RN package"

Commit message: moved board on schema to same sheet
Connections:
- wire segments 113 -> 114
Other:
- note removed: "Add extra capacitor for AVCC"
- note removed: "Make use of the internal pull-ups of the microcontoller"
- note removed: "We could use the internal pull-up of the uC,\nso no need to place these external pull-up resistors.\nBut in case of problems we can place them any-way."
- moved on the sheet: C1001, C1002, C1003, C1004, C1005, C1006, D1001, D1002, D1003, D1004, J1005, JP1001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

Commit message: Rearanged sheets
Changed lines of the file:
@@
 $Descr A4 11693 8268
 encoding utf-8
-Sheet 8 7
+Sheet 4 7
 Title ""
 Date ""
@@
 txd
 $Comp
-L power:GND #PWR01014
+L power:GND #PWR0106
 U 1 1 5F893C9D
 P 2500 5400
-F 0 "#PWR01014" H 2500 5150 50  0001 C CNN
+F 0 "#PWR0106" H 2500 5150 50  0001 C CNN
 F 1 "GND" H 2505 5227 50  0000 C CNN
 F 2 "" H 2500 5400 50  0001 C CNN
@@
 $EndComp
 $Comp
-L power:GND #PWR01005
+L power:GND #PWR0107
 U 1 1 5F894B42
 P 1000 2900
-F 0 "#PWR01005" H 1000 2650 50  0001 C CNN
+F 0 "#PWR0107" H 1000 2650 50  0001 C CNN
 F 1 "GND" H 1005 2727 50  0000 C CNN
 F 2 "" H 1000 2900 50  0001 C CNN
@@
 $EndComp
 $Comp
-L power:GND #PWR01004
+L power:GND #PWR0108
 U 1 1 5F89C743
 P 2100 1750
-F 0 "#PWR01004" H 2100 1500 50  0001 C CNN
+F 0 "#PWR0108" H 2100 1500 50  0001 C CNN
 F 1 "GND" H 2105 1577 50  0000 C CNN
 F 2 "" H 2100 1750 50  0001 C CNN
@@
 $EndComp
 $Comp
-L power:GND #PWR01018
+L power:GND #PWR0109
 U 1 1 5F8AD40C
 P 9500 4950
-F 0 "#PWR01018" H 9500 4700 50  0001 C CNN
+F 0 "#PWR0109" H 9500 4700 50  0001 C CNN
 F 1 "GND" H 9505 4777 50  0000 C CNN
 F 2 "" H 9500 4950 50  0001 C CNN
@@
 $EndComp
 $Comp
-L power:+5V #PWR01011
+L power:+5V #PWR0110
 U 1 1 5F8AED11
 P 9500 3650
-F 0 "#PWR01011" H 9500 3500 50  0001 C CNN
+F 0 "#PWR0110" H 9500 3500 50  0001 C CNN
 F 1 "+5V" H 9515 3823 50  0000 C CNN
 F 2 "" H 9500 3650 50  0001 C CNN
@@
 $EndComp
 $Comp
-L power:GND #PWR01016
+L power:GND #PWR0111
 U 1 1 5F8B3A11
 P 7000 4750
-F 0 "#PWR01016" H 7000 4500 50  0001 C CNN
+F 0 "#PWR0111" H 7000 4500 50  0001 C CNN
 F 1 "GND" H 7005 4577 50  0000 C CNN
 F 2 "" H 7000 4750 50  0001 C CNN
@@
 	5250 2700 5250 2850
 $Comp
-L power:GND #PWR01003
+L power:GND #PWR0112
 U 1 1 5F8A0649
 P 5250 2850
-F 0 "#PWR01003" H 5250 2600 50  0001 C CNN
+F 0 "#PWR0112" H 5250 2600 50  0001 C CNN
 F 1 "GND" V 5255 2722 50  0000 R CNN
 F 2 "" H 5250 2850 50  0001 C CNN
@@
 U 1 1 5F89EAE1
 P 5100 3000
-F 0 "C1004" H 5000 3100 50  0000 L CNN
-F 1 "22pF" H 5000 2900 50  0000 L CNN
+F 0 "C1004" H 4750 3050 50  0000 L CNN
+F 1 "22pF" H 4800 2950 50  0000 L CNN
 F 2 "Capacitor_SMD:C_0805_2012Metric_Pad1.18x1.45mm_HandSolder" H 5138 2850 50  0001 C CNN
 F 3 "~" H 5100 3000 50  0001 C CNN
@@
 U 1 1 5F89DB56
 P 4950 2850
-F 0 "Y1001" H 4950 3118 50  0000 C CNN
-F 1 "14.7456Mhz" H 4950 3027 50  0000 C CNN
+F 0 "Y1001" H 4950 3000 50  0000 C CNN
+F 1 "14.7456Mhz" V 5150 3000 50  0000 C CNN
 F 2 "Crystal:Crystal_HC49-U_Vertical" H 4950 2850 50  0001 C CNN
 F 3 "~" H 4950 2850 50  0001 C CNN
@@
 $EndComp
 $Comp
-L power:+5V #PWR01012
+L power:+5V #PWR0113
 U 1 1 5F8B3F3B
 P 7000 3650
-F 0 "#PWR01012" H 7000 3500 50  0001 C CNN
+F 0 "#PWR0113" H 7000 3500 50  0001 C CNN
 F 1 "+5V" H 7015 3823 50  0000 C CNN
 F 2 "" H 7000 3650 50  0001 C CNN
@@
 $EndComp
 $Comp
-L power:GND #PWR0101
+L power:GND #PWR0114
 U 1 1 5F887A44
 P 7500 2700
-F 0 "#PWR0101" H 7500 2450 50  0001 C CNN
+F 0 "#PWR0114" H 7500 2450 50  0001 C CNN
 F 1 "GND" V 7505 2572 50  0000 R CNN
 F 2 "" H 7500 2700 50  0001 C CNN
@@
 	9550 1400 9550 1800
 $Comp
-L power:GND #PWR0102
+L power:GND #PWR0115
 U 1 1 5F8BEA07
 P 9550 2700
-F 0 "#PWR0102" H 9550 2450 50  0001 C CNN
+F 0 "#PWR0115" H 9550 2450 50  0001 C CNN
 F 1 "GND" V 9555 2572 50  0000 R CNN
 F 2 "" H 9550 2700 50  0001 C CNN
@@
 	5950 6400 5950 6500
 $Comp
-L power:+5V #PWR01007
+L power:+5V #PWR0116
 U 1 1 5F896AEE
 P 5600 6400
-F 0 "#PWR01007" H 5600 6250 50  0001 C CNN
+F 0 "#PWR0116" H 5600 6250 50  0001 C CNN
 F 1 "+5V" H 5615 6573 50  0000 C CNN
 F 2 "" H 5600 6400 50  0001 C CNN
@@
 $EndComp
 $Comp
-L power:+5V #PWR01006
+L power:+5V #PWR0117
 U 1 1 5F8967CB
 P 5950 6400
-F 0 "#PWR01006" H 5950 6250 50  0001 C CNN
+F 0 "#PWR0117" H 5950 6250 50  0001 C CNN
 F 1 "+5V" H 5965 6573 50  0000 C CNN
 F 2 "" H 5950 6400 50  0001 C CNN
@@
 $EndComp
 $Comp
-L power:GND #PWR01009
+L power:GND #PWR0118
 U 1 1 5FD8DA85
 P 3100 7100
-F 0 "#PWR01009" H 3100 6850 50  0001 C CNN
+F 0 "#PWR0118" H 3100 6850 50  0001 C CNN
 F 1 "GND" H 3105 6927 50  0000 C CNN
 F 2 "" H 3100 7100 50  0001 C CNN
@@
 	3100 7100 3100 7000
 $Comp
-L power:+5V #PWR01008
+L power:+5V #PWR0119
 U 1 1 5FD9311B
 P 3100 6300
-F 0 "#PWR01008" H 3100 6150 50  0001 C CNN
+F 0 "#PWR0119" H 3100 6150 50  0001 C CNN
 F 1 "+5V" H 3115 6473 50  0000 C CNN
 F 2 "" H 3100 6300 50  0001 C CNN
@@
 	3100 3100 4000 3100
 $Comp
-L power:GND #PWR01013
+L power:GND #PWR0120
 U 1 1 5F9F6882
 P 2900 1750
-F 0 "#PWR01013" H 2900 1500 50  0001 C CNN
+F 0 "#PWR0120" H 2900 1500 50  0001 C CNN
 F 1 "GND" H 2905 1577 50  0000 C CNN
 F 2 "" H 2900 1750 50  0001 C CNN
@@
 $EndComp
 $Comp
-L power:+5V #PWR01001
+L power:+5V #PWR0121
 U 1 1 5F895448
 P 2550 1150
-F 0 "#PWR01001" H 2550 1000 50  0001 C CNN
+F 0 "#PWR0121" H 2550 1000 50  0001 C CNN
 F 1 "+5V" H 2565 1323 50  0000 C CNN
 F 2 "" H 2550 1150 50  0001 C CNN
