File: LedBarController/Microcontroller.sch (KiCad schematic (older format))
At the start: 24 parts, among them J1005 ISP, SW1001 reset, U1001 ATmega328P-AU, U1002 AT24C256, Y1001 14.7456Mhz

Commit message: Reanotate
Parts:
- renumbered C1001 to C401, C1006 to C402, C1002 to C403, C1003 to C404, C1004 to C405, C1005 to C406, D1001 to D401, D1002 to D402, D1003 to D403, D1004 to D404, J1005 to J401, JP1001 to JP401, JP1002 to JP402, JP1003 to JP403, JP1004 to JP404, JP1005 to JP405, R1006 to R401, R1003 to R402, R1002 to R403, RN1001 to RN401, SW1001 to SW401, U1001 to U401, U1002 to U402, Y1001 to Y401

Commit message: Updated footprints and Fab layer
Parts:
- U401: footprint Package_QFP:TQFP-32_7x7mm_P0.8mm -> LedBarController:TQFP-32_7x7mm_P0.8mm_corner_cutoff
- Y401: footprint Crystal:Crystal_HC49-U_Vertical -> LedBarController:Crystal_HC49-U_Vertical_tight_fit
Changed lines of the file:
@@
 F 0 "Y401" H 4950 3000 50  0000 C CNN
 F 1 "14.7456Mhz" V 5150 3000 50  0000 C CNN
-F 2 "Crystal:Crystal_HC49-U_Vertical" H 4950 2850 50  0001 C CNN
+F 2 "LedBarController:Crystal_HC49-U_Vertical_tight_fit" H 4950 2850 50  0001 C CNN
 F 3 "~" H 4950 2850 50  0001 C CNN
 F 4 "RTC_SUPPORTED" H 4950 2850 50  0001 C CNN "Feature"
@@
 F 0 "U401" H 2850 1900 50  0000 C CNN
 F 1 "ATmega328P-AU" H 2900 1800 50  0000 C CNN
-F 2 "Package_QFP:TQFP-32_7x7mm_P0.8mm" H 2500 3400 50  0001 C CIN
+F 2 "LedBarController:TQFP-32_7x7mm_P0.8mm_corner_cutoff" H 2500 3400 50  0001 C CIN
 F 3 "http://ww1.microchip.com/downloads/en/DeviceDoc/ATmega328_P%20AVR%20MCU%20with%20picoPower%20Technology%20Data%20Sheet%2040001984A.pdf" H 2500 3400 50  0001 C CNN
 F 4 "UC" H 2500 3400 50  0001 C CNN "Feature"

Commit message: Replaced 470R for 10k resistor to make the LED less bright
Parts:
- RN401: value 470R -> 10k
Changed lines of the file:
@@
 P 6750 1400
 F 0 "RN401" V 6543 1400 50  0000 C CNN
-F 1 "470R" V 6634 1400 50  0000 C CNN
+F 1 "10k" V 6634 1400 50  0000 C CNN
 F 2 "Resistor_SMD:R_Array_Concave_4x0603" V 6670 1400 50  0001 C CNN
 F 3 "http://www.vishay.com/docs/31509/csc.pdf" H 6750 1400 50  0001 C CNN
@@
 P 6750 1800
 F 0 "RN401" V 6543 1800 50  0000 C CNN
-F 1 "470R" V 6634 1800 50  0000 C CNN
+F 1 "10k" V 6634 1800 50  0000 C CNN
 F 2 "Resistor_SMD:R_Array_Concave_4x0603" V 6670 1800 50  0001 C CNN
 F 3 "http://www.vishay.com/docs/31509/csc.pdf" H 6750 1800 50  0001 C CNN
@@
 P 6750 2200
 F 0 "RN401" V 6543 2200 50  0000 C CNN
-F 1 "470R" V 6634 2200 50  0000 C CNN
+F 1 "10k" V 6634 2200 50  0000 C CNN
 F 2 "Resistor_SMD:R_Array_Concave_4x0603" V 6670 2200 50  0001 C CNN
 F 3 "http://www.vishay.com/docs/31509/csc.pdf" H 6750 2200 50  0001 C CNN
@@
 P 6750 2600
 F 0 "RN401" V 6543 2600 50  0000 C CNN
-F 1 "470R" V 6634 2600 50  0000 C CNN
+F 1 "10k" V 6634 2600 50  0000 C CNN
 F 2 "Resistor_SMD:R_Array_Concave_4x0603" V 6670 2600 50  0001 C CNN
 F 3 "http://www.vishay.com/docs/31509/csc.pdf" H 6750 2600 50  0001 C CNN

Commit message: Added Arduino pin-numbers to ATMega328 symbol
Parts:
- U401: symbol MCU_Microchip_ATmega:ATmega328P-AU -> LedBarController:ATmega48PV-10AU-arduino-atmega48pv-10au-arduino-LedBarController-rescue
Changed lines of the file:
@@
 $EndComp
 $Comp
-L MCU_Microchip_ATmega:ATmega328P-AU U401
+L LedBarController:ATmega48PV-10AU-arduino-atmega48pv-10au-arduino-LedBarController-rescue U401
 U 1 1 5F8297C2
 P 2500 3400
+AR Path="/5F8297C2" Ref="U401"  Part="1"
+AR Path="/602F109A/602FDBCD/5F8297C2" Ref="U401"  Part="1"
 F 0 "U401" H 2850 1900 50  0000 C CNN
 F 1 "ATmega328P-AU" H 2900 1800 50  0000 C CNN

Commit message: Added more testpoints
Parts:
- added TP401: dbg1, symbol Connector:TestPoint
- added TP402: dbg2, symbol Connector:TestPoint
- added TP403: scl, symbol Connector:TestPoint
- added TP404: sda, symbol Connector:TestPoint
- added TP405: reset, symbol Connector:TestPoint
- added TP406: ~button, symbol Connector:TestPoint
Connections:
- net labels added: button, debug1, debug2, ~button
- wire segments 114 -> 122
- no-connect marks 4 -> 2
Changed lines of the file:
@@
 Text Label 9100 4250 0    50   ~ 0
 reset
-Text HLabel 4000 3100 2    50   Input ~ 0
-~button~
 Wire Wire Line
 	4000 2300 3100 2300
@@
 sda
 Wire Wire Line
-	5600 7000 6350 7000
-Wire Wire Line
 	5600 6800 5600 7000
-Wire Wire Line
-	5950 7100 6350 7100
 Wire Wire Line
 	5950 6800 5950 7100
@@
 	-1   0    0    -1
 $EndComp
-Text HLabel 6350 7000 2    50   Output ~ 0
-scl
 Text HLabel 6350 7100 2    50   BiDi ~ 0
 sda
@@
 	1    0    0    -1
 $EndComp
-NoConn ~ 3100 3300
 NoConn ~ 1900 2500
 $Comp
@@
 Wire Wire Line
 	4000 4500 3100 4500
-NoConn ~ 3100 3200
 Wire Wire Line
 	9350 1000 9550 1000
@@
 Wire Wire Line
 	2600 1500 2600 1900
+Wire Wire Line
+	3100 3200 3900 3200
+Wire Wire Line
+	3100 3300 3900 3300
+Text Label 3500 3300 0    50   ~ 0
+debug2
+$Comp
+L Connector:TestPoint TP401
+U 1 1 607A0A42
+P 3900 3200
+F 0 "TP401" V 3900 3388 50  0000 L CNN
+F 1 "dbg1" V 3945 3388 50  0001 L CNN
+F 2 "" H 4100 3200 50  0001 C CNN
+F 3 "~" H 4100 3200 50  0001 C CNN
+	1    3900 3200
+	0    1    1    0
+$EndComp
+$Comp
+L Connector:TestPoint TP402
+U 1 1 607A1F2C
+P 3900 3300
+F 0 "TP402" V 3900 3488 50  0000 L CNN
+F 1 "dbg2" V 3945 3488 50  0001 L CNN
+F 2 "" H 4100 3300 50  0001 C CNN
+F 3 "~" H 4100 3300 50  0001 C CNN
+	1    3900 3300
+	0    1    1    0
+$EndComp
+Text Label 3500 3200 0    50   ~ 0
+debug1
+Text HLabel 6350 7000 2    50   Output ~ 0
+scl
+$Comp
+L Connector:TestPoint TP405
+U 1 1 607D2CC2
+P 9600 4250
+F 0 "TP405" V 9554 4438 50  0000 L CNN
+F 1 "reset" V 9645 4438 50  0000 L CNN
+F 2 "" H 9800 4250 50  0001 C CNN
+F 3 "~" H 9800 4250 50  0001 C CNN
+	1    9600 4250
+	0    1    1    0
+$EndComp
+Wire Wire Line
+	9600 4250 9500 4250
+$Comp
+L Connector:TestPoint TP403
+U 1 1 607DEDB6
+P 5600 7150
+F 0 "TP403" H 5542 7176 50  0000 R CNN
+F 1 "scl" H 5542 7267 50  0000 R CNN
+F 2 "" H 5800 7150 50  0001 C CNN
+F 3 "~" H 5800 7150 50  0001 C CNN
+	1    5600 7150
+	-1   0    0    1
+$EndComp
+$Comp
+L Connector:TestPoint TP404
+U 1 1 607E3DF5
+P 5950 7150
+F 0 "TP404" H 5892 7176 50  0000 R CNN
+F 1 "sda" H 5892 7267 50  0000 R CNN
+F 2 "" H 6150 7150 50  0001 C CNN
+F 3 "~" H 6150 7150 50  0001 C CNN
+	1    5950 7150
+	-1   0    0    1
+$EndComp
+Wire Wire Line
+	5600 7000 6350 7000
+Wire Wire Line
+	5950 7100 6350 7100
+Wire Wire Line
+	5600 7000 5600 7150
+Wire Wire Line
+	5950 7100 5950 7150
+Text Label 3500 3100 0    50   ~ 0
+button
+Text HLabel 10000 6000 2    50   Input ~ 0
+~button~
+Wire Wire Line
+	9000 6000 9500 6000
+Text Label 9050 6000 0    50   ~ 0
+~button
+$Comp
+L Connector:TestPoint TP406
+U 1 1 60873ACA
+P 9500 5950
+F 0 "TP406" H 9558 6074 50  0000 L CNN
+F 1 "~button" H 9558 5976 50  0000 L CNN
+F 2 "" H 9700 5950 50  0001 C CNN
+F 3 "~" H 9700 5950 50  0001 C CNN
+	1    9500 5950
+	1    0    0    -1
+$EndComp
+Wire Wire Line
+	9500 5950 9500 6000
+Connection ~ 9500 6000
+Wire Wire Line
+	9500 6000 10000 6000
 $EndSCHEMATC
