File: LedBarController/RS485.sch (KiCad schematic (older format))
At the start: 10 parts, among them J201 Conn_01x04, U201 MAX485E

Commit message: Work in progress
Other:
- note added: "TODO: jumper for end-resistor\nTODO: 2nd connector, one for each side"
Changed lines of the file:
@@
 Wire Wire Line
 	7000 3500 7000 3550
+Text Notes 2900 4150 0    50   ~ 0
+TODO: jumper for end-resistor\nTODO: 2nd connector, one for each side
 $EndSCHEMATC

Commit message: Restarted PCB
Parts:
- added J1301: Conn_01x04, Connector_JST:JST_PH_S4B-PH-K_1x04_P2.00mm_Horizontal, symbol Connector_Generic:Conn_01x04
- added JP1301: Jumper_2_Bridged, Connector_PinHeader_2.54mm:PinHeader_1x02_P2.54mm_Vertical, symbol Jumper:Jumper_2_Bridged
- renumbered J201 to J1302, R201 to R1301, R202 to R1302, R203 to R1303, TP201 to TP1301, TP202 to TP1302, TP204 to TP1303, TP203 to TP1304, TP205 to TP1305, U201 to U1301
Connections:
- net +5V: now also J1301.4 (Pin_4)
- net A: now also J1301.2 (Pin_2)
- net B: now also J1301.3 (Pin_3), JP1301.1 (A); no longer R1302.1
- net GND: now also J1301.1 (Pin_1)
- new net: JP1301.2 (B), R1302.1
Other:
- note removed: "TODO: jumper for end-resistor\nTODO: 2nd connector, one for each side"
- moved on the sheet: J1302, R1301, R1302, R1303, TP1301, TP1304

Commit message: Pwm circuit routed (no plane yet)
Parts:
- removed J1301, J1302: Conn_01x04, Connector_JST:JST_PH_S4B-PH-K_1x04_P2.00mm_Horizontal, symbol Connector_Generic:Conn_01x04
- added J1301, J1302: Screw_Terminal_01x03, TerminalBlock_TE-Connectivity:TerminalBlock_TE_282834-3_1x03_P2.54mm_Horizontal, symbol Connector:Screw_Terminal_01x03
Connections:
- net A: now also J1301.2 (Pin_2), J1302.2 (Pin_2)
- net B: now also J1301.1 (Pin_1), J1302.3 (Pin_3)
- net GND: now also J1301.3 (Pin_3), J1302.1 (Pin_1)
Changed lines of the file:
@@
-$EndComp
-$Comp
-L Connector_Generic:Conn_01x04 J1302
-U 1 1 5F7BCC5A
-P 3350 3300
-F 0 "J1302" H 3350 3550 50  0000 C CNN
-F 1 "Conn_01x04" V 3500 3250 50  0000 C CNN
-F 2 "Connector_JST:JST_PH_S4B-PH-K_1x04_P2.00mm_Horizontal" H 3350 3300 50  0001 C CNN
-F 3 "~" H 3350 3300 50  0001 C CNN
-	1    3350 3300
-	-1   0    0    1
 $EndComp
 $Comp
@@
 Wire Wire Line
 	5000 3200 5000 3350
-$Comp
-L Connector_Generic:Conn_01x04 J1301
-U 1 1 5F80B945
-P 4350 3300
-F 0 "J1301" H 4350 3550 50  0000 C CNN
-F 1 "Conn_01x04" V 4500 3250 50  0000 C CNN
-F 2 "Connector_JST:JST_PH_S4B-PH-K_1x04_P2.00mm_Horizontal" H 4350 3300 50  0001 C CNN
-F 3 "~" H 4350 3300 50  0001 C CNN
-	1    4350 3300
-	1    0    0    1
-$EndComp
 Wire Wire Line
 	4000 2500 4000 3200
@@
 	1    0    0    -1
 $EndComp
-$Comp
-L power:+5V #PWR01303
-U 1 1 5F81AA3E
-P 3700 2950
-F 0 "#PWR01303" H 3700 2800 50  0001 C CNN
-F 1 "+5V" H 3715 3123 50  0000 C CNN
-F 2 "" H 3700 2950 50  0001 C CNN
-F 3 "" H 3700 2950 50  0001 C CNN
-	1    3700 2950
-	1    0    0    -1
-$EndComp
-Wire Wire Line
-	3700 2950 3700 3100
 Wire Wire Line
 	3700 3550 3700 3400
@@
 	4000 4000 4500 4000
 Wire Wire Line
-	3550 3100 3700 3100
-Wire Wire Line
 	3550 3400 3700 3400
 Connection ~ 3700 3400
 Wire Wire Line
 	3700 3400 4150 3400
-Connection ~ 3700 3100
-Wire Wire Line
-	3700 3100 4150 3100
+$Comp
+L Connector:Screw_Terminal_01x03 J1301
+U 1 1 5F9ABD9D
+P 3350 3300
+F 0 "J1301" H 3268 3617 50  0000 C CNN
+F 1 "Screw_Terminal_01x03" H 3268 3526 50  0000 C CNN
+F 2 "TerminalBlock_TE-Connectivity:TerminalBlock_TE_282834-3_1x03_P2.54mm_Horizontal" H 3350 3300 50  0001 C CNN
+F 3 "~" H 3350 3300 50  0001 C CNN
+	1    3350 3300
+	-1   0    0    -1
+$EndComp
+$Comp
+L Connector:Screw_Terminal_01x03 J1302
+U 1 1 5F9AB4F9
+P 4350 3300
+F 0 "J1302" H 4268 2975 50  0000 C CNN
+F 1 "Screw_Terminal_01x03" H 4268 3066 50  0000 C CNN
+F 2 "TerminalBlock_TE-Connectivity:TerminalBlock_TE_282834-3_1x03_P2.54mm_Horizontal" H 4350 3300 50  0001 C CNN
+F 3 "~" H 4350 3300 50  0001 C CNN
+	1    4350 3300
+	1    0    0    1
+$EndComp
 $EndSCHEMATC

Commit message: Added capacitor for DS1307 and changed package of MAX485
Parts:
- U1301: footprint Package_TO_SOT_SMD:SOT-23-8_Handsoldering -> Package_SO:SOP-8_3.76x4.96mm_P1.27mm
Changed lines of the file:
@@
 F 0 "U1301" H 5750 3750 50  0000 C CNN
 F 1 "MAX485E" H 5750 3650 50  0000 C CNN
-F 2 "Package_TO_SOT_SMD:SOT-23-8_Handsoldering" H 6000 2500 50  0001 C CNN
+F 2 "Package_SO:SOP-8_3.76x4.96mm_P1.27mm" H 6000 2500 50  0001 C CNN
 F 3 "https://datasheets.maximintegrated.com/en/ds/MAX1487E-MAX491E.pdf" H 6000 3250 50  0001 C CNN
 	1    6000 3200

Commit message: Updated labels in schematic and moved RTC to sub-schematic
Connections:
- net Rx renamed rxd
- net Tx renamed txd
- net TxEn renamed tx_en
Changed lines of the file:
@@
 $Descr A4 11693 8268
 encoding utf-8
-Sheet 13 13
+Sheet 13 14
 Title ""
 Date ""
@@
 $EndComp
 Text HLabel 7400 4000 2    50   Input ~ 0
-TxEn
-Text HLabel 7400 3000 2    50   Output ~ 0
-Rx
+tx_en
 Text HLabel 7400 3500 2    50   Input ~ 0
-Tx
+txd
 Wire Wire Line
 	5000 2000 5000 2100
@@
 	1    0    0    1
 $EndComp
+Text HLabel 7400 3000 2    50   Output ~ 0
+rxd
 $EndSCHEMATC

Commit message: Added missing capacitor for MAX485
Parts:
- added C1301: 0.1uF, Capacitor_SMD:C_0805_2012Metric_Pad1.18x1.45mm_HandSolder, symbol Device:C
Connections:
- net +5V: now also C1301.1
- net GND: now also C1301.2
Changed lines of the file:
@@
 Text HLabel 7400 3000 2    50   Output ~ 0
 rxd
+$Comp
+L Device:C C1301
+U 1 1 5FE4FDAD
+P 6850 1950
+F 0 "C1301" H 6965 1996 50  0000 L CNN
+F 1 "0.1uF" H 6965 1905 50  0000 L CNN
+F 2 "Capacitor_SMD:C_0805_2012Metric_Pad1.18x1.45mm_HandSolder" H 6888 1800 50  0001 C CNN
+F 3 "~" H 6850 1950 50  0001 C CNN
+	1    6850 1950
+	1    0    0    -1
+$EndComp
+$Comp
+L power:GND #PWR01307
+U 1 1 5FE50064
+P 6850 2300
+F 0 "#PWR01307" H 6850 2050 50  0001 C CNN
+F 1 "GND" H 6855 2127 50  0000 C CNN
+F 2 "" H 6850 2300 50  0001 C CNN
+F 3 "" H 6850 2300 50  0001 C CNN
+	1    6850 2300
+	1    0    0    -1
+$EndComp
+$Comp
+L power:+5V #PWR01303
+U 1 1 5FE5053C
+P 6850 1600
+F 0 "#PWR01303" H 6850 1450 50  0001 C CNN
+F 1 "+5V" H 6865 1773 50  0000 C CNN
+F 2 "" H 6850 1600 50  0001 C CNN
+F 3 "" H 6850 1600 50  0001 C CNN
+	1    6850 1600
+	1    0    0    -1
+$EndComp
+Wire Wire Line
+	6850 1600 6850 1800
+Wire Wire Line
+	6850 2100 6850 2300
 $EndSCHEMATC

Commit message: Routed LEDs and solder jumpers, renumbered diodes (and LEDs) on microcontroller schematic
Changed lines of the file:
@@
 P 3350 3300
 F 0 "J1301" H 3268 3617 50  0000 C CNN
-F 1 "Screw_Terminal_01x03" H 3268 3526 50  0000 C CNN
+F 1 "Screw_Terminal_01x03" H 3268 3526 50  0001 C CNN
 F 2 "TerminalBlock_TE-Connectivity:TerminalBlock_TE_282834-3_1x03_P2.54mm_Horizontal" H 3350 3300 50  0001 C CNN
 F 3 "~" H 3350 3300 50  0001 C CNN
@@
 P 4350 3300
 F 0 "J1302" H 4268 2975 50  0000 C CNN
-F 1 "Screw_Terminal_01x03" H 4268 3066 50  0000 C CNN
+F 1 "Screw_Terminal_01x03" H 4268 3066 50  0001 C CNN
 F 2 "TerminalBlock_TE-Connectivity:TerminalBlock_TE_282834-3_1x03_P2.54mm_Horizontal" H 4350 3300 50  0001 C CNN
 F 3 "~" H 4350 3300 50  0001 C CNN

Commit message: Work in progress
Parts:
- C1301: Feature (none) -> RS485_SUPPORTED; Price (none) -> 0.0057; is stock (none) -> yes
- J1301: Feature (none) -> RS485_SUPPORTED_1CONN; Price (none) -> 0.202; is stock (none) -> yes
- J1302: Feature (none) -> RS485_SUPPORTED_2CONN; Price (none) -> 0.202; is stock (none) -> yes
- JP1301: Feature (none) -> RS485_SUPPORTED; Price (none) -> 0.0062; is stock (none) -> yes
- R1301, R1303: value 20K -> 1K; Feature (none) -> RS485_SUPPORTED; Price (none) -> 0.0036; is stock (none) -> yes
- R1302: Feature (none) -> RS485_SUPPORTED; Price (none) -> 0.0036; is stock (none) -> yes
- TP1301, TP1302, TP1303, TP1304, TP1305: Feature (none) -> RS485_SUPPORTED; Price (none) -> 0; is stock (none) -> n.a.
- U1301: Feature (none) -> 10V_SUPPORTED; Price (none) -> 0.065; is stock (none) -> no
Changed lines of the file:
@@
 F 2 "Package_SO:SOP-8_3.76x4.96mm_P1.27mm" H 6000 2500 50  0001 C CNN
 F 3 "https://datasheets.maximintegrated.com/en/ds/MAX1487E-MAX491E.pdf" H 6000 3250 50  0001 C CNN
+F 4 "10V_SUPPORTED" H 6000 3200 50  0001 C CNN "Feature"
+F 5 "0.065" H 6000 3200 50  0001 C CNN "Price"
+F 6 "no" H 6000 3200 50  0001 C CNN "is stock"
 	1    6000 3200
 	-1   0    0    -1
@@
 P 5000 4250
 F 0 "R1303" H 5070 4296 50  0000 L CNN
-F 1 "20K" H 5070 4205 50  0000 L CNN
+F 1 "1K" H 5070 4205 50  0000 L CNN
 F 2 "Resistor_SMD:R_0805_2012Metric_Pad1.20x1.40mm_HandSolder" V 4930 4250 50  0001 C CNN
 F 3 "~" H 5000 4250 50  0001 C CNN
+F 4 "RS485_SUPPORTED" H 5000 4250 50  0001 C CNN "Feature"
+F 5 "0.0036" H 5000 4250 50  0001 C CNN "Price"
+F 6 "yes" H 5000 4250 50  0001 C CNN "is stock"
 	1    5000 4250
 	1    0    0    -1
@@
 P 5000 2250
 F 0 "R1301" H 5070 2296 50  0000 L CNN
-F 1 "20K" H 5070 2205 50  0000 L CNN
+F 1 "1K" H 5070 2205 50  0000 L CNN
 F 2 "Resistor_SMD:R_0805_2012Metric_Pad1.20x1.40mm_HandSolder" V 4930 2250 50  0001 C CNN
 F 3 "~" H 5000 2250 50  0001 C CNN
+F 4 "RS485_SUPPORTED" H 5000 2250 50  0001 C CNN "Feature"
+F 5 "0.0036" H 5000 2250 50  0001 C CNN "Price"
+F 6 "yes" H 5000 2250 50  0001 C CNN "is stock"
 	1    5000 2250
 	1    0    0    -1
@@
 F 2 "Resistor_SMD:R_0805_2012Metric_Pad1.20x1.40mm_HandSolder" V 4930 3500 50  0001 C CNN
 F 3 "~" H 5000 3500 50  0001 C CNN
+F 4 "RS485_SUPPORTED" H 5000 3500 50  0001 C CNN "Feature"
+F 5 "0.0036" H 5000 3500 50  0001 C CNN "Price"
+F 6 "yes" H 5000 3500 50  0001 C CNN "is stock"
 	1    5000 3500
 	1    0    0    -1
@@
 F 2 "TestPoint:TestPoint_Pad_D1.0mm" H 7200 2950 50  0001 C CNN
 F 3 "~" H 7200 2950 50  0001 C CNN
+F 4 "RS485_SUPPORTED" H 7000 2950 50  0001 C CNN "Feature"
+F 5 "0" H 7000 2950 50  0001 C CNN "Price"
+F 6 "n.a." H 7000 2950 50  0001 C CNN "is stock"
 	1    7000 2950
 	1    0    0    -1
@@
 F 2 "TestPoint:TestPoint_Pad_D1.0mm" H 7200 3550 50  0001 C CNN
 F 3 "~" H 7200 3550 50  0001 C CNN
+F 4 "RS485_SUPPORTED" H 7000 3550 50  0001 C CNN "Feature"
+F 5 "0" H 7000 3550 50  0001 C CNN "Price"
+F 6 "n.a." H 7000 3550 50  0001 C CNN "is stock"
 	1    7000 3550
 	-1   0    0    1
@@
 F 2 "TestPoint:TestPoint_Pad_D1.0mm" H 6700 4050 50  0001 C CNN
 F 3 "~" H 6700 4050 50  0001 C CNN
+F 4 "RS485_SUPPORTED" H 6500 4050 50  0001 C CNN "Feature"
+F 5 "0" H 6500 4050 50  0001 C CNN "Price"
+F 6 "n.a." H 6500 4050 50  0001 C CNN "is stock"
 	1    6500 4050
 	-1   0    0    1
@@
 F 2 "TestPoint:TestPoint_Pad_D1.0mm" H 4700 2450 50  0001 C CNN
 F 3 "~" H 4700 2450 50  0001 C CNN
+F 4 "RS485_SUPPORTED" H 4500 2450 50  0001 C CNN "Feature"
+F 5 "0" H 4500 2450 50  0001 C CNN "Price"
+F 6 "n.a." H 4500 2450 50  0001 C CNN "is stock"
 	1    4500 2450
 	1    0    0    -1
@@
 F 2 "TestPoint:TestPoint_Pad_D1.0mm" H 4700 4050 50  0001 C CNN
 F 3 "~" H 4700 4050 50  0001 C CNN
+F 4 "RS485_SUPPORTED" H 4500 4050 50  0001 C CNN "Feature"
+F 5 "0" H 4500 4050 50  0001 C CNN "Price"
+F 6 "n.a." H 4500 4050 50  0001 C CNN "is stock"
 	1    4500 4050
 	-1   0    0    1
@@
 F 2 "Connector_PinHeader_2.54mm:PinHeader_1x02_P2.54mm_Vertical" H 5000 3000 50  0001 C CNN
 F 3 "~" H 5000 3000 50  0001 C CNN
+F 4 "RS485_SUPPORTED" H 5000 3000 50  0001 C CNN "Feature"
+F 5 "0.0062" H 5000 3000 50  0001 C CNN "Price"
+F 6 "yes" H 5000 3000 50  0001 C CNN "is stock"
 	1    5000 3000
 	0    1    1    0
@@
 F 2 "TerminalBlock_TE-Connectivity:TerminalBlock_TE_282834-3_1x03_P2.54mm_Horizontal" H 3350 3300 50  0001 C CNN
 F 3 "~" H 3350 3300 50  0001 C CNN
+F 4 "RS485_SUPPORTED_1CONN" H 3350 3300 50  0001 C CNN "Feature"
+F 5 "0.202" H 3350 3300 50  0001 C CNN "Price"
+F 6 "yes" H 3350 3300 50  0001 C CNN "is stock"
 	1    3350 3300
 	-1   0    0    -1
@@
 F 2 "TerminalBlock_TE-Connectivity:TerminalBlock_TE_282834-3_1x03_P2.54mm_Horizontal" H 4350 3300 50  0001 C CNN
 F 3 "~" H 4350 3300 50  0001 C CNN
+F 4 "RS485_SUPPORTED_2CONN" H 4350 3300 50  0001 C CNN "Feature"
+F 5 "0.202" H 4350 3300 50  0001 C CNN "Price"
+F 6 "yes" H 4350 3300 50  0001 C CNN "is stock"
 	1    4350 3300
 	1    0    0    1
@@
 F 2 "Capacitor_SMD:C_0805_2012Metric_Pad1.18x1.45mm_HandSolder" H 6888 1800 50  0001 C CNN
 F 3 "~" H 6850 1950 50  0001 C CNN
+F 4 "RS485_SUPPORTED" H 6850 1950 50  0001 C CNN "Feature"
+F 5 "0.0057" H 6850 1950 50  0001 C CNN "Price"
+F 6 "yes" H 6850 1950 50  0001 C CNN "is stock"
 	1    6850 1950
 	1    0    0    -1
