File: LedBarController/RS485.sch (KiCad schematic (older format))
At the start: 13 parts, among them J1301 Screw_Terminal_01x03, J1302 Screw_Terminal_01x03, U1301 MAX485E

Commit message: Reduced circuit by remove extra features. Routed whole board. Needs refinement
Parts:
- removed J1302: Screw_Terminal_01x03, TerminalBlock_TE-Connectivity:TerminalBlock_TE_282834-3_1x03_P2.54mm_Horizontal, symbol Connector:Screw_Terminal_01x03
- removed TP1302: Rx, TestPoint:TestPoint_Pad_D1.0mm, symbol Connector:TestPoint
- removed TP1303: Tx, TestPoint:TestPoint_Pad_D1.0mm, symbol Connector:TestPoint
- removed TP1305: TxEn, TestPoint:TestPoint_Pad_D1.0mm, symbol Connector:TestPoint
Changed lines of the file:
@@
 $Descr A4 11693 8268
 encoding utf-8
-Sheet 13 14
+Sheet 12 13
 Title ""
 Date ""
@@
 	4500 4000 5000 4000
 $Comp
-L Connector:TestPoint TP1302
-U 1 1 5FA67E8C
-P 7000 2950
-F 0 "TP1302" H 7058 3068 50  0000 L CNN
-F 1 "Rx" H 7058 2977 50  0000 L CNN
-F 2 "TestPoint:TestPoint_Pad_D1.0mm" H 7200 2950 50  0001 C CNN
-F 3 "~" H 7200 2950 50  0001 C CNN
-F 4 "RS485_SUPPORTED" H 7000 2950 50  0001 C CNN "Feature"
-F 5 "0" H 7000 2950 50  0001 C CNN "Price"
-F 6 "n.a." H 7000 2950 50  0001 C CNN "is stock"
-	1    7000 2950
-	1    0    0    -1
-$EndComp
-$Comp
-L Connector:TestPoint TP1303
-U 1 1 5FA6827F
-P 7000 3550
-F 0 "TP1303" H 6942 3576 50  0000 R CNN
-F 1 "Tx" H 6942 3667 50  0000 R CNN
-F 2 "TestPoint:TestPoint_Pad_D1.0mm" H 7200 3550 50  0001 C CNN
-F 3 "~" H 7200 3550 50  0001 C CNN
-F 4 "RS485_SUPPORTED" H 7000 3550 50  0001 C CNN "Feature"
-F 5 "0" H 7000 3550 50  0001 C CNN "Price"
-F 6 "n.a." H 7000 3550 50  0001 C CNN "is stock"
-	1    7000 3550
-	-1   0    0    1
-$EndComp
-$Comp
-L Connector:TestPoint TP1305
-U 1 1 5FA685D1
-P 6500 4050
-F 0 "TP1305" H 6442 4076 50  0000 R CNN
-F 1 "TxEn" H 6442 4167 50  0000 R CNN
-F 2 "TestPoint:TestPoint_Pad_D1.0mm" H 6700 4050 50  0001 C CNN
-F 3 "~" H 6700 4050 50  0001 C CNN
-F 4 "RS485_SUPPORTED" H 6500 4050 50  0001 C CNN "Feature"
-F 5 "0" H 6500 4050 50  0001 C CNN "Price"
-F 6 "n.a." H 6500 4050 50  0001 C CNN "is stock"
-	1    6500 4050
-	-1   0    0    1
-$EndComp
-$Comp
 L Connector:TestPoint TP1301
 U 1 1 5FA6885F
@@
 $EndComp
 Connection ~ 4500 4000
-Connection ~ 7000 3000
-Connection ~ 6500 4000
 Wire Wire Line
 	4500 4000 4500 4050
@@
 	4500 2450 4500 2500
 Connection ~ 4500 2500
-Wire Wire Line
-	6500 4050 6500 4000
-Wire Wire Line
-	7000 2950 7000 3000
 Text Label 3550 3200 0    50   ~ 0
 B
@@
 Wire Wire Line
 	7400 3500 7000 3500
-Connection ~ 7000 3500
-Wire Wire Line
-	7000 3500 7000 3550
 $Comp
 L Jumper:Jumper_2_Bridged JP1301
@@
 Wire Wire Line
 	4000 2500 4000 3200
-Wire Wire Line
-	4000 3200 4150 3200
 $Comp
 L power:GND #PWR01304
@@
 Wire Wire Line
 	3550 3200 4000 3200
-Connection ~ 4000 3200
 Wire Wire Line
 	3550 3300 4000 3300
@@
 Wire Wire Line
 	4000 3300 4000 4000
-Connection ~ 4000 3300
-Wire Wire Line
-	4000 3300 4150 3300
 Wire Wire Line
 	4000 4000 4500 4000
 Wire Wire Line
 	3550 3400 3700 3400
-Connection ~ 3700 3400
-Wire Wire Line
-	3700 3400 4150 3400
-$Comp
-L Connector:Screw_Terminal_01x03 J1301
-U 1 1 5F9ABD9D
-P 3350 3300
-F 0 "J1301" H 3268 3617 50  0000 C CNN
-F 1 "Screw_Terminal_01x03" H 3268 3526 50  0001 C CNN
-F 2 "TerminalBlock_TE-Connectivity:TerminalBlock_TE_282834-3_1x03_P2.54mm_Horizontal" H 3350 3300 50  0001 C CNN
-F 3 "~" H 3350 3300 50  0001 C CNN
-F 4 "RS485_SUPPORTED_1CONN" H 3350 3300 50  0001 C CNN "Feature"
-F 5 "0.202" H 3350 3300 50  0001 C CNN "Price"
-F 6 "yes" H 3350 3300 50  0001 C CNN "is stock"
-	1    3350 3300
-	-1   0    0    -1
-$EndComp
-$Comp
-L Connector:Screw_Terminal_01x03 J1302
-U 1 1 5F9AB4F9
-P 4350 3300
-F 0 "J1302" H 4268 2975 50  0000 C CNN
-F 1 "Screw_Terminal_01x03" H 4268 3066 50  0001 C CNN
-F 2 "TerminalBlock_TE-Connectivity:TerminalBlock_TE_282834-3_1x03_P2.54mm_Horizontal" H 4350 3300 50  0001 C CNN
-F 3 "~" H 4350 3300 50  0001 C CNN
-F 4 "RS485_SUPPORTED_2CONN" H 4350 3300 50  0001 C CNN "Feature"
-F 5 "0.202" H 4350 3300 50  0001 C CNN "Price"
-F 6 "yes" H 4350 3300 50  0001 C CNN "is stock"
-	1    4350 3300
-	1    0    0    1
-$EndComp
 Text HLabel 7400 3000 2    50   Output ~ 0
 rxd
@@
 Wire Wire Line
 	6850 2100 6850 2300
+$Comp
+L Connector:Screw_Terminal_01x03 J1301
+U 1 1 5F9ABD9D
+P 3350 3300
+F 0 "J1301" H 3350 3500 50  0000 C CNN
+F 1 "Screw_Terminal_01x03" H 3268 3526 50  0001 C CNN
+F 2 "TerminalBlock_TE-Connectivity:TerminalBlock_TE_282834-3_1x03_P2.54mm_Horizontal" H 3350 3300 50  0001 C CNN
+F 3 "~" H 3350 3300 50  0001 C CNN
+F 4 "RS485_SUPPORTED_1CONN" H 3350 3300 50  0001 C CNN "Feature"
+F 5 "0.202" H 3350 3300 50  0001 C CNN "Price"
+F 6 "yes" H 3350 3300 50  0001 C CNN "is stock"
+	1    3350 3300
+	-1   0    0    -1
+$EndComp
 $EndSCHEMATC

Commit message: Reanotate
Parts:
- renumbered C1301 to C501, J1301 to J501, JP1301 to JP501, R1301 to R501, R1302 to R502, R1303 to R503, TP1301 to TP501, TP1304 to TP502, U1301 to U501
Changed lines of the file:
@@
 $EndDescr
 $Comp
-L Interface_UART:MAX485E U1301
+L Interface_UART:MAX485E U501
 U 1 1 5F7B8096
 P 6000 3200
-F 0 "U1301" H 5750 3750 50  0000 C CNN
+F 0 "U501" H 5750 3750 50  0000 C CNN
 F 1 "MAX485E" H 5750 3650 50  0000 C CNN
 F 2 "Package_SO:SOP-8_3.76x4.96mm_P1.27mm" H 6000 2500 50  0001 C CNN
@@
 $EndComp
 $Comp
-L power:GND #PWR0122
+L power:GND #PWR0506
 U 1 1 5F7B92E7
 P 6000 4000
-F 0 "#PWR0122" H 6000 3750 50  0001 C CNN
+F 0 "#PWR0506" H 6000 3750 50  0001 C CNN
 F 1 "GND" H 6005 3827 50  0000 C CNN
 F 2 "" H 6000 4000 50  0001 C CNN
@@
 $EndComp
 $Comp
-L power:+5V #PWR0123
+L power:+5V #PWR0504
 U 1 1 5F7B9C6C
 P 6000 2500
-F 0 "#PWR0123" H 6000 2350 50  0001 C CNN
+F 0 "#PWR0504" H 6000 2350 50  0001 C CNN
 F 1 "+5V" H 6015 2673 50  0000 C CNN
 F 2 "" H 6000 2500 50  0001 C CNN
@@
 $EndComp
 $Comp
-L Device:R R1303
+L Device:R R503
 U 1 1 5F7BA62C
 P 5000 4250
-F 0 "R1303" H 5070 4296 50  0000 L CNN
+F 0 "R503" H 5070 4296 50  0000 L CNN
 F 1 "1K" H 5070 4205 50  0000 L CNN
 F 2 "Resistor_SMD:R_0805_2012Metric_Pad1.20x1.40mm_HandSolder" V 4930 4250 50  0001 C CNN
@@
 $EndComp
 $Comp
-L Device:R R1301
+L Device:R R501
 U 1 1 5F7BA295
 P 5000 2250
-F 0 "R1301" H 5070 2296 50  0000 L CNN
+F 0 "R501" H 5070 2296 50  0000 L CNN
 F 1 "1K" H 5070 2205 50  0000 L CNN
 F 2 "Resistor_SMD:R_0805_2012Metric_Pad1.20x1.40mm_HandSolder" V 4930 2250 50  0001 C CNN
@@
 $EndComp
 $Comp
-L power:GND #PWR0124
+L power:GND #PWR0502
 U 1 1 5F7BC240
 P 5000 2000
-F 0 "#PWR0124" H 5000 1750 50  0001 C CNN
+F 0 "#PWR0502" H 5000 1750 50  0001 C CNN
 F 1 "GND" H 5005 1827 50  0000 C CNN
 F 2 "" H 5000 2000 50  0001 C CNN
@@
 $EndComp
 $Comp
-L power:+5V #PWR0125
+L power:+5V #PWR0507
 U 1 1 5F7BB859
 P 5000 4500
-F 0 "#PWR0125" H 5000 4350 50  0001 C CNN
+F 0 "#PWR0507" H 5000 4350 50  0001 C CNN
 F 1 "+5V" H 5015 4673 50  0000 C CNN
 F 2 "" H 5000 4500 50  0001 C CNN
@@
 $EndComp
 $Comp
-L Device:R R1302
+L Device:R R502
 U 1 1 5F7BC04A
 P 5000 3500
-F 0 "R1302" H 5070 3546 50  0000 L CNN
+F 0 "R502" H 5070 3546 50  0000 L CNN
 F 1 "120" H 5070 3455 50  0000 L CNN
 F 2 "Resistor_SMD:R_0805_2012Metric_Pad1.20x1.40mm_HandSolder" V 4930 3500 50  0001 C CNN
@@
 	4500 4000 5000 4000
 $Comp
-L Connector:TestPoint TP1301
+L Connector:TestPoint TP501
 U 1 1 5FA6885F
 P 4500 2450
-F 0 "TP1301" H 4558 2568 50  0000 L CNN
+F 0 "TP501" H 4558 2568 50  0000 L CNN
 F 1 "B" H 4558 2477 50  0000 L CNN
 F 2 "TestPoint:TestPoint_Pad_D1.0mm" H 4700 2450 50  0001 C CNN
@@
 $EndComp
 $Comp
-L Connector:TestPoint TP1304
+L Connector:TestPoint TP502
 U 1 1 5FA68C0E
 P 4500 4050
-F 0 "TP1304" H 4442 4076 50  0000 R CNN
+F 0 "TP502" H 4442 4076 50  0000 R CNN
 F 1 "A" H 4442 4167 50  0000 R CNN
 F 2 "TestPoint:TestPoint_Pad_D1.0mm" H 4700 4050 50  0001 C CNN
@@
 	7400 3500 7000 3500
 $Comp
-L Jumper:Jumper_2_Bridged JP1301
+L Jumper:Jumper_2_Bridged JP501
 U 1 1 5F804235
 P 5000 3000
-F 0 "JP1301" V 5000 3058 50  0000 L CNN
+F 0 "JP501" V 5000 3058 50  0000 L CNN
 F 1 "Jumper_2_Bridged" V 5045 3058 50  0001 L CNN
 F 2 "Connector_PinHeader_2.54mm:PinHeader_1x02_P2.54mm_Vertical" H 5000 3000 50  0001 C CNN
@@
 	4000 2500 4000 3200
 $Comp
-L power:GND #PWR0126
+L power:GND #PWR0505
 U 1 1 5F81A772
 P 3700 3550
-F 0 "#PWR0126" H 3700 3300 50  0001 C CNN
+F 0 "#PWR0505" H 3700 3300 50  0001 C CNN
 F 1 "GND" H 3705 3377 50  0000 C CNN
 F 2 "" H 3700 3550 50  0001 C CNN
@@
 rxd
 $Comp
-L Device:C C1301
+L Device:C C501
 U 1 1 5FE4FDAD
 P 6850 1950
-F 0 "C1301" H 6965 1996 50  0000 L CNN
+F 0 "C501" H 6965 1996 50  0000 L CNN
 F 1 "0.1uF" H 6965 1905 50  0000 L CNN
 F 2 "Capacitor_SMD:C_0805_2012Metric_Pad1.18x1.45mm_HandSolder" H 6888 1800 50  0001 C CNN
@@
 $EndComp
 $Comp
-L power:GND #PWR0127
+L power:GND #PWR0503
 U 1 1 5FE50064
 P 6850 2300
-F 0 "#PWR0127" H 6850 2050 50  0001 C CNN
+F 0 "#PWR0503" H 6850 2050 50  0001 C CNN
 F 1 "GND" H 6855 2127 50  0000 C CNN
 F 2 "" H 6850 2300 50  0001 C CNN
@@
 $EndComp
 $Comp
-L power:+5V #PWR0128
+L power:+5V #PWR0501
 U 1 1 5FE5053C
 P 6850 1600
-F 0 "#PWR0128" H 6850 1450 50  0001 C CNN
+F 0 "#PWR0501" H 6850 1450 50  0001 C CNN
 F 1 "+5V" H 6865 1773 50  0000 C CNN
 F 2 "" H 6850 1600 50  0001 C CNN
@@
 	6850 2100 6850 2300
 $Comp
-L Connector:Screw_Terminal_01x03 J1301
+L Connector:Screw_Terminal_01x03 J501
 U 1 1 5F9ABD9D
 P 3350 3300
-F 0 "J1301" H 3350 3500 50  0000 C CNN
+F 0 "J501" H 3350 3500 50  0000 C CNN
 F 1 "Screw_Terminal_01x03" H 3268 3526 50  0001 C CNN
 F 2 "TerminalBlock_TE-Connectivity:TerminalBlock_TE_282834-3_1x03_P2.54mm_Horizontal" H 3350 3300 50  0001 C CNN

Commit message: Added more testpoints
Parts:
- added TP503: tx_en, symbol Connector:TestPoint
- added TP504: rxd, symbol Connector:TestPoint
- added TP505: txd, symbol Connector:TestPoint
Connections:
- net rxd: now also TP504.1
- net tx_en: now also TP503.1
- net txd: now also TP505.1
Changed lines of the file:
@@
 Wire Wire Line
 	6500 3300 6500 4000
-Wire Wire Line
-	6500 4000 7400 4000
 Connection ~ 6500 3300
 Wire Wire Line
@@
 	-1   0    0    -1
 $EndComp
+Wire Wire Line
+	6500 4000 7400 4000
+$Comp
+L Connector:TestPoint TP504
+U 1 1 607DBA66
+P 7000 2950
+F 0 "TP504" H 7058 3068 50  0000 L CNN
+F 1 "rxd" H 7058 2977 50  0000 L CNN
+F 2 "" H 7200 2950 50  0001 C CNN
+F 3 "~" H 7200 2950 50  0001 C CNN
+	1    7000 2950
+	1    0    0    -1
+$EndComp
+Wire Wire Line
+	7000 2950 7000 3000
+Connection ~ 7000 3000
+$Comp
+L Connector:TestPoint TP505
+U 1 1 607DCB5D
+P 7000 3550
+F 0 "TP505" H 6942 3576 50  0000 R CNN
+F 1 "txd" H 6942 3667 50  0000 R CNN
+F 2 "" H 7200 3550 50  0001 C CNN
+F 3 "~" H 7200 3550 50  0001 C CNN
+	1    7000 3550
+	-1   0    0    1
+$EndComp
+Wire Wire Line
+	7000 3500 7000 3550
+Connection ~ 7000 3500
+$Comp
+L Connector:TestPoint TP503
+U 1 1 607DD7B7
+P 6500 4050
+F 0 "TP503" H 6442 4076 50  0000 R CNN
+F 1 "tx_en" H 6442 4167 50  0000 R CNN
+F 2 "" H 6700 4050 50  0001 C CNN
+F 3 "~" H 6700 4050 50  0001 C CNN
+	1    6500 4050
+	-1   0    0    1
+$EndComp
+Wire Wire Line
+	6500 4000 6500 4050
+Connection ~ 6500 4000
 $EndSCHEMATC
