File: LedBarController/RTC.sch (KiCad schematic (older format))
At the start: 8 parts, among them U1401 DS1307ZN+, Y1401 32.768kHz

Commit message: Work in progress
Parts:
- C1401: value 0.47uF/5.5V -> 0.47F/5.5V; footprint (none) -> LedBarController:CP_Disc_D11.5mm_H12.3mm_P4.7mm_Vertical; Feature (none) -> RTC_SUPPORTED_BACKEDUP; Price (none) -> 0.376; is stock (none) -> yes
- C1402: value 100nF -> 0.1uF; Feature (none) -> RTC_SUPPORTED_BACKEDUP; Price (none) -> 0.0057; is stock (none) -> yes
- C1403: Feature (none) -> RTC_SUPPORTED; Price (none) -> 0.0057; is stock (none) -> yes
- D1401: Feature (none) -> RTC_SUPPORTED_BACKEDUP; Price (none) -> 0.0152; is stock (none) -> no
- R1401: Feature (none) -> RTC_SUPPORTED_BACKEDUP; Price (none) -> 0.0036; is stock (none) -> yes
- R1402: Feature (none) -> RTC_SUPPORTED; Price (none) -> 0.0036; is stock (none) -> yes
- U1401: Feature (none) -> RTC_SUPPORTED; Price (none) -> 0.098; is stock (none) -> no
- Y1401: Feature (none) -> UC; Price (none) -> 0.0618; is stock (none) -> yes
Changed lines of the file:
@@
 F 2 "Package_SO:SOIC-8_3.9x4.9mm_P1.27mm" H 6200 4050 50  0001 C CNN
 F 3 "https://datasheets.maximintegrated.com/en/ds/DS1307.pdf" H 6200 4550 50  0001 C CNN
+F 4 "RTC_SUPPORTED" H 6200 4550 50  0001 C CNN "Feature"
+F 5 "0.098" H 6200 4550 50  0001 C CNN "Price"
+F 6 "no" H 6200 4550 50  0001 C CNN "is stock"
 	1    6200 4550
 	1    0    0    -1
@@
 F 2 "Crystal:Crystal_DS26_D2.0mm_L6.0mm_Vertical" H 5500 4750 50  0001 C CNN
 F 3 "~" H 5500 4750 50  0001 C CNN
+F 4 "UC" H 5500 4750 50  0001 C CNN "Feature"
+F 5 "0.0618" H 5500 4750 50  0001 C CNN "Price"
+F 6 "yes" H 5500 4750 50  0001 C CNN "is stock"
 	1    5500 4750
 	1    0    0    -1
@@
 F 2 "Resistor_SMD:R_0805_2012Metric_Pad1.20x1.40mm_HandSolder" V 6930 4150 50  0001 C CNN
 F 3 "~" H 7000 4150 50  0001 C CNN
+F 4 "RTC_SUPPORTED" H 7000 4150 50  0001 C CNN "Feature"
+F 5 "0.0036" H 7000 4150 50  0001 C CNN "Price"
+F 6 "yes" H 7000 4150 50  0001 C CNN "is stock"
 	1    7000 4150
 	1    0    0    -1
@@
 AR Path="/5FDC6C57/5FDEB048" Ref="C1402"  Part="1"
 F 0 "C1402" H 9065 2946 50  0000 L CNN
-F 1 "100nF" H 9065 2855 50  0000 L CNN
+F 1 "0.1uF" H 9065 2855 50  0000 L CNN
 F 2 "Capacitor_SMD:C_0805_2012Metric_Pad1.18x1.45mm_HandSolder" H 8988 2750 50  0001 C CNN
 F 3 "~" H 8950 2900 50  0001 C CNN
+F 4 "RTC_SUPPORTED_BACKEDUP" H 8950 2900 50  0001 C CNN "Feature"
+F 5 "0.0057" H 8950 2900 50  0001 C CNN "Price"
+F 6 "yes" H 8950 2900 50  0001 C CNN "is stock"
 	1    8950 2900
 	1    0    0    -1
@@
 AR Path="/5FDC6C57/5FDEB04E" Ref="C1401"  Part="1"
 F 0 "C1401" H 8318 2946 50  0000 L CNN
-F 1 "0.47uF/5.5V" H 8318 2855 50  0000 L CNN
-F 2 "" H 8238 2750 50  0001 C CNN
+F 1 "0.47F/5.5V" H 8318 2855 50  0000 L CNN
+F 2 "LedBarController:CP_Disc_D11.5mm_H12.3mm_P4.7mm_Vertical" H 8238 2750 50  0001 C CNN
 F 3 "~" H 8200 2900 50  0001 C CNN
+F 4 "RTC_SUPPORTED_BACKEDUP" H 8200 2900 50  0001 C CNN "Feature"
+F 5 "0.376" H 8200 2900 50  0001 C CNN "Price"
+F 6 "yes" H 8200 2900 50  0001 C CNN "is stock"
 	1    8200 2900
 	1    0    0    -1
@@
 F 2 "Resistor_SMD:R_0805_2012Metric_Pad1.20x1.40mm_HandSolder" V 7680 2600 50  0001 C CNN
 F 3 "~" H 7750 2600 50  0001 C CNN
+F 4 "RTC_SUPPORTED_BACKEDUP" H 7750 2600 50  0001 C CNN "Feature"
+F 5 "0.0036" H 7750 2600 50  0001 C CNN "Price"
+F 6 "yes" H 7750 2600 50  0001 C CNN "is stock"
 	1    7750 2600
 	0    1    1    0
@@
 F 2 "Diode_SMD:D_SOD-123" H 8950 2300 50  0001 C CNN
 F 3 "~" H 8950 2300 50  0001 C CNN
+F 4 "RTC_SUPPORTED_BACKEDUP" H 8950 2300 50  0001 C CNN "Feature"
+F 5 "0.0152" H 8950 2300 50  0001 C CNN "Price"
+F 6 "no" H 8950 2300 50  0001 C CNN "is stock"
 	1    8950 2300
 	0    -1   -1   0
@@
 F 2 "Capacitor_SMD:C_0805_2012Metric_Pad1.18x1.45mm_HandSolder" H 4488 3200 50  0001 C CNN
 F 3 "~" H 4450 3350 50  0001 C CNN
+F 4 "RTC_SUPPORTED" H 4450 3350 50  0001 C CNN "Feature"
+F 5 "0.0057" H 4450 3350 50  0001 C CNN "Price"
+F 6 "yes" H 4450 3350 50  0001 C CNN "is stock"
 	1    4450 3350
 	1    0    0    -1
