File: LedBarController/Power.sch (KiCad schematic (older format))
At the start: 21 parts, among them J301 Barrel_Jack_Switch, Q301 FQP47P06, U301 AMS1117-5.0

Commit message: Restarted PCB
Parts:
- removed C306: C, Capacitor_SMD:C_0805_2012Metric_Pad1.18x1.45mm_HandSolder, symbol Device:C
- removed D302: D, Diode_SMD:D_1206_3216Metric_Pad1.42x1.75mm_HandSolder, symbol Device:D
- removed R304, R305: R, Resistor_SMD:R_0805_2012Metric_Pad1.20x1.40mm_HandSolder, symbol Device:R
- renumbered C301 to C1201, C302 to C1202, C303 to C1203, C304 to C1204, C305 to C1205, D301 to D1201, D303 to D1202, F301 to F1201, J301 to J1201, Q301 to Q1201, R301 to R1201, R302 to R1202, R303 to R1203, TP301 to TP1201, TP302 to TP1202, TP303 to TP1203, U301 to U1201

Commit message: Routed Power circuit
Parts:
- C1205: value 100uF/10V -> 47uF/50V; footprint Capacitor_THT:CP_Radial_D4.0mm_P2.00mm -> Capacitor_SMD:C_1206_3216Metric_Pad1.33x1.80mm_HandSolder
- D1202: footprint LED_SMD:LED_1206_3216Metric_Pad1.42x1.75mm_HandSolder -> LED_THT:LED_D3.0mm
Changed lines of the file:
@@
 P 7500 4000
 F 0 "C1205" H 7618 4046 50  0000 L CNN
-F 1 "100uF/10V" H 7618 3955 50  0000 L CNN
-F 2 "Capacitor_THT:CP_Radial_D4.0mm_P2.00mm" H 7538 3850 50  0001 C CNN
+F 1 "47uF/50V" H 7618 3955 50  0000 L CNN
+F 2 "Capacitor_SMD:C_1206_3216Metric_Pad1.33x1.80mm_HandSolder" H 7538 3850 50  0001 C CNN
 F 3 "~" H 7500 4000 50  0001 C CNN
 	1    7500 4000
@@
 F 0 "D1202" V 8039 4132 50  0000 R CNN
 F 1 "LED" V 7948 4132 50  0000 R CNN
-F 2 "LED_SMD:LED_1206_3216Metric_Pad1.42x1.75mm_HandSolder" H 8000 4250 50  0001 C CNN
+F 2 "LED_THT:LED_D3.0mm" H 8000 4250 50  0001 C CNN
 F 3 "~" H 8000 4250 50  0001 C CNN
 	1    8000 4250

Commit message: Added INA219 current/voltage sensor
Parts:
- added C1206: 1uF/ceramic, Capacitor_SMD:C_0805_2012Metric_Pad1.18x1.45mm_HandSolder, symbol Device:C
- added C1207: 0.1uF, Capacitor_SMD:C_0805_2012Metric_Pad1.18x1.45mm_HandSolder, symbol Device:C
- added R1204, R1205: 10R, Resistor_SMD:R_0805_2012Metric_Pad1.20x1.40mm_HandSolder, symbol Device:R
- added R1206: R001/2W, Resistor_SMD:R_2512_6332Metric_Pad1.40x3.35mm_HandSolder, symbol Device:R
- added U1202: INA219AxD, Package_SO:SOIC-8_3.9x4.9mm_P1.27mm, symbol Analog_ADC:INA219AxD
- C1204: footprint Capacitor_THT:CP_Radial_D6.3mm_P2.50mm -> Capacitor_SMD:C_1206_3216Metric_Pad1.33x1.80mm_HandSolder
Connections:
- net +5V: now also U1202.5 (VS)
- net GND: now also C1207.2, U1202.1 (A1), U1202.2 (A0), U1202.6 (GND)
- net VDD: now also C1206.1, C1207.1, R1205.1, R1206.1; no longer C1201.1, D1201.1 (K), Q1201.3 (S)
- new net: C1201.1, C1206.2, D1201.1 (K), Q1201.3 (S), R1204.1, R1206.2
- new net: R1205.2, U1202.7 (IN-)
- new net: R1204.2, U1202.8 (IN+)
- new net scl: U1202.4 (SCL)
- new net sda: U1202.3 (SDA)
Other:
- moved on the sheet: C1202, C1203, C1204, C1205, D1202, R1201, R1203, TP1201, TP1202, TP1203, U1201

Commit message: Work in progress
Parts:
- added C1208: 0.1uF, Capacitor_SMD:C_0805_2012Metric_Pad1.18x1.45mm_HandSolder, symbol Device:C
- C1201: Feature (none) -> POWER; Price (none) -> 0.0057; is stock (none) -> yes
- C1202, C1203: value C -> 0.1uF; Feature (none) -> POWER; Price (none) -> 0.0057; is stock (none) -> yes
- C1204: value 100uF/35V -> 10uF/35V; footprint Capacitor_SMD:C_1206_3216Metric_Pad1.33x1.80mm_HandSolder -> Capacitor_Tantalum_SMD:CP_EIA-6032-28_Kemet-C_Pad2.25x2.35mm_HandSolder; Feature (none) -> POWER; Price (none) -> 0.139; is stock (none) -> no
- C1205: value 47uF/50V -> 10uF/10V; footprint Capacitor_SMD:C_1206_3216Metric_Pad1.33x1.80mm_HandSolder -> Capacitor_Tantalum_SMD:CP_EIA-3216-18_Kemet-A_Pad1.58x1.35mm_HandSolder; Feature (none) -> POWER; Price (none) -> 0.19; is stock (none) -> no
- C1206: value 1uF/ceramic -> 1uF; Feature (none) -> INA219_SUPPORTED_FILTERED; Price (none) -> 0.015; is stock (none) -> no
- C1207: Feature (none) -> INA219_SUPPORTED_FILTERED; Price (none) -> 0.0057; is stock (none) -> yes
- D1201: Feature (none) -> REVERSEPOLARITY_SUPPORTED; Price (none) -> 0.0073; is stock (none) -> yes
- D1202: value LED -> Blue; Feature (none) -> POWER; Price (none) -> 0.00675; is stock (none) -> yes
- F1201: value Fuse -> 5A; Feature (none) -> POWER; Price (none) -> 0.1474; is stock (none) -> yes
- J1201: Feature (none) -> POWER; Price (none) -> 0.0472; is stock (none) -> yes
- Q1201: Feature (none) -> REVERSEPOLARITY_SUPPORTED; Price (none) -> 0.386; is stock (none) -> no
- R1201: Feature (none) -> POWER; Price (none) -> 0.056; is stock (none) -> no
- R1202: Feature (none) -> REVERSEPOLARITY_SUPPORTED; Price (none) -> 0.0036; is stock (none) -> yes
- R1203: value 330 -> 470R; Feature (none) -> POWER; Price (none) -> 0.0036; is stock (none) -> yes
- R1204, R1205: Feature (none) -> INA219_SUPPORTED; Price (none) -> 0.0036; is stock (none) -> yes
- R1206: Feature (none) -> INA219; Price (none) -> 0.0794; is stock (none) -> no
- TP1201, TP1202, TP1203: Feature (none) -> POWER; Price (none) -> 0; is stock (none) -> n.a.
- U1201: Feature (none) -> POWER; Price (none) -> 0.0254; is stock (none) -> yes
- U1202: Feature (none) -> INA219; Price (none) -> 1.506; is stock (none) -> no
Connections:
- net +5V: now also C1208.1
- net GND: now also C1208.2
Changed lines of the file:
@@
 F 2 "Connector_BarrelJack:BarrelJack_CUI_PJ-102AH_Horizontal" H 2750 3710 50  0001 C CNN
 F 3 "~" H 2750 3710 50  0001 C CNN
+F 4 "POWER" H 2700 3750 50  0001 C CNN "Feature"
+F 5 "0.0472" H 2700 3750 50  0001 C CNN "Price"
+F 6 "yes" H 2700 3750 50  0001 C CNN "is stock"
 	1    2700 3750
 	1    0    0    -1
@@
 P 3250 3000
 F 0 "F1201" V 3053 3000 50  0000 C CNN
-F 1 "Fuse" V 3144 3000 50  0000 C CNN
+F 1 "5A" V 3144 3000 50  0000 C CNN
 F 2 "Fuse:Fuseholder_Cylinder-5x20mm_Stelvio-Kontek_PTF78_Horizontal_Open" V 3180 3000 50  0001 C CNN
 F 3 "~" H 3250 3000 50  0001 C CNN
+F 4 "POWER" H 3250 3000 50  0001 C CNN "Feature"
+F 5 "0.1474" H 3250 3000 50  0001 C CNN "Price"
+F 6 "yes" H 3250 3000 50  0001 C CNN "is stock"
 	1    3250 3000
 	0    1    1    0
@@
 P 7500 3750
 F 0 "C1202" H 7615 3796 50  0000 L CNN
-F 1 "C" H 7615 3705 50  0000 L CNN
+F 1 "0.1uF" H 7615 3705 50  0000 L CNN
 F 2 "Capacitor_SMD:C_0805_2012Metric_Pad1.18x1.45mm_HandSolder" H 7538 3600 50  0001 C CNN
 F 3 "~" H 7500 3750 50  0001 C CNN
+F 4 "POWER" H 7500 3750 50  0001 C CNN "Feature"
+F 5 "0.0057" H 7500 3750 50  0001 C CNN "Price"
+F 6 "yes" H 7500 3750 50  0001 C CNN "is stock"
 	1    7500 3750
 	1    0    0    -1
@@
 P 8500 3750
 F 0 "C1203" H 8615 3796 50  0000 L CNN
-F 1 "C" H 8615 3705 50  0000 L CNN
+F 1 "0.1uF" H 8615 3705 50  0000 L CNN
 F 2 "Capacitor_SMD:C_0805_2012Metric_Pad1.18x1.45mm_HandSolder" H 8538 3600 50  0001 C CNN
 F 3 "~" H 8500 3750 50  0001 C CNN
+F 4 "POWER" H 8500 3750 50  0001 C CNN "Feature"
+F 5 "0.0057" H 8500 3750 50  0001 C CNN "Price"
+F 6 "yes" H 8500 3750 50  0001 C CNN "is stock"
 	1    8500 3750
 	1    0    0    -1
@@
 P 7000 4000
 F 0 "C1204" H 7118 4046 50  0000 L CNN
-F 1 "100uF/35V" H 7118 3955 50  0000 L CNN
-F 2 "Capacitor_SMD:C_1206_3216Metric_Pad1.33x1.80mm_HandSolder" H 7038 3850 50  0001 C CNN
+F 1 "10uF/35V" H 7118 3955 50  0000 L CNN
+F 2 "Capacitor_Tantalum_SMD:CP_EIA-6032-28_Kemet-C_Pad2.25x2.35mm_HandSolder" H 7038 3850 50  0001 C CNN
 F 3 "~" H 7000 4000 50  0001 C CNN
+F 4 "POWER" H 7000 4000 50  0001 C CNN "Feature"
+F 5 "0.139" H 7000 4000 50  0001 C CNN "Price"
+F 6 "no" H 7000 4000 50  0001 C CNN "is stock"
 	1    7000 4000
 	1    0    0    -1
@@
 P 9000 4000
 F 0 "C1205" H 9118 4046 50  0000 L CNN
-F 1 "47uF/50V" H 9118 3955 50  0000 L CNN
-F 2 "Capacitor_SMD:C_1206_3216Metric_Pad1.33x1.80mm_HandSolder" H 9038 3850 50  0001 C CNN
+F 1 "10uF/10V" H 9118 3955 50  0000 L CNN
+F 2 "Capacitor_Tantalum_SMD:CP_EIA-3216-18_Kemet-A_Pad1.58x1.35mm_HandSolder" H 9038 3850 50  0001 C CNN
 F 3 "~" H 9000 4000 50  0001 C CNN
+F 4 "POWER" H 9000 4000 50  0001 C CNN "Feature"
+F 5 "0.19" H 9000 4000 50  0001 C CNN "Price"
+F 6 "no" H 9000 4000 50  0001 C CNN "is stock"
 	1    9000 4000
 	1    0    0    -1
@@
 F 2 "Resistor_SMD:R_1812_4532Metric_Pad1.30x3.40mm_HandSolder" V 6930 3250 50  0001 C CNN
 F 3 "~" H 7000 3250 50  0001 C CNN
+F 4 "POWER" H 7000 3250 50  0001 C CNN "Feature"
+F 5 "0.056" H 7000 3250 50  0001 C CNN "Price"
+F 6 "no" H 7000 3250 50  0001 C CNN "is stock"
 	1    7000 3250
 	-1   0    0    1
@@
 F 2 "Package_TO_SOT_SMD:SOT-223-3_TabPin2" H 8000 3700 50  0001 C CNN
 F 3 "http://www.advanced-monolithic.com/pdf/ds1117.pdf" H 8100 3250 50  0001 C CNN
+F 4 "POWER" H 8000 3500 50  0001 C CNN "Feature"
+F 5 "0.0254" H 8000 3500 50  0001 C CNN "Price"
+F 6 "yes" H 8000 3500 50  0001 C CNN "is stock"
 	1    8000 3500
 	1    0    0    -1
@@
 F 2 "Capacitor_SMD:C_0805_2012Metric_Pad1.18x1.45mm_HandSolder" H 5038 3600 50  0001 C CNN
 F 3 "~" H 5000 3750 50  0001 C CNN
+F 4 "POWER" H 5000 3750 50  0001 C CNN "Feature"
+F 5 "0.0057" H 5000 3750 50  0001 C CNN "Price"
+F 6 "yes" H 5000 3750 50  0001 C CNN "is stock"
 	1    5000 3750
 	1    0    0    -1
@@
 P 9500 3750
 F 0 "R1203" H 9570 3796 50  0000 L CNN
-F 1 "330" H 9570 3705 50  0000 L CNN
+F 1 "470R" H 9570 3705 50  0000 L CNN
 F 2 "Resistor_SMD:R_0805_2012Metric_Pad1.20x1.40mm_HandSolder" V 9430 3750 50  0001 C CNN
 F 3 "~" H 9500 3750 50  0001 C CNN
+F 4 "POWER" H 9500 3750 50  0001 C CNN "Feature"
+F 5 "0.0036" H 9500 3750 50  0001 C CNN "Price"
+F 6 "yes" H 9500 3750 50  0001 C CNN "is stock"
 	1    9500 3750
 	1    0    0    -1
@@
 P 9500 4250
 F 0 "D1202" V 9539 4132 50  0000 R CNN
-F 1 "LED" V 9448 4132 50  0000 R CNN
+F 1 "Blue" V 9448 4132 50  0000 R CNN
 F 2 "LED_THT:LED_D3.0mm" H 9500 4250 50  0001 C CNN
 F 3 "~" H 9500 4250 50  0001 C CNN
+F 4 "POWER" H 9500 4250 50  0001 C CNN "Feature"
+F 5 "0.00675" H 9500 4250 50  0001 C CNN "Price"
+F 6 "yes" H 9500 4250 50  0001 C CNN "is stock"
 	1    9500 4250
 	0    -1   -1   0
@@
 F 2 "TestPoint:TestPoint_Pad_D1.0mm" H 9700 3500 50  0001 C CNN
 F 3 "~" H 9700 3500 50  0001 C CNN
+F 4 "POWER" H 9500 3500 50  0001 C CNN "Feature"
+F 5 "0" H 9500 3500 50  0001 C CNN "Price"
+F 6 "n.a." H 9500 3500 50  0001 C CNN "is stock"
 	1    9500 3500
 	1    0    0    -1
@@
 F 2 "TestPoint:TestPoint_Pad_D1.0mm" H 7500 2950 50  0001 C CNN
 F 3 "~" H 7500 2950 50  0001 C CNN
+F 4 "POWER" H 7300 2950 50  0001 C CNN "Feature"
+F 5 "0" H 7300 2950 50  0001 C CNN "Price"
+F 6 "n.a." H 7300 2950 50  0001 C CNN "is stock"
 	1    7300 2950
 	1    0    0    -1
@@
 F 2 "TestPoint:TestPoint_Pad_D1.0mm" H 9200 4600 50  0001 C CNN
 F 3 "~" H 9200 4600 50  0001 C CNN
+F 4 "POWER" H 9000 4600 50  0001 C CNN "Feature"
+F 5 "0" H 9000 4600 50  0001 C CNN "Price"
+F 6 "n.a." H 9000 4600 50  0001 C CNN "is stock"
 	1    9000 4600
 	-1   0    0    1
@@
 F 2 "Package_TO_SOT_THT:TO-220-3_Vertical" H 4200 3200 50  0001 C CNN
 F 3 "~" H 4000 3100 50  0001 C CNN
+F 4 "REVERSEPOLARITY_SUPPORTED" H 4000 3100 50  0001 C CNN "Feature"
+F 5 "0.386" H 4000 3100 50  0001 C CNN "Price"
+F 6 "no" H 4000 3100 50  0001 C CNN "is stock"
 	1    4000 3100
 	0    -1   -1   0
@@
 F 2 "Diode_SMD:D_1206_3216Metric_Pad1.42x1.75mm_HandSolder" H 4500 3250 50  0001 C CNN
 F 3 "~" H 4500 3250 50  0001 C CNN
+F 4 "REVERSEPOLARITY_SUPPORTED" H 4500 3250 50  0001 C CNN "Feature"
+F 5 "0.0073" H 4500 3250 50  0001 C CNN "Price"
+F 6 "yes" H 4500 3250 50  0001 C CNN "is stock"
 	1    4500 3250
 	0    1    1    0
@@
 F 2 "Resistor_SMD:R_0805_2012Metric_Pad1.20x1.40mm_HandSolder" V 3930 3750 50  0001 C CNN
 F 3 "~" H 4000 3750 50  0001 C CNN
+F 4 "REVERSEPOLARITY_SUPPORTED" H 4000 3750 50  0001 C CNN "Feature"
+F 5 "0.0036" H 4000 3750 50  0001 C CNN "Price"
+F 6 "yes" H 4000 3750 50  0001 C CNN "is stock"
 	1    4000 3750
 	1    0    0    -1
@@
 F 2 "Resistor_SMD:R_2512_6332Metric_Pad1.40x3.35mm_HandSolder" V 5930 3000 50  0001 C CNN
 F 3 "~" H 6000 3000 50  0001 C CNN
+F 4 "INA219" H 6000 3000 50  0001 C CNN "Feature"
+F 5 "0.0794" H 6000 3000 50  0001 C CNN "Price"
+F 6 "no" H 6000 3000 50  0001 C CNN "is stock"
 	1    6000 3000
 	0    1    1    0
@@
 F 2 "Package_SO:SOIC-8_3.9x4.9mm_P1.27mm" H 8100 1350 50  0001 C CNN
 F 3 "http://www.ti.com/lit/ds/symlink/ina219.pdf" H 7650 1600 50  0001 C CNN
+F 4 "INA219" H 7300 1700 50  0001 C CNN "Feature"
+F 5 "1.506" H 7300 1700 50  0001 C CNN "Price"
+F 6 "no" H 7300 1700 50  0001 C CNN "is stock"
 	1    7300 1700
 	1    0    0    -1
@@
 $EndComp
 Wire Wire Line
-	7300 1100 7300 1300
+	7300 1100 7300 1200
 Wire Wire Line
 	7300 2100 7300 2200
@@
 P 6000 2500
 F 0 "C1206" V 5748 2500 50  0000 C CNN
-F 1 "1uF/ceramic" V 5839 2500 50  0000 C CNN
+F 1 "1uF" V 5839 2500 50  0000 C CNN
 F 2 "Capacitor_SMD:C_0805_2012Metric_Pad1.18x1.45mm_HandSolder" H 6038 2350 50  0001 C CNN
 F 3 "~" H 6000 2500 50  0001 C CNN
+F 4 "INA219_SUPPORTED_FILTERED" H 6000 2500 50  0001 C CNN "Feature"
+F 5 "0.015" H 6000 2500 50  0001 C CNN "Price"
+F 6 "no" H 6000 2500 50  0001 C CNN "is stock"
 	1    6000 2500
 	0    1    1    0
@@
 F 2 "Resistor_SMD:R_0805_2012Metric_Pad1.20x1.40mm_HandSolder" V 6080 2000 50  0001 C CNN
 F 3 "~" H 6150 2000 50  0001 C CNN
+F 4 "INA219_SUPPORTED" H 6150 2000 50  0001 C CNN "Feature"
+F 5 "0.0036" H 6150 2000 50  0001 C CNN "Price"
+F 6 "yes" H 6150 2000 50  0001 C CNN "is stock"
 	1    6150 2000
 	-1   0    0    1
@@
 F 2 "Resistor_SMD:R_0805_2012Metric_Pad1.20x1.40mm_HandSolder" V 5780 2000 50  0001 C CNN
 F 3 "~" H 5850 2000 50  0001 C CNN
+F 4 "INA219_SUPPORTED" H 5850 2000 50  0001 C CNN "Feature"
+F 5 "0.0036" H 5850 2000 50  0001 C CNN "Price"
+F 6 "yes" H 5850 2000 50  0001 C CNN "is stock"
 	1    5850 2000
 	-1   0    0    1
@@
 F 2 "Capacitor_SMD:C_0805_2012Metric_Pad1.18x1.45mm_HandSolder" H 6538 3600 50  0001 C CNN
 F 3 "~" H 6500 3750 50  0001 C CNN
+F 4 "INA219_SUPPORTED_FILTERED" H 6500 3750 50  0001 C CNN "Feature"
+F 5 "0.0057" H 6500 3750 50  0001 C CNN "Price"
+F 6 "yes" H 6500 3750 50  0001 C CNN "is stock"
 	1    6500 3750
 	1    0    0    -1
@@
 Wire Wire Line
 	6500 3000 7000 3000
+$Comp
+L Device:C C1208
+U 1 1 5F9AC8D5
+P 8500 1650
+F 0 "C1208" H 8615 1696 50  0000 L CNN
+F 1 "0.1uF" H 8615 1605 50  0000 L CNN
+F 2 "Capacitor_SMD:C_0805_2012Metric_Pad1.18x1.45mm_HandSolder" H 8538 1500 50  0001 C CNN
+F 3 "~" H 8500 1650 50  0001 C CNN
+F 4 "0.0057" H 8500 1650 50  0001 C CNN "Price"
+F 5 "yes" H 8500 1650 50  0001 C CNN "is stock"
+	1    8500 1650
+	1    0    0    -1
+$EndComp
+Wire Wire Line
+	7300 1200 8500 1200
+Wire Wire Line
+	8500 1200 8500 1500
+Connection ~ 7300 1200
+Wire Wire Line
+	7300 1200 7300 1300
+Wire Wire Line
+	8500 2100 7700 2100
+Connection ~ 7700 2100
+Wire Wire Line
+	8500 1800 8500 2100
 $EndSCHEMATC

Commit message: Reduced circuit by remove extra features. Routed whole board. Needs refinement
Parts:
- D1202: footprint LED_THT:LED_D3.0mm -> LED_SMD:LED_0805_2012Metric_Pad1.15x1.40mm_HandSolder
Changed lines of the file:
@@
 $Descr A4 11693 8268
 encoding utf-8
-Sheet 12 14
+Sheet 11 13
 Title ""
 Date ""
@@
 F 0 "D1202" V 9539 4132 50  0000 R CNN
 F 1 "Blue" V 9448 4132 50  0000 R CNN
-F 2 "LED_THT:LED_D3.0mm" H 9500 4250 50  0001 C CNN
+F 2 "LED_SMD:LED_0805_2012Metric_Pad1.15x1.40mm_HandSolder" H 9500 4250 50  0001 C CNN
 F 3 "~" H 9500 4250 50  0001 C CNN
 F 4 "POWER" H 9500 4250 50  0001 C CNN "Feature"

Commit message: Added surge protection
Parts:
- added D1203: SMBJ30CA CK, Diode_SMD:D_SMB_Handsoldering, symbol Device:D_TVS
Connections:
- net GND: now also D1203.2 (A2)
- net at F1201.1, Q1201.2 (D): now also D1203.1 (A1)
Other:
- moved on the sheet: C1201, D1201, Q1201, R1202
Changed lines of the file:
@@
 L Device:C C1201
 U 1 1 5F7F8388
-P 5000 3750
-F 0 "C1201" H 5115 3796 50  0000 L CNN
-F 1 "0.1uF" H 5115 3705 50  0000 L CNN
-F 2 "Capacitor_SMD:C_0805_2012Metric_Pad1.18x1.45mm_HandSolder" H 5038 3600 50  0001 C CNN
-F 3 "~" H 5000 3750 50  0001 C CNN
-F 4 "POWER" H 5000 3750 50  0001 C CNN "Feature"
-F 5 "0.0057" H 5000 3750 50  0001 C CNN "Price"
-F 6 "yes" H 5000 3750 50  0001 C CNN "is stock"
-	1    5000 3750
+P 5500 3750
+F 0 "C1201" H 5615 3796 50  0000 L CNN
+F 1 "0.1uF" H 5615 3705 50  0000 L CNN
+F 2 "Capacitor_SMD:C_0805_2012Metric_Pad1.18x1.45mm_HandSolder" H 5538 3600 50  0001 C CNN
+F 3 "~" H 5500 3750 50  0001 C CNN
+F 4 "POWER" H 5500 3750 50  0001 C CNN "Feature"
+F 5 "0.0057" H 5500 3750 50  0001 C CNN "Price"
+F 6 "yes" H 5500 3750 50  0001 C CNN "is stock"
+	1    5500 3750
 	1    0    0    -1
 $EndComp
@@
 Wire Wire Line
 	7000 3000 7000 3100
-Wire Wire Line
-	5000 3000 5000 3600
-Connection ~ 5000 3000
-Wire Wire Line
-	5000 3900 5000 4500
-Connection ~ 5000 4500
 $Comp
 L power:PWR_FLAG #FLG01203
 U 1 1 5F820B2B
-P 5000 4500
-F 0 "#FLG01203" H 5000 4575 50  0001 C CNN
-F 1 "PWR_FLAG" H 5000 4673 50  0001 C CNN
-F 2 "" H 5000 4500 50  0001 C CNN
-F 3 "~" H 5000 4500 50  0001 C CNN
-	1    5000 4500
+P 5500 4500
+F 0 "#FLG01203" H 5500 4575 50  0001 C CNN
+F 1 "PWR_FLAG" H 5500 4673 50  0001 C CNN
+F 2 "" H 5500 4500 50  0001 C CNN
+F 3 "~" H 5500 4500 50  0001 C CNN
+	1    5500 4500
 	-1   0    0    1
 $EndComp
@@
 L Device:Q_PMOS_GDS Q1201
 U 1 1 5FA735DA
-P 4000 3100
-F 0 "Q1201" V 4342 3100 50  0000 C CNN
-F 1 "FQP47P06" V 4251 3100 50  0000 C CNN
-F 2 "Package_TO_SOT_THT:TO-220-3_Vertical" H 4200 3200 50  0001 C CNN
-F 3 "~" H 4000 3100 50  0001 C CNN
-F 4 "REVERSEPOLARITY_SUPPORTED" H 4000 3100 50  0001 C CNN "Feature"
-F 5 "0.386" H 4000 3100 50  0001 C CNN "Price"
-F 6 "no" H 4000 3100 50  0001 C CNN "is stock"
-	1    4000 3100
+P 4500 3100
+F 0 "Q1201" V 4842 3100 50  0000 C CNN
+F 1 "FQP47P06" V 4751 3100 50  0000 C CNN
+F 2 "Package_TO_SOT_THT:TO-220-3_Vertical" H 4700 3200 50  0001 C CNN
+F 3 "~" H 4500 3100 50  0001 C CNN
+F 4 "REVERSEPOLARITY_SUPPORTED" H 4500 3100 50  0001 C CNN "Feature"
+F 5 "0.386" H 4500 3100 50  0001 C CNN "Price"
+F 6 "no" H 4500 3100 50  0001 C CNN "is stock"
+	1    4500 3100
 	0    -1   -1   0
 $EndComp
 Wire Wire Line
-	3400 3000 3800 3000
-Wire Wire Line
-	3000 4500 4000 4500
+	3500 4500 4500 4500
 $Comp
 L Device:D_Zener D1201
 U 1 1 5FA7B9A0
-P 4500 3250
-F 0 "D1201" V 4450 3000 50  0000 L CNN
-F 1 "10V" V 4550 3050 50  0000 L CNN
-F 2 "Diode_SMD:D_1206_3216Metric_Pad1.42x1.75mm_HandSolder" H 4500 3250 50  0001 C CNN
-F 3 "~" H 4500 3250 50  0001 C CNN
-F 4 "REVERSEPOLARITY_SUPPORTED" H 4500 3250 50  0001 C CNN "Feature"
-F 5 "0.0073" H 4500 3250 50  0001 C CNN "Price"
-F 6 "yes" H 4500 3250 50  0001 C CNN "is stock"
-	1    4500 3250
+P 5000 3250
+F 0 "D1201" V 4950 3000 50  0000 L CNN
+F 1 "10V" V 5050 3050 50  0000 L CNN
+F 2 "Diode_SMD:D_1206_3216Metric_Pad1.42x1.75mm_HandSolder" H 5000 3250 50  0001 C CNN
+F 3 "~" H 5000 3250 50  0001 C CNN
+F 4 "REVERSEPOLARITY_SUPPORTED" H 5000 3250 50  0001 C CNN "Feature"
+F 5 "0.0073" H 5000 3250 50  0001 C CNN "Price"
+F 6 "yes" H 5000 3250 50  0001 C CNN "is stock"
+	1    5000 3250
 	0    1    1    0
 $EndComp
@@
 L Device:R R1202
 U 1 1 5FA7CE6E
-P 4000 3750
-F 0 "R1202" H 4070 3796 50  0000 L CNN
-F 1 "100k" H 4070 3705 50  0000 L CNN
-F 2 "Resistor_SMD:R_0805_2012Metric_Pad1.20x1.40mm_HandSolder" V 3930 3750 50  0001 C CNN
-F 3 "~" H 4000 3750 50  0001 C CNN
-F 4 "REVERSEPOLARITY_SUPPORTED" H 4000 3750 50  0001 C CNN "Feature"
-F 5 "0.0036" H 4000 3750 50  0001 C CNN "Price"
-F 6 "yes" H 4000 3750 50  0001 C CNN "is stock"
-	1    4000 3750
-	1    0    0    -1
-$EndComp
-Wire Wire Line
-	4200 3000 4500 3000
-Wire Wire Line
-	4500 3100 4500 3000
-Connection ~ 4500 3000
-Wire Wire Line
-	4500 3000 5000 3000
-Wire Wire Line
-	4500 3400 4500 3500
-Wire Wire Line
-	4500 3500 4000 3500
-Wire Wire Line
-	4000 3500 4000 3300
-Wire Wire Line
-	4000 3500 4000 3600
-Connection ~ 4000 3500
-Wire Wire Line
-	4000 3900 4000 4500
-Connection ~ 4000 4500
-Wire Wire Line
-	4000 4500 5000 4500
+P 4500 3750
+F 0 "R1202" H 4570 3796 50  0000 L CNN
+F 1 "100k" H 4570 3705 50  0000 L CNN
+F 2 "Resistor_SMD:R_0805_2012Metric_Pad1.20x1.40mm_HandSolder" V 4430 3750 50  0001 C CNN
+F 3 "~" H 4500 3750 50  0001 C CNN
+F 4 "REVERSEPOLARITY_SUPPORTED" H 4500 3750 50  0001 C CNN "Feature"
+F 5 "0.0036" H 4500 3750 50  0001 C CNN "Price"
+F 6 "yes" H 4500 3750 50  0001 C CNN "is stock"
+	1    4500 3750
+	1    0    0    -1
+$EndComp
+Wire Wire Line
+	4700 3000 5000 3000
+Wire Wire Line
+	5000 3100 5000 3000
+Wire Wire Line
+	5000 3400 5000 3500
+Wire Wire Line
+	5000 3500 4500 3500
+Wire Wire Line
+	4500 3500 4500 3300
+Wire Wire Line
+	4500 3500 4500 3600
+Connection ~ 4500 3500
+Wire Wire Line
+	4500 3900 4500 4500
+Connection ~ 4500 4500
+Wire Wire Line
+	4500 4500 5500 4500
 Wire Notes Line
-	3750 2500 4750 2500
+	4250 2500 5250 2500
 Wire Notes Line
-	4750 2500 4750 4000
+	5250 2500 5250 4000
 Wire Notes Line
-	4750 4000 3750 4000
+	5250 4000 4250 4000
 Wire Notes Line
-	3750 4000 3750 2500
-Text Notes 3750 2500 0    50   ~ 0
+	4250 4000 4250 2500
+Text Notes 4250 2500 0    50   ~ 0
 Reverse voltage protection
 Wire Wire Line
@@
 Wire Wire Line
 	5850 1600 6900 1600
-Wire Wire Line
-	5000 3000 5850 3000
 Connection ~ 5850 3000
 Wire Wire Line
@@
 Text HLabel 8000 1600 2    50   Input ~ 0
 scl
-Wire Wire Line
-	5000 4500 6500 4500
 $Comp
 L Device:C C1207
@@
 Wire Wire Line
 	8500 1800 8500 2100
+$Comp
+L Device:D_TVS D1203
+U 1 1 5FC9A3E5
+P 3500 3750
+F 0 "D1203" V 3454 3830 50  0000 L CNN
+F 1 "SMBJ30CA CK" V 3545 3830 50  0000 L CNN
+F 2 "Diode_SMD:D_SMB_Handsoldering" H 3500 3750 50  0001 C CNN
+F 3 "~" H 3500 3750 50  0001 C CNN
+	1    3500 3750
+	0    1    1    0
+$EndComp
+Wire Wire Line
+	5500 3600 5500 3000
+Wire Wire Line
+	5500 3000 5850 3000
+Wire Wire Line
+	5500 3900 5500 4500
+Wire Wire Line
+	5500 4500 6500 4500
+Connection ~ 5500 4500
+Wire Wire Line
+	5000 3000 5500 3000
+Connection ~ 5000 3000
+Connection ~ 5500 3000
+Wire Wire Line
+	3400 3000 3500 3000
+Wire Wire Line
+	3000 4500 3500 4500
+Wire Wire Line
+	3500 4500 3500 3900
+Connection ~ 3500 4500
+Wire Wire Line
+	3500 3600 3500 3000
+Connection ~ 3500 3000
+Wire Wire Line
+	3500 3000 4300 3000
 $EndSCHEMATC
