File: LedBarController/Power.sch (KiCad schematic (older format))
At the start: 25 parts, among them J1201 Barrel_Jack_Switch, Q1201 FQP47P06, U1201 AMS1117-5.0, U1202 INA219AxD

Commit message: Route complete
Parts:
- D1203: Price (none) -> 0.1; is stock (none) -> no
Changed lines of the file:
@@
 F 2 "Diode_SMD:D_SMB_Handsoldering" H 3000 3750 50  0001 C CNN
 F 3 "~" H 3000 3750 50  0001 C CNN
+F 4 "0.1" H 3000 3750 50  0001 C CNN "Price"
+F 5 "no" H 3000 3750 50  0001 C CNN "is stock"
 	1    3000 3750
 	0    1    1    0

Commit message: moved board on schema to same sheet
Other:
- note added: "Over current and voltage protection"
- note added: "Voltage and current measurement"
- moved on the sheet: C1201, C1202, C1203, C1204, C1205, C1206, C1207, C1208, D1201, D1202, D1203, F1201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

Commit message: Reanotate
Parts:
- renumbered C1208 to C301, C1206 to C302, C1201 to C303, C1207 to C304, C1202 to C305, C1203 to C306, C1204 to C307, C1205 to C308, D1201 to D301, D1203 to D302, D1202 to D303, F1201 to F301, J1201 to J301, Q1201 to Q301, R1204 to R301, R1205 to R302, R1206 to R303, R1201 to R304, R1202 to R305, R1203 to R306, TP1201 to TP301, TP1202 to TP302, TP1203 to TP303, U1202 to U301, U1201 to U302
Changed lines of the file:
@@
 $EndDescr
 $Comp
-L power:VDD #PWR0101
+L power:VDD #PWR0303
 U 1 1 5F7CB8F6
 P 7000 3900
-F 0 "#PWR0101" H 7000 3750 50  0001 C CNN
+F 0 "#PWR0303" H 7000 3750 50  0001 C CNN
 F 1 "VDD" H 7015 4073 50  0000 C CNN
 F 2 "" H 7000 3900 50  0001 C CNN
@@
 $EndComp
 $Comp
-L Device:C C1202
+L Device:C C305
 U 1 1 5F7CE3F6
 P 7500 4750
-F 0 "C1202" H 7615 4796 50  0000 L CNN
+F 0 "C305" H 7615 4796 50  0000 L CNN
 F 1 "0.1uF" H 7615 4705 50  0000 L CNN
 F 2 "Capacitor_SMD:C_0805_2012Metric_Pad1.18x1.45mm_HandSolder" H 7538 4600 50  0001 C CNN
@@
 $EndComp
 $Comp
-L Device:C C1203
+L Device:C C306
 U 1 1 5F7CE9E9
 P 8500 4750
-F 0 "C1203" H 8615 4796 50  0000 L CNN
+F 0 "C306" H 8615 4796 50  0000 L CNN
 F 1 "0.1uF" H 8615 4705 50  0000 L CNN
 F 2 "Capacitor_SMD:C_0805_2012Metric_Pad1.18x1.45mm_HandSolder" H 8538 4600 50  0001 C CNN
@@
 $EndComp
 $Comp
-L Device:CP C1204
+L Device:CP C307
 U 1 1 5F7CF0E4
 P 7000 5000
-F 0 "C1204" H 7118 5046 50  0000 L CNN
+F 0 "C307" H 7118 5046 50  0000 L CNN
 F 1 "10uF/35V" H 7118 4955 50  0000 L CNN
 F 2 "Capacitor_Tantalum_SMD:CP_EIA-6032-28_Kemet-C_Pad2.25x2.35mm_HandSolder" H 7038 4850 50  0001 C CNN
@@
 $EndComp
 $Comp
-L Device:CP C1205
+L Device:CP C308
 U 1 1 5F7CF5E6
 P 9000 5000
-F 0 "C1205" H 9118 5046 50  0000 L CNN
+F 0 "C308" H 9118 5046 50  0000 L CNN
 F 1 "10uF/10V" H 9118 4955 50  0000 L CNN
 F 2 "Capacitor_Tantalum_SMD:CP_EIA-3216-18_Kemet-A_Pad1.58x1.35mm_HandSolder" H 9038 4850 50  0001 C CNN
@@
 	8500 5000 8500 4900
 $Comp
-L Device:R R1201
+L Device:R R304
 U 1 1 5F7D081A
 P 7000 4250
-F 0 "R1201" H 6930 4204 50  0000 R CNN
+F 0 "R304" H 6930 4204 50  0000 R CNN
 F 1 "100, 1W" H 6930 4295 50  0000 R CNN
 F 2 "Resistor_SMD:R_1812_4532Metric_Pad1.30x3.40mm_HandSolder" V 6930 4250 50  0001 C CNN
@@
 $EndComp
 $Comp
-L Regulator_Linear:AMS1117-5.0 U1201
+L Regulator_Linear:AMS1117-5.0 U302
 U 1 1 5F7CD4A1
 P 8000 4500
-F 0 "U1201" H 8000 4742 50  0000 C CNN
+F 0 "U302" H 8000 4742 50  0000 C CNN
 F 1 "AMS1117-5.0" H 8000 4651 50  0000 C CNN
 F 2 "Package_TO_SOT_SMD:SOT-223-3_TabPin2" H 8000 4700 50  0001 C CNN
@@
 Connection ~ 7000 4500
 $Comp
-L power:GND #PWR0102
+L power:GND #PWR0305
 U 1 1 5F7DD625
 P 8000 5500
-F 0 "#PWR0102" H 8000 5250 50  0001 C CNN
+F 0 "#PWR0305" H 8000 5250 50  0001 C CNN
 F 1 "GND" H 8005 5327 50  0000 C CNN
 F 2 "" H 8000 5500 50  0001 C CNN
@@
 $EndComp
 $Comp
-L power:+5V #PWR0103
+L power:+5V #PWR0304
 U 1 1 5F7DDB93
 P 9000 4500
-F 0 "#PWR0103" H 9000 4350 50  0001 C CNN
+F 0 "#PWR0304" H 9000 4350 50  0001 C CNN
 F 1 "+5V" H 9015 4673 50  0000 C CNN
 F 2 "" H 9000 4500 50  0001 C CNN
@@
 Connection ~ 7000 5500
 $Comp
-L Device:C C1201
+L Device:C C303
 U 1 1 5F7F8388
 P 5500 4750
-F 0 "C1201" H 5615 4796 50  0000 L CNN
+F 0 "C303" H 5615 4796 50  0000 L CNN
 F 1 "0.1uF" H 5615 4705 50  0000 L CNN
 F 2 "Capacitor_SMD:C_0805_2012Metric_Pad1.18x1.45mm_HandSolder" H 5538 4600 50  0001 C CNN
@@
 	7000 4000 7000 4100
 $Comp
-L power:PWR_FLAG #FLG0101
+L power:PWR_FLAG #FLG0303
 U 1 1 5F820B2B
 P 5500 5500
-F 0 "#FLG0101" H 5500 5575 50  0001 C CNN
+F 0 "#FLG0303" H 5500 5575 50  0001 C CNN
 F 1 "PWR_FLAG" H 5500 5673 50  0001 C CNN
 F 2 "" H 5500 5500 50  0001 C CNN
@@
 $EndComp
 $Comp
-L power:PWR_FLAG #FLG0102
+L power:PWR_FLAG #FLG0301
 U 1 1 5F81FA3E
 P 6500 4000
-F 0 "#FLG0102" H 6500 4075 50  0001 C CNN
+F 0 "#FLG0301" H 6500 4075 50  0001 C CNN
 F 1 "PWR_FLAG" H 6500 4173 50  0001 C CNN
 F 2 "" H 6500 4000 50  0001 C CNN
@@
 $EndComp
 $Comp
-L power:PWR_FLAG #FLG0103
+L power:PWR_FLAG #FLG0302
 U 1 1 5F826114
 P 7500 4500
-F 0 "#FLG0103" H 7500 4575 50  0001 C CNN
+F 0 "#FLG0302" H 7500 4575 50  0001 C CNN
 F 1 "PWR_FLAG" H 7500 4673 50  0001 C CNN
 F 2 "" H 7500 4500 50  0001 C CNN
@@
 $EndComp
 $Comp
-L Device:R R1203
+L Device:R R306
 U 1 1 5F959CE5
 P 9500 4750
-F 0 "R1203" H 9570 4796 50  0000 L CNN
+F 0 "R306" H 9570 4796 50  0000 L CNN
 F 1 "470R" H 9570 4705 50  0000 L CNN
 F 2 "Resistor_SMD:R_0805_2012Metric_Pad1.20x1.40mm_HandSolder" V 9430 4750 50  0001 C CNN
@@
 $EndComp
 $Comp
-L Device:LED D1202
+L Device:LED D303
 U 1 1 5F95A723
 P 9500 5250
-F 0 "D1202" V 9539 5132 50  0000 R CNN
+F 0 "D303" V 9539 5132 50  0000 R CNN
 F 1 "Blue" V 9448 5132 50  0000 R CNN
 F 2 "LED_SMD:LED_0805_2012Metric_Pad1.15x1.40mm_HandSolder" H 9500 5250 50  0001 C CNN
@@
 Connection ~ 9000 5500
 $Comp
-L Connector:TestPoint TP1202
+L Connector:TestPoint TP302
 U 1 1 5FA64F76
 P 9500 4500
-F 0 "TP1202" H 9558 4618 50  0000 L CNN
+F 0 "TP302" H 9558 4618 50  0000 L CNN
 F 1 "5V+" H 9558 4527 50  0000 L CNN
 F 2 "TestPoint:TestPoint_Pad_D1.0mm" H 9700 4500 50  0001 C CNN
@@
 Connection ~ 9500 4500
 $Comp
-L Connector:TestPoint TP1201
+L Connector:TestPoint TP301
 U 1 1 5FA6537E
 P 7300 3950
-F 0 "TP1201" H 7358 4068 50  0000 L CNN
+F 0 "TP301" H 7358 4068 50  0000 L CNN
 F 1 "VDD" H 7358 3977 50  0000 L CNN
 F 2 "TestPoint:TestPoint_Pad_D1.0mm" H 7500 3950 50  0001 C CNN
@@
 	7300 4000 7300 3950
 $Comp
-L Connector:TestPoint TP1203
+L Connector:TestPoint TP303
 U 1 1 5FA66AC1
 P 9000 5600
-F 0 "TP1203" H 8942 5626 50  0000 R CNN
+F 0 "TP303" H 8942 5626 50  0000 R CNN
 F 1 "GND" H 8942 5717 50  0000 R CNN
 F 2 "TestPoint:TestPoint_Pad_D1.0mm" H 9200 5600 50  0001 C CNN
@@
 $EndComp
 $Comp
-L Device:Q_PMOS_GDS Q1201
+L Device:Q_PMOS_GDS Q301
 U 1 1 5FA735DA
 P 4500 4100
-F 0 "Q1201" V 4842 4100 50  0000 C CNN
+F 0 "Q301" V 4842 4100 50  0000 C CNN
 F 1 "FQP47P06" V 4751 4100 50  0000 C CNN
 F 2 "Package_TO_SOT_THT:TO-220-3_Vertical" H 4700 4200 50  0001 C CNN
@@
 $EndComp
 $Comp
-L Device:D_Zener D1201
+L Device:D_Zener D301
 U 1 1 5FA7B9A0
 P 5000 4250
-F 0 "D1201" V 4950 4000 50  0000 L CNN
+F 0 "D301" V 4950 4000 50  0000 L CNN
 F 1 "10V" V 5050 4050 50  0000 L CNN
 F 2 "Diode_SMD:D_1206_3216Metric_Pad1.42x1.75mm_HandSolder" H 5000 4250 50  0001 C CNN
@@
 $EndComp
 $Comp
-L Device:R R1202
+L Device:R R305
 U 1 1 5FA7CE6E
 P 4500 4750
-F 0 "R1202" H 4570 4796 50  0000 L CNN
+F 0 "R305" H 4570 4796 50  0000 L CNN
 F 1 "100k" H 4570 4705 50  0000 L CNN
 F 2 "Resistor_SMD:R_0805_2012Metric_Pad1.20x1.40mm_HandSolder" V 4430 4750 50  0001 C CNN
@@
 	9000 5500 9000 5600
 $Comp
-L Device:R R1206
+L Device:R R303
 U 1 1 5F8905AC
 P 6000 4000
-F 0 "R1206" V 5900 4000 50  0000 C CNN
+F 0 "R303" V 5900 4000 50  0000 C CNN
 F 1 "R001/2W" V 6100 4000 50  0000 C CNN
 F 2 "Resistor_SMD:R_2512_6332Metric_Pad1.40x3.35mm_HandSolder" V 5930 4000 50  0001 C CNN
@@
 $EndComp
 $Comp
-L Analog_ADC:INA219AxD U1202
+L Analog_ADC:INA219AxD U301
 U 1 1 5F891052
 P 7300 2550
-F 0 "U1202" H 7100 2950 50  0000 C CNN
+F 0 "U301" H 7100 2950 50  0000 C CNN
 F 1 "INA219AxD" H 7600 2950 50  0000 C CNN
 F 2 "Package_SO:SOIC-8_3.9x4.9mm_P1.27mm" H 8100 2200 50  0001 C CNN
@@
 	6150 4000 6500 4000
 $Comp
-L power:GND #PWR0104
+L power:GND #PWR0302
 U 1 1 5F895D32
 P 7300 3050
-F 0 "#PWR0104" H 7300 2800 50  0001 C CNN
+F 0 "#PWR0302" H 7300 2800 50  0001 C CNN
 F 1 "GND" H 7305 2877 50  0000 C CNN
 F 2 "" H 7300 3050 50  0001 C CNN
@@
 $EndComp
 $Comp
-L power:+5V #PWR0105
+L power:+5V #PWR0301
 U 1 1 5F89611F
 P 7300 1950
-F 0 "#PWR0105" H 7300 1800 50  0001 C CNN
+F 0 "#PWR0301" H 7300 1800 50  0001 C CNN
 F 1 "+5V" H 7315 2123 50  0000 C CNN
 F 2 "" H 7300 1950 50  0001 C CNN
@@
 Connection ~ 7300 2950
 $Comp
-L Device:C C1206
+L Device:C C302
 U 1 1 5F89A068
 P 6000 3350
-F 0 "C1206" V 5748 3350 50  0000 C CNN
+F 0 "C302" V 5748 3350 50  0000 C CNN
 F 1 "1uF" V 5839 3350 50  0000 C CNN
 F 2 "Capacitor_SMD:C_0805_2012Metric_Pad1.18x1.45mm_HandSolder" H 6038 3200 50  0001 C CNN
@@
 $EndComp
 $Comp
-L Device:R R1205
+L Device:R R302
 U 1 1 5F89AEA9
 P 6150 2850
-F 0 "R1205" H 6080 2804 50  0000 R CNN
+F 0 "R302" H 6080 2804 50  0000 R CNN
 F 1 "10R" H 6080 2895 50  0000 R CNN
 F 2 "Resistor_SMD:R_0805_2012Metric_Pad1.20x1.40mm_HandSolder" V 6080 2850 50  0001 C CNN
@@
 $EndComp
 $Comp
-L Device:R R1204
+L Device:R R301
 U 1 1 5F89AA2D
 P 5850 2850
-F 0 "R1204" H 6150 2800 50  0000 R CNN
+F 0 "R301" H 6150 2800 50  0000 R CNN
 F 1 "10R" H 6100 2900 50  0000 R CNN
 F 2 "Resistor_SMD:R_0805_2012Metric_Pad1.20x1.40mm_HandSolder" V 5780 2850 50  0001 C CNN
@@
 scl
 $Comp
-L Device:C C1207
+L Device:C C304
 U 1 1 5F8B3D1B
 P 6500 4750
-F 0 "C1207" H 6615 4796 50  0000 L CNN
+F 0 "C304" H 6615 4796 50  0000 L CNN
 F 1 "0.1uF" H 6615 4705 50  0000 L CNN
 F 2 "Capacitor_SMD:C_0805_2012Metric_Pad1.18x1.45mm_HandSolder" H 6538 4600 50  0001 C CNN
@@
 	6500 4000 7000 4000
 $Comp
-L Device:C C1208
+L Device:C C301
 U 1 1 5F9AC8D5
 P 8500 2500
-F 0 "C1208" H 8615 2546 50  0000 L CNN
+F 0 "C301" H 8615 2546 50  0000 L CNN
 F 1 "0.1uF" H 8615 2455 50  0000 L CNN
 F 2 "Capacitor_SMD:C_0805_2012Metric_Pad1.18x1.45mm_HandSolder" H 8538 2350 50  0001 C CNN
@@
 	3400 4000 3500 4000
 $Comp
-L Device:D_TVS D1203
+L Device:D_TVS D302
 U 1 1 5FC9A3E5
 P 3500 4750
-F 0 "D1203" V 3450 4450 50  0000 L CNN
+F 0 "D302" V 3450 4450 50  0000 L CNN
 F 1 "SMBJ30CA CK /SMBJ15CA BM" V 3550 3550 50  0000 L CNN
 F 2 "Diode_SMD:D_SMB_Handsoldering" H 3500 4750 50  0001 C CNN
@@
 	2000 4650 2000 4000
 $Comp
-L Device:Fuse F1201
+L Device:Fuse F301
 U 1 1 5F7CC4D4
 P 3250 4000
-F 0 "F1201" V 3053 4000 50  0000 C CNN
+F 0 "F301" V 3053 4000 50  0000 C CNN
 F 1 "max. 5A F" V 3144 4000 50  0000 C CNN
 F 2 "Fuse:Fuseholder_Cylinder-5x20mm_Stelvio-Kontek_PTF78_Horizontal_Open" V 3180 4000 50  0001 C CNN
@@
 NoConn ~ 2000 4750
 $Comp
-L Connector:Barrel_Jack_Switch J1201
+L Connector:Barrel_Jack_Switch J301
 U 1 1 5F7C9FB6
 P 1700 4750
-F 0 "J1201" H 1757 5067 50  0000 C CNN
+F 0 "J301" H 1757 5067 50  0000 C CNN
 F 1 "Barrel_Jack_Switch" H 1757 4976 50  0000 C CNN
 F 2 "Connector_BarrelJack:BarrelJack_CUI_PJ-102AH_Horizontal" H 1750 4710 50  0001 C CNN

Commit message: Updated footprints and Fab layer
Parts:
- F301: footprint Fuse:Fuseholder_Cylinder-5x20mm_Stelvio-Kontek_PTF78_Horizontal_Open -> LedBarController:Fuseholder_Cylinder-5x20mm_BLX_A_Horizontal
Changed lines of the file:
@@
 F 0 "F301" V 3053 4000 50  0000 C CNN
 F 1 "max. 5A F" V 3144 4000 50  0000 C CNN
-F 2 "Fuse:Fuseholder_Cylinder-5x20mm_Stelvio-Kontek_PTF78_Horizontal_Open" V 3180 4000 50  0001 C CNN
+F 2 "LedBarController:Fuseholder_Cylinder-5x20mm_BLX_A_Horizontal" V 3180 4000 50  0001 C CNN
 F 3 "~" H 3250 4000 50  0001 C CNN
 F 4 "POWER" H 3250 4000 50  0001 C CNN "Feature"

Commit message: Removed Revere voltage protection circuit. I gets to hot! Replaced VTS diode from bidirectional to directional
Parts:
- removed D301: 10V, Diode_SMD:D_1206_3216Metric_Pad1.42x1.75mm_HandSolder, symbol Device:D_Zener
- removed Q301: FQP47P06, Package_TO_SOT_THT:TO-220-3_Vertical, symbol Device:Q_PMOS_GDS
- removed R305: 100k, Resistor_SMD:R_0805_2012Metric_Pad1.20x1.40mm_HandSolder, symbol Device:R
- D302: value SMBJ30CA CK /SMBJ15CA BM -> SMBJ15A; symbol Device:D_TVS -> Diode:Z2SMBxxx
Connections:
- net surge_bypass: now also C302.2, C303.1, R301.1, R303.2
Other:
- note removed: "Reverse voltage protection"
- moved on the sheet: D302, F301, J301
Changed lines of the file:
@@
 	-1   0    0    1
 $EndComp
-$Comp
-L Device:Q_PMOS_GDS Q301
-U 1 1 5FA735DA
-P 4500 4100
-F 0 "Q301" V 4842 4100 50  0000 C CNN
-F 1 "FQP47P06" V 4751 4100 50  0000 C CNN
-F 2 "Package_TO_SOT_THT:TO-220-3_Vertical" H 4700 4200 50  0001 C CNN
-F 3 "~" H 4500 4100 50  0001 C CNN
-F 4 "REVERSEPOLARITY_SUPPORTED" H 4500 4100 50  0001 C CNN "Feature"
-F 5 "0.386" H 4500 4100 50  0001 C CNN "Price"
-F 6 "no" H 4500 4100 50  0001 C CNN "is stock"
-	1    4500 4100
-	0    -1   -1   0
-$EndComp
-$Comp
-L Device:D_Zener D301
-U 1 1 5FA7B9A0
-P 5000 4250
-F 0 "D301" V 4950 4000 50  0000 L CNN
-F 1 "10V" V 5050 4050 50  0000 L CNN
-F 2 "Diode_SMD:D_1206_3216Metric_Pad1.42x1.75mm_HandSolder" H 5000 4250 50  0001 C CNN
-F 3 "~" H 5000 4250 50  0001 C CNN
-F 4 "REVERSEPOLARITY_SUPPORTED" H 5000 4250 50  0001 C CNN "Feature"
-F 5 "0.0073" H 5000 4250 50  0001 C CNN "Price"
-F 6 "yes" H 5000 4250 50  0001 C CNN "is stock"
-	1    5000 4250
-	0    1    1    0
-$EndComp
-$Comp
-L Device:R R305
-U 1 1 5FA7CE6E
-P 4500 4750
-F 0 "R305" H 4570 4796 50  0000 L CNN
-F 1 "100k" H 4570 4705 50  0000 L CNN
-F 2 "Resistor_SMD:R_0805_2012Metric_Pad1.20x1.40mm_HandSolder" V 4430 4750 50  0001 C CNN
-F 3 "~" H 4500 4750 50  0001 C CNN
-F 4 "REVERSEPOLARITY_SUPPORTED" H 4500 4750 50  0001 C CNN "Feature"
-F 5 "0.0036" H 4500 4750 50  0001 C CNN "Price"
-F 6 "yes" H 4500 4750 50  0001 C CNN "is stock"
-	1    4500 4750
-	1    0    0    -1
-$EndComp
-Wire Wire Line
-	4700 4000 5000 4000
-Wire Wire Line
-	5000 4100 5000 4000
-Wire Wire Line
-	5000 4400 5000 4500
-Wire Wire Line
-	5000 4500 4500 4500
-Wire Wire Line
-	4500 4500 4500 4300
-Wire Wire Line
-	4500 4500 4500 4600
-Connection ~ 4500 4500
-Wire Wire Line
-	4500 4900 4500 5500
-Wire Wire Line
-	4500 5500 5500 5500
-Wire Notes Line
-	4250 3500 5250 3500
-Wire Notes Line
-	5250 3500 5250 5000
-Wire Notes Line
-	5250 5000 4250 5000
-Wire Notes Line
-	4250 5000 4250 3500
-Text Notes 4250 3500 0    50   ~ 0
-Reverse voltage protection
 Wire Wire Line
 	9000 5500 9000 5600
@@
 	5500 5500 6500 5500
 Connection ~ 5500 5500
-Wire Wire Line
-	5000 4000 5500 4000
-Connection ~ 5000 4000
 Connection ~ 5500 4000
-Text Label 3500 4550 1    50   ~ 0
+Text Label 4700 4550 1    50   ~ 0
 surge_bypass
 Wire Wire Line
-	3500 4600 3500 4000
-Wire Wire Line
-	3500 5500 3500 4900
-Wire Wire Line
-	3400 4000 3500 4000
-$Comp
-L Device:D_TVS D302
+	4700 4600 4700 4000
+Wire Wire Line
+	4700 5500 4700 4900
+Wire Wire Line
+	4600 4000 4700 4000
+$Comp
+L Diode:Z2SMBxxx D302
 U 1 1 5FC9A3E5
-P 3500 4750
-F 0 "D302" V 3450 4450 50  0000 L CNN
-F 1 "SMBJ30CA CK /SMBJ15CA BM" V 3550 3550 50  0000 L CNN
-F 2 "Diode_SMD:D_SMB_Handsoldering" H 3500 4750 50  0001 C CNN
-F 3 "~" H 3500 4750 50  0001 C CNN
-F 4 "0.1" H 3500 4750 50  0001 C CNN "Price"
-F 5 "no" H 3500 4750 50  0001 C CNN "is stock"
-	1    3500 4750
-	0    1    1    0
-$EndComp
-Wire Wire Line
-	2000 4850 2000 5500
-Wire Wire Line
-	2000 4650 2000 4000
+P 4700 4750
+F 0 "D302" V 4650 4450 50  0000 L CNN
+F 1 "SMBJ15A" V 4750 4350 50  0000 L CNN
+F 2 "Diode_SMD:D_SMB_Handsoldering" H 4700 4750 50  0001 C CNN
+F 3 "~" H 4700 4750 50  0001 C CNN
+F 4 "0.1" H 4700 4750 50  0001 C CNN "Price"
+F 5 "no" H 4700 4750 50  0001 C CNN "is stock"
+	1    4700 4750
+	0    1    1    0
+$EndComp
+Wire Wire Line
+	3200 4850 3200 5500
+Wire Wire Line
+	3200 4650 3200 4000
 $Comp
 L Device:Fuse F301
 U 1 1 5F7CC4D4
-P 3250 4000
-F 0 "F301" V 3053 4000 50  0000 C CNN
-F 1 "max. 5A F" V 3144 4000 50  0000 C CNN
-F 2 "LedBarController:Fuseholder_Cylinder-5x20mm_BLX_A_Horizontal" V 3180 4000 50  0001 C CNN
-F 3 "~" H 3250 4000 50  0001 C CNN
-F 4 "POWER" H 3250 4000 50  0001 C CNN "Feature"
-F 5 "0.1474" H 3250 4000 50  0001 C CNN "Price"
-F 6 "yes" H 3250 4000 50  0001 C CNN "is stock"
-	1    3250 4000
-	0    1    1    0
-$EndComp
-NoConn ~ 2000 4750
+P 4450 4000
+F 0 "F301" V 4253 4000 50  0000 C CNN
+F 1 "max. 5A F" V 4344 4000 50  0000 C CNN
+F 2 "LedBarController:Fuseholder_Cylinder-5x20mm_BLX_A_Horizontal" V 4380 4000 50  0001 C CNN
+F 3 "~" H 4450 4000 50  0001 C CNN
+F 4 "POWER" H 4450 4000 50  0001 C CNN "Feature"
+F 5 "0.1474" H 4450 4000 50  0001 C CNN "Price"
+F 6 "yes" H 4450 4000 50  0001 C CNN "is stock"
+	1    4450 4000
+	0    1    1    0
+$EndComp
+NoConn ~ 3200 4750
 $Comp
 L Connector:Barrel_Jack_Switch J301
 U 1 1 5F7C9FB6
-P 1700 4750
-F 0 "J301" H 1757 5067 50  0000 C CNN
-F 1 "Barrel_Jack_Switch" H 1757 4976 50  0000 C CNN
-F 2 "Connector_BarrelJack:BarrelJack_CUI_PJ-102AH_Horizontal" H 1750 4710 50  0001 C CNN
-F 3 "~" H 1750 4710 50  0001 C CNN
-F 4 "POWER" H 1700 4750 50  0001 C CNN "Feature"
-F 5 "0.0472" H 1700 4750 50  0001 C CNN "Price"
-F 6 "yes" H 1700 4750 50  0001 C CNN "is stock"
-	1    1700 4750
-	1    0    0    -1
-$EndComp
-Wire Wire Line
-	2000 4000 3100 4000
-Wire Wire Line
-	2000 5500 3500 5500
-Wire Wire Line
-	3500 4000 4300 4000
-Connection ~ 3500 4000
-Wire Wire Line
-	4500 5500 3500 5500
-Connection ~ 4500 5500
-Connection ~ 3500 5500
-Wire Notes Line
-	2250 3500 3750 3500
-Wire Notes Line
-	3750 3500 3750 5000
-Wire Notes Line
-	3750 5000 2250 5000
-Wire Notes Line
-	2250 5000 2250 3500
-Text Notes 2250 3500 0    50   ~ 0
+P 2900 4750
+F 0 "J301" H 2957 5067 50  0000 C CNN
+F 1 "Barrel_Jack_Switch" H 2957 4976 50  0000 C CNN
+F 2 "Connector_BarrelJack:BarrelJack_CUI_PJ-102AH_Horizontal" H 2950 4710 50  0001 C CNN
+F 3 "~" H 2950 4710 50  0001 C CNN
+F 4 "POWER" H 2900 4750 50  0001 C CNN "Feature"
+F 5 "0.0472" H 2900 4750 50  0001 C CNN "Price"
+F 6 "yes" H 2900 4750 50  0001 C CNN "is stock"
+	1    2900 4750
+	1    0    0    -1
+$EndComp
+Wire Wire Line
+	3200 4000 4300 4000
+Wire Wire Line
+	3200 5500 4700 5500
+Wire Notes Line
+	3450 3500 4950 3500
+Wire Notes Line
+	4950 3500 4950 5000
+Wire Notes Line
+	4950 5000 3450 5000
+Wire Notes Line
+	3450 5000 3450 3500
+Text Notes 3450 3500 0    50   ~ 0
 Over current and voltage protection
 Wire Wire Line
@@
 Text Notes 5500 1500 0    50   ~ 0
 Voltage and current measurement
+Wire Wire Line
+	4700 4000 5500 4000
+Connection ~ 4700 4000
+Wire Wire Line
+	4700 5500 5500 5500
+Connection ~ 4700 5500
 $EndSCHEMATC

Commit message: Changed address for INA219 from 0x40 to 0x44
Connections:
- net +5V: now also U301.1 (A1)
- net GND: no longer U301.1 (A1)
Changed lines of the file:
@@
 Wire Wire Line
 	7300 2950 7300 3050
-Wire Wire Line
-	7700 2650 7700 2750
-Wire Wire Line
-	7700 2950 7300 2950
-Connection ~ 7700 2750
-Wire Wire Line
-	7700 2750 7700 2950
 Connection ~ 7300 2950
 $Comp
@@
 $EndComp
 Wire Wire Line
-	7300 2050 8500 2050
+	7300 2050 7850 2050
 Wire Wire Line
 	8500 2050 8500 2350
@@
 Wire Wire Line
 	7300 2050 7300 2150
-Wire Wire Line
-	8500 2950 7700 2950
-Connection ~ 7700 2950
 Wire Wire Line
 	8500 2650 8500 2950
@@
 	4700 5500 5500 5500
 Connection ~ 4700 5500
+Wire Wire Line
+	7300 2950 7850 2950
+Wire Wire Line
+	7700 2750 7850 2750
+Wire Wire Line
+	7850 2750 7850 2950
+Connection ~ 7850 2950
+Wire Wire Line
+	7850 2950 8500 2950
+Wire Wire Line
+	7700 2650 7850 2650
+Wire Wire Line
+	7850 2650 7850 2050
+Connection ~ 7850 2050
+Wire Wire Line
+	7850 2050 8500 2050
 $EndSCHEMATC
