File: LedBarController/Power.sch (KiCad schematic (older format))
At the start: 22 parts, among them J301 Barrel_Jack_Switch, U301 INA219AxD, U302 AMS1117-5.0

Commit message: Replaced 470R for 10k resistor to make the LED less bright
Parts:
- R306: value 470R -> 10k
Changed lines of the file:
@@
 P 9500 4750
 F 0 "R306" H 9570 4796 50  0000 L CNN
-F 1 "470R" H 9570 4705 50  0000 L CNN
+F 1 "10k" H 9570 4705 50  0000 L CNN
 F 2 "Resistor_SMD:R_0805_2012Metric_Pad1.20x1.40mm_HandSolder" V 9430 4750 50  0001 C CNN
 F 3 "~" H 9500 4750 50  0001 C CNN
