File: LedBarController/PWM.sch (KiCad schematic (older format))
At the start: 2 parts, among them U601 PCA9685PW

Commit message: Restarted PCB
Parts:
- added C201, C204: 0.1uF, Capacitor_SMD:C_0805_2012Metric_Pad1.18x1.45mm_HandSolder, symbol Device:C
- added C202, C205: 470uF/35V, Capacitor_THT:CP_Radial_D13.0mm_P5.00mm, symbol Device:CP
- added J201, J203: Conn_01x05, Connector_PinHeader_2.00mm:PinHeader_1x05_P2.00mm_Vertical, symbol Connector_Generic:Conn_01x05
- added J202: Conn_02x07_Odd_Even, Connector_PinSocket_2.00mm:PinSocket_2x07_P2.00mm_Vertical, symbol Connector_Generic:Conn_02x07_Odd_Even
- renumbered C601 to C203, U601 to U201
Connections:
- net GND: now also C201.2, C202.2, C204.2, C205.2, J202.14 (Pin_14)
- net strip1_b_out: now also J201.4 (Pin_4)
- net strip1_g_out: now also J201.2 (Pin_2)
- net strip1_r_out: now also J201.3 (Pin_3)
- net strip1_w_out: now also J201.5 (Pin_5)
- net strip2_b_out: now also J202.10 (Pin_10)
- net strip2_g_out: now also J202.6 (Pin_6)
- net strip2_r_out: now also J202.8 (Pin_8)
- net strip2_w_out: now also J202.12 (Pin_12)
- net strip3_b_out: now also J202.9 (Pin_9)
- net strip3_g_out: now also J202.5 (Pin_5)
- net strip3_r_out: now also J202.7 (Pin_7)
- net strip3_w_out: now also J202.11 (Pin_11)
- net strip4_b_out: now also J203.4 (Pin_4)
- net strip4_g_out: now also J203.2 (Pin_2)
- net strip4_r_out: now also J203.3 (Pin_3)
- net strip4_w_out: now also J203.5 (Pin_5)
- new net VDD: C201.1, C202.1, C204.1, C205.1, J201.1 (Pin_1), J202.1 (Pin_1), J202.2 (Pin_2), J202.3 (Pin_3), J202.4 (Pin_4), J203.1 (Pin_1)
- new net button: J202.13 (Pin_13)
Other:
- moved on the sheet: C203, U201

Commit message: Just before reverse order of strips
Connections:
- net strip2_b_out: now also J202.9 (Pin_9); no longer J202.10 (Pin_10)
- net strip2_g_out: now also J202.5 (Pin_5); no longer J202.6 (Pin_6)
- net strip2_r_out: now also J202.7 (Pin_7); no longer J202.8 (Pin_8)
- net strip2_w_out: now also J202.11 (Pin_11); no longer J202.12 (Pin_12)
- net strip3_b_out: now also J202.10 (Pin_10); no longer J202.9 (Pin_9)
- net strip3_g_out: now also J202.6 (Pin_6); no longer J202.5 (Pin_5)
- net strip3_r_out: now also J202.8 (Pin_8); no longer J202.7 (Pin_7)
- net strip3_w_out: now also J202.12 (Pin_12); no longer J202.11 (Pin_11)
Changed lines of the file:
@@
 Wire Wire Line
 	9050 5300 9300 5300
-Wire Wire Line
-	8600 3350 8600 3250
-$Comp
-L Connector_Generic:Conn_02x07_Odd_Even J?
-U 1 1 5F880FC8
-P 8300 3650
-AR Path="/5F92F971/5F880FC8" Ref="J?"  Part="1"
-AR Path="/5F8F2E1B/5F880FC8" Ref="J202"  Part="1"
-F 0 "J202" H 8350 4075 50  0000 C CNN
-F 1 "Conn_02x07_Odd_Even" H 8350 4076 50  0001 C CNN
-F 2 "Connector_PinSocket_2.00mm:PinSocket_2x07_P2.00mm_Vertical" H 8300 3650 50  0001 C CNN
-F 3 "~" H 8300 3650 50  0001 C CNN
-	1    8300 3650
-	0    -1   -1   0
-$EndComp
 $Comp
 L power:GND #PWR?
 U 1 1 5F880FC2
-P 8600 3250
+P 8600 3950
 AR Path="/5F92F971/5F880FC2" Ref="#PWR?"  Part="1"
 AR Path="/5F8F2E1B/5F880FC2" Ref="#PWR0206"  Part="1"
-F 0 "#PWR0206" H 8600 3000 50  0001 C CNN
-F 1 "GND" H 8605 3077 50  0000 C CNN
-F 2 "" H 8600 3250 50  0001 C CNN
-F 3 "" H 8600 3250 50  0001 C CNN
-	1    8600 3250
-	-1   0    0    1
+F 0 "#PWR0206" H 8600 3700 50  0001 C CNN
+F 1 "GND" H 8605 3777 50  0000 C CNN
+F 2 "" H 8600 3950 50  0001 C CNN
+F 3 "" H 8600 3950 50  0001 C CNN
+	1    8600 3950
+	1    0    0    -1
 $EndComp
 Wire Wire Line
@@
 Wire Wire Line
 	6500 2950 8500 2950
-Text HLabel 8700 3950 2    50   Output ~ 0
-button
-Wire Wire Line
-	8600 3850 8600 3950
-Wire Wire Line
-	8600 3950 8700 3950
+Wire Wire Line
+	8600 3250 8700 3250
 Wire Wire Line
 	8200 3350 8200 2750
@@
 Wire Wire Line
 	6500 4250 8300 4250
-Wire Wire Line
-	8200 3850 8200 4350
-Wire Wire Line
-	8300 4250 8300 3850
-Wire Wire Line
-	8400 3850 8400 4450
-Wire Wire Line
-	8500 4550 8500 3850
 Wire Wire Line
 	5500 4250 5100 4250
@@
 F1 "SideStrip.sch" 50
 $EndSheet
+Wire Wire Line
+	8300 4250 8300 3850
+Wire Wire Line
+	8200 3850 8200 4350
+Wire Wire Line
+	8500 4550 8500 3850
+Wire Wire Line
+	8400 3850 8400 4450
+$Comp
+L Connector_Generic:Conn_02x07_Odd_Even J?
+U 1 1 5F880FC8
+P 8300 3550
+AR Path="/5F92F971/5F880FC8" Ref="J?"  Part="1"
+AR Path="/5F8F2E1B/5F880FC8" Ref="J202"  Part="1"
+F 0 "J202" H 8350 3975 50  0000 C CNN
+F 1 "Conn_02x07_Odd_Even" H 8350 3976 50  0001 C CNN
+F 2 "Connector_PinSocket_2.00mm:PinSocket_2x07_P2.00mm_Vertical" H 8300 3550 50  0001 C CNN
+F 3 "~" H 8300 3550 50  0001 C CNN
+	1    8300 3550
+	0    -1   1    0
+$EndComp
+Text HLabel 8700 3250 2    50   Output ~ 0
+button
+Wire Wire Line
+	8600 3950 8600 3850
+Wire Wire Line
+	8600 3350 8600 3250
 $EndSCHEMATC

Commit message: Before moving down the center connector
Connections:
- net GND: now also J202.13 (Pin_13); no longer J202.14 (Pin_14)
- net button: now also J202.14 (Pin_14); no longer J202.13 (Pin_13)
- net strip2_b_out: now also J202.10 (Pin_10); no longer J202.9 (Pin_9)
- net strip2_g_out: now also J202.6 (Pin_6); no longer J202.5 (Pin_5)
- net strip2_r_out: now also J202.8 (Pin_8); no longer J202.7 (Pin_7)
- net strip2_w_out: now also J202.12 (Pin_12); no longer J202.11 (Pin_11)
- net strip3_b_out: now also J202.9 (Pin_9); no longer J202.10 (Pin_10)
- net strip3_g_out: now also J202.5 (Pin_5); no longer J202.6 (Pin_6)
- net strip3_r_out: now also J202.7 (Pin_7); no longer J202.8 (Pin_8)
- net strip3_w_out: now also J202.11 (Pin_11); no longer J202.12 (Pin_12)
Changed lines of the file:
@@
 L Connector_Generic:Conn_02x07_Odd_Even J?
 U 1 1 5F880FC8
-P 8300 3550
+P 8300 3650
 AR Path="/5F92F971/5F880FC8" Ref="J?"  Part="1"
 AR Path="/5F8F2E1B/5F880FC8" Ref="J202"  Part="1"
-F 0 "J202" H 8350 3975 50  0000 C CNN
-F 1 "Conn_02x07_Odd_Even" H 8350 3976 50  0001 C CNN
-F 2 "Connector_PinSocket_2.00mm:PinSocket_2x07_P2.00mm_Vertical" H 8300 3550 50  0001 C CNN
-F 3 "~" H 8300 3550 50  0001 C CNN
-	1    8300 3550
-	0    -1   1    0
+F 0 "J202" H 8350 4075 50  0000 C CNN
+F 1 "Conn_02x07_Odd_Even" H 8350 4076 50  0001 C CNN
+F 2 "Connector_PinSocket_2.00mm:PinSocket_2x07_P2.00mm_Vertical" H 8300 3650 50  0001 C CNN
+F 3 "~" H 8300 3650 50  0001 C CNN
+	1    8300 3650
+	0    -1   -1   0
 $EndComp
 Text HLabel 8700 3250 2    50   Output ~ 0

Commit message: Changed components and moved center connector upwards
Connections:
- net +5V: no longer U201.1 (A0), U201.3 (A2), U201.5 (A4)
- net GND: now also U201.1 (A0), U201.3 (A2), U201.5 (A4)
Changed lines of the file:
@@
 Connection ~ 2100 3850
 Wire Wire Line
-	2100 3050 2100 3850
+	2100 3050 2100 3750
 Wire Wire Line
 	3000 2150 3000 2550
 Wire Wire Line
 	1700 3150 2300 3150
-Wire Wire Line
-	2200 3750 2200 3950
-Connection ~ 2200 3750
-Wire Wire Line
-	2300 3750 2200 3750
-Wire Wire Line
-	2200 3950 2200 4150
-Connection ~ 2200 3950
-Wire Wire Line
-	2300 3950 2200 3950
-Wire Wire Line
-	2200 4150 2300 4150
-Wire Wire Line
-	2200 3650 2200 3750
-$Comp
-L power:+5V #PWR0207
-U 1 1 5F85CEB7
-P 2200 3650
-F 0 "#PWR0207" H 2200 3500 50  0001 C CNN
-F 1 "+5V" H 2215 3823 50  0000 C CNN
-F 2 "" H 2200 3650 50  0001 C CNN
-F 3 "" H 2200 3650 50  0001 C CNN
-	1    2200 3650
-	1    0    0    -1
-$EndComp
 Wire Wire Line
 	2100 4250 2100 4900
@@
 	2300 4250 2100 4250
 Wire Wire Line
-	2100 4050 2100 4250
+	2100 4050 2100 4150
 Connection ~ 2100 4050
 Wire Wire Line
 	2300 4050 2100 4050
 Wire Wire Line
-	2100 3850 2100 4050
+	2100 3850 2100 3950
 Wire Wire Line
 	2300 3850 2100 3850
@@
 Wire Wire Line
 	8600 3350 8600 3250
+Wire Wire Line
+	2300 3750 2100 3750
+Connection ~ 2100 3750
+Wire Wire Line
+	2100 3750 2100 3850
+Wire Wire Line
+	2300 3950 2100 3950
+Connection ~ 2100 3950
+Wire Wire Line
+	2100 3950 2100 4050
+Wire Wire Line
+	2300 4150 2100 4150
+Connection ~ 2100 4150
+Wire Wire Line
+	2100 4150 2100 4250
 $EndSCHEMATC

Commit message: Updated labels in schematic and moved RTC to sub-schematic
Connections:
- net I2C_SCL renamed scl
- net I2C_SDA renamed sda
- net ~OE renamed ~oe
Changed lines of the file:
@@
 $Descr A4 11693 8268
 encoding utf-8
-Sheet 2 13
+Sheet 2 14
 Title ""
 Date ""
@@
 $EndComp
 Text HLabel 1700 3150 0    50   Input ~ 0
-~OE
+~oe
 Wire Wire Line
 	1700 2950 2300 2950
@@
 $EndComp
 Text HLabel 1700 2950 0    50   BiDi ~ 0
-I2C_SDA
+sda
 Text HLabel 1700 2850 0    50   Output ~ 0
-I2C_SCL
+scl
 $Comp
 L Driver_LED:PCA9685PW U201

Commit message: Work in progress
Parts:
- C201, C204: Feature (none) -> PWM_SUPPORTED; Price (none) -> 0.0057; is stock (none) -> yes
- C202, C205: Feature (none) -> PWM_SUPPORTED; Price (none) -> 0.0656; is stock (none) -> no
- C203: value C -> 0.1uF; Feature (none) -> PWM_SUPPORTED; Price (none) -> 0.0057; is stock (none) -> yes
- J201, J203: value Conn_01x05 -> Female pitch strip 1x7 pins 2.0mm pitch; Feature (none) -> PWM_SUPPORTED_4STRIPS; Price (none) -> 0.14; is stock (none) -> yes
- J202: value Conn_02x07_Odd_Even -> Female 2x7 pins 2.0mm pitch; Feature (none) -> PWM_SUPPORTED_2STRIPS; Price (none) -> 0.0595; is stock (none) -> no
- U201: Feature (none) -> PWM_SUPPORTED; Price (none) -> 1.157; is stock (none) -> yes
Changed lines of the file:
@@
 P 1600 4450
 F 0 "C203" H 1715 4496 50  0000 L CNN
-F 1 "C" H 1715 4405 50  0000 L CNN
+F 1 "0.1uF" H 1715 4405 50  0000 L CNN
 F 2 "Capacitor_SMD:C_0805_2012Metric_Pad1.18x1.45mm_HandSolder" H 1638 4300 50  0001 C CNN
 F 3 "~" H 1600 4450 50  0001 C CNN
+F 4 "PWM_SUPPORTED" H 1600 4450 50  0001 C CNN "Feature"
+F 5 "0.0057" H 1600 4450 50  0001 C CNN "Price"
+F 6 "yes" H 1600 4450 50  0001 C CNN "is stock"
 	1    1600 4450
 	1    0    0    -1
@@
 F 2 "Package_SO:TSSOP-28_4.4x9.7mm_P0.65mm" H 3025 2575 50  0001 L CNN
 F 3 "http://www.nxp.com/documents/data_sheet/PCA9685.pdf" H 2600 4250 50  0001 C CNN
+F 4 "PWM_SUPPORTED" H 3000 3550 50  0001 C CNN "Feature"
+F 5 "1.157" H 3000 3550 50  0001 C CNN "Price"
+F 6 "yes" H 3000 3550 50  0001 C CNN "is stock"
 	1    3000 3550
 	1    0    0    -1
@@
 F 2 "Capacitor_THT:CP_Radial_D13.0mm_P5.00mm" H 9388 2100 50  0001 C CNN
 F 3 "~" H 9350 2250 50  0001 C CNN
+F 4 "PWM_SUPPORTED" H 9350 2250 50  0001 C CNN "Feature"
+F 5 "0.0656" H 9350 2250 50  0001 C CNN "Price"
+F 6 "no" H 9350 2250 50  0001 C CNN "is stock"
 	1    9350 2250
 	1    0    0    -1
@@
 F 2 "Capacitor_SMD:C_0805_2012Metric_Pad1.18x1.45mm_HandSolder" H 8888 2100 50  0001 C CNN
 F 3 "~" H 8850 2250 50  0001 C CNN
+F 4 "PWM_SUPPORTED" H 8850 2250 50  0001 C CNN "Feature"
+F 5 "0.0057" H 8850 2250 50  0001 C CNN "Price"
+F 6 "yes" H 8850 2250 50  0001 C CNN "is stock"
 	1    8850 2250
 	1    0    0    -1
@@
 F 2 "Capacitor_THT:CP_Radial_D13.0mm_P5.00mm" H 9338 4900 50  0001 C CNN
 F 3 "~" H 9300 5050 50  0001 C CNN
+F 4 "PWM_SUPPORTED" H 9300 5050 50  0001 C CNN "Feature"
+F 5 "0.0656" H 9300 5050 50  0001 C CNN "Price"
+F 6 "no" H 9300 5050 50  0001 C CNN "is stock"
 	1    9300 5050
 	1    0    0    -1
@@
 F 2 "Capacitor_SMD:C_0805_2012Metric_Pad1.18x1.45mm_HandSolder" H 8838 4900 50  0001 C CNN
 F 3 "~" H 8800 5050 50  0001 C CNN
+F 4 "PWM_SUPPORTED" H 8800 5050 50  0001 C CNN "Feature"
+F 5 "0.0057" H 8800 5050 50  0001 C CNN "Price"
+F 6 "yes" H 8800 5050 50  0001 C CNN "is stock"
 	1    8800 5050
 	1    0    0    -1
@@
 AR Path="/5F8F2E1B/5F9D9614" Ref="J203"  Part="1"
 F 0 "J203" H 8330 6192 50  0000 L CNN
-F 1 "Conn_01x05" H 8000 5850 50  0000 L CNN
+F 1 "Female pitch strip 1x7 pins 2.0mm pitch" H 8000 5850 50  0000 L CNN
 F 2 "Connector_PinHeader_2.00mm:PinHeader_1x05_P2.00mm_Vertical" H 8250 6150 50  0001 C CNN
 F 3 "~" H 8250 6150 50  0001 C CNN
+F 4 "PWM_SUPPORTED_4STRIPS" H 8250 6150 50  0001 C CNN "Feature"
+F 5 "0.14" H 8250 6150 50  0001 C CNN "Price"
+F 6 "yes" H 8250 6150 50  0001 C CNN "is stock"
 	1    8250 6150
 	0    -1   1    0
@@
 AR Path="/5F8F2E1B/5F85865B" Ref="J201"  Part="1"
 F 0 "J201" H 8330 1092 50  0000 L CNN
-F 1 "Conn_01x05" H 8330 1001 50  0000 L CNN
+F 1 "Female pitch strip 1x7 pins 2.0mm pitch" H 8330 1001 50  0000 L CNN
 F 2 "Connector_PinHeader_2.00mm:PinHeader_1x05_P2.00mm_Vertical" H 8250 1050 50  0001 C CNN
 F 3 "~" H 8250 1050 50  0001 C CNN
+F 4 "PWM_SUPPORTED_4STRIPS" H 8250 1050 50  0001 C CNN "Feature"
+F 5 "0.14" H 8250 1050 50  0001 C CNN "Price"
+F 6 "yes" H 8250 1050 50  0001 C CNN "is stock"
 	1    8250 1050
 	0    -1   -1   0
@@
 AR Path="/5F8F2E1B/5F880FC8" Ref="J202"  Part="1"
 F 0 "J202" H 8350 4075 50  0000 C CNN
-F 1 "Conn_02x07_Odd_Even" H 8350 4076 50  0001 C CNN
+F 1 "Female 2x7 pins 2.0mm pitch" H 8350 4076 50  0001 C CNN
 F 2 "Connector_PinSocket_2.00mm:PinSocket_2x07_P2.00mm_Vertical" H 8300 3650 50  0001 C CNN
 F 3 "~" H 8300 3650 50  0001 C CNN
+F 4 "PWM_SUPPORTED_2STRIPS" H 8300 3650 50  0001 C CNN "Feature"
+F 5 "0.0595" H 8300 3650 50  0001 C CNN "Price"
+F 6 "no" H 8300 3650 50  0001 C CNN "is stock"
 	1    8300 3650
 	0    -1   -1   0

Commit message: Route complete
Connections:
- net button renamed ~button~
Changed lines of the file:
@@
 $EndComp
 Text HLabel 8700 3250 2    50   Output ~ 0
-button
+~button~
 Wire Wire Line
 	8600 3950 8600 3850
