File: LedBarController/PWM.sch (KiCad schematic (older format))
At the start: 9 parts, among them J201 Female pitch strip 1x7 pins 2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, J202 Female 2x7 pins 2.0mm pitch, J203 Female pitch strip 1x7 pins 2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, U201 PCA9685PW

Commit message: moved board on schema to same sheet
Other:
- note added: "Left"
Changed lines of the file:
@@
 $Descr A4 11693 8268
 encoding utf-8
-Sheet 2 13
+Sheet 2 11
 Title ""
 Date ""
@@
 	8050 5850 8050 5950
 $Sheet
-S 9500 1000 1050 500
-U 5FA33522
-F0 "SideStrip_left" 50
-F1 "SideStrip.sch" 50
-$EndSheet
-$Sheet
 S 9500 3000 1000 1000
 U 5FA33E59
 F0 "CenterStrips" 50
 F1 "CenterStrips.sch" 50
-$EndSheet
-$Sheet
-S 9450 5550 1050 450
-U 5FA34085
-F0 "SideStrip_right" 50
-F1 "SideStrip.sch" 50
 $EndSheet
 Wire Wire Line
@@
 Wire Wire Line
 	2100 4150 2100 4250
+Text Notes 10050 6100 0    50   ~ 0
+Left
 $EndSCHEMATC

Commit message: Moved FETs to PWM sheet
Parts:
- added Q301, Q302, Q303, Q304, Q401, Q402, Q403, Q404, Q501, Q502, Q503, Q504, Q601, Q602, Q603, Q604: Si2302DS, Package_TO_SOT_SMD:SOT-23_Handsoldering, symbol Device:Q_NMOS_GSD
Connections:
- wire segments 134 -> 152
Other:
- note removed: "Left"
- moved on the sheet: C201, C202, C203, C204, C205, J201, J202, J203, U201

Commit message: Reanotate
Parts:
- renumbered C203 to C601, C201 to C602, C202 to C603, C204 to C604, C205 to C605, J201 to J601, J202 to J602, J203 to J603, Q301 to Q601, Q302 to Q602, Q303 to Q603, Q304 to Q604, Q401 to Q605, Q402 to Q606, Q403 to Q607, Q404 to Q608, Q501 to Q609, Q502 to Q610, Q503 to Q611, Q504 to Q612, Q601 to Q613, Q602 to Q614, Q603 to Q615, Q604 to Q616, U201 to U601
