File: LedBarController/PWM.sch (KiCad schematic (older format))
At the start: 25 parts, among them J601 Female pitch strip 1x7 pins 2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, J602 Female 2x7 pins 2.0mm pitch, J603 Female pitch strip 1x7 pins 2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, Q601 Si2302DS, Q602 Si2302DS, Q603 Si2302DS, Q604 Si2302DS, Q605 Si2302DS, Q606 Si2302DS, Q607 Si2302DS, Q608 Si2302DS, Q609 Si2302DS, Q610 Si2302DS, Q611 Si2302DS, Q612 Si2302DS, Q613 Si2302DS, Q614 Si2302DS, Q615 Si2302DS, Q616 Si2302DS, U601 PCA9685PW

Commit message: Changed size and value of Capacitor C603 and C605
Parts:
- C603, C605: value 470uF/35V -> 1000uF/16V; footprint Capacitor_THT:CP_Radial_D13.0mm_P5.00mm -> Capacitor_THT:CP_Radial_D10.0mm_P5.00mm
Changed lines of the file:
@@
 AR Path="/602F109A/6030A14B/5F83AB7E" Ref="C603"  Part="1"
 F 0 "C603" H 4618 5946 50  0000 L CNN
-F 1 "470uF/35V" H 4618 5855 50  0000 L CNN
-F 2 "Capacitor_THT:CP_Radial_D13.0mm_P5.00mm" H 4538 5750 50  0001 C CNN
+F 1 "1000uF/16V" H 4618 5855 50  0000 L CNN
+F 2 "Capacitor_THT:CP_Radial_D10.0mm_P5.00mm" H 4538 5750 50  0001 C CNN
 F 3 "~" H 4500 5900 50  0001 C CNN
 F 4 "PWM_SUPPORTED" H 4500 5900 50  0001 C CNN "Feature"
@@
 AR Path="/602F109A/6030A14B/5F83D76F" Ref="C605"  Part="1"
 F 0 "C605" H 8118 5996 50  0000 L CNN
-F 1 "470uF/35V" H 8118 5905 50  0000 L CNN
-F 2 "Capacitor_THT:CP_Radial_D13.0mm_P5.00mm" H 8038 5800 50  0001 C CNN
+F 1 "1000uF/16V" H 8118 5905 50  0000 L CNN
+F 2 "Capacitor_THT:CP_Radial_D10.0mm_P5.00mm" H 8038 5800 50  0001 C CNN
 F 3 "~" H 8000 5950 50  0001 C CNN
 F 4 "PWM_SUPPORTED" H 8000 5950 50  0001 C CNN "Feature"

Commit message: Added more testpoints
Parts:
- added TP601: ~oe, symbol Connector:TestPoint
Connections:
- wire segments 152 -> 154
Changed lines of the file:
@@
 	3000 1200 3000 1600
 Wire Wire Line
-	1700 2200 2300 2200
+	1700 2200 1800 2200
 Wire Wire Line
 	2100 3300 2100 3950
@@
 Wire Wire Line
 	7750 5450 9350 5450
+$Comp
+L Connector:TestPoint TP601
+U 1 1 60820EF9
+P 1800 2250
+F 0 "TP601" H 1742 2270 50  0000 R CNN
+F 1 "~oe" H 1742 2368 50  0000 R CNN
+F 2 "" H 2000 2250 50  0001 C CNN
+F 3 "~" H 2000 2250 50  0001 C CNN
+	1    1800 2250
+	-1   0    0    1
+$EndComp
+Wire Wire Line
+	1800 2250 1800 2200
+Connection ~ 1800 2200
+Wire Wire Line
+	1800 2200 2300 2200
 $EndSCHEMATC
