File: LedBarController/0-10V.sch (KiCad schematic (older format))
At the start: 20 parts, among them J1101 Conn_01x02, J1102 Conn_01x02, U1101 LM358

Commit message: Work in progress
Parts:
- C1101: value 0.1uF -> 1uF; Feature (none) -> 10V_SUPPORTED_1CH; Price (none) -> 0.015; is stock (none) -> no
- C1102: value C -> 0.1uF; Feature (none) -> 10V_SUPPORTED; Price (none) -> 0.0057; is stock (none) -> yes
- C1103: value 0.1uF -> 1uF; Feature (none) -> 10V_SUPPORTED_2CH; Price (none) -> 0.015; is stock (none) -> no
- C1104: value C -> 0.1uF; Feature (none) -> 10V_SUPPORTED_1CH; Price (none) -> 0.0057; is stock (none) -> yes
- C1105: value C -> 0.1uF; Feature (none) -> 10V_SUPPORTED_2CH; Price (none) -> 0.0057; is stock (none) -> yes
- J1101: Feature (none) -> 10V_SUPPORTED_1CH; Price (none) -> 0.0097; is stock (none) -> yes
- J1102: Feature (none) -> 10V_SUPPORTED_2CH; Price (none) -> 0.0097; is stock (none) -> yes
- R1101: value 1k -> 10k; Feature (none) -> 10V_SUPPORTED_1CH; Price (none) -> 0.0036; is stock (none) -> yes
- R1102, R1103, R1104: Feature (none) -> 10V_SUPPORTED_1CH; Price (none) -> 0.0036; is stock (none) -> yes
- R1105: value 1k -> 10k; Feature (none) -> 10V_SUPPORTED_2CH; Price (none) -> 0.0036; is stock (none) -> yes
- R1106, R1107, R1108: Feature (none) -> 10V_SUPPORTED_2CH; Price (none) -> 0.0036; is stock (none) -> yes
- TP1101: value 0-10Va1 -> a1; Feature (none) -> 10V_SUPPORTED_1CH; Price (none) -> 0; is stock (none) -> n.a.
- TP1102: value 0-10Vd1 -> d1; Feature (none) -> 10V_SUPPORTED_1CH; Price (none) -> 0; is stock (none) -> n.a.
- TP1103: value 0-10Va2 -> a2; Feature (none) -> 10V_SUPPORTED_2CH; Price (none) -> 0; is stock (none) -> n.a.
- TP1104: value 0-10Vd2 -> d2; Feature (none) -> 10V_SUPPORTED_2CH; Price (none) -> 0; is stock (none) -> n.a.
- U1101: value LM358 -> LM358DR; Feature (none) -> 10V_SUPPORTED; Price (none) -> 0.033; is stock (none) -> no
Changed lines of the file:
@@
 P 6050 2100
 F 0 "U1101" H 6050 2467 50  0000 C CNN
-F 1 "LM358" H 6050 2376 50  0000 C CNN
+F 1 "LM358DR" H 6050 2376 50  0000 C CNN
 F 2 "Package_SO:SOIC-8_3.9x4.9mm_P1.27mm" H 6050 2100 50  0001 C CNN
 F 3 "http://www.ti.com/lit/ds/symlink/lm2904-n.pdf" H 6050 2100 50  0001 C CNN
+F 4 "10V_SUPPORTED" H 6050 2100 50  0001 C CNN "Feature"
+F 5 "0.033" H 6050 2100 50  0001 C CNN "Price"
+F 6 "no" H 6050 2100 50  0001 C CNN "is stock"
 	1    6050 2100
 	1    0    0    -1
@@
 P 4750 2000
 F 0 "R1101" V 4543 2000 50  0000 C CNN
-F 1 "1k" V 4634 2000 50  0000 C CNN
+F 1 "10k" V 4634 2000 50  0000 C CNN
 F 2 "Resistor_SMD:R_0805_2012Metric_Pad1.20x1.40mm_HandSolder" V 4680 2000 50  0001 C CNN
 F 3 "~" H 4750 2000 50  0001 C CNN
+F 4 "10V_SUPPORTED_1CH" H 4750 2000 50  0001 C CNN "Feature"
+F 5 "0.0036" H 4750 2000 50  0001 C CNN "Price"
+F 6 "yes" H 4750 2000 50  0001 C CNN "is stock"
 	1    4750 2000
 	0    1    1    0
@@
 P 9500 4000
 F 0 "C1102" H 9615 4046 50  0000 L CNN
-F 1 "C" H 9615 3955 50  0000 L CNN
+F 1 "0.1uF" H 9615 3955 50  0000 L CNN
 F 2 "Capacitor_SMD:C_0805_2012Metric_Pad1.18x1.45mm_HandSolder" H 9538 3850 50  0001 C CNN
 F 3 "~" H 9500 4000 50  0001 C CNN
+F 4 "10V_SUPPORTED" H 9500 4000 50  0001 C CNN "Feature"
+F 5 "0.0057" H 9500 4000 50  0001 C CNN "Price"
+F 6 "yes" H 9500 4000 50  0001 C CNN "is stock"
 	1    9500 4000
 	1    0    0    -1
@@
 P 10100 4000
 F 0 "U1101" H 10058 4046 50  0000 L CNN
-F 1 "LM358" H 10058 3955 50  0000 L CNN
+F 1 "LM358DR" H 10058 3955 50  0000 L CNN
 F 2 "Package_SO:SOIC-8_3.9x4.9mm_P1.27mm" H 10100 4000 50  0001 C CNN
 F 3 "http://www.ti.com/lit/ds/symlink/lm2904-n.pdf" H 10100 4000 50  0001 C CNN
+F 4 "10V_SUPPORTED" H 10100 4000 50  0001 C CNN "Feature"
+F 5 "0.033" H 10100 4000 50  0001 C CNN "Price"
+F 6 "no" H 10100 4000 50  0001 C CNN "is stock"
 	3    10100 4000
 	1    0    0    -1
@@
 P 5000 2250
 F 0 "C1101" H 5115 2296 50  0000 L CNN
-F 1 "0.1uF" H 5115 2205 50  0000 L CNN
+F 1 "1uF" H 5115 2205 50  0000 L CNN
 F 2 "Capacitor_SMD:C_0805_2012Metric_Pad1.18x1.45mm_HandSolder" H 5038 2100 50  0001 C CNN
 F 3 "~" H 5000 2250 50  0001 C CNN
+F 4 "10V_SUPPORTED_1CH" H 5000 2250 50  0001 C CNN "Feature"
+F 5 "0.015" H 5000 2250 50  0001 C CNN "Price"
+F 6 "no" H 5000 2250 50  0001 C CNN "is stock"
 	1    5000 2250
 	1    0    0    -1
@@
 F 2 "Resistor_SMD:R_0805_2012Metric_Pad1.20x1.40mm_HandSolder" V 6430 2800 50  0001 C CNN
 F 3 "~" H 6500 2800 50  0001 C CNN
+F 4 "10V_SUPPORTED_1CH" H 6500 2800 50  0001 C CNN "Feature"
+F 5 "0.0036" H 6500 2800 50  0001 C CNN "Price"
+F 6 "yes" H 6500 2800 50  0001 C CNN "is stock"
 	1    6500 2800
 	-1   0    0    1
@@
 F 2 "Resistor_SMD:R_0805_2012Metric_Pad1.20x1.40mm_HandSolder" V 6430 3300 50  0001 C CNN
 F 3 "~" H 6500 3300 50  0001 C CNN
+F 4 "10V_SUPPORTED_1CH" H 6500 3300 50  0001 C CNN "Feature"
+F 5 "0.0036" H 6500 3300 50  0001 C CNN "Price"
+F 6 "yes" H 6500 3300 50  0001 C CNN "is stock"
 	1    6500 3300
 	-1   0    0    1
@@
 F 2 "Connector_JST:JST_PH_S2B-PH-K_1x02_P2.00mm_Horizontal" H 7350 2500 50  0001 C CNN
 F 3 "~" H 7350 2500 50  0001 C CNN
+F 4 "10V_SUPPORTED_1CH" H 7350 2500 50  0001 C CNN "Feature"
+F 5 "0.0097" H 7350 2500 50  0001 C CNN "Price"
+F 6 "yes" H 7350 2500 50  0001 C CNN "is stock"
 	1    7350 2500
 	1    0    0    -1
@@
 P 4250 1450
 F 0 "TP1101" H 4308 1568 50  0000 L CNN
-F 1 "0-10Va1" H 4308 1477 50  0000 L CNN
+F 1 "a1" H 4308 1477 50  0000 L CNN
 F 2 "TestPoint:TestPoint_Pad_D1.0mm" H 4450 1450 50  0001 C CNN
 F 3 "~" H 4450 1450 50  0001 C CNN
+F 4 "10V_SUPPORTED_1CH" H 4250 1450 50  0001 C CNN "Feature"
+F 5 "0" H 4250 1450 50  0001 C CNN "Price"
+F 6 "n.a." H 4250 1450 50  0001 C CNN "is stock"
 	1    4250 1450
 	1    0    0    -1
@@
 P 4250 1950
 F 0 "TP1102" H 4308 2068 50  0000 L CNN
-F 1 "0-10Vd1" H 4308 1977 50  0000 L CNN
+F 1 "d1" H 4308 1977 50  0000 L CNN
 F 2 "TestPoint:TestPoint_Pad_D1.0mm" H 4450 1950 50  0001 C CNN
 F 3 "~" H 4450 1950 50  0001 C CNN
+F 4 "10V_SUPPORTED_1CH" H 4250 1950 50  0001 C CNN "Feature"
+F 5 "0" H 4250 1950 50  0001 C CNN "Price"
+F 6 "n.a." H 4250 1950 50  0001 C CNN "is stock"
 	1    4250 1950
 	1    0    0    -1
@@
 F 2 "Resistor_SMD:R_0805_2012Metric_Pad1.20x1.40mm_HandSolder" V 6430 2300 50  0001 C CNN
 F 3 "~" H 6500 2300 50  0001 C CNN
+F 4 "10V_SUPPORTED_1CH" H 6500 2300 50  0001 C CNN "Feature"
+F 5 "0.0036" H 6500 2300 50  0001 C CNN "Price"
+F 6 "yes" H 6500 2300 50  0001 C CNN "is stock"
 	1    6500 2300
 	-1   0    0    1
@@
 F 2 "Resistor_SMD:R_0805_2012Metric_Pad1.20x1.40mm_HandSolder" V 6430 5300 50  0001 C CNN
 F 3 "~" H 6500 5300 50  0001 C CNN
+F 4 "10V_SUPPORTED_2CH" H 6500 5300 50  0001 C CNN "Feature"
+F 5 "0.0036" H 6500 5300 50  0001 C CNN "Price"
+F 6 "yes" H 6500 5300 50  0001 C CNN "is stock"
 	1    6500 5300
 	-1   0    0    1
@@
 F 2 "Resistor_SMD:R_0805_2012Metric_Pad1.20x1.40mm_HandSolder" V 6430 5800 50  0001 C CNN
 F 3 "~" H 6500 5800 50  0001 C CNN
+F 4 "10V_SUPPORTED_2CH" H 6500 5800 50  0001 C CNN "Feature"
+F 5 "0.0036" H 6500 5800 50  0001 C CNN "Price"
+F 6 "yes" H 6500 5800 50  0001 C CNN "is stock"
 	1    6500 5800
 	-1   0    0    1
@@
 F 2 "Connector_JST:JST_PH_B2B-PH-K_1x02_P2.00mm_Vertical" H 7350 5000 50  0001 C CNN
 F 3 "~" H 7350 5000 50  0001 C CNN
+F 4 "10V_SUPPORTED_2CH" H 7350 5000 50  0001 C CNN "Feature"
+F 5 "0.0097" H 7350 5000 50  0001 C CNN "Price"
+F 6 "yes" H 7350 5000 50  0001 C CNN "is stock"
 	1    7350 5000
 	1    0    0    -1
@@
 F 2 "Resistor_SMD:R_0805_2012Metric_Pad1.20x1.40mm_HandSolder" V 6430 4800 50  0001 C CNN
 F 3 "~" H 6500 4800 50  0001 C CNN
+F 4 "10V_SUPPORTED_2CH" H 6500 4800 50  0001 C CNN "Feature"
+F 5 "0.0036" H 6500 4800 50  0001 C CNN "Price"
+F 6 "yes" H 6500 4800 50  0001 C CNN "is stock"
 	1    6500 4800
 	-1   0    0    1
@@
 P 4250 4450
 F 0 "TP1104" H 4308 4568 50  0000 L CNN
-F 1 "0-10Vd2" H 4308 4477 50  0000 L CNN
+F 1 "d2" H 4308 4477 50  0000 L CNN
 F 2 "TestPoint:TestPoint_Pad_D1.0mm" H 4450 4450 50  0001 C CNN
 F 3 "~" H 4450 4450 50  0001 C CNN
+F 4 "10V_SUPPORTED_2CH" H 4250 4450 50  0001 C CNN "Feature"
+F 5 "0" H 4250 4450 50  0001 C CNN "Price"
+F 6 "n.a." H 4250 4450 50  0001 C CNN "is stock"
 	1    4250 4450
 	1    0    0    -1
@@
 P 4250 3950
 F 0 "TP1103" H 4308 4068 50  0000 L CNN
-F 1 "0-10Va2" H 4308 3977 50  0000 L CNN
+F 1 "a2" H 4308 3977 50  0000 L CNN
 F 2 "TestPoint:TestPoint_Pad_D1.0mm" H 4450 3950 50  0001 C CNN
 F 3 "~" H 4450 3950 50  0001 C CNN
+F 4 "10V_SUPPORTED_2CH" H 4250 3950 50  0001 C CNN "Feature"
+F 5 "0" H 4250 3950 50  0001 C CNN "Price"
+F 6 "n.a." H 4250 3950 50  0001 C CNN "is stock"
 	1    4250 3950
 	1    0    0    -1
@@
 P 5000 4750
 F 0 "C1103" H 5115 4796 50  0000 L CNN
-F 1 "0.1uF" H 5115 4705 50  0000 L CNN
+F 1 "1uF" H 5115 4705 50  0000 L CNN
 F 2 "Capacitor_SMD:C_0805_2012Metric_Pad1.18x1.45mm_HandSolder" H 5038 4600 50  0001 C CNN
 F 3 "~" H 5000 4750 50  0001 C CNN
+F 4 "10V_SUPPORTED_2CH" H 5000 4750 50  0001 C CNN "Feature"
+F 5 "0.015" H 5000 4750 50  0001 C CNN "Price"
+F 6 "no" H 5000 4750 50  0001 C CNN "is stock"
 	1    5000 4750
 	1    0    0    -1
@@
 P 4750 4500
 F 0 "R1105" V 4543 4500 50  0000 C CNN
-F 1 "1k" V 4634 4500 50  0000 C CNN
+F 1 "10k" V 4634 4500 50  0000 C CNN
 F 2 "Resistor_SMD:R_0805_2012Metric_Pad1.20x1.40mm_HandSolder" V 4680 4500 50  0001 C CNN
 F 3 "~" H 4750 4500 50  0001 C CNN
+F 4 "10V_SUPPORTED_2CH" H 4750 4500 50  0001 C CNN "Feature"
+F 5 "0.0036" H 4750 4500 50  0001 C CNN "Price"
+F 6 "yes" H 4750 4500 50  0001 C CNN "is stock"
 	1    4750 4500
 	0    1    1    0
@@
 P 6050 4600
 F 0 "U1101" H 6050 4967 50  0000 C CNN
-F 1 "LM358" H 6050 4876 50  0000 C CNN
+F 1 "LM358DR" H 6050 4876 50  0000 C CNN
 F 2 "Package_SO:SOIC-8_3.9x4.9mm_P1.27mm" H 6050 4600 50  0001 C CNN
 F 3 "http://www.ti.com/lit/ds/symlink/lm2904-n.pdf" H 6050 4600 50  0001 C CNN
+F 4 "10V_SUPPORTED" H 6050 4600 50  0001 C CNN "Feature"
+F 5 "0.033" H 6050 4600 50  0001 C CNN "Price"
+F 6 "no" H 6050 4600 50  0001 C CNN "is stock"
 	2    6050 4600
 	1    0    0    -1
@@
 P 7000 4750
 F 0 "C1105" H 7115 4796 50  0000 L CNN
-F 1 "C" H 7115 4705 50  0000 L CNN
+F 1 "0.1uF" H 7115 4705 50  0000 L CNN
 F 2 "Capacitor_SMD:C_0805_2012Metric_Pad1.18x1.45mm_HandSolder" H 7038 4600 50  0001 C CNN
 F 3 "~" H 7000 4750 50  0001 C CNN
+F 4 "10V_SUPPORTED_2CH" H 7000 4750 50  0001 C CNN "Feature"
+F 5 "0.0057" H 7000 4750 50  0001 C CNN "Price"
+F 6 "yes" H 7000 4750 50  0001 C CNN "is stock"
 	1    7000 4750
 	1    0    0    -1
@@
 P 7000 2250
 F 0 "C1104" H 7115 2296 50  0000 L CNN
-F 1 "C" H 7115 2205 50  0000 L CNN
+F 1 "0.1uF" H 7115 2205 50  0000 L CNN
 F 2 "Capacitor_SMD:C_0805_2012Metric_Pad1.18x1.45mm_HandSolder" H 7038 2100 50  0001 C CNN
 F 3 "~" H 7000 2250 50  0001 C CNN
+F 4 "10V_SUPPORTED_1CH" H 7000 2250 50  0001 C CNN "Feature"
+F 5 "0.0057" H 7000 2250 50  0001 C CNN "Price"
+F 6 "yes" H 7000 2250 50  0001 C CNN "is stock"
 	1    7000 2250
 	1    0    0    -1
