File: LedBarController/0-10V.sch (KiCad schematic (older format))
At the start: 16 parts, among them J1101 Conn_01x02, J1102 Conn_01x02, U1101 LM393

Commit message: Reanotate
Parts:
- renumbered C1101 to C701, C1104 to C702, C1102 to C703, C1103 to C704, C1105 to C705, J1101 to J701, J1102 to J702, R1101 to R701, R1102 to R702, R1103 to R703, R1104 to R704, R1105 to R705, R1106 to R706, R1107 to R707, R1108 to R708, U1101 to U701
Changed lines of the file:
@@
 $EndDescr
 $Comp
-L Amplifier_Operational:LM358 U1101
+L Amplifier_Operational:LM358 U701
 U 1 1 5F7CF7BB
 P 6050 2100
-F 0 "U1101" H 6050 2467 50  0000 C CNN
+F 0 "U701" H 6050 2467 50  0000 C CNN
 F 1 "LM393" H 6050 2376 50  0000 C CNN
 F 2 "Package_SO:SOIC-8_3.9x4.9mm_P1.27mm" H 6050 2100 50  0001 C CNN
@@
 $EndComp
 $Comp
-L Device:R R1101
+L Device:R R701
 U 1 1 5F7CF150
 P 4750 2000
-F 0 "R1101" V 4543 2000 50  0000 C CNN
+F 0 "R701" V 4543 2000 50  0000 C CNN
 F 1 "10k" V 4634 2000 50  0000 C CNN
 F 2 "Resistor_SMD:R_0805_2012Metric_Pad1.20x1.40mm_HandSolder" V 4680 2000 50  0001 C CNN
@@
 $EndComp
 $Comp
-L power:GND #PWR0159
+L power:GND #PWR0707
 U 1 1 5F7D11A9
 P 9500 4750
-F 0 "#PWR0159" H 9500 4500 50  0001 C CNN
+F 0 "#PWR0707" H 9500 4500 50  0001 C CNN
 F 1 "GND" H 9505 4577 50  0000 C CNN
 F 2 "" H 9500 4750 50  0001 C CNN
@@
 $EndComp
 $Comp
-L power:VDD #PWR0160
+L power:VDD #PWR0704
 U 1 1 5F7D28E4
 P 9500 3250
-F 0 "#PWR0160" H 9500 3100 50  0001 C CNN
+F 0 "#PWR0704" H 9500 3100 50  0001 C CNN
 F 1 "VDD" H 9515 3423 50  0000 C CNN
 F 2 "" H 9500 3250 50  0001 C CNN
@@
 $EndComp
 $Comp
-L Device:C C1102
+L Device:C C703
 U 1 1 5F7D3020
 P 9500 4000
-F 0 "C1102" H 9615 4046 50  0000 L CNN
+F 0 "C703" H 9615 4046 50  0000 L CNN
 F 1 "0.1uF" H 9615 3955 50  0000 L CNN
 F 2 "Capacitor_SMD:C_0805_2012Metric_Pad1.18x1.45mm_HandSolder" H 9538 3850 50  0001 C CNN
@@
 $EndComp
 $Comp
-L Amplifier_Operational:LM358 U1101
+L Amplifier_Operational:LM358 U701
 U 3 1 5F7CF10E
 P 10100 4000
-F 0 "U1101" H 10058 4046 50  0000 L CNN
+F 0 "U701" H 10058 4046 50  0000 L CNN
 F 1 "LM393" H 10058 3955 50  0000 L CNN
 F 2 "Package_SO:SOIC-8_3.9x4.9mm_P1.27mm" H 10100 4000 50  0001 C CNN
@@
 pwm1
 $Comp
-L Device:C C1101
+L Device:C C701
 U 1 1 5F7DE73D
 P 5000 2250
-F 0 "C1101" H 5115 2296 50  0000 L CNN
+F 0 "C701" H 5115 2296 50  0000 L CNN
 F 1 "1uF" H 5115 2205 50  0000 L CNN
 F 2 "Capacitor_SMD:C_0805_2012Metric_Pad1.18x1.45mm_HandSolder" H 5038 2100 50  0001 C CNN
@@
 	5000 2000 5000 2100
 $Comp
-L power:GND #PWR0161
+L power:GND #PWR0702
 U 1 1 5F7E0414
 P 5000 2500
-F 0 "#PWR0161" H 5000 2250 50  0001 C CNN
+F 0 "#PWR0702" H 5000 2250 50  0001 C CNN
 F 1 "GND" H 5005 2327 50  0000 C CNN
 F 2 "" H 5000 2500 50  0001 C CNN
@@
 Connection ~ 5000 2000
 $Comp
-L Device:R R1103
+L Device:R R703
 U 1 1 5F7E4BB1
 P 6500 2800
-F 0 "R1103" H 6430 2754 50  0000 R CNN
+F 0 "R703" H 6430 2754 50  0000 R CNN
 F 1 "10k" H 6430 2845 50  0000 R CNN
 F 2 "Resistor_SMD:R_0805_2012Metric_Pad1.20x1.40mm_HandSolder" V 6430 2800 50  0001 C CNN
@@
 $EndComp
 $Comp
-L Device:R R1104
+L Device:R R704
 U 1 1 5F7E5039
 P 6500 3300
-F 0 "R1104" H 6430 3254 50  0000 R CNN
+F 0 "R704" H 6430 3254 50  0000 R CNN
 F 1 "10k" H 6430 3345 50  0000 R CNN
 F 2 "Resistor_SMD:R_0805_2012Metric_Pad1.20x1.40mm_HandSolder" V 6430 3300 50  0001 C CNN
@@
 	6500 3050 6500 3150
 $Comp
-L power:GND #PWR0162
+L power:GND #PWR0705
 U 1 1 5F7E7493
 P 6500 3550
-F 0 "#PWR0162" H 6500 3300 50  0001 C CNN
+F 0 "#PWR0705" H 6500 3300 50  0001 C CNN
 F 1 "GND" H 6505 3377 50  0000 C CNN
 F 2 "" H 6500 3550 50  0001 C CNN
@@
 	6500 3450 6500 3550
 $Comp
-L Connector_Generic:Conn_01x02 J1101
+L Connector_Generic:Conn_01x02 J701
 U 1 1 5F80EAFE
 P 7350 2500
-F 0 "J1101" H 7430 2492 50  0000 L CNN
+F 0 "J701" H 7430 2492 50  0000 L CNN
 F 1 "Conn_01x02" H 7430 2401 50  0000 L CNN
 F 2 "TerminalBlock_TE-Connectivity:TerminalBlock_TE_282834-2_1x02_P2.54mm_Horizontal" H 7350 2500 50  0001 C CNN
@@
 $EndComp
 $Comp
-L power:GND #PWR0163
+L power:GND #PWR0703
 U 1 1 5F8114A7
 P 7000 2750
-F 0 "#PWR0163" H 7000 2500 50  0001 C CNN
+F 0 "#PWR0703" H 7000 2500 50  0001 C CNN
 F 1 "GND" H 7005 2577 50  0000 C CNN
 F 2 "" H 7000 2750 50  0001 C CNN
@@
 	7000 2600 7000 2750
 $Comp
-L Device:R R1102
+L Device:R R702
 U 1 1 5F837482
 P 6500 2300
-F 0 "R1102" H 6430 2254 50  0000 R CNN
+F 0 "R702" H 6430 2254 50  0000 R CNN
 F 1 "1k" H 6430 2345 50  0000 R CNN
 F 2 "Resistor_SMD:R_0805_2012Metric_Pad1.20x1.40mm_HandSolder" V 6430 2300 50  0001 C CNN
@@
 	6500 2950 6500 3050
 $Comp
-L Device:C C1104
+L Device:C C702
 U 1 1 5F9C8781
 P 7000 2250
-F 0 "C1104" H 7115 2296 50  0000 L CNN
+F 0 "C702" H 7115 2296 50  0000 L CNN
 F 1 "0.1uF" H 7115 2205 50  0000 L CNN
 F 2 "Capacitor_SMD:C_0805_2012Metric_Pad1.18x1.45mm_HandSolder" H 7038 2100 50  0001 C CNN
@@
 	7000 2500 7150 2500
 $Comp
-L power:GND #PWR0164
+L power:GND #PWR0701
 U 1 1 5F9CDC23
 P 7000 2000
-F 0 "#PWR0164" H 7000 1750 50  0001 C CNN
+F 0 "#PWR0701" H 7000 1750 50  0001 C CNN
 F 1 "GND" H 7005 1827 50  0000 C CNN
 F 2 "" H 7000 2000 50  0001 C CNN
@@
 	7000 2000 7000 2100
 $Comp
-L Amplifier_Operational:LM358 U1101
+L Amplifier_Operational:LM358 U701
 U 2 1 5F7CEF2E
 P 6050 4600
-F 0 "U1101" H 6050 4967 50  0000 C CNN
+F 0 "U701" H 6050 4967 50  0000 C CNN
 F 1 "LM393" H 6050 4876 50  0000 C CNN
 F 2 "Package_SO:SOIC-8_3.9x4.9mm_P1.27mm" H 6050 4600 50  0001 C CNN
@@
 	5500 4700 5750 4700
 $Comp
-L Device:R R1105
+L Device:R R705
 U 1 1 5FEE3D26
 P 4750 4500
-F 0 "R1105" V 4543 4500 50  0000 C CNN
+F 0 "R705" V 4543 4500 50  0000 C CNN
 F 1 "10k" V 4634 4500 50  0000 C CNN
 F 2 "Resistor_SMD:R_0805_2012Metric_Pad1.20x1.40mm_HandSolder" V 4680 4500 50  0001 C CNN
@@
 pwm2
 $Comp
-L Device:C C1103
+L Device:C C704
 U 1 1 5FEE3D30
 P 5000 4750
-F 0 "C1103" H 5115 4796 50  0000 L CNN
+F 0 "C704" H 5115 4796 50  0000 L CNN
 F 1 "1uF" H 5115 4705 50  0000 L CNN
 F 2 "Capacitor_SMD:C_0805_2012Metric_Pad1.18x1.45mm_HandSolder" H 5038 4600 50  0001 C CNN
@@
 	5000 4500 5000 4600
 $Comp
-L power:GND #PWR0165
+L power:GND #PWR0708
 U 1 1 5FEE3D38
 P 5000 5000
-F 0 "#PWR0165" H 5000 4750 50  0001 C CNN
+F 0 "#PWR0708" H 5000 4750 50  0001 C CNN
 F 1 "GND" H 5005 4827 50  0000 C CNN
 F 2 "" H 5000 5000 50  0001 C CNN
@@
 Connection ~ 5000 4500
 $Comp
-L Device:R R1107
+L Device:R R707
 U 1 1 5FEE9ACA
 P 6500 5300
-F 0 "R1107" H 6430 5254 50  0000 R CNN
+F 0 "R707" H 6430 5254 50  0000 R CNN
 F 1 "10k" H 6430 5345 50  0000 R CNN
 F 2 "Resistor_SMD:R_0805_2012Metric_Pad1.20x1.40mm_HandSolder" V 6430 5300 50  0001 C CNN
@@
 $EndComp
 $Comp
-L Device:R R1108
+L Device:R R708
 U 1 1 5FEE9AD3
 P 6500 5800
-F 0 "R1108" H 6430 5754 50  0000 R CNN
+F 0 "R708" H 6430 5754 50  0000 R CNN
 F 1 "10k" H 6430 5845 50  0000 R CNN
 F 2 "Resistor_SMD:R_0805_2012Metric_Pad1.20x1.40mm_HandSolder" V 6430 5800 50  0001 C CNN
@@
 	6500 5550 6500 5650
 $Comp
-L power:GND #PWR0166
+L power:GND #PWR0710
 U 1 1 5FEE9ADC
 P 6500 6050
-F 0 "#PWR0166" H 6500 5800 50  0001 C CNN
+F 0 "#PWR0710" H 6500 5800 50  0001 C CNN
 F 1 "GND" H 6505 5877 50  0000 C CNN
 F 2 "" H 6500 6050 50  0001 C CNN
@@
 	6500 5950 6500 6050
 $Comp
-L Connector_Generic:Conn_01x02 J1102
+L Connector_Generic:Conn_01x02 J702
 U 1 1 5FEE9AE6
 P 7350 5000
-F 0 "J1102" H 7430 4992 50  0000 L CNN
+F 0 "J702" H 7430 4992 50  0000 L CNN
 F 1 "Conn_01x02" H 7430 4901 50  0000 L CNN
 F 2 "TerminalBlock_TE-Connectivity:TerminalBlock_TE_282834-2_1x02_P2.54mm_Horizontal" H 7350 5000 50  0001 C CNN
@@
 $EndComp
 $Comp
-L power:GND #PWR0167
+L power:GND #PWR0709
 U 1 1 5FEE9AEC
 P 7000 5250
-F 0 "#PWR0167" H 7000 5000 50  0001 C CNN
+F 0 "#PWR0709" H 7000 5000 50  0001 C CNN
 F 1 "GND" H 7005 5077 50  0000 C CNN
 F 2 "" H 7000 5250 50  0001 C CNN
@@
 	7000 5100 7000 5250
 $Comp
-L Device:R R1106
+L Device:R R706
 U 1 1 5FEE9AF7
 P 6500 4800
-F 0 "R1106" H 6430 4754 50  0000 R CNN
+F 0 "R706" H 6430 4754 50  0000 R CNN
 F 1 "1k" H 6430 4845 50  0000 R CNN
 F 2 "Resistor_SMD:R_0805_2012Metric_Pad1.20x1.40mm_HandSolder" V 6430 4800 50  0001 C CNN
@@
 	6500 5450 6500 5550
 $Comp
-L Device:C C1105
+L Device:C C705
 U 1 1 5FEE9B07
 P 7000 4750
-F 0 "C1105" H 7115 4796 50  0000 L CNN
+F 0 "C705" H 7115 4796 50  0000 L CNN
 F 1 "0.1uF" H 7115 4705 50  0000 L CNN
 F 2 "Capacitor_SMD:C_0805_2012Metric_Pad1.18x1.45mm_HandSolder" H 7038 4600 50  0001 C CNN
@@
 	7000 5000 7150 5000
 $Comp
-L power:GND #PWR0168
+L power:GND #PWR0706
 U 1 1 5FEE9B10
 P 7000 4500
-F 0 "#PWR0168" H 7000 4250 50  0001 C CNN
+F 0 "#PWR0706" H 7000 4250 50  0001 C CNN
 F 1 "GND" H 7005 4327 50  0000 C CNN
 F 2 "" H 7000 4500 50  0001 C CNN
