File: LedBarController/0-10V.sch (KiCad schematic (older format))
At the start: 16 parts, among them J701 Conn_01x02, J702 Conn_01x02, U701 LM393

Commit message: Improved RC filter for 1-10V
Parts:
- R701, R705: value 10k -> 100k
Changed lines of the file:
@@
 P 4750 2400
 F 0 "R701" V 4543 2400 50  0000 C CNN
-F 1 "10k" V 4634 2400 50  0000 C CNN
+F 1 "100k" V 4634 2400 50  0000 C CNN
 F 2 "Resistor_SMD:R_0805_2012Metric_Pad1.20x1.40mm_HandSolder" V 4680 2400 50  0001 C CNN
 F 3 "~" H 4750 2400 50  0001 C CNN
@@
 P 4750 4900
 F 0 "R705" V 4543 4900 50  0000 C CNN
-F 1 "10k" V 4634 4900 50  0000 C CNN
+F 1 "100k" V 4634 4900 50  0000 C CNN
 F 2 "Resistor_SMD:R_0805_2012Metric_Pad1.20x1.40mm_HandSolder" V 4680 4900 50  0001 C CNN
 F 3 "~" H 4750 4900 50  0001 C CNN

Commit message: Added more testpoints
Parts:
- added TP701: pwm1, symbol Connector:TestPoint
- added TP702: pwm2, symbol Connector:TestPoint
- added TP703: a1, symbol Connector:TestPoint
- added TP704: a2, symbol Connector:TestPoint
- added TP705: ao1, symbol Connector:TestPoint
- added TP706: ao2, symbol Connector:TestPoint
Connections:
- net pwm1: now also TP701.1
- net pwm2: now also TP702.1
- net at C704.1, R705.1, U701.5 (+): now also TP704.1
- net at C705.2, J702.1 (Pin_1), R706.1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: now also TP706.1
- net at C701.1, R701.1, U701.3 (+): now also TP703.1
- net at C702.2, J701.1 (Pin_1), R702.1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: now also TP705.1
Other:
- moved on the sheet: C702, C705, J701, J702
Changed lines of the file:
@@
 L Connector_Generic:Conn_01x02 J701
 U 1 1 5F80EAFE
-P 7350 2500
-F 0 "J701" H 7430 2492 50  0000 L CNN
-F 1 "Conn_01x02" H 7430 2401 50  0000 L CNN
-F 2 "TerminalBlock_TE-Connectivity:TerminalBlock_TE_282834-2_1x02_P2.54mm_Horizontal" H 7350 2500 50  0001 C CNN
-F 3 "~" H 7350 2500 50  0001 C CNN
-F 4 "10V_SUPPORTED_1CH" H 7350 2500 50  0001 C CNN "Feature"
-F 5 "0.0097" H 7350 2500 50  0001 C CNN "Price"
-F 6 "yes" H 7350 2500 50  0001 C CNN "is stock"
-	1    7350 2500
+P 7850 2500
+F 0 "J701" H 7930 2492 50  0000 L CNN
+F 1 "Conn_01x02" H 7930 2401 50  0000 L CNN
+F 2 "TerminalBlock_TE-Connectivity:TerminalBlock_TE_282834-2_1x02_P2.54mm_Horizontal" H 7850 2500 50  0001 C CNN
+F 3 "~" H 7850 2500 50  0001 C CNN
+F 4 "10V_SUPPORTED_1CH" H 7850 2500 50  0001 C CNN "Feature"
+F 5 "0.0097" H 7850 2500 50  0001 C CNN "Price"
+F 6 "yes" H 7850 2500 50  0001 C CNN "is stock"
+	1    7850 2500
 	1    0    0    -1
 $EndComp
@@
 L power:GND #PWR0703
 U 1 1 5F8114A7
-P 7000 2750
-F 0 "#PWR0703" H 7000 2500 50  0001 C CNN
-F 1 "GND" H 7005 2577 50  0000 C CNN
-F 2 "" H 7000 2750 50  0001 C CNN
-F 3 "" H 7000 2750 50  0001 C CNN
-	1    7000 2750
-	1    0    0    -1
-$EndComp
-Wire Wire Line
-	7150 2600 7000 2600
-Wire Wire Line
-	7000 2600 7000 2750
+P 7500 3000
+F 0 "#PWR0703" H 7500 2750 50  0001 C CNN
+F 1 "GND" H 7505 2827 50  0000 C CNN
+F 2 "" H 7500 3000 50  0001 C CNN
+F 3 "" H 7500 3000 50  0001 C CNN
+	1    7500 3000
+	1    0    0    -1
+$EndComp
+Wire Wire Line
+	7650 2600 7500 2600
+Wire Wire Line
+	7500 2600 7500 3000
 $Comp
 L Device:R R702
@@
 Wire Wire Line
 	5500 2600 5500 3050
-Wire Wire Line
-	6500 2500 7000 2500
 Connection ~ 6500 2500
 Wire Wire Line
@@
 Wire Wire Line
 	6500 2950 6500 3050
-$Comp
-L Device:C C702
-U 1 1 5F9C8781
-P 7000 2250
-F 0 "C702" H 7115 2296 50  0000 L CNN
-F 1 "0.1uF" H 7115 2205 50  0000 L CNN
-F 2 "Capacitor_SMD:C_0805_2012Metric_Pad1.18x1.45mm_HandSolder" H 7038 2100 50  0001 C CNN
-F 3 "~" H 7000 2250 50  0001 C CNN
-F 4 "10V_SUPPORTED_1CH" H 7000 2250 50  0001 C CNN "Feature"
-F 5 "0.0057" H 7000 2250 50  0001 C CNN "Price"
-F 6 "yes" H 7000 2250 50  0001 C CNN "is stock"
-	1    7000 2250
-	1    0    0    -1
-$EndComp
-Wire Wire Line
-	7000 2400 7000 2500
-Connection ~ 7000 2500
-Wire Wire Line
-	7000 2500 7150 2500
-$Comp
-L power:GND #PWR0701
-U 1 1 5F9CDC23
-P 7000 2000
-F 0 "#PWR0701" H 7000 1750 50  0001 C CNN
-F 1 "GND" H 7005 1827 50  0000 C CNN
-F 2 "" H 7000 2000 50  0001 C CNN
-F 3 "" H 7000 2000 50  0001 C CNN
-	1    7000 2000
-	-1   0    0    1
-$EndComp
-Wire Wire Line
-	7000 2000 7000 2100
 $Comp
 L Amplifier_Operational:LM358 U701
@@
 L Connector_Generic:Conn_01x02 J702
 U 1 1 5FEE9AE6
-P 7350 5000
-F 0 "J702" H 7430 4992 50  0000 L CNN
-F 1 "Conn_01x02" H 7430 4901 50  0000 L CNN
-F 2 "TerminalBlock_TE-Connectivity:TerminalBlock_TE_282834-2_1x02_P2.54mm_Horizontal" H 7350 5000 50  0001 C CNN
-F 3 "~" H 7350 5000 50  0001 C CNN
-F 4 "10V_SUPPORTED_1CH" H 7350 5000 50  0001 C CNN "Feature"
-F 5 "0.0097" H 7350 5000 50  0001 C CNN "Price"
-F 6 "yes" H 7350 5000 50  0001 C CNN "is stock"
-	1    7350 5000
+P 7850 5000
+F 0 "J702" H 7930 4992 50  0000 L CNN
+F 1 "Conn_01x02" H 7930 4901 50  0000 L CNN
+F 2 "TerminalBlock_TE-Connectivity:TerminalBlock_TE_282834-2_1x02_P2.54mm_Horizontal" H 7850 5000 50  0001 C CNN
+F 3 "~" H 7850 5000 50  0001 C CNN
+F 4 "10V_SUPPORTED_1CH" H 7850 5000 50  0001 C CNN "Feature"
+F 5 "0.0097" H 7850 5000 50  0001 C CNN "Price"
+F 6 "yes" H 7850 5000 50  0001 C CNN "is stock"
+	1    7850 5000
 	1    0    0    -1
 $EndComp
@@
 L power:GND #PWR0709
 U 1 1 5FEE9AEC
-P 7000 5250
-F 0 "#PWR0709" H 7000 5000 50  0001 C CNN
-F 1 "GND" H 7005 5077 50  0000 C CNN
-F 2 "" H 7000 5250 50  0001 C CNN
-F 3 "" H 7000 5250 50  0001 C CNN
-	1    7000 5250
-	1    0    0    -1
-$EndComp
-Wire Wire Line
-	7150 5100 7000 5100
-Wire Wire Line
-	7000 5100 7000 5250
+P 7500 5500
+F 0 "#PWR0709" H 7500 5250 50  0001 C CNN
+F 1 "GND" H 7505 5327 50  0000 C CNN
+F 2 "" H 7500 5500 50  0001 C CNN
+F 3 "" H 7500 5500 50  0001 C CNN
+	1    7500 5500
+	1    0    0    -1
+$EndComp
+Wire Wire Line
+	7650 5100 7500 5100
+Wire Wire Line
+	7500 5100 7500 5500
 $Comp
 L Device:R R706
@@
 	-1   0    0    1
 $EndComp
-Wire Wire Line
-	6500 5000 7000 5000
 Connection ~ 6500 5000
 Wire Wire Line
@@
 L Device:C C705
 U 1 1 5FEE9B07
-P 7000 4750
-F 0 "C705" H 7115 4796 50  0000 L CNN
-F 1 "0.1uF" H 7115 4705 50  0000 L CNN
-F 2 "Capacitor_SMD:C_0805_2012Metric_Pad1.18x1.45mm_HandSolder" H 7038 4600 50  0001 C CNN
-F 3 "~" H 7000 4750 50  0001 C CNN
-F 4 "10V_SUPPORTED_1CH" H 7000 4750 50  0001 C CNN "Feature"
-F 5 "0.0057" H 7000 4750 50  0001 C CNN "Price"
-F 6 "yes" H 7000 4750 50  0001 C CNN "is stock"
-	1    7000 4750
-	1    0    0    -1
-$EndComp
-Wire Wire Line
-	7000 4900 7000 5000
-Connection ~ 7000 5000
-Wire Wire Line
-	7000 5000 7150 5000
+P 7000 5250
+F 0 "C705" H 6900 5300 50  0000 R CNN
+F 1 "0.1uF" H 6900 5200 50  0000 R CNN
+F 2 "Capacitor_SMD:C_0805_2012Metric_Pad1.18x1.45mm_HandSolder" H 7038 5100 50  0001 C CNN
+F 3 "~" H 7000 5250 50  0001 C CNN
+F 4 "10V_SUPPORTED_1CH" H 7000 5250 50  0001 C CNN "Feature"
+F 5 "0.0057" H 7000 5250 50  0001 C CNN "Price"
+F 6 "yes" H 7000 5250 50  0001 C CNN "is stock"
+	1    7000 5250
+	-1   0    0    1
+$EndComp
+Wire Wire Line
+	7000 5100 7000 5000
 $Comp
 L power:GND #PWR0706
 U 1 1 5FEE9B10
-P 7000 4500
-F 0 "#PWR0706" H 7000 4250 50  0001 C CNN
-F 1 "GND" H 7005 4327 50  0000 C CNN
-F 2 "" H 7000 4500 50  0001 C CNN
-F 3 "" H 7000 4500 50  0001 C CNN
-	1    7000 4500
-	-1   0    0    1
-$EndComp
-Wire Wire Line
-	7000 4500 7000 4600
+P 7000 5500
+F 0 "#PWR0706" H 7000 5250 50  0001 C CNN
+F 1 "GND" H 7005 5327 50  0000 C CNN
+F 2 "" H 7000 5500 50  0001 C CNN
+F 3 "" H 7000 5500 50  0001 C CNN
+	1    7000 5500
+	1    0    0    -1
+$EndComp
+Wire Wire Line
+	7000 5500 7000 5400
 Wire Wire Line
 	5500 5100 5500 5550
 Wire Wire Line
-	4000 2400 4600 2400
-Wire Wire Line
-	4000 4900 4600 4900
+	4000 2400 4150 2400
+Wire Wire Line
+	4000 4900 4150 4900
 $Comp
 L power:VDD #PWR0101
@@
 Wire Wire Line
 	6500 2100 6500 2000
+$Comp
+L Connector:TestPoint TP701
+U 1 1 607F410D
+P 4150 2350
+F 0 "TP701" H 4208 2468 50  0000 L CNN
+F 1 "pwm1" H 4208 2377 50  0000 L CNN
+F 2 "" H 4350 2350 50  0001 C CNN
+F 3 "~" H 4350 2350 50  0001 C CNN
+	1    4150 2350
+	1    0    0    -1
+$EndComp
+Wire Wire Line
+	4150 2350 4150 2400
+Connection ~ 4150 2400
+Wire Wire Line
+	4150 2400 4600 2400
+$Comp
+L Connector:TestPoint TP703
+U 1 1 607F5B5B
+P 5000 2350
+F 0 "TP703" H 5058 2468 50  0000 L CNN
+F 1 "a1" H 5058 2377 50  0000 L CNN
+F 2 "" H 5200 2350 50  0001 C CNN
+F 3 "~" H 5200 2350 50  0001 C CNN
+	1    5000 2350
+	1    0    0    -1
+$EndComp
+Wire Wire Line
+	7000 3000 7000 2900
+$Comp
+L power:GND #PWR0701
+U 1 1 5F9CDC23
+P 7000 3000
+F 0 "#PWR0701" H 7000 2750 50  0001 C CNN
+F 1 "GND" H 7005 2827 50  0000 C CNN
+F 2 "" H 7000 3000 50  0001 C CNN
+F 3 "" H 7000 3000 50  0001 C CNN
+	1    7000 3000
+	1    0    0    -1
+$EndComp
+$Comp
+L Device:C C702
+U 1 1 5F9C8781
+P 7000 2750
+F 0 "C702" H 6900 2800 50  0000 R CNN
+F 1 "0.1uF" H 6900 2700 50  0000 R CNN
+F 2 "Capacitor_SMD:C_0805_2012Metric_Pad1.18x1.45mm_HandSolder" H 7038 2600 50  0001 C CNN
+F 3 "~" H 7000 2750 50  0001 C CNN
+F 4 "10V_SUPPORTED_1CH" H 7000 2750 50  0001 C CNN "Feature"
+F 5 "0.0057" H 7000 2750 50  0001 C CNN "Price"
+F 6 "yes" H 7000 2750 50  0001 C CNN "is stock"
+	1    7000 2750
+	-1   0    0    1
+$EndComp
+Wire Wire Line
+	6500 2500 7000 2500
+Connection ~ 7000 2500
+Wire Wire Line
+	7000 2500 7000 2600
+$Comp
+L Connector:TestPoint TP705
+U 1 1 60805502
+P 7000 2350
+F 0 "TP705" H 7058 2468 50  0000 L CNN
+F 1 "ao1" H 7058 2377 50  0000 L CNN
+F 2 "" H 7200 2350 50  0001 C CNN
+F 3 "~" H 7200 2350 50  0001 C CNN
+	1    7000 2350
+	1    0    0    -1
+$EndComp
+Wire Wire Line
+	7000 2350 7000 2500
+Wire Wire Line
+	5000 2350 5000 2400
+Wire Wire Line
+	6500 5000 7000 5000
+Connection ~ 7000 5000
+$Comp
+L Connector:TestPoint TP706
+U 1 1 6081125F
+P 7000 4850
+F 0 "TP706" H 7058 4968 50  0000 L CNN
+F 1 "ao2" H 7058 4877 50  0000 L CNN
+F 2 "" H 7200 4850 50  0001 C CNN
+F 3 "~" H 7200 4850 50  0001 C CNN
+	1    7000 4850
+	1    0    0    -1
+$EndComp
+Wire Wire Line
+	7000 4850 7000 5000
+$Comp
+L Connector:TestPoint TP704
+U 1 1 608129B8
+P 5000 4850
+F 0 "TP704" H 5058 4968 50  0000 L CNN
+F 1 "a2" H 5058 4877 50  0000 L CNN
+F 2 "" H 5200 4850 50  0001 C CNN
+F 3 "~" H 5200 4850 50  0001 C CNN
+	1    5000 4850
+	1    0    0    -1
+$EndComp
+$Comp
+L Connector:TestPoint TP702
+U 1 1 608131ED
+P 4150 4850
+F 0 "TP702" H 4208 4968 50  0000 L CNN
+F 1 "pwm2" H 4208 4877 50  0000 L CNN
+F 2 "" H 4350 4850 50  0001 C CNN
+F 3 "~" H 4350 4850 50  0001 C CNN
+	1    4150 4850
+	1    0    0    -1
+$EndComp
+Wire Wire Line
+	4150 4850 4150 4900
+Connection ~ 4150 4900
+Wire Wire Line
+	4150 4900 4600 4900
+Wire Wire Line
+	5000 4850 5000 4900
+Wire Wire Line
+	7000 2500 7650 2500
+Wire Wire Line
+	7000 5000 7650 5000
 $EndSCHEMATC
