File: LedBarController/SideStrip.sch (KiCad schematic (older format))
At the start: 4 parts, among them J1301 Conn_01x05, J1302 Conn_01x05, J1303 Conn_01x05, J1304 Conn_01x05

Commit message: Work in progress
Connections:
- no-connect marks 1 -> 0
Changed lines of the file:
@@
 Text HLabel 3900 2950 0    50   Input ~ 0
 white
-NoConn ~ 3700 1900
 $Comp
 L Connector_Generic:Conn_01x05 J1301

Commit message: Restarted PCB
Parts:
- removed J1301: Conn_01x05, Connector_PinHeader_2.00mm:PinHeader_1x05_P2.00mm_Vertical, symbol Connector_Generic:Conn_01x05
- renumbered J1302 to J701, J1303 to J702, J1304 to J703
Other:
- note removed: "Speparate PCB"
Changed lines of the file:
@@
 $Descr A4 11693 8268
 encoding utf-8
-Sheet 11 13
+Sheet 16 13
 Title ""
 Date ""
@@
 Comment4 ""
 $EndDescr
-Text HLabel 3900 2750 0    50   Input ~ 0
-red
-Text HLabel 3900 2650 0    50   Input ~ 0
-green
-Text HLabel 3900 2850 0    50   Input ~ 0
-blue
-Text HLabel 3900 2950 0    50   Input ~ 0
-white
 $Comp
-L Connector_Generic:Conn_01x05 J1301
-U 1 1 5F96CE6F
-P 4500 2750
-AR Path="/5F92F348/5F96CE6F" Ref="J1301"  Part="1"
-AR Path="/5F92F3F9/5F96CE6F" Ref="J1101"  Part="1"
-F 0 "J1101" H 4580 2792 50  0000 L CNN
-F 1 "Conn_01x05" H 4580 2701 50  0000 L CNN
-F 2 "Connector_PinHeader_2.00mm:PinHeader_1x05_P2.00mm_Vertical" H 4500 2750 50  0001 C CNN
-F 3 "~" H 4500 2750 50  0001 C CNN
-	1    4500 2750
-	1    0    0    -1
-$EndComp
-$Comp
-L power:VDD #PWR01301
-U 1 1 5F96DC01
-P 4000 2300
-AR Path="/5F92F348/5F96DC01" Ref="#PWR01301"  Part="1"
-AR Path="/5F92F3F9/5F96DC01" Ref="#PWR01101"  Part="1"
-F 0 "#PWR01101" H 4000 2150 50  0001 C CNN
-F 1 "VDD" H 4015 2473 50  0000 C CNN
-F 2 "" H 4000 2300 50  0001 C CNN
-F 3 "" H 4000 2300 50  0001 C CNN
-	1    4000 2300
-	1    0    0    -1
-$EndComp
-Wire Wire Line
-	4000 2300 4000 2550
-Wire Wire Line
-	4000 2550 4300 2550
-Wire Wire Line
-	3900 2650 4300 2650
-Wire Wire Line
-	4300 2750 3900 2750
-Wire Wire Line
-	3900 2850 4300 2850
-Wire Wire Line
-	4300 2950 3900 2950
-$Comp
-L Connector_Generic:Conn_01x05 J1302
+L Connector_Generic:Conn_01x05 J?
 U 1 1 5F96E4A9
 P 6000 2750
-AR Path="/5F92F348/5F96E4A9" Ref="J1302"  Part="1"
-AR Path="/5F92F3F9/5F96E4A9" Ref="J1102"  Part="1"
-F 0 "J1102" H 5918 3167 50  0000 C CNN
+AR Path="/5F92F348/5F96E4A9" Ref="J?"  Part="1"
+AR Path="/5F92F3F9/5F96E4A9" Ref="J?"  Part="1"
+AR Path="/5F8F2E1B/5FA33522/5F96E4A9" Ref="J701"  Part="1"
+AR Path="/5F8F2E1B/5FA34085/5F96E4A9" Ref="J901"  Part="1"
+F 0 "J901" H 5918 3167 50  0000 C CNN
 F 1 "Conn_01x05" H 5918 3076 50  0000 C CNN
 F 2 "Connector_PinHeader_2.00mm:PinHeader_1x05_P2.00mm_Vertical" H 6000 2750 50  0001 C CNN
@@
 $EndComp
 $Comp
-L Connector_Generic:Conn_01x05 J1303
+L Connector_Generic:Conn_01x05 J?
 U 1 1 5F96EB0B
 P 7500 2750
-AR Path="/5F92F348/5F96EB0B" Ref="J1303"  Part="1"
-AR Path="/5F92F3F9/5F96EB0B" Ref="J1103"  Part="1"
-F 0 "J1103" H 7450 3050 50  0000 L CNN
+AR Path="/5F92F348/5F96EB0B" Ref="J?"  Part="1"
+AR Path="/5F92F3F9/5F96EB0B" Ref="J?"  Part="1"
+AR Path="/5F8F2E1B/5FA33522/5F96EB0B" Ref="J702"  Part="1"
+AR Path="/5F8F2E1B/5FA34085/5F96EB0B" Ref="J902"  Part="1"
+F 0 "J902" H 7450 3050 50  0000 L CNN
 F 1 "Conn_01x05" H 7450 3150 50  0000 L CNN
 F 2 "Connector_PinHeader_2.00mm:PinHeader_1x05_P2.00mm_Vertical" H 7500 2750 50  0001 C CNN
@@
 $EndComp
 $Comp
-L Connector_Generic:Conn_01x05 J1304
+L Connector_Generic:Conn_01x05 J?
 U 1 1 5F96F581
 P 7500 3750
-AR Path="/5F92F348/5F96F581" Ref="J1304"  Part="1"
-AR Path="/5F92F3F9/5F96F581" Ref="J1104"  Part="1"
-F 0 "J1104" H 7450 4050 50  0000 L CNN
+AR Path="/5F92F348/5F96F581" Ref="J?"  Part="1"
+AR Path="/5F92F3F9/5F96F581" Ref="J?"  Part="1"
+AR Path="/5F8F2E1B/5FA33522/5F96F581" Ref="J703"  Part="1"
+AR Path="/5F8F2E1B/5FA34085/5F96F581" Ref="J903"  Part="1"
+F 0 "J903" H 7450 4050 50  0000 L CNN
 F 1 "Conn_01x05" H 7450 4150 50  0000 L CNN
 F 2 "Connector_PinHeader_2.00mm:PinHeader_1x05_P2.00mm_Vertical" H 7500 3750 50  0001 C CNN
@@
 	6200 2950 7200 2950
 Connection ~ 7200 2950
-Wire Notes Line
-	5500 2000 5500 4500
-Wire Notes Line
-	5500 4500 8000 4500
-Wire Notes Line
-	8000 4500 8000 2000
-Wire Notes Line
-	8000 2000 5500 2000
-Text Notes 5500 2000 0    50   ~ 0
-Speparate PCB
 Text Label 6250 2650 0    50   ~ 0
 green_

Commit message: Work in progress
Parts:
- J701: value Conn_01x05 -> Male pitch strip 1x7 pins 2.0mm pitch; Feature (none) -> PWM_SUPPORTED_4STRIPS; Price (none) -> 0.016; is stock (none) -> yes
- J702, J703: Feature (none) -> PWM_SUPPORTED_4STRIPS; Price (none) -> 0; is stock (none) -> no
Changed lines of the file:
@@
 $Descr A4 11693 8268
 encoding utf-8
-Sheet 16 14
+Sheet 7 14
 Title ""
 Date ""
@@
 AR Path="/5F8F2E1B/5FA34085/5F96E4A9" Ref="J901"  Part="1"
 F 0 "J901" H 5918 3167 50  0000 C CNN
-F 1 "Conn_01x05" H 5918 3076 50  0000 C CNN
+F 1 "Male pitch strip 1x7 pins 2.0mm pitch" H 5918 3076 50  0000 C CNN
 F 2 "Connector_PinHeader_2.00mm:PinHeader_1x05_P2.00mm_Vertical" H 6000 2750 50  0001 C CNN
 F 3 "~" H 6000 2750 50  0001 C CNN
+F 4 "PWM_SUPPORTED_4STRIPS" H 6000 2750 50  0001 C CNN "Feature"
+F 5 "0.016" H 6000 2750 50  0001 C CNN "Price"
+F 6 "yes" H 6000 2750 50  0001 C CNN "is stock"
 	1    6000 2750
 	-1   0    0    -1
@@
 F 2 "Connector_PinHeader_2.00mm:PinHeader_1x05_P2.00mm_Vertical" H 7500 2750 50  0001 C CNN
 F 3 "~" H 7500 2750 50  0001 C CNN
+F 4 "PWM_SUPPORTED_4STRIPS" H 7500 2750 50  0001 C CNN "Feature"
+F 5 "0" H 7500 2750 50  0001 C CNN "Price"
+F 6 "no" H 7500 2750 50  0001 C CNN "is stock"
 	1    7500 2750
 	1    0    0    -1
@@
 F 2 "Connector_PinHeader_2.00mm:PinHeader_1x05_P2.00mm_Vertical" H 7500 3750 50  0001 C CNN
 F 3 "~" H 7500 3750 50  0001 C CNN
+F 4 "PWM_SUPPORTED_4STRIPS" H 7500 3750 50  0001 C CNN "Feature"
+F 5 "0" H 7500 3750 50  0001 C CNN "Price"
+F 6 "no" H 7500 3750 50  0001 C CNN "is stock"
 	1    7500 3750
 	1    0    0    -1

Commit message: moved board on schema to same sheet
Parts:
- added J? (x2): Male pitch strip 1x7 pins 2.0mm pitch, Connector_PinHeader_2.00mm:PinHeader_1x05_P2.00mm_Vertical, symbol Connector_Generic:Conn_01x05
- J702, J703: footprint Connector_PinHeader_2.00mm:PinHeader_1x05_P2.00mm_Vertical -> LedBarController:LED_Strip_10mm_5pins_Left
Connections:
- new net: J?.1 (Pin_1), J?.1 (Pin_1)
- new net: J?.2 (Pin_2), J?.2 (Pin_2)
- new net: J?.3 (Pin_3), J?.3 (Pin_3)
- new net: J?.4 (Pin_4), J?.4 (Pin_4)
- new net: J?.5 (Pin_5), J?.5 (Pin_5)
Other:
- moved on the sheet: J901, J902, J903
Changed lines of the file:
@@
 $Descr A4 11693 8268
 encoding utf-8
-Sheet 9 13
+Sheet 8 12
 Title ""
 Date ""
@@
 L Connector_Generic:Conn_01x05 J?
 U 1 1 5F96E4A9
-P 6000 2750
+P 6500 2750
 AR Path="/5F92F348/5F96E4A9" Ref="J?"  Part="1"
 AR Path="/5F92F3F9/5F96E4A9" Ref="J?"  Part="1"
 AR Path="/5F8F2E1B/5FA33522/5F96E4A9" Ref="J701"  Part="1"
 AR Path="/5F8F2E1B/5FA34085/5F96E4A9" Ref="J901"  Part="1"
-F 0 "J901" H 5918 3167 50  0000 C CNN
-F 1 "Male pitch strip 1x7 pins 2.0mm pitch" H 5918 3076 50  0000 C CNN
-F 2 "Connector_PinHeader_2.00mm:PinHeader_1x05_P2.00mm_Vertical" H 6000 2750 50  0001 C CNN
-F 3 "~" H 6000 2750 50  0001 C CNN
-F 4 "PWM_SUPPORTED_4STRIPS" H 6000 2750 50  0001 C CNN "Feature"
-F 5 "0.016" H 6000 2750 50  0001 C CNN "Price"
-F 6 "yes" H 6000 2750 50  0001 C CNN "is stock"
-	1    6000 2750
+F 0 "J901" H 6418 3167 50  0000 C CNN
+F 1 "Male pitch strip 1x7 pins 2.0mm pitch" H 6418 3076 50  0000 C CNN
+F 2 "Connector_PinHeader_2.00mm:PinHeader_1x05_P2.00mm_Vertical" H 6500 2750 50  0001 C CNN
+F 3 "~" H 6500 2750 50  0001 C CNN
+F 4 "PWM_SUPPORTED_4STRIPS" H 6500 2750 50  0001 C CNN "Feature"
+F 5 "0.016" H 6500 2750 50  0001 C CNN "Price"
+F 6 "yes" H 6500 2750 50  0001 C CNN "is stock"
+	1    6500 2750
 	-1   0    0    -1
 $EndComp
@@
 L Connector_Generic:Conn_01x05 J?
 U 1 1 5F96EB0B
-P 7500 2750
+P 8000 2750
 AR Path="/5F92F348/5F96EB0B" Ref="J?"  Part="1"
 AR Path="/5F92F3F9/5F96EB0B" Ref="J?"  Part="1"
 AR Path="/5F8F2E1B/5FA33522/5F96EB0B" Ref="J702"  Part="1"
 AR Path="/5F8F2E1B/5FA34085/5F96EB0B" Ref="J902"  Part="1"
-F 0 "J902" H 7450 3050 50  0000 L CNN
-F 1 "Conn_01x05" H 7450 3150 50  0000 L CNN
-F 2 "Connector_PinHeader_2.00mm:PinHeader_1x05_P2.00mm_Vertical" H 7500 2750 50  0001 C CNN
-F 3 "~" H 7500 2750 50  0001 C CNN
-F 4 "PWM_SUPPORTED_4STRIPS" H 7500 2750 50  0001 C CNN "Feature"
-F 5 "0" H 7500 2750 50  0001 C CNN "Price"
-F 6 "no" H 7500 2750 50  0001 C CNN "is stock"
-	1    7500 2750
+F 0 "J902" H 7950 3050 50  0000 L CNN
+F 1 "Conn_01x05" H 7950 3150 50  0000 L CNN
+F 2 "LedBarController:LED_Strip_10mm_5pins_Left" H 8000 2750 50  0001 C CNN
+F 3 "~" H 8000 2750 50  0001 C CNN
+F 4 "PWM_SUPPORTED_4STRIPS" H 8000 2750 50  0001 C CNN "Feature"
+F 5 "0" H 8000 2750 50  0001 C CNN "Price"
+F 6 "no" H 8000 2750 50  0001 C CNN "is stock"
+	1    8000 2750
 	1    0    0    -1
 $EndComp
@@
 L Connector_Generic:Conn_01x05 J?
 U 1 1 5F96F581
-P 7500 3750
+P 8000 3750
 AR Path="/5F92F348/5F96F581" Ref="J?"  Part="1"
 AR Path="/5F92F3F9/5F96F581" Ref="J?"  Part="1"
 AR Path="/5F8F2E1B/5FA33522/5F96F581" Ref="J703"  Part="1"
 AR Path="/5F8F2E1B/5FA34085/5F96F581" Ref="J903"  Part="1"
-F 0 "J903" H 7450 4050 50  0000 L CNN
-F 1 "Conn_01x05" H 7450 4150 50  0000 L CNN
-F 2 "Connector_PinHeader_2.00mm:PinHeader_1x05_P2.00mm_Vertical" H 7500 3750 50  0001 C CNN
-F 3 "~" H 7500 3750 50  0001 C CNN
-F 4 "PWM_SUPPORTED_4STRIPS" H 7500 3750 50  0001 C CNN "Feature"
-F 5 "0" H 7500 3750 50  0001 C CNN "Price"
-F 6 "no" H 7500 3750 50  0001 C CNN "is stock"
-	1    7500 3750
+F 0 "J903" H 7950 4050 50  0000 L CNN
+F 1 "Conn_01x05" H 7950 4150 50  0000 L CNN
+F 2 "LedBarController:LED_Strip_10mm_5pins_Left" H 8000 3750 50  0001 C CNN
+F 3 "~" H 8000 3750 50  0001 C CNN
+F 4 "PWM_SUPPORTED_4STRIPS" H 8000 3750 50  0001 C CNN "Feature"
+F 5 "0" H 8000 3750 50  0001 C CNN "Price"
+F 6 "no" H 8000 3750 50  0001 C CNN "is stock"
+	1    8000 3750
 	1    0    0    -1
 $EndComp
 Wire Wire Line
-	7300 2950 7200 2950
+	7800 2950 7700 2950
 Wire Wire Line
-	7200 2950 7200 3950
+	7700 2950 7700 3950
 Wire Wire Line
-	7200 3950 7300 3950
+	7700 3950 7800 3950
 Wire Wire Line
-	7300 3850 7100 3850
+	7800 3850 7600 3850
 Wire Wire Line
-	7100 3850 7100 2850
+	7600 3850 7600 2850
 Wire Wire Line
-	7100 2850 7300 2850
+	7600 2850 7800 2850
 Wire Wire Line
-	7300 2750 7000 2750
+	7800 2750 7500 2750
 Wire Wire Line
-	7000 2750 7000 3750
+	7500 2750 7500 3750
 Wire Wire Line
-	7000 3750 7300 3750
+	7500 3750 7800 3750
 Wire Wire Line
-	7300 3650 6900 3650
+	7800 3650 7400 3650
 Wire Wire Line
-	6900 3650 6900 2650
+	7400 3650 7400 2650
 Wire Wire Line
-	6900 2650 7300 2650
+	7400 2650 7800 2650
 Wire Wire Line
-	7300 3550 6800 3550
+	7800 3550 7300 3550
 Wire Wire Line
-	6800 2550 7300 2550
+	7300 2550 7800 2550
 Wire Wire Line
-	6200 2550 6800 2550
-Connection ~ 6800 2550
+	6700 2550 7300 2550
+Connection ~ 7300 2550
 Wire Wire Line
-	6800 3550 6800 2550
+	7300 3550 7300 2550
 Wire Wire Line
-	6200 2650 6900 2650
-Connection ~ 6900 2650
+	6700 2650 7400 2650
+Connection ~ 7400 2650
 Wire Wire Line
-	6200 2750 7000 2750
-Connection ~ 7000 2750
+	6700 2750 7500 2750
+Connection ~ 7500 2750
 Wire Wire Line
-	6200 2850 7100 2850
-Connection ~ 7100 2850
+	6700 2850 7600 2850
+Connection ~ 7600 2850
 Wire Wire Line
-	6200 2950 7200 2950
-Connection ~ 7200 2950
-Text Label 6250 2650 0    50   ~ 0
+	6700 2950 7700 2950
+Connection ~ 7700 2950
+Text Label 6750 2650 0    50   ~ 0
 green_
-Text Label 6250 2750 0    50   ~ 0
+Text Label 6750 2750 0    50   ~ 0
 red_
-Text Label 6250 2850 0    50   ~ 0
+Text Label 6750 2850 0    50   ~ 0
 blue_
-Text Label 6250 2950 0    50   ~ 0
+Text Label 6750 2950 0    50   ~ 0
 white_
-Text Label 6250 2550 0    50   ~ 0
+Text Label 6750 2550 0    50   ~ 0
 VDD_
+$Comp
+L Connector_Generic:Conn_01x05 J?
+U 1 1 5FC02B67
+P 4500 2750
+AR Path="/5F92F348/5FC02B67" Ref="J?"  Part="1"
+AR Path="/5F92F3F9/5FC02B67" Ref="J?"  Part="1"
+AR Path="/5F8F2E1B/5FA33522/5FC02B67" Ref="J?"  Part="1"
+AR Path="/5F8F2E1B/5FA34085/5FC02B67" Ref="J?"  Part="1"
+F 0 "J?" H 4418 3167 50  0000 C CNN
+F 1 "Male pitch strip 1x7 pins 2.0mm pitch" H 4418 3076 50  0000 C CNN
+F 2 "Connector_PinHeader_2.00mm:PinHeader_1x05_P2.00mm_Vertical" H 4500 2750 50  0001 C CNN
+F 3 "~" H 4500 2750 50  0001 C CNN
+F 4 "PWM_SUPPORTED_4STRIPS" H 4500 2750 50  0001 C CNN "Feature"
+F 5 "0.016" H 4500 2750 50  0001 C CNN "Price"
+F 6 "yes" H 4500 2750 50  0001 C CNN "is stock"
+	1    4500 2750
+	1    0    0    -1
+$EndComp
+$Comp
+L Connector_Generic:Conn_01x05 J?
+U 1 1 5FC037F4
+P 2500 2750
+AR Path="/5F92F348/5FC037F4" Ref="J?"  Part="1"
+AR Path="/5F92F3F9/5FC037F4" Ref="J?"  Part="1"
+AR Path="/5F8F2E1B/5FA33522/5FC037F4" Ref="J?"  Part="1"
+AR Path="/5F8F2E1B/5FA34085/5FC037F4" Ref="J?"  Part="1"
+F 0 "J?" H 2418 3167 50  0000 C CNN
+F 1 "Male pitch strip 1x7 pins 2.0mm pitch" H 2418 3076 50  0000 C CNN
+F 2 "Connector_PinHeader_2.00mm:PinHeader_1x05_P2.00mm_Vertical" H 2500 2750 50  0001 C CNN
+F 3 "~" H 2500 2750 50  0001 C CNN
+F 4 "PWM_SUPPORTED_4STRIPS" H 2500 2750 50  0001 C CNN "Feature"
+F 5 "0.016" H 2500 2750 50  0001 C CNN "Price"
+F 6 "yes" H 2500 2750 50  0001 C CNN "is stock"
+	1    2500 2750
+	-1   0    0    -1
+$EndComp
+Wire Wire Line
+	2700 2550 4300 2550
+Wire Wire Line
+	2700 2650 4300 2650
+Wire Wire Line
+	2700 2750 4300 2750
+Wire Wire Line
+	2700 2850 4300 2850
+Wire Wire Line
+	2700 2950 4300 2950
 $EndSCHEMATC
