File: LedBarController/CenterStrips.sch (KiCad schematic (older format))
At the start: 7 parts, among them J1201 Conn_02x07_Odd_Even, J1202 Conn_02x07_Odd_Even, J1203 Conn_01x05, J1204 Conn_01x05, J1205 Conn_01x05, J1206 Conn_01x05, SW1201 SW_Push

Commit message: Restarted PCB
Parts:
- removed J1201: Conn_02x07_Odd_Even, Connector_PinSocket_2.00mm:PinSocket_2x07_P2.00mm_Vertical, symbol Connector_Generic:Conn_02x07_Odd_Even
- renumbered J1203 to J801, J1202 to J802, J1205 to J803, J1204 to J804, J1206 to J805, SW1201 to SW801
Other:
- note removed: "Separate PCB"
- moved on the sheet: J801, J802, J803, J804, J805, SW801

Commit message: Changed components and moved center connector upwards
Parts:
- SW801: footprint Button_Switch_SMD:SW_Push_1P1T_NO_CK_KSC7xxJ -> Button_Switch_SMD:SW_SPST_SKQG_WithStem
Changed lines of the file:
@@
 $Descr A4 11693 8268
 encoding utf-8
-Sheet 12 13
+Sheet 8 13
 Title ""
 Date ""
@@
 F 0 "SW801" H 5500 4385 50  0000 C CNN
 F 1 "SW_Push" H 5500 4294 50  0000 C CNN
-F 2 "Button_Switch_SMD:SW_Push_1P1T_NO_CK_KSC7xxJ" H 5500 4300 50  0001 C CNN
+F 2 "Button_Switch_SMD:SW_SPST_SKQG_WithStem" H 5500 4300 50  0001 C CNN
 F 3 "~" H 5500 4300 50  0001 C CNN
 	1    5500 4100

Commit message: Work in progress
Parts:
- J801, J803, J804, J805: Feature (none) -> PWM_SUPPORTED_2STRIPS; Price (none) -> 0; is stock (none) -> no
- J802: value Conn_02x07_Odd_Even -> Male pitch strip 2x7pins 2.0mm pitch; Feature (none) -> PWM_SUPPORTED_2STRIPS; Price (none) -> 0.055; is stock (none) -> no
- SW801: value SW_Push -> 4x42.3mm PCB Tactile Push Button Switch; Feature (none) -> PWM_SUPPORTED_2STRIPS; Price (none) -> 0.0356; is stock (none) -> no
Changed lines of the file:
@@
 F 2 "Connector_PinHeader_2.00mm:PinHeader_1x05_P2.00mm_Vertical" H 7050 4350 50  0001 C CNN
 F 3 "~" H 7050 4350 50  0001 C CNN
+F 4 "PWM_SUPPORTED_2STRIPS" H 7050 4350 50  0001 C CNN "Feature"
+F 5 "0" H 7050 4350 50  0001 C CNN "Price"
+F 6 "no" H 7050 4350 50  0001 C CNN "is stock"
 	1    7050 4350
 	1    0    0    -1
@@
 F 2 "Connector_PinHeader_2.00mm:PinHeader_1x05_P2.00mm_Vertical" H 7050 3350 50  0001 C CNN
 F 3 "~" H 7050 3350 50  0001 C CNN
+F 4 "PWM_SUPPORTED_2STRIPS" H 7050 3350 50  0001 C CNN "Feature"
+F 5 "0" H 7050 3350 50  0001 C CNN "Price"
+F 6 "no" H 7050 3350 50  0001 C CNN "is stock"
 	1    7050 3350
 	1    0    0    -1
@@
 F 2 "Connector_PinHeader_2.00mm:PinHeader_1x05_P2.00mm_Vertical" H 3950 3350 50  0001 C CNN
 F 3 "~" H 3950 3350 50  0001 C CNN
+F 4 "PWM_SUPPORTED_2STRIPS" H 3950 3350 50  0001 C CNN "Feature"
+F 5 "0" H 3950 3350 50  0001 C CNN "Price"
+F 6 "no" H 3950 3350 50  0001 C CNN "is stock"
 	1    3950 3350
 	-1   0    0    -1
@@
 F 2 "Connector_PinHeader_2.00mm:PinHeader_1x05_P2.00mm_Vertical" H 3950 4350 50  0001 C CNN
 F 3 "~" H 3950 4350 50  0001 C CNN
+F 4 "PWM_SUPPORTED_2STRIPS" H 3950 4350 50  0001 C CNN "Feature"
+F 5 "0" H 3950 4350 50  0001 C CNN "Price"
+F 6 "no" H 3950 4350 50  0001 C CNN "is stock"
 	1    3950 4350
 	-1   0    0    -1
@@
 AR Path="/5F8F2E1B/5FA33E59/5F9BC931" Ref="SW801"  Part="1"
 F 0 "SW801" H 5500 4385 50  0000 C CNN
-F 1 "SW_Push" H 5500 4294 50  0000 C CNN
+F 1 "4x42.3mm PCB Tactile Push Button Switch" H 5500 4294 50  0000 C CNN
 F 2 "Button_Switch_SMD:SW_SPST_SKQG_WithStem" H 5500 4300 50  0001 C CNN
 F 3 "~" H 5500 4300 50  0001 C CNN
+F 4 "PWM_SUPPORTED_2STRIPS" H 5500 4100 50  0001 C CNN "Feature"
+F 5 "0.0356" H 5500 4100 50  0001 C CNN "Price"
+F 6 "no" H 5500 4100 50  0001 C CNN "is stock"
 	1    5500 4100
 	1    0    0    -1
@@
 AR Path="/5F8F2E1B/5FA33E59/5F9CBA33" Ref="J802"  Part="1"
 F 0 "J802" H 5500 3775 50  0000 C CNN
-F 1 "Conn_02x07_Odd_Even" H 5500 3776 50  0001 C CNN
+F 1 "Male pitch strip 2x7pins 2.0mm pitch" H 5500 3776 50  0001 C CNN
 F 2 "Connector_PinHeader_2.00mm:PinHeader_2x07_P2.00mm_Vertical" H 5450 3350 50  0001 C CNN
 F 3 "~" H 5450 3350 50  0001 C CNN
+F 4 "PWM_SUPPORTED_2STRIPS" H 5450 3350 50  0001 C CNN "Feature"
+F 5 "0.055" H 5450 3350 50  0001 C CNN "Price"
+F 6 "no" H 5450 3350 50  0001 C CNN "is stock"
 	1    5450 3350
 	1    0    0    -1

Commit message: Route complete
Connections:
- net button_ renamed ~button~_
Changed lines of the file:
@@
 AR Path="/5F92F971/5F9BC931" Ref="SW?"  Part="1"
 AR Path="/5F8F2E1B/5FA33E59/5F9BC931" Ref="SW801"  Part="1"
-F 0 "SW801" H 5500 4385 50  0000 C CNN
-F 1 "4x42.3mm PCB Tactile Push Button Switch" H 5500 4294 50  0000 C CNN
+F 0 "SW801" H 5500 4250 50  0000 C CNN
+F 1 "4x42.3mm PCB Tactile Push Button Switch" H 5500 4000 50  0000 C CNN
 F 2 "Button_Switch_SMD:SW_SPST_SKQG_WithStem" H 5500 4300 50  0001 C CNN
 F 3 "~" H 5500 4300 50  0001 C CNN
@@
 GND_
 Text Label 5200 3850 2    50   ~ 0
-button_
+~button~_
 $EndSCHEMATC

Commit message: moved board on schema to same sheet
Parts:
- added J701, J704, J901, J905: Male pitch strip 1x7 pins 2.0mm pitch, Connector_PinHeader_2.00mm:PinHeader_1x05_P2.00mm_Vertical, symbol Connector_Generic:Conn_01x05
- added J702, J703: Conn_01x05, LedBarController:LED_Strip_10mm_5pins_Left, symbol Connector_Generic:Conn_01x05
- added J705: Male pitch strip 1x7 pins 2.0mm pitch, LedBarController:LED_Strip_10mm_5pins_Right, symbol Connector_Generic:Conn_01x05
- added J902, J903: Conn_01x05, LedBarController:LED_Strip_10mm_5pins_Right, symbol Connector_Generic:Conn_01x05
- added J904: Male pitch strip 1x7 pins 2.0mm pitch, LedBarController:LED_Strip_10mm_5pins_Left, symbol Connector_Generic:Conn_01x05
- J801, J804: footprint Connector_PinHeader_2.00mm:PinHeader_1x05_P2.00mm_Vertical -> LedBarController:LED_Strip_10mm_5pins_Left
- J803, J805: footprint Connector_PinHeader_2.00mm:PinHeader_1x05_P2.00mm_Vertical -> LedBarController:LED_Strip_10mm_5pins_Right
Connections:
- net GND_ renamed ~button~
- net VDD_ renamed center_front_vdd
- net blue_left_ renamed center_front_l_blue
- net center_front_l_blue: now also J802.10 (Pin_10); no longer J802.9 (Pin_9)
- net blue_right_ renamed center_front_r_blue
- net center_front_r_blue: now also J802.9 (Pin_9); no longer J802.10 (Pin_10)
- net green_left_ renamed center_front_l_green
- net center_front_l_green: now also J802.6 (Pin_6); no longer J802.5 (Pin_5)
- net green_right_ renamed center_front_r_green
- net center_front_r_green: now also J802.5 (Pin_5); no longer J802.6 (Pin_6)
- net red_left_ renamed center_front_l_red
- net center_front_l_red: now also J802.8 (Pin_8); no longer J802.7 (Pin_7)
- net red_right_ renamed center_front_r_red
- net center_front_r_red: now also J802.7 (Pin_7); no longer J802.8 (Pin_8)
- net white_left_ renamed center_front_l_white
- net center_front_l_white: now also J802.12 (Pin_12); no longer J802.11 (Pin_11)
- net white_right_ renamed center_front_r_white
- net center_front_r_white: now also J802.11 (Pin_11); no longer J802.12 (Pin_12)
- net ~button~_ renamed gnd
- new net blue_left_front: J701.4 (Pin_4), J702.4 (Pin_4), J703.4 (Pin_4)
- new net left_back_blue: J704.4 (Pin_4), J705.4 (Pin_4)
- new net left_back_green: J704.2 (Pin_2), J705.2 (Pin_2)
- new net left_back_red: J704.3 (Pin_3), J705.3 (Pin_3)
- new net left_back_vdd: J704.1 (Pin_1), J705.1 (Pin_1)
- new net left_back_white: J704.5 (Pin_5), J705.5 (Pin_5)
- new net left_front_green: J701.2 (Pin_2), J702.2 (Pin_2), J703.2 (Pin_2)
- new net left_front_vdd: J701.1 (Pin_1), J702.1 (Pin_1), J703.1 (Pin_1)
- new net red_left_front: J701.3 (Pin_3), J702.3 (Pin_3), J703.3 (Pin_3)
- new net right_back_blue: J904.4 (Pin_4), J905.4 (Pin_4)
- new net right_back_green: J904.2 (Pin_2), J905.2 (Pin_2)
- new net right_back_red: J904.3 (Pin_3), J905.3 (Pin_3)
- new net right_back_vdd: J904.1 (Pin_1), J905.1 (Pin_1)
- new net right_back_white: J904.5 (Pin_5), J905.5 (Pin_5)
- new net right_front_blue: J901.4 (Pin_4), J902.4 (Pin_4), J903.4 (Pin_4)
- new net right_front_green: J901.2 (Pin_2), J902.2 (Pin_2), J903.2 (Pin_2)
- new net right_front_red: J901.3 (Pin_3), J902.3 (Pin_3), J903.3 (Pin_3)
- new net right_front_vdd: J901.1 (Pin_1), J902.1 (Pin_1), J903.1 (Pin_1)
- new net right_front_white: J901.5 (Pin_5), J902.5 (Pin_5), J903.5 (Pin_5)
- new net white_left_front: J701.5 (Pin_5), J702.5 (Pin_5), J703.5 (Pin_5)
Other:
- note added: "Board: Center Front"
- note added: "Board: Left Back"
- note added: "Board: Left Front"
- note added: "Board: Right Back"
- note added: "Board: Right Front"
- moved on the sheet: J801, J802, J803, J804, J805, SW801
