File: LedBarController/LedBarController.sch (KiCad schematic (older format))
At the start: 0 parts

Commit message: Restarted PCB
Changed lines of the file:
@@
 Comment4 ""
 $EndDescr
+Wire Wire Line
+	6800 3600 6500 3600
+Wire Wire Line
+	6800 2100 6800 3600
+Wire Wire Line
+	8000 2100 6800 2100
+Wire Wire Line
+	6900 2200 8000 2200
+Wire Wire Line
+	6900 3700 6900 2200
+Wire Wire Line
+	6500 3700 6900 3700
+Wire Wire Line
+	7100 2400 8000 2400
+Wire Wire Line
+	7100 3900 7100 2400
+Wire Wire Line
+	6500 3900 7100 3900
+Wire Wire Line
+	7500 3850 7500 4250
+Wire Wire Line
+	8000 3850 7500 3850
+Wire Wire Line
+	6500 4250 7500 4250
 $Sheet
-S 2000 4000 1000 500
+S 8000 2000 1000 2000
+U 5F8F2E1B
+F0 "PWM" 50
+F1 "PWM.sch" 50
+F2 "~OE" I L 8000 2400 50
+F3 "I2C_SDA" B L 8000 2200 50
+F4 "I2C_SCL" O L 8000 2100 50
+F5 "button" O L 8000 3850 50
+$EndSheet
+Wire Wire Line
+	6500 4900 8000 4900
+Wire Wire Line
+	6500 4800 8000 4800
+Wire Wire Line
+	6500 4700 8000 4700
+Wire Wire Line
+	6500 4600 8000 4600
+Wire Wire Line
+	4500 3700 5500 3700
+Wire Wire Line
+	4500 3600 5500 3600
+$Sheet
+S 5500 3500 1000 1500
+U 5F829319
+F0 "Microcontroller" 50
+F1 "Microcontroller.sch" 50
+F2 "Rx" I L 5500 3600 50
+F3 "Tx" O L 5500 3700 50
+F4 "TxEn" O L 5500 3900 50
+F5 "I2C_SDA" B R 6500 3700 50
+F6 "I2C_SCL" O R 6500 3600 50
+F7 "~PWM_OE" O R 6500 3900 50
+F8 "0_10V_dout_1" O R 6500 4600 50
+F9 "0_10V_dout_2" O R 6500 4800 50
+F10 "0_10V_ain_1" I R 6500 4700 50
+F11 "0_10V_ain_2" I R 6500 4900 50
+F12 "button" I R 6500 4250 50
+$EndSheet
+Wire Wire Line
+	4500 3900 5500 3900
+$Sheet
+S 8000 4500 1000 500
+U 5F8293F0
+F0 "0-10V" 50
+F1 "0-10V.sch" 50
+F2 "0-10Vd1" I L 8000 4600 50
+F3 "0-10Va1" O L 8000 4700 50
+F4 "0-10Vd2" I L 8000 4800 50
+F5 "0-10Va2" O L 8000 4900 50
+$EndSheet
+$Sheet
+S 3500 2000 1000 500
+U 5F7C8D58
+F0 "Power" 50
+F1 "Power.sch" 50
+$EndSheet
+$Sheet
+S 3500 3500 1000 500
 U 5F7B7D30
 F0 "RS485" 50
 F1 "RS485.sch" 50
-F2 "TxEn" I R 3000 4400 50
-F3 "Rx" O R 3000 4100 50
-F4 "Tx" I R 3000 4200 50
+F2 "TxEn" I R 4500 3900 50
+F3 "Rx" O R 4500 3600 50
+F4 "Tx" I R 4500 3700 50
 $EndSheet
-$Sheet
-S 2000 5000 1000 500
-U 5F7C8D58
-F0 "Power" 50
-F1 "Power.sch" 50
-F2 "ADC1" O R 3000 5250 50
-$EndSheet
-$Sheet
-S 6500 5000 1000 500
-U 5F8293F0
-F0 "0-10V" 50
-F1 "0-10V.sch" 50
-F2 "0-10Vd1" I L 6500 5100 50
-F3 "0-10Va1" O L 6500 5200 50
-F4 "0-10Vd2" I L 6500 5300 50
-F5 "0-10Va2" O L 6500 5400 50
-$EndSheet
-Wire Wire Line
-	3000 4400 4000 4400
-Wire Wire Line
-	3000 5250 3500 5250
-Wire Wire Line
-	3500 5250 3500 4800
-Wire Wire Line
-	3500 4800 4000 4800
-$Sheet
-S 4000 4000 1000 1500
-U 5F829319
-F0 "Microcontroller" 50
-F1 "Microcontroller.sch" 50
-F2 "Rx" I L 4000 4100 50
-F3 "Tx" O L 4000 4200 50
-F4 "TxEn" O L 4000 4400 50
-F5 "I2C_SDA" B R 5000 4200 50
-F6 "I2C_SCL" O R 5000 4100 50
-F7 "~PWM_OE" O R 5000 4400 50
-F8 "ADC1" I L 4000 4800 50
-F9 "0_10V_dout_1" O R 5000 5100 50
-F10 "0_10V_dout_2" O R 5000 5300 50
-F11 "0_10V_ain_1" I R 5000 5200 50
-F12 "0_10V_ain_2" I R 5000 5400 50
-F13 "button" I R 5000 4750 50
-$EndSheet
-Wire Wire Line
-	3000 4100 4000 4100
-Wire Wire Line
-	3000 4200 4000 4200
-$Sheet
-S 6500 2500 1000 2000
-U 5F8F2E1B
-F0 "PWM" 50
-F1 "PWM.sch" 50
-F2 "strip1_r_out" O R 7500 2600 50
-F3 "strip1_g_out" O R 7500 2700 50
-F4 "strip1_b_out" O R 7500 2800 50
-F5 "strip1_w_out" O R 7500 2900 50
-F6 "~OE" I L 6500 4400 50
-F7 "I2C_SDA" B L 6500 4200 50
-F8 "I2C_SCL" O L 6500 4100 50
-F9 "strip2_r_out" O R 7500 3100 50
-F10 "strip2_g_out" O R 7500 3200 50
-F11 "strip2_b_out" O R 7500 3300 50
-F12 "strip2_w_out" O R 7500 3400 50
-F13 "strip3_r_out" O R 7500 3600 50
-F14 "strip3_g_out" O R 7500 3700 50
-F15 "strip3_b_out" O R 7500 3800 50
-F16 "strip3_w_out" O R 7500 3900 50
-F17 "strip4_r_out" O R 7500 4100 50
-F18 "strip4_g_out" O R 7500 4200 50
-F19 "strip4_b_out" O R 7500 4300 50
-F20 "strip4_w_out" O R 7500 4400 50
-$EndSheet
-$Sheet
-S 9500 5000 1000 500
-U 5F92F3F9
-F0 "SideStrip_right" 50
-F1 "SideStrip.sch" 50
-F2 "red" I L 9500 5100 50
-F3 "green" I L 9500 5200 50
-F4 "blue" I L 9500 5300 50
-F5 "white" I L 9500 5400 50
-$EndSheet
-$Sheet
-S 9500 3000 1000 1500
-U 5F92F971
-F0 "CenterStrips" 50
-F1 "CenterStrips.sch" 50
-F2 "red_left" I L 9500 3100 50
-F3 "green_left" I L 9500 3200 50
-F4 "blue_left" I L 9500 3300 50
-F5 "while_left" I L 9500 3400 50
-F6 "red_right" I L 9500 3600 50
-F7 "green_right" I L 9500 3700 50
-F8 "blue_right" I L 9500 3800 50
-F9 "white_right" I L 9500 3900 50
-F10 "button" O L 9500 4400 50
-$EndSheet
-Wire Wire Line
-	8200 2600 8200 2100
-Wire Wire Line
-	8200 2100 9500 2100
-Wire Wire Line
-	8300 2700 8300 2200
-Wire Wire Line
-	8300 2200 9500 2200
-Wire Wire Line
-	8400 2800 8400 2300
-Wire Wire Line
-	8400 2300 9500 2300
-Wire Wire Line
-	8500 2900 8500 2400
-Wire Wire Line
-	8500 2400 9500 2400
-Wire Wire Line
-	8200 4400 8200 5400
-Wire Wire Line
-	8200 5400 9500 5400
-Wire Wire Line
-	8300 4300 8300 5300
-Wire Wire Line
-	8300 5300 9500 5300
-Wire Wire Line
-	8400 4200 8400 5200
-Wire Wire Line
-	8400 5200 9500 5200
-Wire Wire Line
-	8500 4100 8500 5100
-Wire Wire Line
-	8500 5100 9500 5100
-$Sheet
-S 9500 2000 1000 500
-U 5F92F348
-F0 "SideStrip_left" 50
-F1 "SideStrip.sch" 50
-F2 "red" I L 9500 2100 50
-F3 "green" I L 9500 2200 50
-F4 "blue" I L 9500 2300 50
-F5 "white" I L 9500 2400 50
-$EndSheet
-Wire Wire Line
-	5000 4100 6500 4100
-Wire Wire Line
-	5000 4200 6500 4200
-Wire Wire Line
-	5000 4400 6500 4400
-Wire Wire Line
-	5000 4750 9000 4750
-Wire Wire Line
-	9000 4750 9000 4400
-Wire Wire Line
-	9000 4400 9500 4400
-Wire Wire Line
-	5000 5100 6500 5100
-Wire Wire Line
-	5000 5200 6500 5200
-Wire Wire Line
-	5000 5300 6500 5300
-Wire Wire Line
-	5000 5400 6500 5400
-Wire Wire Line
-	7500 2600 8200 2600
-Wire Wire Line
-	7500 2700 8300 2700
-Wire Wire Line
-	7500 2800 8400 2800
-Wire Wire Line
-	7500 2900 8500 2900
-Wire Wire Line
-	7500 3100 9500 3100
-Wire Wire Line
-	7500 3200 9500 3200
-Wire Wire Line
-	7500 3300 9500 3300
-Wire Wire Line
-	7500 3400 9500 3400
-Wire Wire Line
-	7500 3600 9500 3600
-Wire Wire Line
-	7500 3700 9500 3700
-Wire Wire Line
-	7500 3800 9500 3800
-Wire Wire Line
-	7500 3900 9500 3900
-Wire Wire Line
-	7500 4100 8500 4100
-Wire Wire Line
-	7500 4200 8400 4200
-Wire Wire Line
-	7500 4300 8300 4300
-Wire Wire Line
-	7500 4400 8200 4400
 $EndSCHEMATC

Commit message: Updated schematic, added ds1307, replaced gpio-headers for LEDs and solder-jumpers and remove ISP-connector
Changed lines of the file:
@@
 F0 "Microcontroller" 50
 F1 "Microcontroller.sch" 50
-F2 "Rx" I L 5500 3600 50
-F3 "Tx" O L 5500 3700 50
-F4 "TxEn" O L 5500 3900 50
-F5 "I2C_SDA" B R 6500 3700 50
-F6 "I2C_SCL" O R 6500 3600 50
-F7 "~PWM_OE" O R 6500 3900 50
-F8 "0_10V_dout_1" O R 6500 4600 50
-F9 "0_10V_dout_2" O R 6500 4800 50
-F10 "0_10V_ain_1" I R 6500 4700 50
-F11 "0_10V_ain_2" I R 6500 4900 50
+F2 "txd" O L 5500 3700 50
+F3 "I2C_SDA" B R 6500 3700 50
+F4 "I2C_SCL" O R 6500 3600 50
+F5 "~pwm_OE" O R 6500 3900 50
+F6 "0_10v_dout_1" O R 6500 4600 50
+F7 "0_10v_dout_2" O R 6500 4800 50
+F8 "0_10v_ain_1" I R 6500 4700 50
+F9 "0_10v_ain_2" I R 6500 4900 50
+F10 "rxd" I L 5500 3600 50
+F11 "tx_en" O L 5500 3900 50
 F12 "button" I R 6500 4250 50
 $EndSheet

Commit message: Updated labels in schematic and moved RTC to sub-schematic
Changed lines of the file:
@@
 $Descr A4 11693 8268
 encoding utf-8
-Sheet 1 13
+Sheet 1 14
 Title ""
 Date ""
@@
 $EndDescr
 Wire Wire Line
-	6800 3600 6500 3600
+	7200 3600 6300 3600
 Wire Wire Line
-	6800 2100 6800 3600
+	7200 2100 7200 3600
 Wire Wire Line
-	8000 2100 6800 2100
+	8000 2100 7200 2100
 Wire Wire Line
-	6900 2200 8000 2200
+	7300 2200 8000 2200
 Wire Wire Line
-	6900 3700 6900 2200
+	7300 3700 7300 2200
 Wire Wire Line
-	6500 3700 6900 3700
+	6300 3700 7300 3700
 Wire Wire Line
-	7100 2400 8000 2400
+	7500 2400 8000 2400
 Wire Wire Line
-	7100 3900 7100 2400
+	7500 3900 7500 2400
 Wire Wire Line
-	6500 3900 7100 3900
+	6300 3900 7500 3900
 Wire Wire Line
-	7500 3850 7500 4250
+	7700 3850 7700 4250
 Wire Wire Line
-	8000 3850 7500 3850
+	8000 3850 7700 3850
 Wire Wire Line
-	6500 4250 7500 4250
+	6300 4250 7700 4250
 $Sheet
 S 8000 2000 1000 2000
@@
 F0 "PWM" 50
 F1 "PWM.sch" 50
-F2 "~OE" I L 8000 2400 50
-F3 "I2C_SDA" B L 8000 2200 50
-F4 "I2C_SCL" O L 8000 2100 50
-F5 "button" O L 8000 3850 50
+F2 "button" O L 8000 3850 50
+F3 "~oe" I L 8000 2400 50
+F4 "sda" B L 8000 2200 50
+F5 "scl" O L 8000 2100 50
 $EndSheet
 Wire Wire Line
-	6500 4900 8000 4900
+	4500 3700 5300 3700
 Wire Wire Line
-	6500 4800 8000 4800
-Wire Wire Line
-	6500 4700 8000 4700
-Wire Wire Line
-	6500 4600 8000 4600
-Wire Wire Line
-	4500 3700 5500 3700
-Wire Wire Line
-	4500 3600 5500 3600
+	4500 3600 5300 3600
 $Sheet
-S 5500 3500 1000 1500
+S 5300 3500 1000 1750
 U 5F829319
 F0 "Microcontroller" 50
 F1 "Microcontroller.sch" 50
-F2 "txd" O L 5500 3700 50
-F3 "I2C_SDA" B R 6500 3700 50
-F4 "I2C_SCL" O R 6500 3600 50
-F5 "~pwm_OE" O R 6500 3900 50
-F6 "0_10v_dout_1" O R 6500 4600 50
-F7 "0_10v_dout_2" O R 6500 4800 50
-F8 "0_10v_ain_1" I R 6500 4700 50
-F9 "0_10v_ain_2" I R 6500 4900 50
-F10 "rxd" I L 5500 3600 50
-F11 "tx_en" O L 5500 3900 50
-F12 "button" I R 6500 4250 50
+F2 "txd" O L 5300 3700 50
+F3 "0_10v_dout_1" O R 6300 4800 50
+F4 "0_10v_dout_2" O R 6300 5000 50
+F5 "0_10v_ain_1" I R 6300 4900 50
+F6 "0_10v_ain_2" I R 6300 5100 50
+F7 "rxd" I L 5300 3600 50
+F8 "tx_en" O L 5300 3900 50
+F9 "button" I R 6300 4250 50
+F10 "scl" O R 6300 3600 50
+F11 "sda" B R 6300 3700 50
+F12 "rtc_sqw" O R 6300 4450 50
+F13 "~pwm_oe" O R 6300 3900 50
 $EndSheet
 Wire Wire Line
-	4500 3900 5500 3900
+	4500 3900 5300 3900
 $Sheet
-S 8000 4500 1000 500
+S 8000 5500 1000 500
 U 5F8293F0
 F0 "0-10V" 50
 F1 "0-10V.sch" 50
-F2 "0-10Vd1" I L 8000 4600 50
-F3 "0-10Va1" O L 8000 4700 50
-F4 "0-10Vd2" I L 8000 4800 50
-F5 "0-10Va2" O L 8000 4900 50
+F2 "dout_1" I L 8000 5600 50
+F3 "ain_1" O L 8000 5700 50
+F4 "ain_2" O L 8000 5900 50
+F5 "dout_2" I L 8000 5800 50
 $EndSheet
 $Sheet
@@
 F0 "RS485" 50
 F1 "RS485.sch" 50
-F2 "TxEn" I R 4500 3900 50
-F3 "Rx" O R 4500 3600 50
-F4 "Tx" I R 4500 3700 50
+F2 "tx_en" I R 4500 3900 50
+F3 "txd" I R 4500 3700 50
+F4 "rxd" O R 4500 3600 50
+$EndSheet
+Wire Wire Line
+	7300 3700 7300 4700
+Wire Wire Line
+	7300 4700 8000 4700
+Connection ~ 7300 3700
+Wire Wire Line
+	7200 3600 7200 4600
+Wire Wire Line
+	7200 4600 8000 4600
+Connection ~ 7200 3600
+Wire Wire Line
+	6300 4450 7000 4450
+Wire Wire Line
+	7000 4450 7000 4900
+Wire Wire Line
+	7000 4900 8000 4900
+Wire Wire Line
+	6300 4800 6800 4800
+Wire Wire Line
+	6800 4800 6800 5600
+Wire Wire Line
+	6800 5600 8000 5600
+Wire Wire Line
+	6300 4900 6700 4900
+Wire Wire Line
+	6700 4900 6700 5700
+Wire Wire Line
+	6700 5700 8000 5700
+Wire Wire Line
+	6300 5000 6600 5000
+Wire Wire Line
+	6600 5000 6600 5800
+Wire Wire Line
+	6600 5800 8000 5800
+Wire Wire Line
+	6300 5100 6500 5100
+Wire Wire Line
+	6500 5100 6500 5900
+Wire Wire Line
+	6500 5900 8000 5900
+$Sheet
+S 8000 4500 1000 500
+U 5FDC6C57
+F0 "RTC" 50
+F1 "RTC.sch" 50
+F2 "sqw" O L 8000 4900 50
+F3 "scl" I L 8000 4600 50
+F4 "sda" B L 8000 4700 50
 $EndSheet
 $EndSCHEMATC

Commit message: Added INA219 current/voltage sensor
Changed lines of the file:
@@
 F0 "Power" 50
 F1 "Power.sch" 50
+F2 "scl" I R 4500 2100 50
+F3 "sda" B R 4500 2200 50
 $EndSheet
 $Sheet
@@
 F4 "sda" B L 8000 4700 50
 $EndSheet
+Wire Wire Line
+	7200 2100 4500 2100
+Connection ~ 7200 2100
+Wire Wire Line
+	4500 2200 7300 2200
+Connection ~ 7300 2200
 $EndSCHEMATC

Commit message: Reduced circuit by remove extra features. Routed whole board. Needs refinement
Changed lines of the file:
@@
 $Descr A4 11693 8268
 encoding utf-8
-Sheet 1 14
+Sheet 1 13
 Title ""
 Date ""
@@
 F2 "txd" O L 5300 3700 50
 F3 "0_10v_dout_1" O R 6300 4800 50
-F4 "0_10v_dout_2" O R 6300 5000 50
-F5 "0_10v_ain_1" I R 6300 4900 50
-F6 "0_10v_ain_2" I R 6300 5100 50
-F7 "rxd" I L 5300 3600 50
-F8 "tx_en" O L 5300 3900 50
-F9 "button" I R 6300 4250 50
-F10 "scl" O R 6300 3600 50
-F11 "sda" B R 6300 3700 50
-F12 "rtc_sqw" O R 6300 4450 50
-F13 "~pwm_oe" O R 6300 3900 50
+F4 "0_10v_ain_1" I R 6300 4900 50
+F5 "rxd" I L 5300 3600 50
+F6 "tx_en" O L 5300 3900 50
+F7 "button" I R 6300 4250 50
+F8 "scl" O R 6300 3600 50
+F9 "sda" B R 6300 3700 50
+F10 "~pwm_oe" O R 6300 3900 50
 $EndSheet
 Wire Wire Line
 	4500 3900 5300 3900
-$Sheet
-S 8000 5500 1000 500
-U 5F8293F0
-F0 "0-10V" 50
-F1 "0-10V.sch" 50
-F2 "dout_1" I L 8000 5600 50
-F3 "ain_1" O L 8000 5700 50
-F4 "ain_2" O L 8000 5900 50
-F5 "dout_2" I L 8000 5800 50
-$EndSheet
 $Sheet
 S 3500 2000 1000 500
@@
 $EndSheet
 Wire Wire Line
-	7300 3700 7300 4700
-Wire Wire Line
-	7300 4700 8000 4700
-Connection ~ 7300 3700
-Wire Wire Line
-	7200 3600 7200 4600
-Wire Wire Line
-	7200 4600 8000 4600
-Connection ~ 7200 3600
-Wire Wire Line
-	6300 4450 7000 4450
-Wire Wire Line
-	7000 4450 7000 4900
-Wire Wire Line
-	7000 4900 8000 4900
-Wire Wire Line
 	6300 4800 6800 4800
 Wire Wire Line
@@
 	6700 5700 8000 5700
 Wire Wire Line
-	6300 5000 6600 5000
-Wire Wire Line
-	6600 5000 6600 5800
-Wire Wire Line
-	6600 5800 8000 5800
-Wire Wire Line
-	6300 5100 6500 5100
-Wire Wire Line
-	6500 5100 6500 5900
-Wire Wire Line
-	6500 5900 8000 5900
-$Sheet
-S 8000 4500 1000 500
-U 5FDC6C57
-F0 "RTC" 50
-F1 "RTC.sch" 50
-F2 "sqw" O L 8000 4900 50
-F3 "scl" I L 8000 4600 50
-F4 "sda" B L 8000 4700 50
-$EndSheet
-Wire Wire Line
 	7200 2100 4500 2100
 Connection ~ 7200 2100
@@
 	4500 2200 7300 2200
 Connection ~ 7300 2200
+$Sheet
+S 8000 5500 1000 500
+U 5F8293F0
+F0 "0-10V" 50
+F1 "0-10V.sch" 50
+F2 "dout_1" I L 8000 5600 50
+F3 "ain_1" O L 8000 5700 50
+$EndSheet
 $EndSCHEMATC

Commit message: Route complete
Changed lines of the file:
@@
 F0 "PWM" 50
 F1 "PWM.sch" 50
-F2 "button" O L 8000 3850 50
-F3 "~oe" I L 8000 2400 50
-F4 "sda" B L 8000 2200 50
-F5 "scl" O L 8000 2100 50
+F2 "~oe" I L 8000 2400 50
+F3 "sda" B L 8000 2200 50
+F4 "scl" O L 8000 2100 50
+F5 "~button~" O L 8000 3850 50
 $EndSheet
 Wire Wire Line
@@
 F1 "Microcontroller.sch" 50
 F2 "txd" O L 5300 3700 50
-F3 "0_10v_dout_1" O R 6300 4800 50
-F4 "0_10v_ain_1" I R 6300 4900 50
-F5 "rxd" I L 5300 3600 50
-F6 "tx_en" O L 5300 3900 50
-F7 "button" I R 6300 4250 50
-F8 "scl" O R 6300 3600 50
-F9 "sda" B R 6300 3700 50
-F10 "~pwm_oe" O R 6300 3900 50
+F3 "rxd" I L 5300 3600 50
+F4 "tx_en" O L 5300 3900 50
+F5 "scl" O R 6300 3600 50
+F6 "sda" B R 6300 3700 50
+F7 "~pwm_oe" O R 6300 3900 50
+F8 "pwm1" O R 6300 4800 50
+F9 "pwm2" O R 6300 4900 50
+F10 "~button~" I R 6300 4250 50
 $EndSheet
 Wire Wire Line
@@
 F0 "0-10V" 50
 F1 "0-10V.sch" 50
-F2 "dout_1" I L 8000 5600 50
-F3 "ain_1" O L 8000 5700 50
+F2 "pwm1" I L 8000 5600 50
+F3 "pwm2" I L 8000 5700 50
 $EndSheet
 $EndSCHEMATC
