File: LedBarController/LedBarController.sch (KiCad schematic (older format))
At the start: 0 parts

Commit message: Rearanged sheets
Parts:
- added J701, J704, J901, J905: Male pitch strip 1x7 pins 2.0mm pitch, Connector_PinHeader_2.00mm:PinHeader_1x05_P2.00mm_Vertical, symbol Connector_Generic:Conn_01x05
- added J702, J703, J801, J804: Conn_01x05, LedBarController:LED_Strip_10mm_5pins_Left, symbol Connector_Generic:Conn_01x05
- added J705: Male pitch strip 1x7 pins 2.0mm pitch, LedBarController:LED_Strip_10mm_5pins_Right, symbol Connector_Generic:Conn_01x05
- added J802: Male pitch strip 2x7pins 2.0mm pitch, Connector_PinHeader_2.00mm:PinHeader_2x07_P2.00mm_Vertical, symbol Connector_Generic:Conn_02x07_Odd_Even
- added J803, J805, J902, J903: Conn_01x05, LedBarController:LED_Strip_10mm_5pins_Right, symbol Connector_Generic:Conn_01x05
- added J904: Male pitch strip 1x7 pins 2.0mm pitch, LedBarController:LED_Strip_10mm_5pins_Left, symbol Connector_Generic:Conn_01x05
- added SW801: 4x42.3mm PCB Tactile Push Button Switch, Button_Switch_SMD:SW_SPST_SKQG_WithStem, symbol Switch:SW_Push
Connections:
- new net blue_left_front: J701.4 (Pin_4), J702.4 (Pin_4), J703.4 (Pin_4)
- new net center_front_l_blue: J801.4 (Pin_4), J802.10 (Pin_10), J804.4 (Pin_4)
- new net center_front_l_green: J801.2 (Pin_2), J802.6 (Pin_6), J804.2 (Pin_2)
- new net center_front_l_red: J801.3 (Pin_3), J802.8 (Pin_8), J804.3 (Pin_3)
- new net center_front_l_white: J801.5 (Pin_5), J802.12 (Pin_12), J804.5 (Pin_5)
- new net center_front_r_blue: J802.9 (Pin_9), J803.4 (Pin_4), J805.4 (Pin_4)
- new net center_front_r_green: J802.5 (Pin_5), J803.2 (Pin_2), J805.2 (Pin_2)
- new net center_front_r_red: J802.7 (Pin_7), J803.3 (Pin_3), J805.3 (Pin_3)
- new net center_front_r_white: J802.11 (Pin_11), J803.5 (Pin_5), J805.5 (Pin_5)
- new net center_front_vdd: J801.1 (Pin_1), J802.1 (Pin_1), J802.2 (Pin_2), J802.3 (Pin_3), J802.4 (Pin_4), J803.1 (Pin_1), J804.1 (Pin_1), J805.1 (Pin_1)
- new net gnd: J802.13 (Pin_13), SW801.1
- new net left_back_blue: J704.4 (Pin_4), J705.4 (Pin_4)
- new net left_back_green: J704.2 (Pin_2), J705.2 (Pin_2)
- new net left_back_red: J704.3 (Pin_3), J705.3 (Pin_3)
- new net left_back_vdd: J704.1 (Pin_1), J705.1 (Pin_1)
- new net left_back_white: J704.5 (Pin_5), J705.5 (Pin_5)
- new net left_front_green: J701.2 (Pin_2), J702.2 (Pin_2), J703.2 (Pin_2)
- new net left_front_vdd: J701.1 (Pin_1), J702.1 (Pin_1), J703.1 (Pin_1)
- new net red_left_front: J701.3 (Pin_3), J702.3 (Pin_3), J703.3 (Pin_3)
- new net right_back_blue: J904.4 (Pin_4), J905.4 (Pin_4)
- new net right_back_green: J904.2 (Pin_2), J905.2 (Pin_2)
- new net right_back_red: J904.3 (Pin_3), J905.3 (Pin_3)
- new net right_back_vdd: J904.1 (Pin_1), J905.1 (Pin_1)
- new net right_back_white: J904.5 (Pin_5), J905.5 (Pin_5)
- new net right_front_blue: J901.4 (Pin_4), J902.4 (Pin_4), J903.4 (Pin_4)
- new net right_front_green: J901.2 (Pin_2), J902.2 (Pin_2), J903.2 (Pin_2)
- new net right_front_red: J901.3 (Pin_3), J902.3 (Pin_3), J903.3 (Pin_3)
- new net right_front_vdd: J901.1 (Pin_1), J902.1 (Pin_1), J903.1 (Pin_1)
- new net right_front_white: J901.5 (Pin_5), J902.5 (Pin_5), J903.5 (Pin_5)
- new net white_left_front: J701.5 (Pin_5), J702.5 (Pin_5), J703.5 (Pin_5)
- new net ~button~: J802.14 (Pin_14), SW801.2
Other:
- note added: "Board: Center Front"
- note added: "Board: Left Back"
- note added: "Board: Left Front"
- note added: "Board: Right Back"
- note added: "Board: Right Front"

Commit message: Reanotate
Parts:
- renumbered J704 to J101, J705 to J102, J904 to J103, J905 to J104, J702 to J105, J701 to J106, J801 to J107, J802 to J108, J803 to J109, J901 to J110, J902 to J111, J703 to J112, J804 to J113, J805 to J114, J903 to J115, SW801 to SW101
Changed lines of the file:
@@
 AR Path="/5F92F971/602EA7CB" Ref="J?"  Part="1"
 AR Path="/5F8F2E1B/5FA33E59/602EA7CB" Ref="J?"  Part="1"
-AR Path="/602EA7CB" Ref="J805"  Part="1"
-F 0 "J805" H 7850 5800 50  0000 L CNN
+AR Path="/602EA7CB" Ref="J114"  Part="1"
+F 0 "J114" H 7850 5800 50  0000 L CNN
 F 1 "Conn_01x05" H 8030 5451 50  0001 L CNN
 F 2 "LedBarController:LED_Strip_10mm_5pins_Right" H 7950 5500 50  0001 C CNN
@@
 AR Path="/5F92F971/602EA7D4" Ref="J?"  Part="1"
 AR Path="/5F8F2E1B/5FA33E59/602EA7D4" Ref="J?"  Part="1"
-AR Path="/602EA7D4" Ref="J803"  Part="1"
-F 0 "J803" H 7850 4800 50  0000 L CNN
+AR Path="/602EA7D4" Ref="J109"  Part="1"
+F 0 "J109" H 7850 4800 50  0000 L CNN
 F 1 "Conn_01x05" H 8030 4451 50  0001 L CNN
 F 2 "LedBarController:LED_Strip_10mm_5pins_Right" H 7950 4500 50  0001 C CNN
@@
 AR Path="/5F92F971/602EA7DD" Ref="J?"  Part="1"
 AR Path="/5F8F2E1B/5FA33E59/602EA7DD" Ref="J?"  Part="1"
-AR Path="/602EA7DD" Ref="J801"  Part="1"
-F 0 "J801" H 4100 4800 50  0000 C CNN
+AR Path="/602EA7DD" Ref="J107"  Part="1"
+F 0 "J107" H 4100 4800 50  0000 C CNN
 F 1 "Conn_01x05" H 4018 4826 50  0001 C CNN
 F 2 "LedBarController:LED_Strip_10mm_5pins_Left" H 4100 4500 50  0001 C CNN
@@
 AR Path="/5F92F971/602EA7E6" Ref="J?"  Part="1"
 AR Path="/5F8F2E1B/5FA33E59/602EA7E6" Ref="J?"  Part="1"
-AR Path="/602EA7E6" Ref="J804"  Part="1"
-F 0 "J804" H 4100 5800 50  0000 C CNN
+AR Path="/602EA7E6" Ref="J113"  Part="1"
+F 0 "J113" H 4100 5800 50  0000 C CNN
 F 1 "Conn_01x05" H 4018 5826 50  0001 C CNN
 F 2 "LedBarController:LED_Strip_10mm_5pins_Left" H 4100 5500 50  0001 C CNN
@@
 AR Path="/5F92F971/602EA81D" Ref="SW?"  Part="1"
 AR Path="/5F8F2E1B/5FA33E59/602EA81D" Ref="SW?"  Part="1"
-AR Path="/602EA81D" Ref="SW801"  Part="1"
-F 0 "SW801" H 6000 5400 50  0000 C CNN
+AR Path="/602EA81D" Ref="SW101"  Part="1"
+F 0 "SW101" H 6000 5400 50  0000 C CNN
 F 1 "4x42.3mm PCB Tactile Push Button Switch" H 6000 5150 50  0001 C CNN
 F 2 "Button_Switch_SMD:SW_SPST_SKQG_WithStem" H 6000 5450 50  0001 C CNN
@@
 AR Path="/5F92F971/602EA826" Ref="J?"  Part="1"
 AR Path="/5F8F2E1B/5FA33E59/602EA826" Ref="J?"  Part="1"
-AR Path="/602EA826" Ref="J802"  Part="1"
-F 0 "J802" H 6100 4925 50  0000 C CNN
+AR Path="/602EA826" Ref="J108"  Part="1"
+F 0 "J108" H 6100 4925 50  0000 C CNN
 F 1 "Male pitch strip 2x7pins 2.0mm pitch" H 6100 4926 50  0001 C CNN
 F 2 "Connector_PinHeader_2.00mm:PinHeader_2x07_P2.00mm_Vertical" H 6050 4500 50  0001 C CNN
@@
 AR Path="/5F8F2E1B/5FA34085/602EA83F" Ref="J?"  Part="1"
 AR Path="/5F8F2E1B/5FA33E59/602EA83F" Ref="J?"  Part="1"
-AR Path="/602EA83F" Ref="J701"  Part="1"
-F 0 "J701" H 2850 4800 50  0000 C CNN
+AR Path="/602EA83F" Ref="J106"  Part="1"
+F 0 "J106" H 2850 4800 50  0000 C CNN
 F 1 "Male pitch strip 1x7 pins 2.0mm pitch" H 2768 4826 50  0001 C CNN
 F 2 "Connector_PinHeader_2.00mm:PinHeader_1x05_P2.00mm_Vertical" H 2850 4500 50  0001 C CNN
@@
 AR Path="/5F8F2E1B/5FA34085/602EA848" Ref="J?"  Part="1"
 AR Path="/5F8F2E1B/5FA33E59/602EA848" Ref="J?"  Part="1"
-AR Path="/602EA848" Ref="J702"  Part="1"
-F 0 "J702" H 1150 4800 50  0000 L CNN
+AR Path="/602EA848" Ref="J105"  Part="1"
+F 0 "J105" H 1150 4800 50  0000 L CNN
 F 1 "Conn_01x05" H 1200 4900 50  0001 L CNN
 F 2 "LedBarController:LED_Strip_10mm_5pins_Left" H 1250 4500 50  0001 C CNN
@@
 AR Path="/5F8F2E1B/5FA34085/602EA851" Ref="J?"  Part="1"
 AR Path="/5F8F2E1B/5FA33E59/602EA851" Ref="J?"  Part="1"
-AR Path="/602EA851" Ref="J703"  Part="1"
-F 0 "J703" H 1150 5800 50  0000 L CNN
+AR Path="/602EA851" Ref="J112"  Part="1"
+F 0 "J112" H 1150 5800 50  0000 L CNN
 F 1 "Conn_01x05" H 1200 5900 50  0001 L CNN
 F 2 "LedBarController:LED_Strip_10mm_5pins_Left" H 1250 5500 50  0001 C CNN
@@
 AR Path="/5F8F2E1B/5FA34085/602EA873" Ref="J?"  Part="1"
 AR Path="/5F8F2E1B/5FA33E59/602EA873" Ref="J?"  Part="1"
-AR Path="/602EA873" Ref="J704"  Part="1"
-F 0 "J704" H 1250 3300 50  0000 C CNN
+AR Path="/602EA873" Ref="J101"  Part="1"
+F 0 "J101" H 1250 3300 50  0000 C CNN
 F 1 "Male pitch strip 1x7 pins 2.0mm pitch" H 1168 3326 50  0001 C CNN
 F 2 "Connector_PinHeader_2.00mm:PinHeader_1x05_P2.00mm_Vertical" H 1250 3000 50  0001 C CNN
@@
 AR Path="/5F8F2E1B/5FA34085/602EA881" Ref="J?"  Part="1"
 AR Path="/5F8F2E1B/5FA33E59/602EA881" Ref="J?"  Part="1"
-AR Path="/602EA881" Ref="J705"  Part="1"
-F 0 "J705" H 2750 3300 50  0000 C CNN
+AR Path="/602EA881" Ref="J102"  Part="1"
+F 0 "J102" H 2750 3300 50  0000 C CNN
 F 1 "Male pitch strip 1x7 pins 2.0mm pitch" H 2668 3326 50  0001 C CNN
 F 2 "LedBarController:LED_Strip_10mm_5pins_Right" H 2750 3000 50  0001 C CNN
@@
 AR Path="/5F8F2E1B/5FA34085/602EA88A" Ref="J?"  Part="1"
 AR Path="/5F8F2E1B/5FA33E59/602EA88A" Ref="J?"  Part="1"
-AR Path="/602EA88A" Ref="J901"  Part="1"
-F 0 "J901" H 9150 4800 50  0000 C CNN
+AR Path="/602EA88A" Ref="J110"  Part="1"
+F 0 "J110" H 9150 4800 50  0000 C CNN
 F 1 "Male pitch strip 1x7 pins 2.0mm pitch" H 9068 4826 50  0001 C CNN
 F 2 "Connector_PinHeader_2.00mm:PinHeader_1x05_P2.00mm_Vertical" H 9150 4500 50  0001 C CNN
@@
 AR Path="/5F8F2E1B/5FA34085/602EA893" Ref="J?"  Part="1"
 AR Path="/5F8F2E1B/5FA33E59/602EA893" Ref="J?"  Part="1"
-AR Path="/602EA893" Ref="J902"  Part="1"
-F 0 "J902" H 10650 4800 50  0000 L CNN
+AR Path="/602EA893" Ref="J111"  Part="1"
+F 0 "J111" H 10650 4800 50  0000 L CNN
 F 1 "Conn_01x05" H 10700 4900 50  0001 L CNN
 F 2 "LedBarController:LED_Strip_10mm_5pins_Right" H 10750 4500 50  0001 C CNN
@@
 AR Path="/5F8F2E1B/5FA34085/602EA89C" Ref="J?"  Part="1"
 AR Path="/5F8F2E1B/5FA33E59/602EA89C" Ref="J?"  Part="1"
-AR Path="/602EA89C" Ref="J903"  Part="1"
-F 0 "J903" H 10650 5800 50  0000 L CNN
+AR Path="/602EA89C" Ref="J115"  Part="1"
+F 0 "J115" H 10650 5800 50  0000 L CNN
 F 1 "Conn_01x05" H 10700 5900 50  0001 L CNN
 F 2 "LedBarController:LED_Strip_10mm_5pins_Right" H 10750 5500 50  0001 C CNN
@@
 AR Path="/5F8F2E1B/5FA34085/602EA8BE" Ref="J?"  Part="1"
 AR Path="/5F8F2E1B/5FA33E59/602EA8BE" Ref="J?"  Part="1"
-AR Path="/602EA8BE" Ref="J905"  Part="1"
-F 0 "J905" H 10750 3350 50  0000 C CNN
+AR Path="/602EA8BE" Ref="J104"  Part="1"
+F 0 "J104" H 10750 3350 50  0000 C CNN
 F 1 "Male pitch strip 1x7 pins 2.0mm pitch" H 10668 3326 50  0001 C CNN
 F 2 "Connector_PinHeader_2.00mm:PinHeader_1x05_P2.00mm_Vertical" H 10750 3000 50  0001 C CNN
@@
 AR Path="/5F8F2E1B/5FA34085/602EA8C7" Ref="J?"  Part="1"
 AR Path="/5F8F2E1B/5FA33E59/602EA8C7" Ref="J?"  Part="1"
-AR Path="/602EA8C7" Ref="J904"  Part="1"
-F 0 "J904" H 9250 3350 50  0000 C CNN
+AR Path="/602EA8C7" Ref="J103"  Part="1"
+F 0 "J103" H 9250 3350 50  0000 C CNN
 F 1 "Male pitch strip 1x7 pins 2.0mm pitch" H 9168 3326 50  0001 C CNN
 F 2 "LedBarController:LED_Strip_10mm_5pins_Left" H 9250 3000 50  0001 C CNN

Commit message: Updated footprints and Fab layer
Other:
- note added: "-->"
- note added: "<--"
Changed lines of the file:
@@
 F1 "CenterBack.sch" 50
 $EndSheet
+Text Notes 3250 3000 0    79   ~ 0
+<--
+Text Notes 8750 3000 2    79   ~ 0
+-->
+Text Notes 2000 3900 1    79   ~ 0
+<--
+Text Notes 6050 3850 1    79   ~ 0
+<--
+Text Notes 10100 3850 1    79   ~ 0
+<--
 $EndSCHEMATC

Commit message: Fixed minor issues
Parts:
- removed J101, J104: Male pitch strip 1x7 pins 2.0mm pitch, Connector_PinHeader_2.00mm:PinHeader_1x05_P2.00mm_Vertical, symbol Connector_Generic:Conn_01x05
- removed J102: Male pitch strip 1x7 pins 2.0mm pitch, LedBarController:LED_Strip_10mm_5pins_Right, symbol Connector_Generic:Conn_01x05
- removed J103: Male pitch strip 1x7 pins 2.0mm pitch, LedBarController:LED_Strip_10mm_5pins_Left, symbol Connector_Generic:Conn_01x05
- renumbered J105 to J101, J112 to J102, J106 to J103, J107 to J104, J113 to J105, J108 to J106, J109 to J107, J114 to J108, J110 to J109, J111 to J110, J115 to J111
Other:
- note added: "Wire x 5"
- note removed: "-->"
- note removed: "<--"
- note removed: "Board: Left Back"
- note removed: "Board: Right Back"
